Commit message: Add TF to hande (#38)
* fix: changed repo to local

* fix: urdf hande joints

* feat: add a grasping point

* fix: rebild cntainer .

* fix: gripper point coords

* fix: hande tf

* fix: remove launch

* fix: git ignore

File: src/ur3e_hande_robot_description/urdf/hande.xacro (robot description, xacro)
@@ -99,6 +99,11 @@
       </xacro:cylinder_inertial>
     </link>
+    <link name="grasping_point_link">
+      <visual>
+        <origin rpy="0 0 0" xyz="0 0 0"/>
+       </visual>
+    </link>
     <!-- hande installation -->
-    <joint name="${tf_prefix}joint_finger" type="prismatic">
+    <joint name="${tf_prefix}joint_finger" type="fixed">
       <origin rpy="0 0 0" xyz="0 0 0.099"/>
       <parent link="${tf_prefix}robotiq_hande_base_link"/>
@@ -107,5 +112,5 @@
       <limit effort="130" lower="0" upper="0.025" velocity="0.15"/>
     </joint>
-    <joint name="robotiq_hande_base_to_${tf_prefix}right_finger" type="prismatic">
+    <joint name="robotiq_hande_base_to_${tf_prefix}right_finger" type="fixed">
       <origin rpy="0 0 0" xyz="0 0 0.099"/>
       <parent link="${tf_prefix}robotiq_hande_base_link"/>
@@ -115,4 +120,10 @@
       <mimic joint="${tf_prefix}joint_finger" multiplier="1" offset="0"/>
     </joint>
+    <joint name="${tf_prefix}grasping_point" type="fixed">
+      <origin rpy="0 0 0" xyz="0.0 0.0 0.134"/>
+      <parent link="${tf_prefix}robotiq_hande_base_link"/>
+      <child link="grasping_point_link"/>
+      <axis xyz="0 0 0"/>
+    </joint>
 </xacro:macro>
 </robot>

Commit message: Fix hande urdf (#39)
* fix: changed repo to local

* fix: urdf hande joints

* fix: rebild cntainer .

* fix: gripper point coords

* fix: hande tf

* fix: remove launch

* fix: git ignore

* fix: move the grasping point

* Update src/ur3e_hande_robot_description/urdf/hande.xacro

---------

Co-authored-by: Dr. Phil Maffettone <43007690+maffettone@users.noreply.github.com>

File: src/ur3e_hande_robot_description/urdf/hande.xacro (robot description, xacro)
@@ -39,4 +39,5 @@
   <xacro:property name="finger_radius" value="${sec_inertia_parameters['finger_radius']}" scope="parent"/>
     <!-- customizations to include hande -->
+    <!-- TODO: Add the coupling between the wrist_3_link and robotiq_hande_base_link -->
     <link name="${tf_prefix}robotiq_hande_base_link">
       <visual>
@@ -100,7 +101,4 @@
     </link>
     <link name="grasping_point_link">
-      <visual>
-        <origin rpy="0 0 0" xyz="0 0 0"/>
-       </visual>
     </link>
     <!-- hande installation -->
@@ -121,5 +119,5 @@
     </joint>
     <joint name="${tf_prefix}grasping_point" type="fixed">
-      <origin rpy="0 0 0" xyz="0.0 0.0 0.134"/>
+      <origin rpy="0 0 0" xyz="0.0 0.0 0.15"/>
       <parent link="${tf_prefix}robotiq_hande_base_link"/>
       <child link="grasping_point_link"/>

Commit message: Azure camera integration on to the UR3e arm (#47)
* feat: add cam mount + aruco pose changes

* fix: add missing file

* fix: use one hande for all + spelling + PR fixes

* fix: remove duplicate urdfs

* refac: remove comments

* fix: remove tab spaces from new line

* Update src/ur3e_hande_robot_description/urdf/hande.xacro

---------

Co-authored-by: Dr. Phil Maffettone <43007690+maffettone@users.noreply.github.com>

File: src/ur3e_hande_robot_description/urdf/hande.xacro (robot description, xacro)
@@ -1,13 +1,10 @@
 <?xml version="1.0"?>
-<robot xmlns:xacro="http://wiki.ros.org/xacro" name="$(arg name)">
+<robot xmlns:xacro="http://wiki.ros.org/xacro" name="hande">
 <!--Based on same file and version as the https://github.com/AcutronicRobotics/robotiq_modular_gripper/blob/4e708524e5dd20753f711686eb2cd1017a25a09e/robotiq_hande_gripper_description/urdf/robotiq_hande.urdf.xacro-->
-  <xacro:arg name="name" default="hande"/>
 <xacro:macro name="robotiq_hande" params="
-    name
     tf_prefix
     parent" >
   <xacro:property name="hande_kinematics_params" value="$(find ur3e_hande_robot_description)/config/hande/default_kinematics.yaml"/>
   <xacro:property name="hande_physical_params" value="$(find ur3e_hande_robot_description)/config/hande/physical_parameters.yaml"/>
-  <xacro:property name="hande_visual_params" value="$(find ur3e_hande_robot_description)/config/hande/visual_parameters.yaml"/>
   <xacro:macro name="cylinder_inertial" params="radius length mass *origin">
     <inertial>
@@ -20,5 +17,4 @@
   </xacro:macro>
   <xacro:property name="config_physical_parameters" value="${xacro.load_yaml(hande_physical_params)}"/>
-  <!-- Extract subsections from yaml dictionaries -->
   <xacro:property name="sec_inertia_parameters" value="${config_physical_parameters['inertia_parameters']}" />
   <xacro:property name="intertia_links" value="${sec_inertia_parameters['links']}" scope="parent"/>
@@ -38,10 +34,33 @@
   <xacro:property name="hande_base_radius" value="${sec_inertia_parameters['hande_base_radius']}" scope="parent"/>
   <xacro:property name="finger_radius" value="${sec_inertia_parameters['finger_radius']}" scope="parent"/>
-    <!-- customizations to include hande -->
+  <xacro:property name="scaling_factor_cp" value="1"/>
+    <link name="${tf_prefix}robotiq_coupler">
+      <inertial>
+        <mass value="0.100" />
+        <inertia
+          ixx="6.17674E-05" ixy="0.0" ixz="0.0"
+          iyy="6.17674E-05" iyz="0.0"
+          izz="1.18125E-04"
+        />
+      </inertial>
+      <collision>
+        <geometry>
+          <mesh filename="package://ur3e_hande_robot_description/meshes/hande/collision/coupler.stl" scale="${scaling_factor_cp} ${scaling_factor_cp} ${scaling_factor_cp}" />
+        </geometry>
+      </collision>
+      <visual>
+        <geometry>
+          <mesh filename="package://ur3e_hande_robot_description/meshes/hande/visual/coupler.dae" scale="${scaling_factor_cp} ${scaling_factor_cp} ${scaling_factor_cp}" />
+        </geometry>
+        <material name="Gazebo/Black">
+          <color rgba="0.1 0.1 0.1 1" />
+        </material>
+      </visual>
+    </link>
     <link name="${tf_prefix}robotiq_hande_base_link">
       <visual>
-        <origin xyz="0 0 0" rpy="0 0 0" />
+        <origin xyz="0 0 0" rpy="0 -1.570796 -1.570796" />
         <geometry>
-          <mesh filename="package://ur3e_hande_robot_description/meshes/hande/visual/hand-e.dae" scale="0.001 0.001 0.001" />
+          <mesh filename="package://ur3e_hande_robot_description/meshes/hande/visual/hande.dae" scale="1 1 1" />
         </geometry>
         <material name="Gazebo/Black">
@@ -50,11 +69,10 @@
       </visual>
       <collision>
-        <origin xyz="0 0 0" rpy="0 0 0" />
         <geometry>
-          <mesh filename="package://ur3e_hande_robot_description/meshes/hande/collision/hand-e.stl" scale="0.001 0.001 0.001"/>
+          <mesh filename="package://ur3e_hande_robot_description/meshes/hande/collision/hande.stl" scale="1 1 1"/>
         </geometry>
       </collision>
       <xacro:cylinder_inertial radius="${hande_base_inertia_radius}" length="${hande_base_inertia_length}"  mass="${hande_base_mass}">
-        <origin xyz="0.0 0.0 ${-0.5 * hande_base_inertia_length}" rpy="0 0 0" />
+        <origin xyz="${hande_base_cog}" rpy="0 0 0" />
       </xacro:cylinder_inertial>
     </link>
@@ -76,5 +94,5 @@
       </collision>
       <xacro:cylinder_inertial radius="${left_finger_inertia_radius}" length="${left_finger_inertia_length}"  mass="${left_finger_mass}">
-        <origin xyz="0.0 0.0 ${-0.5 * left_finger_inertia_length}" rpy="0 0 0" />
+        <origin xyz="${finger_cog}" rpy="0 0 0" />
       </xacro:cylinder_inertial>
     </link>
@@ -96,12 +114,16 @@
       </collision>
       <xacro:cylinder_inertial radius="${right_finger_inertia_radius}" length="${right_finger_inertia_length}"  mass="${right_finger_mass}">
-        <origin xyz="0.0 0.0 ${-0.5 * right_finger_inertia_length}" rpy="0 0 0" />
+        <origin xyz="${finger_cog}" rpy="0 0 0" />
       </xacro:cylinder_inertial>
     </link>
     <link name="grasping_point_link">
     </link>
-    <!-- hande installation -->
+    <joint name="robotiq_coupler_joint" type="fixed">
+      <origin xyz="0 0 -0.05" rpy="${pi} 0 ${-pi/2.0}" />
+      <parent link="${tf_prefix}robotiq_coupler"/>
+      <child link="${tf_prefix}robotiq_hande_base_link"/>
+    </joint>
     <joint name="${tf_prefix}joint_finger" type="fixed">
-      <origin rpy="0 0 0" xyz="0 0 0.099"/>
+      <origin rpy="0 0 ${pi/2.0}" xyz="0 0 0.05"/>
       <parent link="${tf_prefix}robotiq_hande_base_link"/>
       <child link="${tf_prefix}left_finger"/>
@@ -110,5 +132,5 @@
     </joint>
     <joint name="robotiq_hande_base_to_${tf_prefix}right_finger" type="fixed">
-      <origin rpy="0 0 0" xyz="0 0 0.099"/>
+      <origin rpy="0 0 ${pi/2.0}" xyz="0 0 0.05"/>
       <parent link="${tf_prefix}robotiq_hande_base_link"/>
       <child link="${tf_prefix}right_finger"/>
@@ -118,5 +140,5 @@
     </joint>
     <joint name="${tf_prefix}grasping_point" type="fixed">
-      <origin rpy="0 0 0" xyz="0.0 0.0 0.15"/>
+      <origin rpy="0 0 0" xyz="0.0 0.0 0.09"/>
       <parent link="${tf_prefix}robotiq_hande_base_link"/>
       <child link="grasping_point_link"/>
