Commit message: switched from ur3e to ur5e

File: src/ur5e_hande_robot_description/urdf/camera_mount.xacro (robot description, xacro)
@@ -2,5 +2,5 @@
 <robot xmlns:xacro="http://www.ros.org/wiki/xacro" name="camera">
 <xacro:macro name="camera_mount">
-  <xacro:property name="mount_physical_params_file" value="$(find ur3e_hande_robot_description)/config/camera_mount/physical_parameters.yaml"/>
+  <xacro:property name="mount_physical_params_file" value="$(find ur5e_hande_robot_description)/config/camera_mount/physical_parameters.yaml"/>
   <xacro:property name="mount_physical_parameters" value="${xacro.load_yaml(mount_physical_params_file)}"/>
   <!-- Mass and Inertial properties -->
@@ -34,5 +34,5 @@
       <origin xyz="0 0 0" rpy="0 0 0"/>
       <geometry>
-        <mesh filename="package://ur3e_hande_robot_description/meshes/camera_mount/visual/ur3e_flange_camera_mount.dae" scale="${scaling_factor} ${scaling_factor} ${scaling_factor}"/>
+        <mesh filename="package://ur5e_hande_robot_description/meshes/camera_mount/visual/ur5e_flange_camera_mount.dae" scale="${scaling_factor} ${scaling_factor} ${scaling_factor}"/>
       </geometry>
       <material name="mat">
@@ -43,5 +43,5 @@
       <origin xyz="0 0 0" rpy="0 0 0"/>
       <geometry>
-        <mesh filename="package://ur3e_hande_robot_description/meshes/camera_mount/collision/ur3e_flange_camera_mount.stl" scale="${scaling_factor} ${scaling_factor} ${scaling_factor}"/>
+        <mesh filename="package://ur5e_hande_robot_description/meshes/camera_mount/collision/ur5e_flange_camera_mount.stl" scale="${scaling_factor} ${scaling_factor} ${scaling_factor}"/>
       </geometry>
     </collision>
@@ -54,5 +54,5 @@
     <visual>
         <geometry>
-          <mesh filename="package://ur3e_hande_robot_description/meshes/camera_mount/visual/azure_kinect.dae" scale="${scaling_factor_cm} ${scaling_factor_cm} ${scaling_factor_cm}" />
+          <mesh filename="package://ur5e_hande_robot_description/meshes/camera_mount/visual/azure_kinect.dae" scale="${scaling_factor_cm} ${scaling_factor_cm} ${scaling_factor_cm}" />
         </geometry>
         <material name="Gazebo/Black">
@@ -62,5 +62,5 @@
     <collision>
       <geometry>
-        <mesh filename="package://ur3e_hande_robot_description/meshes/camera_mount/collision/azure_kinect.stl" scale="${scaling_factor_cm} ${scaling_factor_cm} ${scaling_factor_cm}" />
+        <mesh filename="package://ur5e_hande_robot_description/meshes/camera_mount/collision/azure_kinect.stl" scale="${scaling_factor_cm} ${scaling_factor_cm} ${scaling_factor_cm}" />
       </geometry>
     </collision>

File: src/ur5e_hande_robot_description/urdf/hande.xacro (robot description, xacro)
@@ -5,6 +5,6 @@
     tf_prefix
     parent" >
-  <xacro:property name="hande_kinematics_params" value="$(find ur3e_hande_robot_description)/config/hande/default_kinematics.yaml"/>
-  <xacro:property name="hande_physical_params" value="$(find ur3e_hande_robot_description)/config/hande/physical_parameters.yaml"/>
+  <xacro:property name="hande_kinematics_params" value="$(find ur5e_hande_robot_description)/config/hande/default_kinematics.yaml"/>
+  <xacro:property name="hande_physical_params" value="$(find ur5e_hande_robot_description)/config/hande/physical_parameters.yaml"/>
   <xacro:macro name="cylinder_inertial" params="radius length mass *origin">
     <inertial>
@@ -46,10 +46,10 @@
       <collision>
         <geometry>
-          <mesh filename="package://ur3e_hande_robot_description/meshes/hande/collision/coupler.stl" scale="${scaling_factor_cp} ${scaling_factor_cp} ${scaling_factor_cp}" />
+          <mesh filename="package://ur5e_hande_robot_description/meshes/hande/collision/coupler.stl" scale="${scaling_factor_cp} ${scaling_factor_cp} ${scaling_factor_cp}" />
         </geometry>
       </collision>
       <visual>
         <geometry>
-          <mesh filename="package://ur3e_hande_robot_description/meshes/hande/visual/coupler.dae" scale="${scaling_factor_cp} ${scaling_factor_cp} ${scaling_factor_cp}" />
+          <mesh filename="package://ur5e_hande_robot_description/meshes/hande/visual/coupler.dae" scale="${scaling_factor_cp} ${scaling_factor_cp} ${scaling_factor_cp}" />
         </geometry>
         <material name="Gazebo/Black">
@@ -62,5 +62,5 @@
         <origin xyz="0 0 0" rpy="0 -1.570796 -1.570796" />
         <geometry>
-          <mesh filename="package://ur3e_hande_robot_description/meshes/hande/visual/hande.dae" scale="1 1 1" />
+          <mesh filename="package://ur5e_hande_robot_description/meshes/hande/visual/hande.dae" scale="1 1 1" />
         </geometry>
         <material name="Gazebo/Black">
@@ -70,5 +70,5 @@
       <collision>
         <geometry>
-          <mesh filename="package://ur3e_hande_robot_description/meshes/hande/collision/hande.stl" scale="1 1 1"/>
+          <mesh filename="package://ur5e_hande_robot_description/meshes/hande/collision/hande.stl" scale="1 1 1"/>
         </geometry>
       </collision>
@@ -81,5 +81,5 @@
         <origin rpy="0 0 0" xyz="0 0 0"/>
         <geometry>
-          <mesh filename="package://ur3e_hande_robot_description/meshes/hande/visual/finger_1.dae" scale="0.001 0.001 0.001"/>
+          <mesh filename="package://ur5e_hande_robot_description/meshes/hande/visual/finger_1.dae" scale="0.001 0.001 0.001"/>
         </geometry>
         <material name="Gazebo/Grey">
@@ -90,5 +90,5 @@
         <origin rpy="0 0 0" xyz="0 0 0"/>
         <geometry>
-          <mesh filename="package://ur3e_hande_robot_description/meshes/hande/collision/finger_1.stl" scale="0.001 0.001 0.001"/>
+          <mesh filename="package://ur5e_hande_robot_description/meshes/hande/collision/finger_1.stl" scale="0.001 0.001 0.001"/>
         </geometry>
       </collision>
@@ -101,5 +101,5 @@
         <origin rpy="0 0 0" xyz="0 0 0"/>
         <geometry>
-          <mesh filename="package://ur3e_hande_robot_description/meshes/hande/visual/finger_2.dae" scale="0.001 0.001 0.001"/>
+          <mesh filename="package://ur5e_hande_robot_description/meshes/hande/visual/finger_2.dae" scale="0.001 0.001 0.001"/>
         </geometry>
         <material name="Gazebo/Grey">
@@ -110,5 +110,5 @@
         <origin rpy="0 0 0" xyz="0 0 0"/>
         <geometry>
-          <mesh filename="package://ur3e_hande_robot_description/meshes/hande/collision/finger_2.stl" scale="0.001 0.001 0.001"/>
+          <mesh filename="package://ur5e_hande_robot_description/meshes/hande/collision/finger_2.stl" scale="0.001 0.001 0.001"/>
         </geometry>
       </collision>

File: src/ur5e_hande_robot_description/urdf/ur_with_camera_hande.xacro (robot description, xacro)
@@ -6,9 +6,9 @@
    <!-- import main macro -->
    <xacro:include filename="$(find ur_description)/urdf/ur_macro.xacro"/>
-  <xacro:include filename="$(find ur3e_hande_robot_description)/urdf/hande.xacro"/>
-  <xacro:include filename="$(find ur3e_hande_robot_description)/urdf/camera_mount.xacro"/>
-   <!-- possible 'ur_type' values: ur3, ur3e, ur5, ur5e, ur10, ur10e, ur16e, ur20 -->
+  <xacro:include filename="$(find ur5e_hande_robot_description)/urdf/hande.xacro"/>
+  <xacro:include filename="$(find ur5e_hande_robot_description)/urdf/camera_mount.xacro"/>
+   <!-- possible 'ur_type' values: ur3, ur5e, ur5, ur5e, ur10, ur10e, ur16e, ur20 -->
    <!-- the default value should raise an error in case this was called without defining the type -->
-   <xacro:arg name="ur_type" default="ur3e"/>
+   <xacro:arg name="ur_type" default="ur5e"/>
    <!-- These parameters are from https://github.com/UniversalRobots/Universal_Robots_ROS2_Description/blob/29e90d5095fdf4af99eba3c3eae153d7d5d769c0/urdf/ur.urdf.xacro-->
    <xacro:arg name="tf_prefix" default="" />

File: src/ur5e_hande_robot_description/urdf/ur_with_hande.xacro (robot description, xacro)
@@ -6,8 +6,8 @@
    <!-- import main macro -->
    <xacro:include filename="$(find ur_description)/urdf/ur_macro.xacro"/>
-  <xacro:include filename="$(find ur3e_hande_robot_description)/urdf/hande.xacro"/>
-   <!-- possible 'ur_type' values: ur3, ur3e, ur5, ur5e, ur10, ur10e, ur16e, ur20 -->
+  <xacro:include filename="$(find ur5e_hande_robot_description)/urdf/hande.xacro"/>
+   <!-- possible 'ur_type' values: ur3, ur5e, ur5, ur5e, ur10, ur10e, ur16e, ur20 -->
    <!-- the default value should raise an error in case this was called without defining the type -->
-   <xacro:arg name="ur_type" default="ur3e"/>
+   <xacro:arg name="ur_type" default="ur5e"/>
    <!-- These parameters are from https://github.com/UniversalRobots/Universal_Robots_ROS2_Description/blob/29e90d5095fdf4af99eba3c3eae153d7d5d769c0/urdf/ur.urdf.xacro-->
    <xacro:arg name="tf_prefix" default="" />
