Commit message: new gripper setup

File: src/ur5e_hande_robot_description/urdf/hande.xacro (robot description, xacro)
@@ -1,148 +1,30 @@
 <?xml version="1.0"?>
-<robot xmlns:xacro="http://wiki.ros.org/xacro" name="hande">
-<!--Based on same file and version as the https://github.com/AcutronicRobotics/robotiq_modular_gripper/blob/4e708524e5dd20753f711686eb2cd1017a25a09e/robotiq_hande_gripper_description/urdf/robotiq_hande.urdf.xacro-->
-<xacro:macro name="robotiq_hande" params="
-    tf_prefix
-    parent" >
-  <xacro:property name="hande_kinematics_params" value="$(find ur5e_hande_robot_description)/config/hande/default_kinematics.yaml"/>
-  <xacro:property name="hande_physical_params" value="$(find ur5e_hande_robot_description)/config/hande/physical_parameters.yaml"/>
-  <xacro:macro name="cylinder_inertial" params="radius length mass *origin">
-    <inertial>
-      <mass value="${mass}" />
-      <xacro:insert_block name="origin" />
-      <inertia ixx="${0.0833333 * mass * (3 * radius * radius + length * length)}" ixy="0.0" ixz="0.0"
-        iyy="${0.0833333 * mass * (3 * radius * radius + length * length)}" iyz="0.0"
-        izz="${0.5 * mass * radius * radius}" />
-    </inertial>
+<robot xmlns:xacro="http://ros.org/wiki/xacro">
+  <xacro:arg name="grip_pos_min" default="0"/>
+  <xacro:arg name="grip_pos_max" default="0.025"/>
+  <xacro:arg name="tty" default="/tmp/ttyUR"/>
+  <xacro:arg name="baudrate" default="115200"/>
+  <xacro:arg name="parity" default="N"/>
+  <xacro:arg name="data_bits" default="8"/>
+  <xacro:arg name="stop_bit" default="1"/>
+  <xacro:arg name="slave_id" default="9"/>
+  <xacro:arg name="tf_prefix" default="" />
+  <xacro:include filename="$(find ur5e_hande_robot_description)/urdf/robotiq_hande_gripper.xacro"/>
+  <!-- TODO(issue#34): pass initial position from the YAML file analogous to the ur_definition -->
+  <xacro:macro name="hande" params="parent tf_prefix mock_hardware">
+    <xacro:robotiq_hande_gripper
+      name="robotiq_hande_gripper"
+      tf_prefix="$(arg tf_prefix)"
+      parent="${parent}"
+      grip_pos_min="$(arg grip_pos_min)"
+      grip_pos_max="$(arg grip_pos_max)"
+      tty="$(arg tty)"
+      baudrate="$(arg baudrate)"
+      parity="$(arg parity)"
+      data_bits="$(arg data_bits)"
+      stop_bit="$(arg stop_bit)"
+      slave_id="$(arg slave_id)"
+      use_fake_hardware="$(arg mock_hardware)"
+    />
   </xacro:macro>
-  <xacro:property name="config_physical_parameters" value="${xacro.load_yaml(hande_physical_params)}"/>
-  <xacro:property name="sec_inertia_parameters" value="${config_physical_parameters['inertia_parameters']}" />
-  <xacro:property name="intertia_links" value="${sec_inertia_parameters['links']}" scope="parent"/>
-  <xacro:property name="hande_base_mass" value="${sec_inertia_parameters['hande_base_mass']}" scope="parent"/>
-  <xacro:property name="left_finger_mass" value="${sec_inertia_parameters['left_finger_mass']}" scope="parent"/>
-  <xacro:property name="right_finger_mass" value="${sec_inertia_parameters['right_finger_mass']}" scope="parent"/>
-  <xacro:property name="hande_base_inertia_radius" value="${intertia_links['hande_base']['radius']}" scope="parent"/>
-  <xacro:property name="hande_base_inertia_length" value="${intertia_links['hande_base']['length']}" scope="parent"/>
-  <xacro:property name="left_finger_inertia_radius" value="${intertia_links['left_finger']['radius']}" scope="parent"/>
-  <xacro:property name="left_finger_inertia_length" value="${intertia_links['left_finger']['length']}" scope="parent"/>
-  <xacro:property name="right_finger_inertia_radius" value="${intertia_links['right_finger']['radius']}" scope="parent"/>
-  <xacro:property name="right_finger_inertia_length" value="${intertia_links['right_finger']['length']}" scope="parent"/>
-  <xacro:property name="prop_hande_cog" value="${sec_inertia_parameters['center_of_mass']['hande_cog']}" scope="parent"/>
-  <xacro:property name="prop_finger_cog" value="${sec_inertia_parameters['center_of_mass']['finger_cog']}" scope="parent"/>
-  <xacro:property name="hande_base_cog" value="${prop_hande_cog['x']} ${prop_hande_cog['y']} ${prop_hande_cog['z']}" scope="parent"/>
-  <xacro:property name="finger_cog" value="${prop_finger_cog['x']} ${prop_finger_cog['y']} ${prop_finger_cog['z']}" scope="parent"/>
-  <xacro:property name="hande_base_radius" value="${sec_inertia_parameters['hande_base_radius']}" scope="parent"/>
-  <xacro:property name="finger_radius" value="${sec_inertia_parameters['finger_radius']}" scope="parent"/>
-  <xacro:property name="scaling_factor_cp" value="1"/>
-    <link name="${tf_prefix}robotiq_coupler">
-      <inertial>
-        <mass value="0.100" />
-        <inertia
-          ixx="6.17674E-05" ixy="0.0" ixz="0.0"
-          iyy="6.17674E-05" iyz="0.0"
-          izz="1.18125E-04"
-        />
-      </inertial>
-      <collision>
-        <geometry>
-          <mesh filename="package://ur5e_hande_robot_description/meshes/hande/collision/coupler.stl" scale="${scaling_factor_cp} ${scaling_factor_cp} ${scaling_factor_cp}" />
-        </geometry>
-      </collision>
-      <visual>
-        <geometry>
-          <mesh filename="package://ur5e_hande_robot_description/meshes/hande/visual/coupler.dae" scale="${scaling_factor_cp} ${scaling_factor_cp} ${scaling_factor_cp}" />
-        </geometry>
-        <material name="Gazebo/Black">
-          <color rgba="0.1 0.1 0.1 1" />
-        </material>
-      </visual>
-    </link>
-    <link name="${tf_prefix}robotiq_hande_base_link">
-      <visual>
-        <origin xyz="0 0 0" rpy="0 -1.570796 -1.570796" />
-        <geometry>
-          <mesh filename="package://ur5e_hande_robot_description/meshes/hande/visual/hande.dae" scale="1 1 1" />
-        </geometry>
-        <material name="Gazebo/Black">
-          <color rgba="0.1 0.1 0.1 1" />
-        </material>
-      </visual>
-      <collision>
-        <geometry>
-          <mesh filename="package://ur5e_hande_robot_description/meshes/hande/collision/hande.stl" scale="1 1 1"/>
-        </geometry>
-      </collision>
-      <xacro:cylinder_inertial radius="${hande_base_inertia_radius}" length="${hande_base_inertia_length}"  mass="${hande_base_mass}">
-        <origin xyz="${hande_base_cog}" rpy="0 0 0" />
-      </xacro:cylinder_inertial>
-    </link>
-    <link name="${tf_prefix}left_finger">
-      <visual>
-        <origin rpy="0 0 0" xyz="0 0 0"/>
-        <geometry>
-          <mesh filename="package://ur5e_hande_robot_description/meshes/hande/visual/finger_1.dae" scale="0.001 0.001 0.001"/>
-        </geometry>
-        <material name="Gazebo/Grey">
-          <color rgba="0.1 0.1 0.1 1"/>
-        </material>
-      </visual>
-      <collision>
-        <origin rpy="0 0 0" xyz="0 0 0"/>
-        <geometry>
-          <mesh filename="package://ur5e_hande_robot_description/meshes/hande/collision/finger_1.stl" scale="0.001 0.001 0.001"/>
-        </geometry>
-      </collision>
-      <xacro:cylinder_inertial radius="${left_finger_inertia_radius}" length="${left_finger_inertia_length}"  mass="${left_finger_mass}">
-        <origin xyz="${finger_cog}" rpy="0 0 0" />
-      </xacro:cylinder_inertial>
-    </link>
-    <link name="${tf_prefix}right_finger">
-      <visual>
-        <origin rpy="0 0 0" xyz="0 0 0"/>
-        <geometry>
-          <mesh filename="package://ur5e_hande_robot_description/meshes/hande/visual/finger_2.dae" scale="0.001 0.001 0.001"/>
-        </geometry>
-        <material name="Gazebo/Grey">
-          <color rgba="0.1 0.1 0.1 1"/>
-        </material>
-      </visual>
-      <collision>
-        <origin rpy="0 0 0" xyz="0 0 0"/>
-        <geometry>
-          <mesh filename="package://ur5e_hande_robot_description/meshes/hande/collision/finger_2.stl" scale="0.001 0.001 0.001"/>
-        </geometry>
-      </collision>
-      <xacro:cylinder_inertial radius="${right_finger_inertia_radius}" length="${right_finger_inertia_length}"  mass="${right_finger_mass}">
-        <origin xyz="${finger_cog}" rpy="0 0 0" />
-      </xacro:cylinder_inertial>
-    </link>
-    <link name="grasping_point_link">
-    </link>
-    <joint name="robotiq_coupler_joint" type="fixed">
-      <origin xyz="0 0 -0.05" rpy="${pi} 0 ${-pi/2.0}" />
-      <parent link="${tf_prefix}robotiq_coupler"/>
-      <child link="${tf_prefix}robotiq_hande_base_link"/>
-    </joint>
-    <joint name="${tf_prefix}joint_finger" type="prismatic">
-      <origin rpy="0 0 ${pi/2.0}" xyz="0 0 0.05"/>
-      <parent link="${tf_prefix}robotiq_hande_base_link"/>
-      <child link="${tf_prefix}left_finger"/>
-      <axis xyz="-1 0 0"/>
-      <limit effort="130" lower="0" upper="0.025" velocity="0.15"/>
-    </joint>
-    <joint name="robotiq_hande_base_to_${tf_prefix}right_finger" type="prismatic">
-      <origin rpy="0 0 ${pi/2.0}" xyz="0 0 0.05"/>
-      <parent link="${tf_prefix}robotiq_hande_base_link"/>
-      <child link="${tf_prefix}right_finger"/>
-      <axis xyz="1 0 0"/>
-      <limit effort="130" lower="0" upper="0.025" velocity="0.15"/>
-      <mimic joint="${tf_prefix}joint_finger" multiplier="1" offset="0"/>
-    </joint>
-    <joint name="${tf_prefix}grasping_point" type="fixed">
-      <origin rpy="0 0 0" xyz="0.0 0.0 0.09"/>
-      <parent link="${tf_prefix}robotiq_hande_base_link"/>
-      <child link="grasping_point_link"/>
-      <axis xyz="0 0 0"/>
-    </joint>
-</xacro:macro>
 </robot>

File: src/ur5e_hande_robot_description/urdf/ur_with_camera_hande.xacro (robot description, xacro)
@@ -54,4 +54,6 @@
    <!-- create link fixed to the "map" -->
    <link name="map" />
+   <!-- mock_hardware for gripper  -->
+   <xacro:arg name="mock_hardware" default="false" />
    <!-- arm -->
    <xacro:ur_robot
@@ -94,9 +96,4 @@
      <origin xyz="0 0 0" rpy="0 0 0" />          <!-- position robot in the map -->
    </xacro:ur_robot>
-    <!-- Call the robot gripper -->
-    <xacro:robotiq_hande
-     tf_prefix="$(arg tf_prefix)"
-     parent="map"
-   />
     <xacro:camera_mount
     />
@@ -107,9 +104,5 @@
       <origin xyz="0 0 -0.001" rpy="${pi} 0 -${pi/2}" />
     </joint>
-    <!-- attach the gripper to the arm -->
-    <joint name="$(arg tf_prefix)hande_to_wrist_flange" type="fixed">
-      <parent link="mount" />
-      <child link="$(arg tf_prefix)robotiq_coupler" />
-      <origin xyz="0 -0.013 0" rpy="-${pi/2.0} -${pi} 0" />
-    </joint>
+    <!-- Call the robot gripper -->
+    <xacro:hande parent="mount" tf_prefix="$(arg tf_prefix)" mock_hardware="$(arg mock_hardware)"/>
 </robot>

File: src/ur5e_hande_robot_description/urdf/ur_with_hande.xacro (robot description, xacro)
@@ -6,5 +6,5 @@
    <!-- import main macro -->
    <xacro:include filename="$(find ur_description)/urdf/ur_macro.xacro"/>
-  <xacro:include filename="$(find ur5e_hande_robot_description)/urdf/hande.xacro"/>
+   <xacro:include filename="$(find ur5e_hande_robot_description)/urdf/hande.xacro"/>
    <!-- possible 'ur_type' values: ur3, ur5e, ur5, ur5e, ur10, ur10e, ur16e, ur20 -->
    <!-- the default value should raise an error in case this was called without defining the type -->
@@ -93,23 +93,10 @@
      <origin xyz="0 0 0" rpy="0 0 0" />          <!-- position robot in the map -->
    </xacro:ur_robot>
+    <xacro:arg name="mock_hardware" default="false" />
     <!-- Call the robot gripper -->
-    <xacro:robotiq_hande
+    <xacro:hande
+     parent="$(arg tf_prefix)flange"
      tf_prefix="$(arg tf_prefix)"
-     parent="map"
-   />
-    <!-- attach the gripper to the arm -->
-    <joint name="$(arg tf_prefix)hande_to_wrist_flange" type="fixed">
-      <parent link="$(arg tf_prefix)flange" />
-      <child link="$(arg tf_prefix)robotiq_coupler" />
-      <origin xyz="0.005 0 0" rpy="-${pi/2.0} 0 ${pi/2.0}" />
-    </joint>
-    <ros2_control name="gripper" type="system">
-      <hardware>
-        <plugin>fake_components/GenericSystem</plugin>
-      </hardware>
-      <joint name="joint_finger">
-        <command_interface name="position"/>
-        <state_interface name="position"/>
-      </joint>
-    </ros2_control>
+     mock_hardware="$(arg mock_hardware)">
+    </xacro:hande>
 </robot>

Commit message: new_moveit_config

File: src/ur5e_hande_robot_description/urdf/hande.xacro (robot description, xacro)
@@ -10,10 +10,10 @@
   <xacro:arg name="slave_id" default="9"/>
   <xacro:arg name="tf_prefix" default="" />
-  <xacro:include filename="$(find ur5e_hande_robot_description)/urdf/robotiq_hande_gripper.xacro"/>
+  <xacro:include filename="$(find robotiq_hande_description)/urdf/robotiq_hande_gripper.xacro"/>
   <!-- TODO(issue#34): pass initial position from the YAML file analogous to the ur_definition -->
-  <xacro:macro name="hande" params="parent tf_prefix mock_hardware">
+  <xacro:macro name="hande" params="parent prefix mock_hardware">
     <xacro:robotiq_hande_gripper
       name="robotiq_hande_gripper"
-      tf_prefix="$(arg tf_prefix)"
+      prefix="${prefix}"
       parent="${parent}"
       grip_pos_min="$(arg grip_pos_min)"

File: src/ur5e_hande_robot_description/urdf/ur_with_hande.urdf (robot description, URDF)
Before this commit: robot ur, 18 links, 17 joints
Links:
- link robotiq_hande_coupler: geometry collision cylinder length=0.0169 radius=0.0385; visual mesh filename=package://robotiq_hande_description/meshes/io_coupler.dae
- link robotiq_hande_left_finger: geometry collision mesh filename=package://robotiq_hande_description/meshes/finger_collision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 scale=1.0 1.0 1.0; visual mesh filename=package://robotiq_hande_description/meshes/finger.dae scale=1.0 1.0 1.0
- link robotiq_hande_link: geometry collision cylinder length=0.10690000000000001 radius=0.0385; visual mesh filename=package://robotiq_hande_description/meshes/hande.dae scale=1.0 1.0 1.0
- link robotiq_hande_right_finger: geometry collision mesh filename=package://robotiq_hande_description/meshes/finger_collision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 scale=1.0 1.0 1.0; visual mesh filename=package://robotiq_hande_description/meshes/finger.dae scale=1.0 1.0 1.0

File: src/ur5e_hande_robot_description/urdf/ur_with_hande.xacro (robot description, xacro)
@@ -93,10 +93,10 @@
      <origin xyz="0 0 0" rpy="0 0 0" />          <!-- position robot in the map -->
    </xacro:ur_robot>
-    <xacro:arg name="mock_hardware" default="false" />
+    <xacro:arg name="mock_hardware" default="true" />
     <!-- Call the robot gripper -->
     <xacro:hande
      parent="$(arg tf_prefix)flange"
-     tf_prefix="$(arg tf_prefix)"
-     mock_hardware="$(arg mock_hardware)">
+     prefix="$(arg tf_prefix)"
+     mock_hardware="$(arg use_fake_hardware)">
     </xacro:hande>
 </robot>
