Commit message: new moveit_config with tool exchanger and hande

File: src/ur5e_hande_robot_description/urdf/tool_exchanger.xacro (robot description, xacro)
@@ -1,10 +1,10 @@
 <?xml version="1.0"?>
 <robot xmlns:xacro="http://ros.org/wiki/xacro" name="wingman_toolchanger">
-  <xacro:macro name="tool_exchanger_robot_side" params="parent_link">
-    <link name="tool_exchanger_robot_link">
+  <xacro:macro name="tool_exchanger" params="parent_link">
+    <link name="tool_exchanger">
       <visual>
         <origin xyz="0 0 0" rpy="0 0 0"/>
         <geometry>
-          <mesh filename="package://ur5e_hande_robot_description/meshes/tool_exchanger/robot_side_part.stl"
+          <mesh filename="package://ur5e_hande_robot_description/meshes/tool_exchanger/TE_assembly.stl"
                 scale="0.001 0.001 0.001"/>
         </geometry>
@@ -16,5 +16,5 @@
         <origin xyz="0 0 0" rpy="0 0 0"/>
         <geometry>
-          <mesh filename="package://ur5e_hande_robot_description/meshes/tool_exchanger/robot_side_part.stl"
+          <mesh filename="package://ur5e_hande_robot_description/meshes/tool_exchanger/TE_assembly.stl"
                 scale="0.001 0.001 0.001"/>
         </geometry>
@@ -30,5 +30,5 @@
     <joint name="tool_exchanger_joint" type="fixed">
       <parent link="${parent_link}"/>
-      <child link="tool_exchanger_robot_link"/>
+      <child link="tool_exchanger"/>
       <origin xyz="0.010 0 0" rpy="0 0 ${pi/2}"/>
     </joint>

File: src/ur5e_hande_robot_description/urdf/ur_with_toolexchanger.urdf (robot description, URDF)
Before this commit: robot ur, 14 links, 13 joints
Links:
- removed link tool_exchanger_robot_link
- added link robotiq_hande_coupler, mass 0.119; collision cylinder length=0.0169 radius=0.0385; visual mesh filename=package://robotiq_hande_description/meshes/io_coupler.dae
- added link robotiq_hande_end
- added link robotiq_hande_left_finger, mass 0.03804; collision mesh filename=package://robotiq_hande_description/meshes/finger_collision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 scale=1.0 1.0 1.0; visual mesh filename=package://robotiq_hande_description/meshes/finger.dae scale=1.0 1.0 1.0
- added link robotiq_hande_link, mass 0.86387; collision cylinder length=0.10690000000000001 radius=0.0385; visual mesh filename=package://robotiq_hande_description/meshes/hande.dae scale=1.0 1.0 1.0
- added link robotiq_hande_right_finger, mass 0.03804; collision mesh filename=package://robotiq_hande_description/meshes/finger_collision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 scale=1.0 1.0 1.0; visual mesh filename=package://robotiq_hande_description/meshes/finger.dae scale=1.0 1.0 1.0
- added link tool_exchanger, mass 0.5; collision mesh filename=package://ur5e_hande_robot_description/meshes/tool_exchange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 scale=0.001 0.001 0.001; visual mesh filename=package://ur5e_hande_robot_description/meshes/tool_exchange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 scale=0.001 0.001 0.001
Joints:
- added joint robotiq_hande_base_joint: type fixed, parent robotiq_hande_coupler, child robotiq_hande_link, origin xyz=0 0 0.011 rpy=0 0 0
- added joint robotiq_hande_coupler_joint: type fixed, parent tool_exchanger, child robotiq_hande_coupler, origin xyz=0.0 -0.019 0.0 rpy=1.5708 0 0
- added joint robotiq_hande_end_joint: type fixed, parent robotiq_hande_link, child robotiq_hande_end, origin xyz=0 0 0.14550000000000002 rpy=0 0 0
- added joint robotiq_hande_left_finger_joint: type prismatic, parent robotiq_hande_link, child robotiq_hande_left_finger, origin xyz=0 0 0.099 rpy=0 0 0, axis 1 0 0, limit lower=0 upper=0.025 effort=130 velocity=0.15
- added joint robotiq_hande_right_finger_joint: type prismatic, parent robotiq_hande_link, child robotiq_hande_right_finger, origin xyz=0 0 0.099 rpy=0 0 0, axis -1 0 0, limit lower=0 upper=0.025 effort=130 velocity=0.15, mimic joint=robotiq_hande_left_finger_joint multiplier=1 offset=0
- joint tool_exchanger_joint: child tool_exchanger_robot_link -> tool_exchanger

File: src/ur5e_hande_robot_description/urdf/ur_with_toolexchanger.xacro (robot description, xacro)
@@ -7,4 +7,5 @@
    <xacro:include filename="$(find ur_description)/urdf/ur_macro.xacro"/>
    <xacro:include filename="$(find ur5e_hande_robot_description)/urdf/tool_exchanger.xacro"/>
+   <xacro:include filename="$(find robotiq_hande_description)/urdf/robotiq_hande_gripper.xacro"/>
    <!-- possible 'ur_type' values: ur3, ur5e, ur5, ur5e, ur10, ur10e, ur16e, ur20 -->
    <!-- the default value should raise an error in case this was called without defining the type -->
@@ -94,28 +95,28 @@
      <origin xyz="0 0 0" rpy="0 0 0" />          <!-- position robot in the map -->
    </xacro:ur_robot>
+  <xacro:tool_exchanger parent_link="$(arg tf_prefix)flange"/>
   <!-- hande gripper -->
-    <!-- <xacro:arg name="grip_pos_min" default="0"/>
-    <xacro:arg name="grip_pos_max" default="0.025"/>
-    <xacro:arg name="tty" default="/tmp/ttyUR"/>
-    <xacro:arg name="baudrate" default="115200"/>
-    <xacro:arg name="parity" default="N"/>
-    <xacro:arg name="data_bits" default="8"/>
-    <xacro:arg name="stop_bit" default="1"/>
-    <xacro:arg name="slave_id" default="9"/>
-    <xacro:robotiq_hande_gripper
-      name="robotiq_hande_gripper"
-      prefix="$(arg tf_prefix)"
-      parent="$(arg tf_prefix)flange"
-      grip_pos_min="$(arg grip_pos_min)"
-      grip_pos_max="$(arg grip_pos_max)"
-      tty="$(arg tty)"
-      baudrate="$(arg baudrate)"
-      parity="$(arg parity)"
-      data_bits="$(arg data_bits)"
-      stop_bit="$(arg stop_bit)"
-      slave_id="$(arg slave_id)"
-      use_fake_hardware="$(arg mock_hardware)"
-      xyz="0 0 0"
-      rpy="-1.5708 0 -1.5708"/> -->
-  <xacro:tool_exchanger_robot_side parent_link="$(arg tf_prefix)flange"/>
+  <xacro:arg name="grip_pos_min" default="0"/>
+  <xacro:arg name="grip_pos_max" default="0.025"/>
+  <xacro:arg name="tty" default="/tmp/ttyUR"/>
+  <xacro:arg name="baudrate" default="115200"/>
+  <xacro:arg name="parity" default="N"/>
+  <xacro:arg name="data_bits" default="8"/>
+  <xacro:arg name="stop_bit" default="1"/>
+  <xacro:arg name="slave_id" default="9"/>
+  <xacro:robotiq_hande_gripper
+    name="robotiq_hande_gripper"
+    prefix="$(arg tf_prefix)"
+    parent="tool_exchanger"
+    grip_pos_min="$(arg grip_pos_min)"
+    grip_pos_max="$(arg grip_pos_max)"
+    tty="$(arg tty)"
+    baudrate="$(arg baudrate)"
+    parity="$(arg parity)"
+    data_bits="$(arg data_bits)"
+    stop_bit="$(arg stop_bit)"
+    slave_id="$(arg slave_id)"
+    use_fake_hardware="false"
+    xyz="0.0 -0.019 0.0"
+    rpy="1.5708 0 0"/>
 </robot>
