Commit message: adding ur_standalone

File: src/ur5e_hande_robot_description/urdf/ur_with_epick.xacro (robot description, xacro)
@@ -43,5 +43,5 @@
    <xacro:arg name="tool_tcp_port" default="54321" />
      <!-- Simulation parameters -->
-   <xacro:arg name="use_fake_hardware" default="false" />
+   <xacro:arg name="use_fake_hardware" default="true" />
    <xacro:arg name="fake_sensor_commands" default="false" />
    <xacro:arg name="sim_gazebo" default="false" />

File: src/ur5e_hande_robot_description/urdf/ur_with_hande.urdf (robot description, URDF)
Before this commit: robot ur, 18 links, 17 joints
Links:
- added link tool_exchanger, mass 0.5; collision mesh filename=package://ur5e_hande_robot_description/meshes/tool_exchange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 scale=0.001 0.001 0.001; visual mesh filename=package://ur5e_hande_robot_description/meshes/tool_exchange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 scale=0.001 0.001 0.001
Joints:
- added joint tool_exchanger_joint: type fixed, parent flange, child tool_exchanger, origin xyz=0.010 0 0 rpy=0 0 1.5707963267948966
- joint robotiq_hande_coupler_joint: origin xyz=0 0 0 rpy=-1.5708 0 -1.5708 -> xyz=0.0 -0.019 0.0 rpy=1.5708 0 0; parent flange -> tool_exchanger

File: src/ur5e_hande_robot_description/urdf/ur_with_hande.xacro (robot description, xacro)
@@ -6,4 +6,5 @@
    <!-- import main macro -->
    <xacro:include filename="$(find ur_description)/urdf/ur_macro.xacro"/>
+   <xacro:include filename="$(find ur5e_hande_robot_description)/urdf/tool_exchanger.xacro"/>
    <xacro:include filename="$(find robotiq_hande_description)/urdf/robotiq_hande_gripper.xacro"/>
    <!-- possible 'ur_type' values: ur3, ur5e, ur5, ur5e, ur10, ur10e, ur16e, ur20 -->
@@ -47,4 +48,5 @@
    <xacro:arg name="sim_ignition" default="false" />
    <xacro:arg name="simulation_controllers" default="" />
+   <xacro:arg name="mock_hardware" default="true" />
    <!-- initial position for simulations (Fake Hardware, Gazebo, Ignition) -->
    <xacro:arg name="initial_positions_file" default="$(find ur_description)/config/initial_positions.yaml"/>
@@ -93,27 +95,28 @@
      <origin xyz="0 0 0" rpy="0 0 0" />          <!-- position robot in the map -->
    </xacro:ur_robot>
+  <xacro:tool_exchanger parent_link="$(arg tf_prefix)flange"/>
   <!-- hande gripper -->
-    <xacro:arg name="grip_pos_min" default="0"/>
-    <xacro:arg name="grip_pos_max" default="0.025"/>
-    <xacro:arg name="tty" default="/tmp/ttyUR"/>
-    <xacro:arg name="baudrate" default="115200"/>
-    <xacro:arg name="parity" default="N"/>
-    <xacro:arg name="data_bits" default="8"/>
-    <xacro:arg name="stop_bit" default="1"/>
-    <xacro:arg name="slave_id" default="9"/>
-    <xacro:robotiq_hande_gripper
-      name="robotiq_hande_gripper"
-      prefix="$(arg tf_prefix)"
-      parent="$(arg tf_prefix)flange"
-      grip_pos_min="$(arg grip_pos_min)"
-      grip_pos_max="$(arg grip_pos_max)"
-      tty="$(arg tty)"
-      baudrate="$(arg baudrate)"
-      parity="$(arg parity)"
-      data_bits="$(arg data_bits)"
-      stop_bit="$(arg stop_bit)"
-      slave_id="$(arg slave_id)"
-      use_fake_hardware="false"
-      xyz="0 0 0"
-      rpy="-1.5708 0 -1.5708"/>
+  <xacro:arg name="grip_pos_min" default="0"/>
+  <xacro:arg name="grip_pos_max" default="0.025"/>
+  <xacro:arg name="tty" default="/tmp/ttyUR"/>
+  <xacro:arg name="baudrate" default="115200"/>
+  <xacro:arg name="parity" default="N"/>
+  <xacro:arg name="data_bits" default="8"/>
+  <xacro:arg name="stop_bit" default="1"/>
+  <xacro:arg name="slave_id" default="9"/>
+  <xacro:robotiq_hande_gripper
+    name="robotiq_hande_gripper"
+    prefix="$(arg tf_prefix)"
+    parent="tool_exchanger"
+    grip_pos_min="$(arg grip_pos_min)"
+    grip_pos_max="$(arg grip_pos_max)"
+    tty="$(arg tty)"
+    baudrate="$(arg baudrate)"
+    parity="$(arg parity)"
+    data_bits="$(arg data_bits)"
+    stop_bit="$(arg stop_bit)"
+    slave_id="$(arg slave_id)"
+    use_fake_hardware="$(arg use_fake_hardware)"
+    xyz="0.0 -0.019 0.0"
+    rpy="1.5708 0 0"/>
 </robot>
