Commit message: replace zivid_assembly with smaller file

File: src/ur5e_hande_robot_description/urdf/zivid_camera_mount.xacro (robot description, xacro)
@@ -11,5 +11,5 @@
         <origin xyz="0 0 0" rpy="0 0 0"/>
         <geometry>
-          <mesh filename="package://ur5e_hande_robot_description/meshes/zivid/zivid_assembly.dae"
+          <mesh filename="package://ur5e_hande_robot_description/meshes/zivid/zivid_assembly_decimated.stl"
                 scale="${scale} ${scale} ${scale}"/>
         </geometry>
@@ -21,5 +21,5 @@
         <origin xyz="0 0 0" rpy="0 0 0"/>
         <geometry>
-          <mesh filename="package://ur5e_hande_robot_description/meshes/zivid/zivid_assembly.dae"
+          <mesh filename="package://ur5e_hande_robot_description/meshes/zivid/zivid_assembly_decimated.stl"
                 scale="${scale} ${scale} ${scale}"/>
         </geometry>
