Commit message: remove unused moveit_configs , descriptions add camera to standalone

File: src/ur5e_hande_robot_description/urdf/te_robotside.xacro (robot description, xacro)
@@ -1,5 +1,5 @@
 <?xml version="1.0"?>
 <robot xmlns:xacro="http://ros.org/wiki/xacro" name="wingman_toolchanger_robotside">
-  <xacro:macro name="te_robotside" params="parent_link">
+  <xacro:macro name="te_robotside" params="parent_link xyz:='0.010 0 0' rpy:='0 0 ${pi/2}'">
     <link name="te_robotside">
       <visual>
@@ -31,5 +31,5 @@
       <parent link="${parent_link}"/>
       <child link="te_robotside"/>
-      <origin xyz="0.010 0 0" rpy="0 0 ${pi/2}"/>
+      <origin xyz="${xyz}" rpy="${rpy}"/>
     </joint>
   </xacro:macro>

File: src/ur5e_hande_robot_description/urdf/ur_standalone.urdf (robot description, URDF)
Before this commit: robot ur, 14 links, 13 joints
Links:
- added link zivid_camera, mass 1.1; collision mesh filename=package://ur5e_hande_robot_description/meshes/zivid/zivid_a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 scale=1.0 1.0 1.0; visual mesh filename=package://ur5e_hande_robot_description/meshes/zivid/zivid_a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 scale=1.0 1.0 1.0
Joints:
- added joint zivid_camera_mount_joint: type fixed, parent flange, child zivid_camera, origin xyz=0.025 0 -0.105 rpy=-1.5708 0 -1.5708
- joint elbow_joint: origin xyz=-0.425339544116836 0 0 rpy=3.140592129600155 3.140015588611444 3.141577155253905 -> xyz=-0.425 0 0 rpy=0 0 0
- joint shoulder_lift_joint: origin xyz=5.074781107846515e-05 0 0 rpy=1.5704524934465869 0 -4.384813157010115e-07 -> xyz=0 0 0 rpy=1.570796327 0 0
- joint shoulder_pan_joint: origin xyz=0 0 0.1626011910349399 rpy=0 0 5.644671548406254e-08 -> xyz=0 0 0.1625 rpy=0 0 0
- joint te_robotside_joint: origin xyz=0.010 0 0 rpy=0 0 1.5707963267948966 -> xyz=0 -0.105 0 rpy=-1.5708 0 0; parent flange -> zivid_camera
- joint wrist_1_joint: origin xyz=-0.39212480859428955 -0.0007090153706380207 0.13387434235334733 rpy=0.005296076374611026 0.001323324865500051 4.849956441084167e-06 -> xyz=-0.3922 0 0.1333 rpy=0 0 0
- joint wrist_2_joint: origin xyz=-3.7545657827714984e-07 -0.0998688315746992 3.565303029367016e-05 rpy=1.5704393282377205 0 2.1955918973817767e-06 -> xyz=0 -0.0997 -2.044881182297852e-11 rpy=1.570796327 0 0
- joint wrist_3_joint: origin xyz=-2.3804544682715832e-05 0.09954804890217026 1.6577536206585414e-05 rpy=1.570962854780489 3.141592653589793 -3.141592619557402 -> xyz=0 0.0996 -2.042830148012698e-11 rpy=1.570796326589793 3.141592653589793 3.141592653589793

File: src/ur5e_hande_robot_description/urdf/ur_standalone.xacro (robot description, xacro)
@@ -6,4 +6,5 @@
    <!-- import main macro -->
    <xacro:include filename="$(find ur_description)/urdf/ur_macro.xacro"/>
+   <xacro:include filename="$(find ur5e_hande_robot_description)/urdf/zivid_camera_mount.xacro"/>
    <xacro:include filename="$(find ur5e_hande_robot_description)/urdf/te_robotside.xacro"/>
    <!-- possible 'ur_type' values: ur3, ur5e, ur5, ur5e, ur10, ur10e, ur16e, ur20 -->
@@ -94,4 +95,7 @@
      <origin xyz="0 0 0" rpy="0 0 0" />          <!-- position robot in the map -->
    </xacro:ur_robot>
-  <xacro:te_robotside parent_link="$(arg tf_prefix)flange"/>
+  <!-- Zivid camera mount attached to flange -->
+  <xacro:zivid_camera_mount parent_link="$(arg tf_prefix)flange" xyz="0.025 0 -0.105" rpy="-1.5708 0 -1.5708"/>
+  <!-- Tool exchanger robotside attached to camera -->
+  <xacro:te_robotside parent_link="zivid_camera" xyz="0 -0.105 0" rpy="-1.5708 0 0"/>
 </robot>
