Commit message: working new grippr with moveit

File: src/ur5e_2fg7_moveit_config/urdf/ur.urdf (robot description, URDF)
Before this commit: robot ur, 16 links, 15 joints
Links:
- removed link gripper_base_link
- removed link gripper_left_finger
- removed link gripper_right_finger
- added link _base_link, mass 0.25; collision mesh filename=package://ur5e_hande_robot_description/meshes/onrobot_2fg7_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 scale=1 1 1; visual mesh filename=package://ur5e_hande_robot_description/meshes/onrobot_2fg7_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 scale=1 1 1
- added link _left_finger, mass 0.1; collision mesh filename=package://ur5e_hande_robot_description/meshes/onrobot_2fg7_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 scale=1.0 1.0 1.0; visual mesh filename=package://ur5e_hande_robot_description/meshes/onrobot_2fg7_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 scale=1.0 1.0 1.0
- added link _right_finger, mass 0.1; collision mesh filename=package://ur5e_hande_robot_description/meshes/onrobot_2fg7_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 scale=1.0 1.0 1.0; visual mesh filename=package://ur5e_hande_robot_description/meshes/onrobot_2fg7_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 scale=1.0 1.0 1.0
Joints:
- removed joint gripper_base_joint
- removed joint gripper_left_finger_joint
- removed joint gripper_right_finger_joint
- added joint 2fg7_to_wrist_flange: type fixed, parent flange, child _base_link, origin xyz=0 0 0 rpy=0 0 0
- added joint _base_joint: type fixed, parent map, child _base_link, origin xyz=0 0 0 rpy=0 0 0
- added joint _left_finger_joint: type prismatic, parent _base_link, child _left_finger, origin xyz=0.10972 0.0175 0 rpy=0.0 0.0 0.0, axis 0 1 0, limit lower=0.0 upper=0.019 effort=1.0 velocity=0.6
- added joint _right_finger_joint: type prismatic, parent _base_link, child _right_finger, origin xyz=0.10972 -0.0175 0 rpy=0.0 0.0 0.0, axis 0 -1 0, limit lower=0.0 upper=0.019 effort=1.0 velocity=0.6, mimic joint=_left_finger_joint multiplier=1.0 offset=0
- joint elbow_joint: origin xyz=-0.425339544116836 0 0 rpy=3.140592129600155 3.140015588611444 3.141577155253905 -> xyz=-0.425 0 0 rpy=0 0 0
- joint shoulder_lift_joint: origin xyz=5.074781107846515e-05 0 0 rpy=1.5704524934465869 0 -4.384813157010115e-07 -> xyz=0 0 0 rpy=1.570796327 0 0
- joint shoulder_pan_joint: origin xyz=0 0 0.1626011910349399 rpy=0 0 5.644671548406254e-08 -> xyz=0 0 0.1625 rpy=0 0 0
- joint wrist_1_joint: origin xyz=-0.39212480859428955 -0.0007090153706380207 0.13387434235334733 rpy=0.005296076374611026 0.001323324865500051 4.849956441084167e-06 -> xyz=-0.3922 0 0.1333 rpy=0 0 0
- joint wrist_2_joint: origin xyz=-3.7545657827714984e-07 -0.0998688315746992 3.565303029367016e-05 rpy=1.5704393282377205 0 2.1955918973817767e-06 -> xyz=0 -0.0997 -2.044881182297852e-11 rpy=1.570796327 0 0
- joint wrist_3_joint: origin xyz=-2.3804544682715832e-05 0.09954804890217026 1.6577536206585414e-05 rpy=1.570962854780489 3.141592653589793 -3.141592619557402 -> xyz=0 0.0996 -2.042830148012698e-11 rpy=1.570796326589793 3.141592653589793 3.141592653589793
