Commit message: change world to map , fixed frame

File: src/ur5e_hande_moveit_config/urdf/ur.urdf (robot description, URDF)
Before this commit: robot ur, 18 links, 17 joints
Links:
- removed link world
- added link map
Joints:
- joint base_joint: parent world -> map

File: src/ur5e_hande_moveit_config/urdf/ur_with_2fg7.urdf (robot description, URDF)
Before this commit: robot ur, 16 links, 16 joints
Links:
- removed link world
- added link map
Joints:
- joint _base_joint: parent world -> map
- joint base_joint: parent world -> map

File: src/ur5e_hande_robot_description/urdf/ur_with_2fg7.xacro (robot description, xacro)
@@ -51,11 +51,11 @@
    <!-- convert to property to use substitution in function -->
    <xacro:property name="initial_positions_file" default="$(arg initial_positions_file)"/>
-   <!-- create link fixed to the "world" -->
-   <link name="world" />
+   <!-- create link fixed to the "map" -->
+   <link name="map" />
    <!-- arm -->
    <xacro:ur_robot
      name="$(arg name)"
      tf_prefix="$(arg tf_prefix)"
-     parent="world"
+     parent="map"
      joint_limits_parameters_file="$(arg joint_limit_params)"
      kinematics_parameters_file="$(arg kinematics_params)"
@@ -91,10 +91,10 @@
      trajectory_port="$(arg trajectory_port)"
      >
-     <origin xyz="0 0 0" rpy="0 0 0" />          <!-- position robot in the world -->
+     <origin xyz="0 0 0" rpy="0 0 0" />          <!-- position robot in the map -->
    </xacro:ur_robot>
     <!-- Call the robot gripper -->
     <xacro:onrobot_2fg7_gripper
      tf_prefix="$(arg tf_prefix)"
-     parent="world">
+     parent="map">
     <origin xyz="0 0 0" rpy="0 0 0" />
     </xacro:onrobot_2fg7_gripper>

File: src/ur5e_hande_robot_description/urdf/ur_with_camera_hande.xacro (robot description, xacro)
@@ -52,11 +52,11 @@
    <!-- convert to property to use substitution in function -->
    <xacro:property name="initial_positions_file" default="$(arg initial_positions_file)"/>
-   <!-- create link fixed to the "world" -->
-   <link name="world" />
+   <!-- create link fixed to the "map" -->
+   <link name="map" />
    <!-- arm -->
    <xacro:ur_robot
      name="$(arg name)"
      tf_prefix="$(arg tf_prefix)"
-     parent="world"
+     parent="map"
      joint_limits_parameters_file="$(find ur_description)/config/$(arg ur_type)/joint_limits.yaml"
      kinematics_parameters_file="$(find ur_description)/config/$(arg ur_type)/default_kinematics.yaml"
@@ -92,10 +92,10 @@
      trajectory_port="$(arg trajectory_port)"
      >
-     <origin xyz="0 0 0" rpy="0 0 0" />          <!-- position robot in the world -->
+     <origin xyz="0 0 0" rpy="0 0 0" />          <!-- position robot in the map -->
    </xacro:ur_robot>
     <!-- Call the robot gripper -->
     <xacro:robotiq_hande
      tf_prefix="$(arg tf_prefix)"
-     parent="world"
+     parent="map"
    />
     <xacro:camera_mount

File: src/ur5e_hande_robot_description/urdf/ur_with_hande.xacro (robot description, xacro)
@@ -51,11 +51,11 @@
    <!-- convert to property to use substitution in function -->
    <xacro:property name="initial_positions_file" default="$(arg initial_positions_file)"/>
-   <!-- create link fixed to the "world" -->
-   <link name="world" />
+   <!-- create link fixed to the "map" -->
+   <link name="map" />
    <!-- arm -->
    <xacro:ur_robot
      name="$(arg name)"
      tf_prefix="$(arg tf_prefix)"
-     parent="world"
+     parent="map"
      joint_limits_parameters_file="$(arg joint_limit_params)"
      kinematics_parameters_file="$(arg kinematics_params)"
@@ -91,10 +91,10 @@
      trajectory_port="$(arg trajectory_port)"
      >
-     <origin xyz="0 0 0" rpy="0 0 0" />          <!-- position robot in the world -->
+     <origin xyz="0 0 0" rpy="0 0 0" />          <!-- position robot in the map -->
    </xacro:ur_robot>
     <!-- Call the robot gripper -->
     <xacro:robotiq_hande
      tf_prefix="$(arg tf_prefix)"
-     parent="world"
+     parent="map"
    />
     <!-- attach the gripper to the arm -->

Commit message: onrobot driver testing

File: src/ur5e_hande_moveit_config/urdf/ur.urdf (robot description, URDF)
Before this commit: robot ur, 18 links, 17 joints
Joints:
- joint joint_finger: limit lower=0 upper=0.025 effort=130 velocity=0.15 -> lower=0.0 upper=0.025 effort=100 velocity=0.15; type fixed -> prismatic
- joint robotiq_hande_base_to_right_finger: limit lower=0 upper=0.025 effort=130 velocity=0.15 -> lower=0.0 upper=0.025 effort=100 velocity=0.15; mimic joint=joint_finger multiplier=1 offset=0 -> joint=joint_finger multiplier=1.0 offset=0.0; type fixed -> prismatic

File: src/ur5e_hande_robot_description/urdf/hande.xacro (robot description, xacro)
@@ -124,5 +124,5 @@
       <child link="${tf_prefix}robotiq_hande_base_link"/>
     </joint>
-    <joint name="${tf_prefix}joint_finger" type="fixed">
+    <joint name="${tf_prefix}joint_finger" type="prismatic">
       <origin rpy="0 0 ${pi/2.0}" xyz="0 0 0.05"/>
       <parent link="${tf_prefix}robotiq_hande_base_link"/>
@@ -131,5 +131,5 @@
       <limit effort="130" lower="0" upper="0.025" velocity="0.15"/>
     </joint>
-    <joint name="robotiq_hande_base_to_${tf_prefix}right_finger" type="fixed">
+    <joint name="robotiq_hande_base_to_${tf_prefix}right_finger" type="prismatic">
       <origin rpy="0 0 ${pi/2.0}" xyz="0 0 0.05"/>
       <parent link="${tf_prefix}robotiq_hande_base_link"/>

File: src/ur5e_hande_robot_description/urdf/ur_with_hande.xacro (robot description, xacro)
@@ -104,3 +104,12 @@
       <origin xyz="0.005 0 0" rpy="-${pi/2.0} 0 ${pi/2.0}" />
     </joint>
+    <ros2_control name="gripper" type="system">
+      <hardware>
+        <plugin>fake_components/GenericSystem</plugin>
+      </hardware>
+      <joint name="joint_finger">
+        <command_interface name="position"/>
+        <state_interface name="position"/>
+      </joint>
+    </ros2_control>
 </robot>

Commit message: changing global frame from 'map' to 'world'

File: src/ur5e_hande_moveit_config/urdf/ur.urdf (robot description, URDF)
Before this commit: robot ur, 18 links, 17 joints
Links:
- removed link map
- added link world
Joints:
- joint base_joint: parent map -> world

File: src/ur5e_hande_robot_description/urdf/ur_with_hande.xacro (robot description, xacro)
@@ -52,10 +52,10 @@
    <xacro:property name="initial_positions_file" default="$(arg initial_positions_file)"/>
    <!-- create link fixed to the "map" -->
-   <link name="map" />
+   <link name="world" />
    <!-- arm -->
    <xacro:ur_robot
      name="$(arg name)"
      tf_prefix="$(arg tf_prefix)"
-     parent="map"
+     parent="world"
      joint_limits_parameters_file="$(arg joint_limit_params)"
      kinematics_parameters_file="$(arg kinematics_params)"
@@ -96,5 +96,5 @@
     <xacro:robotiq_hande
      tf_prefix="$(arg tf_prefix)"
-     parent="map"
+     parent="world"
    />
     <!-- attach the gripper to the arm -->

Commit message: global frame from world to map

File: src/ur5e_hande_moveit_config/urdf/ur.urdf (robot description, URDF)
Before this commit: robot ur, 18 links, 17 joints
Links:
- removed link world
- added link map
Joints:
- joint base_joint: parent world -> map

File: src/ur5e_hande_robot_description/urdf/ur_with_hande.xacro (robot description, xacro)
@@ -52,10 +52,10 @@
    <xacro:property name="initial_positions_file" default="$(arg initial_positions_file)"/>
    <!-- create link fixed to the "map" -->
-   <link name="world" />
+   <link name="map" />
    <!-- arm -->
    <xacro:ur_robot
      name="$(arg name)"
      tf_prefix="$(arg tf_prefix)"
-     parent="world"
+     parent="map"
      joint_limits_parameters_file="$(arg joint_limit_params)"
      kinematics_parameters_file="$(arg kinematics_params)"
@@ -96,5 +96,5 @@
     <xacro:robotiq_hande
      tf_prefix="$(arg tf_prefix)"
-     parent="world"
+     parent="map"
    />
     <!-- attach the gripper to the arm -->
