Commit message: Updated ur_hande_moveit_config

File: src/actual_moveit_config/urdf/ur.urdf (robot description, URDF)
Before this commit: robot ur, 16 links, 16 joints
Links:
- removed link _base_link
- removed link _left_finger
- removed link _right_finger
- added link grasping_point_link
- added link left_finger, mass 0.03804; collision mesh filename=package://ur5e_hande_robot_description/meshes/hande/collisi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 scale=0.001 0.001 0.001; visual mesh filename=package://ur5e_hande_robot_description/meshes/hande/visual/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 scale=0.001 0.001 0.001
- added link right_finger, mass 0.03804; collision mesh filename=package://ur5e_hande_robot_description/meshes/hande/collisi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 scale=0.001 0.001 0.001; visual mesh filename=package://ur5e_hande_robot_description/meshes/hande/visual/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 scale=0.001 0.001 0.001
- added link robotiq_coupler, mass 0.100; collision mesh filename=package://ur5e_hande_robot_description/meshes/hande/collisi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 scale=1 1 1; visual mesh filename=package://ur5e_hande_robot_description/meshes/hande/visual/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 scale=1 1 1
- added link robotiq_hande_base_link, mass 1.4; collision mesh filename=package://ur5e_hande_robot_description/meshes/hande/collisi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 scale=1 1 1; visual mesh filename=package://ur5e_hande_robot_description/meshes/hande/visual/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 scale=1 1 1
Joints:
- removed joint 2fg7_to_wrist_flange
- removed joint _base_joint
- removed joint _left_finger_joint
- removed joint _right_finger_joint
- added joint grasping_point: type fixed, parent robotiq_hande_base_link, child grasping_point_link, origin xyz=0.0 0.0 0.09 rpy=0 0 0, axis 0 0 0
- added joint hande_to_wrist_flange: type fixed, parent flange, child robotiq_coupler, origin xyz=0.005 0 0 rpy=-1.5707963267948966 0 1.5707963267948966
- added joint joint_finger: type prismatic, parent robotiq_hande_base_link, child left_finger, origin xyz=0 0 0.05 rpy=0 0 1.5707963267948966, axis -1 0 0, limit lower=0 upper=0.025 effort=130 velocity=0.15
- added joint robotiq_coupler_joint: type fixed, parent robotiq_coupler, child robotiq_hande_base_link, origin xyz=0 0 -0.05 rpy=3.141592653589793 0 -1.5707963267948966
- added joint robotiq_hande_base_to_right_finger: type prismatic, parent robotiq_hande_base_link, child right_finger, origin xyz=0 0 0.05 rpy=0 0 1.5707963267948966, axis 1 0 0, limit lower=0 upper=0.025 effort=130 velocity=0.15, mimic joint=joint_finger multiplier=1 offset=0
- joint elbow_joint: origin xyz=-0.425 0 0 rpy=0 0 0 -> xyz=-0.425339544116836 0 0 rpy=3.140592129600155 3.140015588611444 3.141577155253905
- joint shoulder_lift_joint: origin xyz=0 0 0 rpy=1.570796327 0 0 -> xyz=5.074781107846515e-05 0 0 rpy=1.5704524934465869 0 -4.384813157010115e-07
- joint shoulder_pan_joint: origin xyz=0 0 0.1625 rpy=0 0 0 -> xyz=0 0 0.1626011910349399 rpy=0 0 5.644671548406254e-08
- joint wrist_1_joint: origin xyz=-0.3922 0 0.1333 rpy=0 0 0 -> xyz=-0.39212480859428955 -0.0007090153706380207 0.13387434235334733 rpy=0.005296076374611026 0.001323324865500051 4.849956441084167e-06
- joint wrist_2_joint: origin xyz=0 -0.0997 -2.044881182297852e-11 rpy=1.570796327 0 0 -> xyz=-3.7545657827714984e-07 -0.0998688315746992 3.565303029367016e-05 rpy=1.5704393282377205 0 2.1955918973817767e-06
- joint wrist_3_joint: origin xyz=0 0.0996 -2.042830148012698e-11 rpy=1.570796326589793 3.141592653589793 3.141592653589793 -> xyz=-2.3804544682715832e-05 0.09954804890217026 1.6577536206585414e-05 rpy=1.570962854780489 3.141592653589793 -3.141592619557402
