Commit message: removed hande.xacro , call directly

File: src/robotiq_hande_description/urdf/robotiq_hande_gripper.xacro (robot description, xacro)
@@ -6,5 +6,22 @@
   <xacro:include filename="$(find robotiq_hande_description)/urdf/robotiq_hande_gripper.ros2_control.xacro"/>
   <xacro:include filename="$(find robotiq_hande_description)/urdf/cylinder_inertial.xacro"/>
-  <xacro:macro name="robotiq_hande_gripper" params="name prefix parent grip_pos_min grip_pos_max tty baudrate parity data_bits stop_bit slave_id use_fake_hardware coupler_mass:=0.119">
+  <xacro:macro
+    name="robotiq_hande_gripper"
+    params="name
+            prefix
+            parent
+            grip_pos_min
+            grip_pos_max
+            tty
+            baudrate
+            parity
+            data_bits
+            stop_bit
+            slave_id
+            use_fake_hardware
+            coupler_mass:=0.119
+            xyz:='0 0 0'
+            rpy:='0 0 0'"
+  >
     <!-- ros2_control parameters  -->
     <xacro:robotiq_hande_ros2_control
@@ -22,6 +39,6 @@
     />
     <!-- Robotiq Hand-E specs -->
-    <!--  + Height added by the IO coupler 11.0mm -->
-    <!--  + Height added by the Hand-E 99.0mm -->
+    <!--  + Height added by the IO coupler: 11.0mm -->
+    <!--  + Height added by the Hand-E: 99.0mm -->
     <!--  + Coupler mass includes the bolts -->
     <xacro:arg name="coupler_height" default="0.011"/>
@@ -32,5 +49,5 @@
     <xacro:arg name="hande_radius" default="0.0375"/>
     <joint name="${prefix}robotiq_hande_coupler_joint" type="fixed">
-      <origin xyz="0 0 0" rpy="-${pi/2} 0 -${pi/2}"/>
+      <origin xyz="${xyz}" rpy="${rpy}"/>
       <parent link="${parent}"/>
       <child link="${prefix}robotiq_hande_coupler"/>

File: src/ur5e_hande_robot_description/urdf/ur_with_hande.xacro (robot description, xacro)
@@ -6,5 +6,5 @@
    <!-- import main macro -->
    <xacro:include filename="$(find ur_description)/urdf/ur_macro.xacro"/>
-   <xacro:include filename="$(find ur5e_hande_robot_description)/urdf/hande.xacro"/>
+   <xacro:include filename="$(find robotiq_hande_description)/urdf/robotiq_hande_gripper.xacro"/>
    <!-- possible 'ur_type' values: ur3, ur5e, ur5, ur5e, ur10, ur10e, ur16e, ur20 -->
    <!-- the default value should raise an error in case this was called without defining the type -->
@@ -94,10 +94,27 @@
      <origin xyz="0 0 0" rpy="0 0 0" />          <!-- position robot in the map -->
    </xacro:ur_robot>
-    <!-- Call the robot gripper -->
-    <xacro:hande
-     parent="$(arg tf_prefix)flange"
-     prefix="$(arg tf_prefix)"
-     mock_hardware="$(arg mock_hardware)">
-    </xacro:hande>
-    <xacro:property name="print_mock_hardware" value="${xacro:log('mock_hardware: ' + str(mock_hardware))}"/>
+  <!-- hande gripper -->
+    <xacro:arg name="grip_pos_min" default="0"/>
+    <xacro:arg name="grip_pos_max" default="0.025"/>
+    <xacro:arg name="tty" default="/tmp/ttyUR"/>
+    <xacro:arg name="baudrate" default="115200"/>
+    <xacro:arg name="parity" default="N"/>
+    <xacro:arg name="data_bits" default="8"/>
+    <xacro:arg name="stop_bit" default="1"/>
+    <xacro:arg name="slave_id" default="9"/>
+    <xacro:robotiq_hande_gripper
+      name="robotiq_hande_gripper"
+      prefix="$(arg tf_prefix)"
+      parent="$(arg tf_prefix)flange"
+      grip_pos_min="$(arg grip_pos_min)"
+      grip_pos_max="$(arg grip_pos_max)"
+      tty="$(arg tty)"
+      baudrate="$(arg baudrate)"
+      parity="$(arg parity)"
+      data_bits="$(arg data_bits)"
+      stop_bit="$(arg stop_bit)"
+      slave_id="$(arg slave_id)"
+      use_fake_hardware="$(arg mock_hardware)"
+      xyz="0 0 0"
+      rpy="-1.5708 0 -1.5708"/>
 </robot>
