Commit message: fixed gripper issues and new compressed dae files

File: src/robotiq_hande_description/urdf/robotiq_hande_gripper.ros2_control.xacro (robot description, xacro)
@@ -1,5 +1,8 @@
 <?xml version="1.0"?>
 <robot xmlns:xacro="http://www.ros.org/wiki/xacro">
-  <xacro:macro name="robotiq_hande_ros2_control" params="name prefix grip_pos_min grip_pos_max tty baudrate parity data_bits stop_bit slave_id use_fake_hardware">
+  <xacro:macro
+    name="robotiq_hande_ros2_control"
+    params="name prefix grip_pos_min grip_pos_max tty_port baudrate parity data_bits stop_bit slave_id frequency_hz create_socat_tty ip_adress port use_fake_hardware"
+  >
     <ros2_control name="${name}" type="system">
       <hardware>
@@ -11,5 +14,5 @@
           <param name="grip_pos_min">${grip_pos_min}</param>
           <param name="grip_pos_max">${grip_pos_max}</param>
-          <param name="tty">${tty}</param>
+          <param name="tty_port">${tty_port}</param>
           <param name="baudrate">${baudrate}</param>
           <param name="parity">${parity}</param>
@@ -17,4 +20,8 @@
           <param name="stop_bit">${stop_bit}</param>
           <param name="slave_id">${slave_id}</param>
+          <param name="frequency_hz">${frequency_hz}</param>
+          <param name="create_socat_tty">${create_socat_tty}</param>
+          <param name="ip_adress">${ip_adress}</param>
+          <param name="port">${port}</param>
         </xacro:unless>
       </hardware>

File: src/robotiq_hande_description/urdf/robotiq_hande_gripper.xacro (robot description, xacro)
@@ -13,5 +13,5 @@
             grip_pos_min
             grip_pos_max
-            tty
+            tty_port
             baudrate
             parity
@@ -20,4 +20,8 @@
             slave_id
             use_fake_hardware
+            frequency_hz:=10
+            create_socat_tty:=false
+            ip_adress:=192.168.100.10
+            port:=54321
             coupler_mass:=0.119
             xyz:='0 0 0'
@@ -30,5 +34,5 @@
       grip_pos_min="${grip_pos_min}"
       grip_pos_max="${grip_pos_max}"
-      tty="${tty}"
+      tty_port="${tty_port}"
       baudrate="${baudrate}"
       parity="${parity}"
@@ -36,4 +40,8 @@
       stop_bit="${stop_bit}"
       slave_id="${slave_id}"
+      frequency_hz="${frequency_hz}"
+      create_socat_tty="${create_socat_tty}"
+      ip_adress="${ip_adress}"
+      port="${port}"
       use_fake_hardware="${use_fake_hardware}"
     />

File: src/ur5e_hande_robot_description/urdf/ur_with_hande.xacro (robot description, xacro)
@@ -99,5 +99,5 @@
   <xacro:arg name="grip_pos_min" default="0"/>
   <xacro:arg name="grip_pos_max" default="0.025"/>
-  <xacro:arg name="tty" default="/tmp/ttyUR"/>
+  <xacro:arg name="tty_port" default="/tmp/ttyUR"/>
   <xacro:arg name="baudrate" default="115200"/>
   <xacro:arg name="parity" default="N"/>
@@ -105,4 +105,7 @@
   <xacro:arg name="stop_bit" default="1"/>
   <xacro:arg name="slave_id" default="9"/>
+  <xacro:arg name="create_socat_tty" default="true"/>
+  <xacro:arg name="ip_adress" default="192.168.1.101"/>
+  <xacro:arg name="port" default="54321"/>
   <xacro:robotiq_hande_gripper
     name="robotiq_hande_gripper"
@@ -111,5 +114,5 @@
     grip_pos_min="$(arg grip_pos_min)"
     grip_pos_max="$(arg grip_pos_max)"
-    tty="$(arg tty)"
+    tty_port="$(arg tty_port)"
     baudrate="$(arg baudrate)"
     parity="$(arg parity)"
@@ -117,6 +120,10 @@
     stop_bit="$(arg stop_bit)"
     slave_id="$(arg slave_id)"
-    use_fake_hardware="true"
+    use_fake_hardware="$(arg use_fake_hardware)"
     xyz="0.0 -0.019 0.0"
-    rpy="1.5708 0 0"/>
+    rpy="1.5708 0 0"
+    create_socat_tty="$(arg create_socat_tty)"
+    ip_adress="$(arg ip_adress)"
+    port="$(arg port)"
+  />
 </robot>

File: src/ur5e_hande_robot_description/urdf/ur_with_hande_no_te.xacro (robot description, xacro)
@@ -96,5 +96,5 @@
     <xacro:arg name="grip_pos_min" default="0"/>
     <xacro:arg name="grip_pos_max" default="0.025"/>
-    <xacro:arg name="tty" default="/tmp/ttyUR"/>
+    <xacro:arg name="tty_port" default="/tmp/ttyUR"/>
     <xacro:arg name="baudrate" default="115200"/>
     <xacro:arg name="parity" default="N"/>
@@ -108,5 +108,5 @@
       grip_pos_min="$(arg grip_pos_min)"
       grip_pos_max="$(arg grip_pos_max)"
-      tty="$(arg tty)"
+      tty_port="$(arg tty_port)"
       baudrate="$(arg baudrate)"
       parity="$(arg parity)"

File: src/ur5e_hande_robot_description/urdf/ur_with_zivid_hande.xacro (robot description, xacro)
@@ -102,5 +102,5 @@
   <xacro:arg name="grip_pos_min" default="0"/>
   <xacro:arg name="grip_pos_max" default="0.025"/>
-  <xacro:arg name="tty" default="/tmp/ttyUR"/>
+  <xacro:arg name="tty_port" default="/tmp/ttyUR"/>
   <xacro:arg name="baudrate" default="115200"/>
   <xacro:arg name="parity" default="N"/>
@@ -108,4 +108,7 @@
   <xacro:arg name="stop_bit" default="1"/>
   <xacro:arg name="slave_id" default="9"/>
+  <xacro:arg name="create_socat_tty" default="true"/>
+  <xacro:arg name="ip_adress" default="192.168.1.101"/>
+  <xacro:arg name="port" default="54321"/>
   <xacro:robotiq_hande_gripper
     name="robotiq_hande_gripper"
@@ -114,5 +117,5 @@
     grip_pos_min="$(arg grip_pos_min)"
     grip_pos_max="$(arg grip_pos_max)"
-    tty="$(arg tty)"
+    tty_port="$(arg tty_port)"
     baudrate="$(arg baudrate)"
     parity="$(arg parity)"
@@ -120,6 +123,10 @@
     stop_bit="$(arg stop_bit)"
     slave_id="$(arg slave_id)"
-    use_fake_hardware="true"
+    use_fake_hardware="$(arg use_fake_hardware)"
     xyz="0 -0.02 0"
-    rpy="-1.5708 0 3.1416"/>
+    rpy="-1.5708 0 3.1416"
+    create_socat_tty="$(arg create_socat_tty)"
+    ip_adress="$(arg ip_adress)"
+    port="$(arg port)"
+  />
 </robot>
