Commit message: Updated launch file

File: src/ur5e_hande_moveit_config/config/ur.ros2_control.xacro (robot description, xacro)
@@ -2,5 +2,5 @@
 <robot xmlns:xacro="http://www.ros.org/wiki/xacro">
     <xacro:macro name="ur_ros2_control" params="name initial_positions_file">
-        <xacro:property name="initial_positions" value="${load_yaml(initial_positions_file)['initial_positions']}"/>
+        <xacro:property name="initial_positions" value="${xacro.load_yaml(initial_positions_file)['initial_positions']}"/>
         <ros2_control name="${name}" type="system">
             <hardware>

File: src/ur5e_hande_robot_description/urdf/ur_with_hande.xacro (robot description, xacro)
@@ -47,4 +47,5 @@
    <xacro:arg name="sim_ignition" default="false" />
    <xacro:arg name="simulation_controllers" default="" />
+   <xacro:arg name="mock_hardware" default="true" />
    <!-- initial position for simulations (Fake Hardware, Gazebo, Ignition) -->
    <xacro:arg name="initial_positions_file" default="$(find ur_description)/config/initial_positions.yaml"/>
@@ -93,10 +94,10 @@
      <origin xyz="0 0 0" rpy="0 0 0" />          <!-- position robot in the map -->
    </xacro:ur_robot>
-    <xacro:arg name="mock_hardware" default="true" />
     <!-- Call the robot gripper -->
     <xacro:hande
      parent="$(arg tf_prefix)flange"
      prefix="$(arg tf_prefix)"
-     mock_hardware="$(arg use_fake_hardware)">
+     mock_hardware="$(arg mock_hardware)">
     </xacro:hande>
+    <xacro:property name="print_mock_hardware" value="${xacro:log('mock_hardware: ' + str(mock_hardware))}"/>
 </robot>

Commit message: adding tool_exchanger for viz

File: src/ur5e_hande_moveit_config/config/ur.ros2_control.xacro (robot description, xacro)
@@ -2,5 +2,5 @@
 <robot xmlns:xacro="http://www.ros.org/wiki/xacro">
     <xacro:macro name="ur_ros2_control" params="name initial_positions_file">
-        <xacro:property name="initial_positions" value="${xacro.load_yaml(initial_positions_file)['initial_positions']}"/>
+        <xacro:property name="initial_positions" value="${load_yaml(initial_positions_file)['initial_positions']}"/>
         <ros2_control name="${name}" type="system">
             <hardware>

File: src/ur5e_hande_robot_description/urdf/ur_with_hande.urdf (robot description, URDF)
Before this commit: robot ur, 18 links, 17 joints
Joints:
- joint robotiq_hande_coupler_joint: origin xyz=0 0 0 rpy=-1.5707963267948966 0 -1.5707963267948966 -> xyz=0 0 0 rpy=-1.5708 0 -1.5708
