Commit message: rename from ur5e_hande_robot_description to ur5e_robot_description

File: src/moveit_configs/ur_standalone_moveit_config/config/ur.urdf.xacro (robot description, xacro)
@@ -3,5 +3,5 @@
     <xacro:arg name="initial_positions_file" default="initial_positions.yaml" />
     <!-- Import ur urdf file -->
-    <xacro:include filename="$(find ur5e_hande_robot_description)/urdf/ur_standalone.urdf" />
+    <xacro:include filename="$(find ur5e_robot_description)/urdf/ur_standalone.urdf" />
     <!-- Import control_xacro -->
     <xacro:include filename="ur.ros2_control.xacro" />

File: src/moveit_configs/ur_zivid_epick_moveit_config/config/ur.urdf.xacro (robot description, xacro)
@@ -3,5 +3,5 @@
     <xacro:arg name="initial_positions_file" default="initial_positions.yaml" />
     <!-- Import ur urdf file -->
-    <xacro:include filename="$(find ur5e_hande_robot_description)/urdf/ur_with_zivid_epick.urdf" />
+    <xacro:include filename="$(find ur5e_robot_description)/urdf/ur_with_zivid_epick.urdf" />
     <!-- Import control_xacro -->
     <xacro:include filename="ur.ros2_control.xacro" />

File: src/moveit_configs/ur_zivid_hande_moveit_config/config/ur.urdf.xacro (robot description, xacro)
@@ -3,5 +3,5 @@
     <xacro:arg name="initial_positions_file" default="initial_positions.yaml" />
     <!-- Import ur urdf file -->
-    <xacro:include filename="$(find ur5e_hande_robot_description)/urdf/ur_with_zivid_hande.urdf" />
+    <xacro:include filename="$(find ur5e_robot_description)/urdf/ur_with_zivid_hande.urdf" />
     <!-- Import control_xacro -->
     <xacro:include filename="ur.ros2_control.xacro" />

File: src/ur5e_hande_moveit_config/config/ur.urdf.xacro (robot description, xacro)
@@ -3,5 +3,5 @@
     <xacro:arg name="initial_positions_file" default="initial_positions.yaml" />
     <!-- Import ur urdf file -->
-    <xacro:include filename="$(find ur5e_hande_robot_description)/urdf/ur_with_hande.urdf" />
+    <xacro:include filename="$(find ur5e_robot_description)/urdf/ur_with_hande.urdf" />
     <!-- Import control_xacro -->
     <xacro:include filename="ur.ros2_control.xacro" />

File: src/ur5e_robot_description/urdf/te_robotside.xacro (robot description, xacro)
@@ -1,11 +1,11 @@
 <?xml version="1.0"?>
-<robot xmlns:xacro="http://ros.org/wiki/xacro" name="tool_block">
-  <xacro:macro name="tool_block" params="parent_link xyz:='0 0 0' rpy:='0 0 0' scale:='0.001' mass:='0.2'">
-    <link name="tool_block">
+<robot xmlns:xacro="http://ros.org/wiki/xacro" name="wingman_toolchanger_robotside">
+  <xacro:macro name="te_robotside" params="parent_link xyz:='0.010 0 0' rpy:='0 0 ${pi/2}'">
+    <link name="te_robotside">
       <visual>
         <origin xyz="0 0 0" rpy="0 0 0"/>
         <geometry>
-          <mesh filename="package://ur5e_hande_robot_description/meshes/tool_exchanger/Tool_block.stl"
-                scale="${scale} ${scale} ${scale}"/>
+          <mesh filename="package://ur5e_robot_description/meshes/tool_exchanger/TE_RobotSide.stl"
+                scale="0.001 0.001 0.001"/>
         </geometry>
         <material name="grey">
@@ -16,10 +16,10 @@
         <origin xyz="0 0 0" rpy="0 0 0"/>
         <geometry>
-          <mesh filename="package://ur5e_hande_robot_description/meshes/tool_exchanger/Tool_block.stl"
-                scale="${scale} ${scale} ${scale}"/>
+          <mesh filename="package://ur5e_robot_description/meshes/tool_exchanger/TE_RobotSide.stl"
+                scale="0.001 0.001 0.001"/>
         </geometry>
       </collision>
       <inertial>
-        <mass value="${mass}"/>
+        <mass value="0.5"/>
         <origin xyz="0 0 0" rpy="0 0 0"/>
         <inertia ixx="0.001" ixy="0.0" ixz="0.0"
@@ -28,7 +28,7 @@
       </inertial>
     </link>
-    <joint name="tool_block_joint" type="fixed">
+    <joint name="te_robotside_joint" type="fixed">
       <parent link="${parent_link}"/>
-      <child link="tool_block"/>
+      <child link="te_robotside"/>
       <origin xyz="${xyz}" rpy="${rpy}"/>
     </joint>

File: src/ur5e_robot_description/urdf/tool_block.xacro (robot description, xacro)
@@ -1,11 +1,11 @@
 <?xml version="1.0"?>
-<robot xmlns:xacro="http://ros.org/wiki/xacro" name="wingman_toolchanger_robotside">
-  <xacro:macro name="te_robotside" params="parent_link xyz:='0.010 0 0' rpy:='0 0 ${pi/2}'">
-    <link name="te_robotside">
+<robot xmlns:xacro="http://ros.org/wiki/xacro" name="tool_block">
+  <xacro:macro name="tool_block" params="parent_link xyz:='0 0 0' rpy:='0 0 0' scale:='0.001' mass:='0.2'">
+    <link name="tool_block">
       <visual>
         <origin xyz="0 0 0" rpy="0 0 0"/>
         <geometry>
-          <mesh filename="package://ur5e_hande_robot_description/meshes/tool_exchanger/TE_RobotSide.stl"
-                scale="0.001 0.001 0.001"/>
+          <mesh filename="package://ur5e_robot_description/meshes/tool_exchanger/Tool_block.stl"
+                scale="${scale} ${scale} ${scale}"/>
         </geometry>
         <material name="grey">
@@ -16,10 +16,10 @@
         <origin xyz="0 0 0" rpy="0 0 0"/>
         <geometry>
-          <mesh filename="package://ur5e_hande_robot_description/meshes/tool_exchanger/TE_RobotSide.stl"
-                scale="0.001 0.001 0.001"/>
+          <mesh filename="package://ur5e_robot_description/meshes/tool_exchanger/Tool_block.stl"
+                scale="${scale} ${scale} ${scale}"/>
         </geometry>
       </collision>
       <inertial>
-        <mass value="0.5"/>
+        <mass value="${mass}"/>
         <origin xyz="0 0 0" rpy="0 0 0"/>
         <inertia ixx="0.001" ixy="0.0" ixz="0.0"
@@ -28,7 +28,7 @@
       </inertial>
     </link>
-    <joint name="te_robotside_joint" type="fixed">
+    <joint name="tool_block_joint" type="fixed">
       <parent link="${parent_link}"/>
-      <child link="te_robotside"/>
+      <child link="tool_block"/>
       <origin xyz="${xyz}" rpy="${rpy}"/>
     </joint>

File: src/ur5e_robot_description/urdf/ur_standalone.urdf (robot description, URDF)
Before this commit: robot ur, 20 links, 19 joints
Links:
- removed link robotiq_hande_coupler
- removed link robotiq_hande_end
- removed link robotiq_hande_left_finger
- removed link robotiq_hande_link
- removed link robotiq_hande_right_finger
- removed link tool_block
- added link te_robotside, mass 0.5; collision mesh filename=package://ur5e_robot_description/meshes/tool_exchanger/TE_R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 scale=0.001 0.001 0.001; visual mesh filename=package://ur5e_robot_description/meshes/tool_exchanger/TE_R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 scale=0.001 0.001 0.001
- link zivid_camera: geometry collision mesh filename=package://ur5e_robot_description/meshes/zivid/zivid_assembl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 scale=1.0 1.0 1.0; visual mesh filename=package://ur5e_robot_description/meshes/zivid/zivid_assembl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 scale=1.0 1.0 1.0
Joints:
- removed joint robotiq_hande_base_joint
- removed joint robotiq_hande_coupler_joint
- removed joint robotiq_hande_end_joint
- removed joint robotiq_hande_left_finger_joint
- removed joint robotiq_hande_right_finger_joint
- removed joint tool_block_joint
- added joint te_robotside_joint: type fixed, parent zivid_camera, child te_robotside, origin xyz=0 -0.105 0 rpy=-1.5708 0 0

File: src/ur5e_robot_description/urdf/ur_standalone.xacro (robot description, xacro)
@@ -6,6 +6,6 @@
    <!-- import main macro -->
    <xacro:include filename="$(find ur_description)/urdf/ur_macro.xacro"/>
-   <xacro:include filename="$(find ur5e_hande_robot_description)/urdf/zivid_camera_mount.xacro"/>
-   <xacro:include filename="$(find ur5e_hande_robot_description)/urdf/te_robotside.xacro"/>
+   <xacro:include filename="$(find ur5e_robot_description)/urdf/zivid_camera_mount.xacro"/>
+   <xacro:include filename="$(find ur5e_robot_description)/urdf/te_robotside.xacro"/>
    <!-- possible 'ur_type' values: ur3, ur5e, ur5, ur5e, ur10, ur10e, ur16e, ur20 -->
    <!-- the default value should raise an error in case this was called without defining the type -->

File: src/ur5e_robot_description/urdf/ur_with_zivid_epick.urdf (robot description, URDF)
Before this commit: robot ur, 15 links, 14 joints
Links:
- removed link te_robotside
- added link epick_base_link
- added link epick_body; collision cylinder length=0.1023 radius=0.044; visual mesh filename=package://epick_description/meshes/visual/epick_body.stl scale=0.001 0.001 0.001
- added link epick_suction_cup; collision cylinder length=0.02 radius=0.012; visual cylinder length=0.02 radius=0.012
- added link epick_tcp
- added link epick_tip
- added link epick_vacuum_state
- added link tool_block, mass 0.2; collision mesh filename=package://ur5e_robot_description/meshes/tool_exchanger/Tool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 scale=0.001 0.001 0.001; visual mesh filename=package://ur5e_robot_description/meshes/tool_exchanger/Tool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 scale=0.001 0.001 0.001
- link zivid_camera: geometry collision mesh filename=package://ur5e_robot_description/meshes/zivid/zivid_assembl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 scale=1.0 1.0 1.0; visual mesh filename=package://ur5e_robot_description/meshes/zivid/zivid_assembl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 scale=1.0 1.0 1.0
Joints:
- removed joint te_robotside_joint
- added joint epick_base_link_to_epick_body: type fixed, parent epick_base_link, child epick_body, origin xyz=0 0 0.05115 rpy=0 0 0
- added joint epick_body_to_epick_suction_cup: type fixed, parent epick_body, child epick_suction_cup, origin xyz=0 0 0.06115 rpy=0 0 0
- added joint epick_suction_cup_to_epick_tip: type fixed, parent epick_suction_cup, child epick_tip, origin xyz=0 0 0.01 rpy=0 0 0
- added joint epick_tip_to_epick_tcp: type fixed, parent epick_tip, child epick_tcp, origin xyz=0 0 -0.0 rpy=0 0 0
- added joint gripper: type revolute, parent epick_tcp, child epick_vacuum_state, origin xyz=0 0 0 rpy=0 0 0, limit lower=0.0 upper=1.0 effort=30 velocity=1.0
- added joint tool_block_joint: type fixed, parent zivid_camera, child tool_block, origin xyz=0 -0.105 0.03 rpy=-1.5708 0 0
- added joint tool_block_to_epick_base_link: type fixed, parent tool_block, child epick_base_link, origin xyz=0 -0.02 0 rpy=-1.5708 0 3.1416

File: src/ur5e_robot_description/urdf/ur_with_zivid_epick.xacro (robot description, xacro)
@@ -1,15 +1,16 @@
 <?xml version="1.0"?>
 <robot xmlns:xacro="http://wiki.ros.org/xacro" name="$(arg name)">
-  <!-- Based on ur_with_hande.xacro; assembles UR robot + Zivid camera mount + HandE gripper
-       Chain: map -> UR -> flange -> zivid_camera_mount -> zivid_camera -> HandE gripper -->
+  <!-- Based on ur_with_hande.xacro; assembles UR robot + Zivid camera mount + EPick gripper
+       Chain: map -> UR -> flange -> zivid_camera_mount -> zivid_camera -> EPick gripper -->
   <!-- robot name parameter -->
   <xacro:arg name="name" default="ur"/>
   <!-- import main macros -->
   <xacro:include filename="$(find ur_description)/urdf/ur_macro.xacro"/>
-  <xacro:include filename="$(find ur5e_hande_robot_description)/urdf/zivid_camera_mount.xacro"/>
-  <xacro:include filename="$(find ur5e_hande_robot_description)/urdf/tool_block.xacro"/>
-  <xacro:include filename="$(find robotiq_hande_description)/urdf/robotiq_hande_gripper.xacro"/>
+  <xacro:include filename="$(find ur5e_robot_description)/urdf/zivid_camera_mount.xacro"/>
+  <xacro:include filename="$(find ur5e_robot_description)/urdf/tool_block.xacro"/>
+  <xacro:include filename="$(find epick_config)/urdf/epick_overlay.xacro"/>
   <!-- possible 'ur_type' values: ur3, ur5e, ur5, ur10, ur10e, ur16e, ur20 -->
   <xacro:arg name="ur_type" default="ur5e"/>
+  <!--. -->
   <!-- Parameters from upstream UR description -->
   <xacro:arg name="tf_prefix" default="" />
@@ -99,34 +100,6 @@
   <!-- Tool block attached to the Zivid camera -->
   <xacro:tool_block parent_link="zivid_camera" xyz="0 -0.105 0.03" rpy="-1.5708 0 0"/>
-  <!-- pos wrt camera / not flange -->
-  <xacro:arg name="grip_pos_min" default="0"/>
-  <xacro:arg name="grip_pos_max" default="0.025"/>
-  <xacro:arg name="tty_port" default="/tmp/ttyUR"/>
-  <xacro:arg name="baudrate" default="115200"/>
-  <xacro:arg name="parity" default="N"/>
-  <xacro:arg name="data_bits" default="8"/>
-  <xacro:arg name="stop_bit" default="1"/>
-  <xacro:arg name="slave_id" default="9"/>
-  <xacro:arg name="create_socat_tty" default="true"/>
-  <xacro:arg name="socat_ip_address" default="192.168.1.101"/>
-  <xacro:arg name="socat_port" default="54321"/>
-  <xacro:robotiq_hande_gripper
-    name="robotiq_hande_gripper"
-    prefix="$(arg tf_prefix)"
-    parent="tool_block"
-    grip_pos_min="$(arg grip_pos_min)"
-    grip_pos_max="$(arg grip_pos_max)"
-    tty_port="$(arg tty_port)"
-    baudrate="$(arg baudrate)"
-    parity="$(arg parity)"
-    data_bits="$(arg data_bits)"
-    stop_bit="$(arg stop_bit)"
-    slave_id="$(arg slave_id)"
-    use_fake_hardware="true"
-    xyz="0 -0.02 0"
-    rpy="-1.5708 0 3.1416"
-    create_socat_tty="$(arg create_socat_tty)"
-    socat_ip_address="$(arg socat_ip_address)"
-    socat_port="$(arg socat_port)"
-  />
+  <xacro:epick_overlay use_fake_hardware="true" parent="tool_block"
+                  origin_xyz="0 -0.02 0"
+                  origin_rpy="-1.5708 0 3.1416"/>
 </robot>

File: src/ur5e_robot_description/urdf/ur_with_zivid_hande.urdf (robot description, URDF)
Before this commit: robot ur, 21 links, 20 joints
Links:
- removed link epick_base_link
- removed link epick_body
- removed link epick_suction_cup
- removed link epick_tcp
- removed link epick_tip
- removed link epick_vacuum_state
- added link robotiq_hande_coupler, mass 0.119; collision cylinder length=0.0169 radius=0.0385; visual mesh filename=package://robotiq_hande_description/meshes/io_coupler.dae
- added link robotiq_hande_end
- added link robotiq_hande_left_finger, mass 0.03804; collision mesh filename=package://robotiq_hande_description/meshes/finger_collision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 scale=1.0 1.0 1.0; visual mesh filename=package://robotiq_hande_description/meshes/finger.dae scale=1.0 1.0 1.0
- added link robotiq_hande_link, mass 0.86387; collision cylinder length=0.10690000000000001 radius=0.0385; visual mesh filename=package://robotiq_hande_description/meshes/hande.dae scale=1.0 1.0 1.0
- added link robotiq_hande_right_finger, mass 0.03804; collision mesh filename=package://robotiq_hande_description/meshes/finger_collision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 scale=1.0 1.0 1.0; visual mesh filename=package://robotiq_hande_description/meshes/finger.dae scale=1.0 1.0 1.0
- link tool_block: geometry collision mesh filename=package://ur5e_robot_description/meshes/tool_exchanger/Tool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 scale=0.001 0.001 0.001; visual mesh filename=package://ur5e_robot_description/meshes/tool_exchanger/Tool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 scale=0.001 0.001 0.001
- link zivid_camera: geometry collision mesh filename=package://ur5e_robot_description/meshes/zivid/zivid_assembl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 scale=1.0 1.0 1.0; visual mesh filename=package://ur5e_robot_description/meshes/zivid/zivid_assembl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 scale=1.0 1.0 1.0
Joints:
- removed joint epick_base_link_to_epick_body
- removed joint epick_body_to_epick_suction_cup
- removed joint epick_suction_cup_to_epick_tip
- removed joint epick_tip_to_epick_tcp
- removed joint gripper
- removed joint tool_block_to_epick_base_link
- added joint robotiq_hande_base_joint: type fixed, parent robotiq_hande_coupler, child robotiq_hande_link, origin xyz=0 0 0.011 rpy=0 0 0
- added joint robotiq_hande_coupler_joint: type fixed, parent tool_block, child robotiq_hande_coupler, origin xyz=0 -0.02 0 rpy=-1.5708 0 3.1416
- added joint robotiq_hande_end_joint: type fixed, parent robotiq_hande_link, child robotiq_hande_end, origin xyz=0 0 0.14550000000000002 rpy=0 0 0
- added joint robotiq_hande_left_finger_joint: type prismatic, parent robotiq_hande_link, child robotiq_hande_left_finger, origin xyz=0 0 0.099 rpy=0 0 0, axis 1 0 0, limit lower=0 upper=0.025 effort=130 velocity=0.15
- added joint robotiq_hande_right_finger_joint: type prismatic, parent robotiq_hande_link, child robotiq_hande_right_finger, origin xyz=0 0 0.099 rpy=0 0 0, axis -1 0 0, limit lower=0 upper=0.025 effort=130 velocity=0.15, mimic joint=robotiq_hande_left_finger_joint multiplier=1 offset=0

File: src/ur5e_robot_description/urdf/ur_with_zivid_hande.xacro (robot description, xacro)
@@ -1,16 +1,15 @@
 <?xml version="1.0"?>
 <robot xmlns:xacro="http://wiki.ros.org/xacro" name="$(arg name)">
-  <!-- Based on ur_with_hande.xacro; assembles UR robot + Zivid camera mount + EPick gripper
-       Chain: map -> UR -> flange -> zivid_camera_mount -> zivid_camera -> EPick gripper -->
+  <!-- Based on ur_with_hande.xacro; assembles UR robot + Zivid camera mount + HandE gripper
+       Chain: map -> UR -> flange -> zivid_camera_mount -> zivid_camera -> HandE gripper -->
   <!-- robot name parameter -->
   <xacro:arg name="name" default="ur"/>
   <!-- import main macros -->
   <xacro:include filename="$(find ur_description)/urdf/ur_macro.xacro"/>
-  <xacro:include filename="$(find ur5e_hande_robot_description)/urdf/zivid_camera_mount.xacro"/>
-  <xacro:include filename="$(find ur5e_hande_robot_description)/urdf/tool_block.xacro"/>
-  <xacro:include filename="$(find epick_config)/urdf/epick_overlay.xacro"/>
+  <xacro:include filename="$(find ur5e_robot_description)/urdf/zivid_camera_mount.xacro"/>
+  <xacro:include filename="$(find ur5e_robot_description)/urdf/tool_block.xacro"/>
+  <xacro:include filename="$(find robotiq_hande_description)/urdf/robotiq_hande_gripper.xacro"/>
   <!-- possible 'ur_type' values: ur3, ur5e, ur5, ur10, ur10e, ur16e, ur20 -->
   <xacro:arg name="ur_type" default="ur5e"/>
-  <!--. -->
   <!-- Parameters from upstream UR description -->
   <xacro:arg name="tf_prefix" default="" />
@@ -100,6 +99,34 @@
   <!-- Tool block attached to the Zivid camera -->
   <xacro:tool_block parent_link="zivid_camera" xyz="0 -0.105 0.03" rpy="-1.5708 0 0"/>
-  <xacro:epick_overlay use_fake_hardware="true" parent="tool_block"
-                  origin_xyz="0 -0.02 0"
-                  origin_rpy="-1.5708 0 3.1416"/>
+  <!-- pos wrt camera / not flange -->
+  <xacro:arg name="grip_pos_min" default="0"/>
+  <xacro:arg name="grip_pos_max" default="0.025"/>
+  <xacro:arg name="tty_port" default="/tmp/ttyUR"/>
+  <xacro:arg name="baudrate" default="115200"/>
+  <xacro:arg name="parity" default="N"/>
+  <xacro:arg name="data_bits" default="8"/>
+  <xacro:arg name="stop_bit" default="1"/>
+  <xacro:arg name="slave_id" default="9"/>
+  <xacro:arg name="create_socat_tty" default="true"/>
+  <xacro:arg name="socat_ip_address" default="192.168.1.101"/>
+  <xacro:arg name="socat_port" default="54321"/>
+  <xacro:robotiq_hande_gripper
+    name="robotiq_hande_gripper"
+    prefix="$(arg tf_prefix)"
+    parent="tool_block"
+    grip_pos_min="$(arg grip_pos_min)"
+    grip_pos_max="$(arg grip_pos_max)"
+    tty_port="$(arg tty_port)"
+    baudrate="$(arg baudrate)"
+    parity="$(arg parity)"
+    data_bits="$(arg data_bits)"
+    stop_bit="$(arg stop_bit)"
+    slave_id="$(arg slave_id)"
+    use_fake_hardware="true"
+    xyz="0 -0.02 0"
+    rpy="-1.5708 0 3.1416"
+    create_socat_tty="$(arg create_socat_tty)"
+    socat_ip_address="$(arg socat_ip_address)"
+    socat_port="$(arg socat_port)"
+  />
 </robot>

File: src/ur5e_robot_description/urdf/zivid_camera_mount.xacro (robot description, xacro)
@@ -11,5 +11,5 @@
         <origin xyz="0 0 0" rpy="0 0 0"/>
         <geometry>
-          <mesh filename="package://ur5e_hande_robot_description/meshes/zivid/zivid_assembly_decimated.stl"
+          <mesh filename="package://ur5e_robot_description/meshes/zivid/zivid_assembly_decimated.stl"
                 scale="${scale} ${scale} ${scale}"/>
         </geometry>
@@ -21,5 +21,5 @@
         <origin xyz="0 0 0" rpy="0 0 0"/>
         <geometry>
-          <mesh filename="package://ur5e_hande_robot_description/meshes/zivid/zivid_assembly_decimated.stl"
+          <mesh filename="package://ur5e_robot_description/meshes/zivid/zivid_assembly_decimated.stl"
                 scale="${scale} ${scale} ${scale}"/>
         </geometry>
