Commit message: working camera

File: src/ur5e_robot_description/urdf/ur_with_zivid_hande.urdf (robot description, URDF)
Before this commit: robot ur, 20 links, 19 joints
Links:
- removed link zivid_camera
- added link robotiq_hande_tcp; visual sphere radius=0.003
- added link zivid_arm_mount, mass 0.5; collision mesh filename=package://ur5e_robot_description/meshes/zivid/zivid_onarm_m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 scale=0.001 0.001 0.001; visual mesh filename=package://ur5e_robot_description/meshes/zivid/zivid_onarm_m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 scale=0.001 0.001 0.001
- added link zivid_base_link; collision mesh filename=package://zivid_description/meshes/collision/zivid_2_plus_c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; visual mesh filename=package://zivid_description/meshes/visual/zivid_2_plus.stl
- added link zivid_optical_frame
Joints:
- removed joint zivid_camera_mount_joint
- added joint mount_to_camera_joint: type fixed, parent zivid_arm_mount, child zivid_base_link, origin xyz=0.025 0.062 -0.049 rpy=0 -1.5708 -1.5708
- added joint robotiq_hande_tcp_joint: type fixed, parent robotiq_hande_end, child robotiq_hande_tcp, origin xyz=0 0 0 rpy=0 0 0
- added joint zivid_arm_mount_joint: type fixed, parent flange, child zivid_arm_mount, origin xyz=0 0 0 rpy=-1.5708 0 -1.5708
- added joint zivid_uncalibrated_optical_joint: type fixed, parent zivid_base_link, child zivid_optical_frame, origin xyz=0.049 0.03202 0.0295 rpy=-1.5707963267948966 0 -1.6144295580947547
- joint tool_block_joint: origin xyz=0 -0.105 0.03 rpy=-1.5708 0 0 -> xyz=0 0 0.03 rpy=-1.5708 0 3.14159; parent zivid_camera -> zivid_arm_mount

File: src/ur5e_robot_description/urdf/ur_with_zivid_hande.xacro (robot description, xacro)
@@ -6,5 +6,5 @@
   <!-- import main macros -->
   <xacro:include filename="$(find ur_description)/urdf/ur_macro.xacro"/>
-  <xacro:include filename="$(find ur5e_robot_description)/urdf/zivid_camera_mount.xacro"/>
+  <xacro:include filename="$(find ur5e_robot_description)/urdf/zivid_modular_mount.xacro"/>
   <xacro:include filename="$(find ur5e_robot_description)/urdf/tool_block.xacro"/>
   <xacro:include filename="$(find robotiq_hande_description)/urdf/robotiq_hande_gripper.xacro"/>
@@ -94,8 +94,12 @@
     <origin xyz="0 0 0" rpy="0 0 0" />
   </xacro:ur_robot>
-  <!-- Camera_mount -->
-  <xacro:zivid_camera_mount parent_link="$(arg tf_prefix)flange" xyz="0.025 0 -0.105" rpy="-1.5708 0 -1.5708"/>
-  <!-- Tool block attached to the Zivid camera -->
-  <xacro:tool_block parent_link="zivid_camera" xyz="0 -0.105 0.03" rpy="-1.5708 0 0"/>
+  <!-- Modular Zivid: Arm Mount + Camera (with calibrated camera position) -->
+  <xacro:zivid_modular_mount
+    parent_link="$(arg tf_prefix)flange"
+    xyz="0 0 0"
+    rpy="-1.5708 0 -1.5708"
+    zivid_model="ZIVID_2_PLUS_MR60"/>
+  <!-- Tool block attached to the Zivid arm mount (not the camera) -->
+  <xacro:tool_block parent_link="zivid_arm_mount" xyz="0 0 0.03" rpy="-1.5708 0 3.14159"/>
   <!-- gripper pos wrt camera    -->
   <xacro:arg name="grip_pos_min" default="0"/>

File: src/ur5e_robot_description/urdf/zivid_camera_mount.xacro (robot description, xacro)
@@ -2,17 +2,9 @@
 <robot xmlns:xacro="http://ros.org/wiki/xacro" name="zivid_camera_mount">
   <!--
-    Zivid 2 Plus MR60 camera mount macro
+    Zivid camera mount macro
     - Modeled after tool_exchanger.xacro style
     - Parameters allow positioning/orientation relative to the parent link
-    - Includes optical frame for vision system compatibility
-    - Configured for Zivid 2 Plus MR60 (with M60 optics)
   -->
   <xacro:macro name="zivid_camera_mount" params="parent_link xyz:='0 0 0' rpy:='0 0 0' scale:='1.0' mass:='1.1'">
-    <!-- Optical center values for Zivid 2 Plus MR60 -->
-    <!-- From official Zivid specs - adjust after hand-eye calibration -->
-    <xacro:property name="optical_center_x" value="0.049" />
-    <xacro:property name="optical_center_y" value="0.03202" />
-    <xacro:property name="optical_center_z" value="0.0295" />
-    <xacro:property name="optical_angle_deg" value="2.5" />
     <link name="zivid_camera">
       <visual>
@@ -46,14 +38,4 @@
       <origin xyz="${xyz}" rpy="${rpy}"/>
     </joint>
-    <!-- Zivid optical frame (measurement/camera frame) -->
-    <!-- This is where point clouds and images are measured from -->
-    <link name="zivid_optical_frame"/>
-    <!-- Optical joint - Uses Zivid 2 Plus MR60 factory specs (uncalibrated) -->
-    <!-- For production accuracy, perform hand-eye calibration and update these values -->
-    <joint name="zivid_optical_joint" type="fixed">
-      <parent link="zivid_camera"/>
-      <child link="zivid_optical_frame"/>
-      <origin xyz="${optical_center_x} ${optical_center_y} ${optical_center_z}" rpy="0 ${optical_angle_deg * 3.14159265 / 180.0} 0"/>
-    </joint>
   </xacro:macro>
 </robot>

Commit message: corrected placement

File: src/ur5e_robot_description/urdf/ur_with_zivid_hande.urdf (robot description, URDF)
Before this commit: robot ur5e, 23 links, 22 joints
Links:
- link zivid_arm_mount: geometry collision mesh filename=package://ur5e_robot_description/meshes/zivid/zivid_custom_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 scale=0.001 0.001 0.001; visual mesh filename=package://ur5e_robot_description/meshes/zivid/zivid_custom_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 scale=1.0 1.0 1.0
Joints:
- joint tool_block_joint: origin xyz=0 0 0.03 rpy=-1.5708 0 3.14159 -> xyz=0 0 0.05 rpy=-1.5708 0 3.14159
- joint zivid_arm_mount_joint: origin xyz=0 0 0 rpy=-1.5708 0 -1.5708 -> xyz=0.005 0 0 rpy=-1.5708 0 -1.5708

File: src/ur5e_robot_description/urdf/ur_with_zivid_hande.xacro (robot description, xacro)
@@ -97,9 +97,9 @@
   <xacro:zivid_modular_mount
     parent_link="$(arg tf_prefix)flange"
-    xyz="0 0 0"
+    xyz="0.005 0 0"
     rpy="-1.5708 0 -1.5708"
     zivid_model="ZIVID_2_PLUS_MR60"/>
   <!-- Tool block attached to the Zivid arm mount (not the camera) -->
-  <xacro:tool_block parent_link="zivid_arm_mount" xyz="0 0 0.03" rpy="-1.5708 0 3.14159"/>
+  <xacro:tool_block parent_link="zivid_arm_mount" xyz="0 0 0.05" rpy="-1.5708 0 3.14159"/>
   <!-- gripper pos wrt camera    -->
   <xacro:arg name="grip_pos_min" default="0"/>

File: src/ur5e_robot_description/urdf/ur_with_zivid_mount.urdf (robot description, URDF)
Before this commit: robot ur5e, 16 links, 15 joints
Links:
- link zivid_arm_mount: geometry collision mesh filename=package://ur5e_robot_description/meshes/zivid/zivid_custom_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 scale=0.001 0.001 0.001; visual mesh filename=package://ur5e_robot_description/meshes/zivid/zivid_custom_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 scale=1.0 1.0 1.0
Joints:
- joint zivid_arm_mount_joint: origin xyz=0 0 0 rpy=-1.5708 0 -1.5708 -> xyz=0.005 0 0 rpy=-1.5708 0 -1.5708

File: src/ur5e_robot_description/urdf/ur_with_zivid_mount.xacro (robot description, xacro)
@@ -95,5 +95,5 @@
   <xacro:zivid_modular_mount
     parent_link="$(arg tf_prefix)flange"
-    xyz="0 0 0"
+    xyz="0.005 0 0"
     rpy="-1.5708 0 -1.5708"
     zivid_model="ZIVID_2_PLUS_MR60"/>

File: src/ur5e_robot_description/urdf/zivid_modular_mount.xacro (robot description, xacro)
@@ -4,14 +4,12 @@
   <xacro:include filename="$(find zivid_description)/urdf/macros/zivid_camera.xacro"/>
   <xacro:macro name="zivid_modular_mount" params="parent_link xyz:='0 0 0' rpy:='0 0 0' zivid_model:='ZIVID_2_PLUS_MR60'">
-    <!-- ============================================= -->
     <!-- ARM MOUNT LINK (Easily replaceable)          -->
-    <!-- ============================================= -->
     <link name="zivid_arm_mount">
       <visual>
         <origin xyz="0 0 0" rpy="0 0 0"/>
         <geometry>
-          <!-- MOUNT MESH - Replace this when Zivid provides new model -->
-          <mesh filename="package://ur5e_robot_description/meshes/zivid/zivid_onarm_mount.stl"
-                scale="0.001 0.001 0.001"/>
+          <!-- MOUNT MESH - Updated with custom mount from Zivid -->
+          <mesh filename="package://ur5e_robot_description/meshes/zivid/zivid_custom_mount.dae"
+                scale="1.0 1.0 1.0"/>
         </geometry>
         <material name="mount_dark">
@@ -22,5 +20,5 @@
         <origin xyz="0 0 0" rpy="0 0 0"/>
         <geometry>
-          <mesh filename="package://ur5e_robot_description/meshes/zivid/zivid_onarm_mount.stl"
+          <mesh filename="package://ur5e_robot_description/meshes/zivid/zivid_custom_mount.dae"
                 scale="0.001 0.001 0.001"/>
         </geometry>
@@ -40,15 +38,11 @@
       <origin xyz="${xyz}" rpy="${rpy}"/>
     </joint>
-    <!-- ============================================= -->
     <!-- ZIVID CAMERA (From official zivid-ros)       -->
-    <!-- ============================================= -->
     <xacro:zivid_camera
       prefix="zivid_"
       model="${zivid_model}"
       field_of_view="false"/>
-    <!-- ============================================= -->
     <!-- Joint: Arm Mount -> Camera                   -->
     <!-- CALIBRATION: Adjust xyz/rpy to match setup   -->
-    <!-- ============================================= -->
     <joint name="mount_to_camera_joint" type="fixed">
       <parent link="zivid_arm_mount"/>
