Commit message: updated xacros and urdfs

File: src/ur5e_robot_description/urdf/te_robotside.xacro (robot description, xacro)
@@ -6,5 +6,5 @@
         <origin xyz="0 0 0" rpy="0 0 0"/>
         <geometry>
-          <mesh filename="package://ur5e_robot_description/meshes/tool_exchanger/TE_RobotSide.stl"
+          <mesh filename="package://ur5e_robot_description/meshes/tool_exchanger/Tool_block_robotside.stl"
                 scale="0.001 0.001 0.001"/>
         </geometry>
@@ -16,5 +16,5 @@
         <origin xyz="0 0 0" rpy="0 0 0"/>
         <geometry>
-          <mesh filename="package://ur5e_robot_description/meshes/tool_exchanger/TE_RobotSide.stl"
+          <mesh filename="package://ur5e_robot_description/meshes/tool_exchanger/Tool_block_robotside.stl"
                 scale="0.001 0.001 0.001"/>
         </geometry>

File: src/ur5e_robot_description/urdf/ur_standalone.urdf (robot description, URDF)
Before this commit: robot ur, 15 links, 14 joints
Links:
- removed link zivid_camera
- added link zivid_arm_mount, mass 0.5; collision mesh filename=package://ur5e_robot_description/meshes/zivid/zivid_custom_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 scale=0.001 0.001 0.001; visual mesh filename=package://ur5e_robot_description/meshes/zivid/zivid_custom_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 scale=1.0 1.0 1.0
- added link zivid_base_link; collision mesh filename=package://zivid_description/meshes/collision/zivid_2_plus_c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; visual mesh filename=package://zivid_description/meshes/visual/zivid_2_plus.stl
- added link zivid_optical_frame
- link te_robotside: geometry collision mesh filename=package://ur5e_robot_description/meshes/tool_exchanger/Tool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 scale=0.001 0.001 0.001; visual mesh filename=package://ur5e_robot_description/meshes/tool_exchanger/Tool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 scale=0.001 0.001 0.001
Joints:
- removed joint zivid_camera_mount_joint
- added joint mount_to_camera_joint: type fixed, parent zivid_arm_mount, child zivid_base_link, origin xyz=0.025 0.062 -0.049 rpy=0 -1.5708 -1.5708
- added joint zivid_arm_mount_joint: type fixed, parent flange, child zivid_arm_mount, origin xyz=0.005 0 0 rpy=-1.5708 0 -1.5708
- added joint zivid_uncalibrated_optical_joint: type fixed, parent zivid_base_link, child zivid_optical_frame, origin xyz=0.049 0.03202 0.0295 rpy=-1.5707963267948966 0 -1.6144295580947547
- joint te_robotside_joint: origin xyz=0 -0.105 0 rpy=-1.5708 0 0 -> xyz=0 0 0.055 rpy=-1.5708 0 3.14159; parent zivid_camera -> zivid_arm_mount

File: src/ur5e_robot_description/urdf/ur_standalone.xacro (robot description, xacro)
@@ -6,5 +6,5 @@
    <!-- import main macro -->
    <xacro:include filename="$(find ur_description)/urdf/ur_macro.xacro"/>
-   <xacro:include filename="$(find ur5e_robot_description)/urdf/zivid_camera_mount.xacro"/>
+   <xacro:include filename="$(find ur5e_robot_description)/urdf/zivid_modular_mount.xacro"/>
    <xacro:include filename="$(find ur5e_robot_description)/urdf/te_robotside.xacro"/>
    <!-- possible 'ur_type' values: ur3, ur5e, ur5, ur5e, ur10, ur10e, ur16e, ur20 -->
@@ -95,7 +95,11 @@
      <origin xyz="0 0 0" rpy="0 0 0" />          <!-- position robot in the map -->
    </xacro:ur_robot>
-  <!-- Zivid camera mount attached to flange -->
-  <xacro:zivid_camera_mount parent_link="$(arg tf_prefix)flange" xyz="0.025 0 -0.105" rpy="-1.5708 0 -1.5708"/>
-  <!-- Tool exchanger robotside attached to camera -->
-  <xacro:te_robotside parent_link="zivid_camera" xyz="0 -0.105 0" rpy="-1.5708 0 0"/>
+  <!-- Modular Zivid: Arm Mount + Camera (with calibrated camera position) -->
+  <xacro:zivid_modular_mount
+    parent_link="$(arg tf_prefix)flange"
+    xyz="0.005 0 0"
+    rpy="-1.5708 0 -1.5708"
+    zivid_model="ZIVID_2_PLUS_MR60"/>
+  <!-- Tool exchanger robotside attached to arm mount (not camera) -->
+  <xacro:te_robotside parent_link="zivid_arm_mount" xyz="0 0 0.055" rpy="-1.5708 0 3.14159"/>
 </robot>

File: src/ur5e_robot_description/urdf/ur_with_zivid_epick.urdf (robot description, URDF)
Before this commit: robot ur, 21 links, 20 joints
Links:
- removed link zivid_camera
- added link zivid_arm_mount, mass 0.5; collision mesh filename=package://ur5e_robot_description/meshes/zivid/zivid_custom_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 scale=0.001 0.001 0.001; visual mesh filename=package://ur5e_robot_description/meshes/zivid/zivid_custom_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 scale=1.0 1.0 1.0
- added link zivid_base_link; collision mesh filename=package://zivid_description/meshes/collision/zivid_2_plus_c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; visual mesh filename=package://zivid_description/meshes/visual/zivid_2_plus.stl
- added link zivid_optical_frame
Joints:
- removed joint zivid_camera_mount_joint
- added joint mount_to_camera_joint: type fixed, parent zivid_arm_mount, child zivid_base_link, origin xyz=0.025 0.062 -0.049 rpy=0 -1.5708 -1.5708
- added joint zivid_arm_mount_joint: type fixed, parent flange, child zivid_arm_mount, origin xyz=0.005 0 0 rpy=-1.5708 0 -1.5708
- added joint zivid_uncalibrated_optical_joint: type fixed, parent zivid_base_link, child zivid_optical_frame, origin xyz=0.049 0.03202 0.0295 rpy=-1.5707963267948966 0 -1.6144295580947547
- joint tool_block_joint: origin xyz=0 -0.105 0.03 rpy=-1.5708 0 0 -> xyz=0 0 0.055 rpy=-1.5708 0 3.14159; parent zivid_camera -> zivid_arm_mount

File: src/ur5e_robot_description/urdf/ur_with_zivid_epick.xacro (robot description, xacro)
@@ -6,5 +6,5 @@
   <!-- import main macros -->
   <xacro:include filename="$(find ur_description)/urdf/ur_macro.xacro"/>
-  <xacro:include filename="$(find ur5e_robot_description)/urdf/zivid_camera_mount.xacro"/>
+  <xacro:include filename="$(find ur5e_robot_description)/urdf/zivid_modular_mount.xacro"/>
   <xacro:include filename="$(find ur5e_robot_description)/urdf/tool_block.xacro"/>
   <xacro:include filename="$(find epick_config)/urdf/epick_overlay.xacro"/>
@@ -95,8 +95,12 @@
     <origin xyz="0 0 0" rpy="0 0 0" />
   </xacro:ur_robot>
-  <!-- Zivid Camera mount -->
-  <xacro:zivid_camera_mount parent_link="$(arg tf_prefix)flange" xyz="0.025 0 -0.105" rpy="-1.5708 0 -1.5708"/>
-  <!-- Tool block attached to the Zivid camera -->
-  <xacro:tool_block parent_link="zivid_camera" xyz="0 -0.105 0.03" rpy="-1.5708 0 0"/>
+  <!-- Modular Zivid: Arm Mount + Camera (with calibrated camera position) -->
+  <xacro:zivid_modular_mount
+    parent_link="$(arg tf_prefix)flange"
+    xyz="0.005 0 0"
+    rpy="-1.5708 0 -1.5708"
+    zivid_model="ZIVID_2_PLUS_MR60"/>
+  <!-- Tool block attached to the Zivid arm mount (not the camera) -->
+  <xacro:tool_block parent_link="zivid_arm_mount" xyz="0 0 0.055" rpy="-1.5708 0 3.14159"/>
   <!-- ZEpick Gripper -->
   <xacro:epick_overlay use_fake_hardware="true" parent="tool_block"

File: src/ur5e_robot_description/urdf/ur_with_zivid_hande.urdf (robot description, URDF)
Before this commit: robot ur5e, 23 links, 22 joints
Joints:
- joint tool_block_joint: origin xyz=0 0 0.05 rpy=-1.5708 0 3.14159 -> xyz=0 0 0.055 rpy=-1.5708 0 3.14159

File: src/ur5e_robot_description/urdf/ur_with_zivid_hande.xacro (robot description, xacro)
@@ -101,5 +101,5 @@
     zivid_model="ZIVID_2_PLUS_MR60"/>
   <!-- Tool block attached to the Zivid arm mount (not the camera) -->
-  <xacro:tool_block parent_link="zivid_arm_mount" xyz="0 0 0.05" rpy="-1.5708 0 3.14159"/>
+  <xacro:tool_block parent_link="zivid_arm_mount" xyz="0 0 0.055" rpy="-1.5708 0 3.14159"/>
   <!-- gripper pos wrt camera    -->
   <xacro:arg name="grip_pos_min" default="0"/>
