Commit message: cleanup

File: src/ur5e_robot_description/urdf/ur_standalone.xacro (robot description, xacro)
@@ -6,5 +6,5 @@
    <!-- import main macro -->
    <xacro:include filename="$(find ur_description)/urdf/ur_macro.xacro"/>
-   <xacro:include filename="$(find ur5e_robot_description)/urdf/zivid_modular_mount.xacro"/>
+   <xacro:include filename="$(find ur5e_robot_description)/urdf/zivid_camera_mount.xacro"/>
    <xacro:include filename="$(find ur5e_robot_description)/urdf/te_robotside.xacro"/>
    <!-- possible 'ur_type' values: ur3, ur5e, ur5, ur5e, ur10, ur10e, ur16e, ur20 -->
@@ -96,5 +96,5 @@
    </xacro:ur_robot>
   <!-- Modular Zivid: Arm Mount + Camera (with calibrated camera position) -->
-  <xacro:zivid_modular_mount
+  <xacro:zivid_camera_mount
     parent_link="$(arg tf_prefix)flange"
     xyz="0.005 0 0"

File: src/ur5e_robot_description/urdf/ur_with_zivid_epick.xacro (robot description, xacro)
@@ -6,5 +6,5 @@
   <!-- import main macros -->
   <xacro:include filename="$(find ur_description)/urdf/ur_macro.xacro"/>
-  <xacro:include filename="$(find ur5e_robot_description)/urdf/zivid_modular_mount.xacro"/>
+  <xacro:include filename="$(find ur5e_robot_description)/urdf/zivid_camera_mount.xacro"/>
   <xacro:include filename="$(find ur5e_robot_description)/urdf/tool_block.xacro"/>
   <xacro:include filename="$(find epick_config)/urdf/epick_overlay.xacro"/>
@@ -96,5 +96,5 @@
   </xacro:ur_robot>
   <!-- Modular Zivid: Arm Mount + Camera (with calibrated camera position) -->
-  <xacro:zivid_modular_mount
+  <xacro:zivid_camera_mount
     parent_link="$(arg tf_prefix)flange"
     xyz="0.005 0 0"

File: src/ur5e_robot_description/urdf/ur_with_zivid_hande.xacro (robot description, xacro)
@@ -6,5 +6,5 @@
   <!-- import main macros -->
   <xacro:include filename="$(find ur_description)/urdf/ur_macro.xacro"/>
-  <xacro:include filename="$(find ur5e_robot_description)/urdf/zivid_modular_mount.xacro"/>
+  <xacro:include filename="$(find ur5e_robot_description)/urdf/zivid_camera_mount.xacro"/>
   <xacro:include filename="$(find ur5e_robot_description)/urdf/tool_block.xacro"/>
   <xacro:include filename="$(find robotiq_hande_description)/urdf/robotiq_hande_gripper.xacro"/>
@@ -95,5 +95,5 @@
   </xacro:ur_robot>
   <!-- Modular Zivid: Arm Mount + Camera (with calibrated camera position) -->
-  <xacro:zivid_modular_mount
+  <xacro:zivid_camera_mount
     parent_link="$(arg tf_prefix)flange"
     xyz="0.005 0 0"

File: src/ur5e_robot_description/urdf/zivid_camera_mount.xacro (robot description, xacro)
@@ -1,19 +1,18 @@
 <?xml version="1.0"?>
 <robot xmlns:xacro="http://ros.org/wiki/xacro" name="zivid_camera_mount">
-  <!--
-    Zivid camera mount macro
-    - Modeled after tool_exchanger.xacro style
-    - Parameters allow positioning/orientation relative to the parent link
-  -->
-  <xacro:macro name="zivid_camera_mount" params="parent_link xyz:='0 0 0' rpy:='0 0 0' scale:='1.0' mass:='1.1'">
-    <link name="zivid_camera">
+  <!-- Import official Zivid camera from zivid-ros -->
+  <xacro:include filename="$(find zivid_description)/urdf/macros/zivid_camera.xacro"/>
+  <xacro:macro name="zivid_camera_mount" params="parent_link xyz:='0 0 0' rpy:='0 0 0' zivid_model:='ZIVID_2_PLUS_MR60'">
+    <!-- ARM MOUNT LINK (Easily replaceable)          -->
+    <link name="zivid_arm_mount">
       <visual>
         <origin xyz="0 0 0" rpy="0 0 0"/>
         <geometry>
-          <mesh filename="package://ur5e_robot_description/meshes/zivid/zivid_assembly_decimated.stl"
-                scale="${scale} ${scale} ${scale}"/>
+          <!-- MOUNT MESH - Updated with custom mount from Zivid -->
+          <mesh filename="package://ur5e_robot_description/meshes/zivid/zivid_custom_mount.dae"
+                scale="1.0 1.0 1.0"/>
         </geometry>
-        <material name="grey">
-          <color rgba="0.5 0.5 0.5 1.0"/>
+        <material name="mount_dark">
+          <color rgba="0.2 0.2 0.2 1.0"/>
         </material>
       </visual>
@@ -21,10 +20,10 @@
         <origin xyz="0 0 0" rpy="0 0 0"/>
         <geometry>
-          <mesh filename="package://ur5e_robot_description/meshes/zivid/zivid_assembly_decimated.stl"
-                scale="${scale} ${scale} ${scale}"/>
+          <mesh filename="package://ur5e_robot_description/meshes/zivid/zivid_custom_mount.dae"
+                scale="0.001 0.001 0.001"/>
         </geometry>
       </collision>
       <inertial>
-        <mass value="${mass}"/>
+        <mass value="0.5"/>  <!-- Approximate arm mount mass -->
         <origin xyz="0 0 0" rpy="0 0 0"/>
         <inertia ixx="0.001" ixy="0.0" ixz="0.0"
@@ -33,8 +32,24 @@
       </inertial>
     </link>
-    <joint name="zivid_camera_mount_joint" type="fixed">
+    <!-- Joint: Flange -> Arm Mount -->
+    <joint name="zivid_arm_mount_joint" type="fixed">
       <parent link="${parent_link}"/>
-      <child link="zivid_camera"/>
+      <child link="zivid_arm_mount"/>
       <origin xyz="${xyz}" rpy="${rpy}"/>
+    </joint>
+    <!-- ZIVID CAMERA (From official zivid-ros)       -->
+    <xacro:zivid_camera
+      prefix="zivid_"
+      model="${zivid_model}"
+      field_of_view="false"/>
+    <!-- Joint: Arm Mount -> Camera                   -->
+    <!-- CALIBRATION: Adjust xyz/rpy to match setup   -->
+    <joint name="mount_to_camera_joint" type="fixed">
+      <parent link="zivid_arm_mount"/>
+      <child link="zivid_base_link"/>
+      <!-- for forward mounted camera bracket -->
+            <!-- <origin xyz="0.025 0.062 0.0" rpy="0 -1.5708 -1.5708"/> -->
+      <!-- for backward mounted camera bracket -->
+      <origin xyz="0.025 0.062 -0.049" rpy="0 -1.5708 -1.5708"/>
     </joint>
   </xacro:macro>
