Commit message: updated zivid camera settings (temp) removed planning scene update,

File: src/ur5e_robot_description/urdf/zivid_camera_mount.xacro (robot description, xacro)
@@ -2,9 +2,17 @@
 <robot xmlns:xacro="http://ros.org/wiki/xacro" name="zivid_camera_mount">
   <!--
-    Zivid camera mount macro
+    Zivid 2 Plus MR60 camera mount macro
     - Modeled after tool_exchanger.xacro style
     - Parameters allow positioning/orientation relative to the parent link
+    - Includes optical frame for vision system compatibility
+    - Configured for Zivid 2 Plus MR60 (with M60 optics)
   -->
   <xacro:macro name="zivid_camera_mount" params="parent_link xyz:='0 0 0' rpy:='0 0 0' scale:='1.0' mass:='1.1'">
+    <!-- Optical center values for Zivid 2 Plus MR60 -->
+    <!-- From official Zivid specs - adjust after hand-eye calibration -->
+    <xacro:property name="optical_center_x" value="0.049" />
+    <xacro:property name="optical_center_y" value="0.03202" />
+    <xacro:property name="optical_center_z" value="0.0295" />
+    <xacro:property name="optical_angle_deg" value="2.5" />
     <link name="zivid_camera">
       <visual>
@@ -38,4 +46,15 @@
       <origin xyz="${xyz}" rpy="${rpy}"/>
     </joint>
+    <!-- Zivid optical frame (measurement/camera frame) -->
+    <!-- This is where point clouds and images are measured from -->
+    <link name="zivid_optical_frame"/>
+    <!-- Optical joint connecting camera body to optical center -->
+    <!-- Based on Zivid specifications - perform hand-eye calibration for precision -->
+    <joint name="zivid_optical_joint" type="fixed">
+      <parent link="zivid_camera"/>
+      <child link="zivid_optical_frame"/>
+      <origin xyz="${optical_center_x} ${optical_center_y} ${optical_center_z}"
+              rpy="${-pi/2} 0 ${-pi/2 - optical_angle_deg*pi/180.0}"/>
+    </joint>
   </xacro:macro>
 </robot>

Commit message: working zivid calib

File: src/ur5e_robot_description/urdf/zivid_camera_mount.xacro (robot description, xacro)
@@ -49,11 +49,9 @@
     <!-- This is where point clouds and images are measured from -->
     <link name="zivid_optical_frame"/>
-    <!-- Optical joint connecting camera body to optical center -->
-    <!-- Based on Zivid specifications - perform hand-eye calibration for precision -->
+    <!-- Optical joint - TEMPORARY: optical frame at camera body origin for testing -->
     <joint name="zivid_optical_joint" type="fixed">
       <parent link="zivid_camera"/>
       <child link="zivid_optical_frame"/>
-      <origin xyz="${optical_center_x} ${optical_center_y} ${optical_center_z}"
-              rpy="${-pi/2} 0 ${-pi/2 - optical_angle_deg*pi/180.0}"/>
+      <origin xyz="0 0 0" rpy="0 0 0"/>
     </joint>
   </xacro:macro>

Commit message: .

File: src/ur5e_robot_description/urdf/zivid_camera_mount.xacro (robot description, xacro)
@@ -49,9 +49,10 @@
     <!-- This is where point clouds and images are measured from -->
     <link name="zivid_optical_frame"/>
-    <!-- Optical joint - TEMPORARY: optical frame at camera body origin for testing -->
+    <!-- Optical joint - Uses Zivid 2 Plus MR60 factory specs (uncalibrated) -->
+    <!-- For production accuracy, perform hand-eye calibration and update these values -->
     <joint name="zivid_optical_joint" type="fixed">
       <parent link="zivid_camera"/>
       <child link="zivid_optical_frame"/>
-      <origin xyz="0 0 0" rpy="0 0 0"/>
+      <origin xyz="${optical_center_x} ${optical_center_y} ${optical_center_z}" rpy="0 ${optical_angle_deg * 3.14159265 / 180.0} 0"/>
     </joint>
   </xacro:macro>

Commit message: `

File: src/ur5e_robot_description/urdf/zivid_camera_mount.xacro (robot description, xacro)
@@ -25,9 +25,9 @@
       </collision>
       <inertial>
-        <mass value="0.5"/>  <!-- Approximate arm mount mass -->
+        <mass value="0.170"/>  <!-- Actual measured mass: 170g -->
         <origin xyz="0 0 0" rpy="0 0 0"/>
-        <inertia ixx="0.001" ixy="0.0" ixz="0.0"
-                 iyy="0.001" iyz="0.0"
-                 izz="0.001"/>
+        <inertia ixx="0.0003" ixy="0.0" ixz="0.0"
+                 iyy="0.0005" iyz="0.0"
+                 izz="0.0006"/>
       </inertial>
     </link>

Commit message: updated zivid camera config

File: src/ur5e_robot_description/urdf/zivid_camera_mount.xacro (robot description, xacro)
@@ -4,5 +4,5 @@
   <xacro:include filename="$(find zivid_description)/urdf/macros/zivid_camera.xacro"/>
   <xacro:macro name="zivid_camera_mount" params="parent_link xyz:='0 0 0' rpy:='0 0 0' zivid_model:='ZIVID_2_PLUS_MR60'">
-    <!-- ARM MOUNT LINK (Easily replaceable)          -->
+    <!-- ARM MOUNT LINK -->
     <link name="zivid_arm_mount">
       <visual>
@@ -25,5 +25,5 @@
       </collision>
       <inertial>
-        <mass value="0.170"/>  <!-- Actual measured mass: 170g -->
+        <mass value="0.170"/>
         <origin xyz="0 0 0" rpy="0 0 0"/>
         <inertia ixx="0.0003" ixy="0.0" ixz="0.0"

Commit message: ur5e_robot_description package clean

File: src/ur5e_robot_description/urdf/zivid_camera_mount.xacro (robot description, xacro)
@@ -44,5 +44,4 @@
       field_of_view="false"/>
     <!-- Joint: Arm Mount -> Camera Base Link -->
-    <!-- CALIBRATED: Using NEW calibration matrix (Z is now positive!) -->
     <!-- Zivid calibration uses tool0 frame per: https://github.com/zivid/zivid-ros/issues/124 -->
     <joint name="mount_to_camera_joint" type="fixed">
@@ -52,6 +51,4 @@
               rpy="0.53964 -1.53712 -2.13794"/>
     </joint>
-    <!-- OLD CALIBRATION VALUES (Z was negative): -->
-    <!-- <origin xyz="0.02234 0.07744 -0.24656" rpy="0.30355 -1.53903 -1.89103"/> -->
   </xacro:macro>
 </robot>
