Commit message: use tool0 instead of flange

File: src/ur5e_robot_description/urdf/ur_standalone.urdf (robot description, URDF)
Before this commit: robot ur5e, 17 links, 16 joints
Links:
- link zivid_arm_mount: mass 0.5 -> 0.170; geometry collision mesh filename=package://ur5e_robot_description/meshes/zivid/zivid_custom_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 scale=1.0 1.0 1.0; visual mesh filename=package://ur5e_robot_description/meshes/zivid/zivid_custom_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 scale=1.0 1.0 1.0
Joints:
- joint mount_to_camera_joint: origin xyz=0.025 0.062 -0.049 rpy=0 -1.5708 -1.5708 -> xyz=0.02803 0.07664 -0.04577 rpy=0.53964 -1.53712 -2.13794
- joint zivid_arm_mount_joint: origin xyz=0.005 0 0 rpy=-1.5708 0 -1.5708 -> xyz=0 0 0.005 rpy=0 0 3.14159; parent flange -> tool0

File: src/ur5e_robot_description/urdf/ur_standalone.xacro (robot description, xacro)
@@ -96,8 +96,9 @@
    </xacro:ur_robot>
   <!-- Modular Zivid: Arm Mount + Camera (with calibrated camera position) -->
+  <!-- Using tool0 instead of flange - Zivid calibration uses tool0 frame -->
   <xacro:zivid_camera_mount
-    parent_link="$(arg tf_prefix)flange"
-    xyz="0.005 0 0"
-    rpy="-1.5708 0 -1.5708"
+    parent_link="$(arg tf_prefix)tool0"
+    xyz="0 0 0.005"
+    rpy="0 0 3.14159"
     zivid_model="ZIVID_2_PLUS_MR60"/>
   <!-- Tool exchanger robotside attached to arm mount (not camera) -->

File: src/ur5e_robot_description/urdf/ur_with_zivid_epick.urdf (robot description, URDF)
Before this commit: robot ur5e, 23 links, 22 joints
Links:
- link zivid_arm_mount: mass 0.5 -> 0.170; geometry collision mesh filename=package://ur5e_robot_description/meshes/zivid/zivid_custom_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 scale=1.0 1.0 1.0; visual mesh filename=package://ur5e_robot_description/meshes/zivid/zivid_custom_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 scale=1.0 1.0 1.0
Joints:
- joint mount_to_camera_joint: origin xyz=0.025 0.062 -0.049 rpy=0 -1.5708 -1.5708 -> xyz=0.02803 0.07664 -0.04577 rpy=0.53964 -1.53712 -2.13794
- joint zivid_arm_mount_joint: origin xyz=0.005 0 0 rpy=-1.5708 0 -1.5708 -> xyz=0 0 0.005 rpy=0 0 3.14159; parent flange -> tool0

File: src/ur5e_robot_description/urdf/ur_with_zivid_epick.xacro (robot description, xacro)
@@ -96,8 +96,9 @@
   </xacro:ur_robot>
   <!-- Modular Zivid: Arm Mount + Camera (with calibrated camera position) -->
+  <!-- Using tool0 instead of flange - Zivid calibration uses tool0 frame -->
   <xacro:zivid_camera_mount
-    parent_link="$(arg tf_prefix)flange"
-    xyz="0.005 0 0"
-    rpy="-1.5708 0 -1.5708"
+    parent_link="$(arg tf_prefix)tool0"
+    xyz="0 0 0.005"
+    rpy="0 0 3.14159"
     zivid_model="ZIVID_2_PLUS_MR60"/>
   <!-- Tool block attached to the Zivid arm mount (not the camera) -->

File: src/ur5e_robot_description/urdf/ur_with_zivid_hande.urdf (robot description, URDF)
Before this commit: robot ur5e, 22 links, 21 joints
Joints:
- joint mount_to_camera_joint: origin xyz=0.02234 0.07744 -0.24656 rpy=0.30355 -1.53903 -1.89103 -> xyz=0.02803 0.07664 -0.04577 rpy=0.53964 -1.53712 -2.13794

File: src/ur5e_robot_description/urdf/ur_with_zivid_pipettor.urdf (robot description, URDF)
Before this commit: robot ur5e, 21 links, 20 joints
Joints:
- joint mount_to_camera_joint: origin xyz=0.025 0.062 -0.049 rpy=0 -1.5708 -1.5708 -> xyz=0.02803 0.07664 -0.04577 rpy=0.53964 -1.53712 -2.13794
- joint zivid_arm_mount_joint: origin xyz=0.005 0 0 rpy=-1.5708 0 -1.5708 -> xyz=0 0 0.005 rpy=0 0 3.14159; parent flange -> tool0

File: src/ur5e_robot_description/urdf/ur_with_zivid_pipettor.xacro (robot description, xacro)
@@ -95,8 +95,9 @@
   </xacro:ur_robot>
   <!-- Modular Zivid: Arm Mount + Camera (with calibrated camera position) -->
+  <!-- Using tool0 instead of flange - Zivid calibration uses tool0 frame -->
   <xacro:zivid_camera_mount
-    parent_link="$(arg tf_prefix)flange"
-    xyz="0.005 0 0"
-    rpy="-1.5708 0 -1.5708"
+    parent_link="$(arg tf_prefix)tool0"
+    xyz="0 0 0.005"
+    rpy="0 0 3.14159"
     zivid_model="ZIVID_2_PLUS_MR60"/>
   <!-- Tool block attached to the Zivid arm mount (not the camera) -->
