Commit message: Refactor to use Zivid camera package, payload support

File: src/custom-ur-descriptions/ur5e_robot_description/urdf/te_robotside.xacro (robot description, xacro)
@@ -6,5 +6,5 @@
         <origin xyz="0 0 0" rpy="0 0 0"/>
         <geometry>
-          <mesh filename="package://ur5e_robot_description/meshes/tool_exchanger/TE_RobotSide.stl"
+          <mesh filename="package://ur5e_robot_description/meshes/tool_exchanger/Tool_block_robotside.stl"
                 scale="0.001 0.001 0.001"/>
         </geometry>
@@ -16,5 +16,5 @@
         <origin xyz="0 0 0" rpy="0 0 0"/>
         <geometry>
-          <mesh filename="package://ur5e_robot_description/meshes/tool_exchanger/TE_RobotSide.stl"
+          <mesh filename="package://ur5e_robot_description/meshes/tool_exchanger/Tool_block_robotside.stl"
                 scale="0.001 0.001 0.001"/>
         </geometry>

File: src/custom-ur-descriptions/ur5e_robot_description/urdf/ur_standalone.xacro (robot description, xacro)
@@ -95,7 +95,11 @@
      <origin xyz="0 0 0" rpy="0 0 0" />          <!-- position robot in the map -->
    </xacro:ur_robot>
-  <!-- Zivid camera mount attached to flange -->
-  <xacro:zivid_camera_mount parent_link="$(arg tf_prefix)flange" xyz="0.025 0 -0.105" rpy="-1.5708 0 -1.5708"/>
-  <!-- Tool exchanger robotside attached to camera -->
-  <xacro:te_robotside parent_link="zivid_camera" xyz="0 -0.105 0" rpy="-1.5708 0 0"/>
+  <!-- Modular Zivid: Arm Mount + Camera (with calibrated camera position) -->
+  <xacro:zivid_camera_mount
+    parent_link="$(arg tf_prefix)flange"
+    xyz="0.005 0 0"
+    rpy="-1.5708 0 -1.5708"
+    zivid_model="ZIVID_2_PLUS_MR60"/>
+  <!-- Tool exchanger robotside attached to arm mount (not camera) -->
+  <xacro:te_robotside parent_link="zivid_arm_mount" xyz="0 0 0.055" rpy="-1.5708 0 3.14159"/>
 </robot>

File: src/custom-ur-descriptions/ur5e_robot_description/urdf/ur_with_zivid_epick.xacro (robot description, xacro)
@@ -95,8 +95,12 @@
     <origin xyz="0 0 0" rpy="0 0 0" />
   </xacro:ur_robot>
-  <!-- Zivid Camera mount -->
-  <xacro:zivid_camera_mount parent_link="$(arg tf_prefix)flange" xyz="0.025 0 -0.105" rpy="-1.5708 0 -1.5708"/>
-  <!-- Tool block attached to the Zivid camera -->
-  <xacro:tool_block parent_link="zivid_camera" xyz="0 -0.105 0.03" rpy="-1.5708 0 0"/>
+  <!-- Modular Zivid: Arm Mount + Camera (with calibrated camera position) -->
+  <xacro:zivid_camera_mount
+    parent_link="$(arg tf_prefix)flange"
+    xyz="0.005 0 0"
+    rpy="-1.5708 0 -1.5708"
+    zivid_model="ZIVID_2_PLUS_MR60"/>
+  <!-- Tool block attached to the Zivid arm mount (not the camera) -->
+  <xacro:tool_block parent_link="zivid_arm_mount" xyz="0 0 0.055" rpy="-1.5708 0 3.14159"/>
   <!-- ZEpick Gripper -->
   <xacro:epick_overlay use_fake_hardware="true" parent="tool_block"

File: src/custom-ur-descriptions/ur5e_robot_description/urdf/ur_with_zivid_hande.xacro (robot description, xacro)
@@ -94,8 +94,12 @@
     <origin xyz="0 0 0" rpy="0 0 0" />
   </xacro:ur_robot>
-  <!-- Camera_mount -->
-  <xacro:zivid_camera_mount parent_link="$(arg tf_prefix)flange" xyz="0.025 0 -0.105" rpy="-1.5708 0 -1.5708"/>
-  <!-- Tool block attached to the Zivid camera -->
-  <xacro:tool_block parent_link="zivid_camera" xyz="0 -0.105 0.03" rpy="-1.5708 0 0"/>
+  <!-- Modular Zivid: Arm Mount + Camera (with calibrated camera position) -->
+  <xacro:zivid_camera_mount
+    parent_link="$(arg tf_prefix)flange"
+    xyz="0.005 0 0"
+    rpy="-1.5708 0 -1.5708"
+    zivid_model="ZIVID_2_PLUS_MR60"/>
+  <!-- Tool block attached to the Zivid arm mount (not the camera) -->
+  <xacro:tool_block parent_link="zivid_arm_mount" xyz="0 0 0.055" rpy="-1.5708 0 3.14159"/>
   <!-- gripper pos wrt camera    -->
   <xacro:arg name="grip_pos_min" default="0"/>

File: src/custom-ur-descriptions/ur5e_robot_description/urdf/zivid_camera_mount.xacro (robot description, xacro)
@@ -1,19 +1,18 @@
 <?xml version="1.0"?>
 <robot xmlns:xacro="http://ros.org/wiki/xacro" name="zivid_camera_mount">
-  <!--
-    Zivid camera mount macro
-    - Modeled after tool_exchanger.xacro style
-    - Parameters allow positioning/orientation relative to the parent link
-  -->
-  <xacro:macro name="zivid_camera_mount" params="parent_link xyz:='0 0 0' rpy:='0 0 0' scale:='1.0' mass:='1.1'">
-    <link name="zivid_camera">
+  <!-- Import official Zivid camera from zivid-ros -->
+  <xacro:include filename="$(find zivid_description)/urdf/macros/zivid_camera.xacro"/>
+  <xacro:macro name="zivid_camera_mount" params="parent_link xyz:='0 0 0' rpy:='0 0 0' zivid_model:='ZIVID_2_PLUS_MR60'">
+    <!-- ARM MOUNT LINK -->
+    <link name="zivid_arm_mount">
       <visual>
         <origin xyz="0 0 0" rpy="0 0 0"/>
         <geometry>
-          <mesh filename="package://ur5e_robot_description/meshes/zivid/zivid_assembly_decimated.stl"
-                scale="${scale} ${scale} ${scale}"/>
+          <!-- MOUNT MESH - Updated with custom mount from Zivid -->
+          <mesh filename="package://ur5e_robot_description/meshes/zivid/zivid_custom_mount.dae"
+                scale="1.0 1.0 1.0"/>
         </geometry>
-        <material name="grey">
-          <color rgba="0.5 0.5 0.5 1.0"/>
+        <material name="mount_dark">
+          <color rgba="0.2 0.2 0.2 1.0"/>
         </material>
       </visual>
@@ -21,20 +20,36 @@
         <origin xyz="0 0 0" rpy="0 0 0"/>
         <geometry>
-          <mesh filename="package://ur5e_robot_description/meshes/zivid/zivid_assembly_decimated.stl"
-                scale="${scale} ${scale} ${scale}"/>
+          <mesh filename="package://ur5e_robot_description/meshes/zivid/zivid_custom_mount.dae"
+                scale="1.0 1.0 1.0"/>
         </geometry>
       </collision>
       <inertial>
-        <mass value="${mass}"/>
+        <mass value="0.170"/>
         <origin xyz="0 0 0" rpy="0 0 0"/>
-        <inertia ixx="0.001" ixy="0.0" ixz="0.0"
-                 iyy="0.001" iyz="0.0"
-                 izz="0.001"/>
+        <inertia ixx="0.0003" ixy="0.0" ixz="0.0"
+                 iyy="0.0005" iyz="0.0"
+                 izz="0.0006"/>
       </inertial>
     </link>
-    <joint name="zivid_camera_mount_joint" type="fixed">
+    <!-- Joint: Flange -> Arm Mount -->
+    <joint name="zivid_arm_mount_joint" type="fixed">
       <parent link="${parent_link}"/>
-      <child link="zivid_camera"/>
+      <child link="zivid_arm_mount"/>
       <origin xyz="${xyz}" rpy="${rpy}"/>
+    </joint>
+    <!-- ZIVID CAMERA (From official zivid-ros)       -->
+    <xacro:zivid_camera
+      prefix="zivid_"
+      model="${zivid_model}"
+      field_of_view="false"/>
+    <!-- Joint: Arm Mount -> Camera                   -->
+    <!-- CALIBRATION: Adjust xyz/rpy to match setup   -->
+    <joint name="mount_to_camera_joint" type="fixed">
+      <parent link="zivid_arm_mount"/>
+      <child link="zivid_base_link"/>
+      <!-- for forward mounted camera bracket -->
+            <!-- <origin xyz="0.025 0.062 0.0" rpy="0 -1.5708 -1.5708"/> -->
+      <!-- for backward mounted camera bracket -->
+      <origin xyz="0.025 0.062 -0.049" rpy="0 -1.5708 -1.5708"/>
     </joint>
   </xacro:macro>

Commit message: uptodate ur5e_robot_description

File: src/custom-ur-descriptions/ur5e_robot_description/urdf/te_robotside.xacro (robot description, xacro)
@@ -1,11 +1,11 @@
 <?xml version="1.0"?>
 <robot xmlns:xacro="http://ros.org/wiki/xacro" name="wingman_toolchanger_robotside">
-  <xacro:macro name="te_robotside" params="parent_link xyz:='0.010 0 0' rpy:='0 0 ${pi/2}'">
+  <xacro:macro name="te_robotside" params="parent_link xyz:='0.010 0 0' rpy:='0 0 ${pi/2}' scale:='0.001' mass:='0.5'">
     <link name="te_robotside">
       <visual>
         <origin xyz="0 0 0" rpy="0 0 0"/>
         <geometry>
-          <mesh filename="package://ur5e_robot_description/meshes/tool_exchanger/TE_RobotSide.stl"
-                scale="0.001 0.001 0.001"/>
+          <mesh filename="package://ur5e_robot_description/meshes/tool_exchanger/Tool_block_robotside.stl"
+                scale="${scale} ${scale} ${scale}"/>
         </geometry>
         <material name="grey">
@@ -16,10 +16,10 @@
         <origin xyz="0 0 0" rpy="0 0 0"/>
         <geometry>
-          <mesh filename="package://ur5e_robot_description/meshes/tool_exchanger/TE_RobotSide.stl"
-                scale="0.001 0.001 0.001"/>
+          <mesh filename="package://ur5e_robot_description/meshes/tool_exchanger/Tool_block_robotside.stl"
+                scale="${scale} ${scale} ${scale}"/>
         </geometry>
       </collision>
       <inertial>
-        <mass value="0.5"/>
+        <mass value="${mass}"/>
         <origin xyz="0 0 0" rpy="0 0 0"/>
         <inertia ixx="0.001" ixy="0.0" ixz="0.0"

File: src/custom-ur-descriptions/ur5e_robot_description/urdf/ur_standalone.urdf (robot description, URDF)
Before this commit: robot ur, 15 links, 14 joints
Links:
- removed link zivid_camera
- added link zivid_arm_mount, mass 0.170; collision mesh filename=package://ur5e_robot_description/meshes/zivid/zivid_custom_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 scale=1.0 1.0 1.0; visual mesh filename=package://ur5e_robot_description/meshes/zivid/zivid_custom_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 scale=1.0 1.0 1.0
- added link zivid_base_link; collision mesh filename=package://zivid_description/meshes/collision/zivid_2_plus_c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; visual mesh filename=package://zivid_description/meshes/visual/zivid_2_plus.stl
- added link zivid_optical_frame
- link te_robotside: geometry collision mesh filename=package://ur5e_robot_description/meshes/tool_exchanger/Tool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 scale=0.001 0.001 0.001; visual mesh filename=package://ur5e_robot_description/meshes/tool_exchanger/Tool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 scale=0.001 0.001 0.001
Joints:
- removed joint zivid_camera_mount_joint
- added joint mount_to_camera_joint: type fixed, parent zivid_arm_mount, child zivid_base_link, origin xyz=0.02803 0.07664 -0.04577 rpy=0.53964 -1.53712 -2.13794
- added joint zivid_arm_mount_joint: type fixed, parent tool0, child zivid_arm_mount, origin xyz=0 0 0.005 rpy=0 0 3.14159
- added joint zivid_uncalibrated_optical_joint: type fixed, parent zivid_base_link, child zivid_optical_frame, origin xyz=0.049 0.03202 0.0295 rpy=-1.5707963267948966 0 -1.6144295580947547
- joint te_robotside_joint: origin xyz=0 -0.105 0 rpy=-1.5708 0 0 -> xyz=0 0 0.055 rpy=-1.5708 0 3.14159; parent zivid_camera -> zivid_arm_mount

File: src/custom-ur-descriptions/ur5e_robot_description/urdf/ur_standalone.xacro (robot description, xacro)
@@ -95,7 +95,12 @@
      <origin xyz="0 0 0" rpy="0 0 0" />          <!-- position robot in the map -->
    </xacro:ur_robot>
-  <!-- Zivid camera mount attached to flange -->
-  <xacro:zivid_camera_mount parent_link="$(arg tf_prefix)flange" xyz="0.025 0 -0.105" rpy="-1.5708 0 -1.5708"/>
-  <!-- Tool exchanger robotside attached to camera -->
-  <xacro:te_robotside parent_link="zivid_camera" xyz="0 -0.105 0" rpy="-1.5708 0 0"/>
+  <!-- Modular Zivid: Arm Mount + Camera (with calibrated camera position) -->
+  <!-- Using tool0 instead of flange - Zivid calibration uses tool0 frame -->
+  <xacro:zivid_camera_mount
+    parent_link="$(arg tf_prefix)tool0"
+    xyz="0 0 0.005"
+    rpy="0 0 3.14159"
+    zivid_model="ZIVID_2_PLUS_MR60"/>
+  <!-- Tool exchanger robotside attached to arm mount (not camera) -->
+  <xacro:te_robotside parent_link="zivid_arm_mount" xyz="0 0 0.055" rpy="-1.5708 0 3.14159"/>
 </robot>

File: src/custom-ur-descriptions/ur5e_robot_description/urdf/ur_with_zivid_epick.xacro (robot description, xacro)
@@ -95,10 +95,15 @@
     <origin xyz="0 0 0" rpy="0 0 0" />
   </xacro:ur_robot>
-  <!-- Zivid Camera mount -->
-  <xacro:zivid_camera_mount parent_link="$(arg tf_prefix)flange" xyz="0.025 0 -0.105" rpy="-1.5708 0 -1.5708"/>
-  <!-- Tool block attached to the Zivid camera -->
-  <xacro:tool_block parent_link="zivid_camera" xyz="0 -0.105 0.03" rpy="-1.5708 0 0"/>
+  <!-- Modular Zivid: Arm Mount + Camera (with calibrated camera position) -->
+  <!-- Using tool0 instead of flange - Zivid calibration uses tool0 frame -->
+  <xacro:zivid_camera_mount
+    parent_link="$(arg tf_prefix)tool0"
+    xyz="0 0 0.005"
+    rpy="0 0 3.14159"
+    zivid_model="ZIVID_2_PLUS_MR60"/>
+  <!-- Tool block attached to the Zivid arm mount (not the camera) -->
+  <xacro:tool_block parent_link="zivid_arm_mount" xyz="0 0 0.055" rpy="-1.5708 0 3.14159"/>
   <!-- ZEpick Gripper -->
-  <xacro:epick_overlay use_fake_hardware="true" parent="tool_block"
+  <xacro:epick_overlay use_fake_hardware="false" parent="tool_block"
                   origin_xyz="0 -0.02 0"
                   origin_rpy="-1.5708 0 3.1416"/>

File: src/custom-ur-descriptions/ur5e_robot_description/urdf/ur_with_zivid_hande.xacro (robot description, xacro)
@@ -94,8 +94,13 @@
     <origin xyz="0 0 0" rpy="0 0 0" />
   </xacro:ur_robot>
-  <!-- Camera_mount -->
-  <xacro:zivid_camera_mount parent_link="$(arg tf_prefix)flange" xyz="0.025 0 -0.105" rpy="-1.5708 0 -1.5708"/>
-  <!-- Tool block attached to the Zivid camera -->
-  <xacro:tool_block parent_link="zivid_camera" xyz="0 -0.105 0.03" rpy="-1.5708 0 0"/>
+  <!-- Modular Zivid: Arm Mount + Camera (with calibrated camera position) -->
+  <!-- Using tool0 instead of flange - Zivid calibration uses tool0 frame -->
+  <xacro:zivid_camera_mount
+    parent_link="$(arg tf_prefix)tool0"
+    xyz="0.00000 0.00000 0.00500"
+    rpy="0.00000 0.00000 3.14159"
+    zivid_model="ZIVID_2_PLUS_MR60"/>
+  <!-- Tool block attached to the Zivid arm mount (not the camera) -->
+  <xacro:tool_block parent_link="zivid_arm_mount" xyz="0 0 0.055" rpy="-1.5708 0 3.14159"/>
   <!-- gripper pos wrt camera    -->
   <xacro:arg name="grip_pos_min" default="0"/>
@@ -122,5 +127,5 @@
     stop_bit="$(arg stop_bit)"
     slave_id="$(arg slave_id)"
-    use_fake_hardware="true"
+    use_fake_hardware="false"
     xyz="0 -0.02 0"
     rpy="-1.5708 0 3.1416"

File: src/custom-ur-descriptions/ur5e_robot_description/urdf/zivid_camera_mount.xacro (robot description, xacro)
@@ -1,19 +1,18 @@
 <?xml version="1.0"?>
 <robot xmlns:xacro="http://ros.org/wiki/xacro" name="zivid_camera_mount">
-  <!--
-    Zivid camera mount macro
-    - Modeled after tool_exchanger.xacro style
-    - Parameters allow positioning/orientation relative to the parent link
-  -->
-  <xacro:macro name="zivid_camera_mount" params="parent_link xyz:='0 0 0' rpy:='0 0 0' scale:='1.0' mass:='1.1'">
-    <link name="zivid_camera">
+  <!-- Import official Zivid camera from zivid-ros -->
+  <xacro:include filename="$(find zivid_description)/urdf/macros/zivid_camera.xacro"/>
+  <xacro:macro name="zivid_camera_mount" params="parent_link xyz:='0 0 0' rpy:='0 0 0' zivid_model:='ZIVID_2_PLUS_MR60'">
+    <!-- ARM MOUNT LINK -->
+    <link name="zivid_arm_mount">
       <visual>
         <origin xyz="0 0 0" rpy="0 0 0"/>
         <geometry>
-          <mesh filename="package://ur5e_robot_description/meshes/zivid/zivid_assembly_decimated.stl"
-                scale="${scale} ${scale} ${scale}"/>
+          <!-- MOUNT MESH - Updated with custom mount from Zivid -->
+          <mesh filename="package://ur5e_robot_description/meshes/zivid/zivid_custom_mount.dae"
+                scale="1.0 1.0 1.0"/>
         </geometry>
-        <material name="grey">
-          <color rgba="0.5 0.5 0.5 1.0"/>
+        <material name="mount_dark">
+          <color rgba="0.2 0.2 0.2 1.0"/>
         </material>
       </visual>
@@ -21,20 +20,34 @@
         <origin xyz="0 0 0" rpy="0 0 0"/>
         <geometry>
-          <mesh filename="package://ur5e_robot_description/meshes/zivid/zivid_assembly_decimated.stl"
-                scale="${scale} ${scale} ${scale}"/>
+          <mesh filename="package://ur5e_robot_description/meshes/zivid/zivid_custom_mount.dae"
+                scale="1.0 1.0 1.0"/>
         </geometry>
       </collision>
       <inertial>
-        <mass value="${mass}"/>
+        <mass value="0.170"/>
         <origin xyz="0 0 0" rpy="0 0 0"/>
-        <inertia ixx="0.001" ixy="0.0" ixz="0.0"
-                 iyy="0.001" iyz="0.0"
-                 izz="0.001"/>
+        <inertia ixx="0.0003" ixy="0.0" ixz="0.0"
+                 iyy="0.0005" iyz="0.0"
+                 izz="0.0006"/>
       </inertial>
     </link>
-    <joint name="zivid_camera_mount_joint" type="fixed">
+    <!-- Joint: Flange -> Arm Mount -->
+    <joint name="zivid_arm_mount_joint" type="fixed">
       <parent link="${parent_link}"/>
-      <child link="zivid_camera"/>
+      <child link="zivid_arm_mount"/>
       <origin xyz="${xyz}" rpy="${rpy}"/>
+    </joint>
+    <!-- ZIVID CAMERA (From official zivid-ros)       -->
+    <xacro:zivid_camera
+      prefix="zivid_"
+      model="${zivid_model}"
+      field_of_view="false"/>
+    <!-- Joint: Arm Mount -> Camera Base Link -->
+    <!-- Zivid calibration uses tool0 frame per: https://github.com/zivid/zivid-ros/issues/124 -->
+    <joint name="mount_to_camera_joint" type="fixed">
+      <parent link="zivid_arm_mount"/>
+      <child link="zivid_base_link"/>
+      <origin xyz="0.02803 0.07664 -0.04577"
+              rpy="0.53964 -1.53712 -2.13794"/>
     </joint>
   </xacro:macro>
