Commit message: new camera/wrist orientation and positioning

File: src/custom-ur-descriptions/ur5e_robot_description/urdf/ur_standalone.xacro (robot description, xacro)
@@ -103,5 +103,5 @@
     parent_link="$(arg tf_prefix)tool0"
     xyz="0 0 0.005"
-    rpy="0 0 3.14159"
+    rpy="0 0 0"
     zivid_model="ZIVID_2_PLUS_MR60"/>
   <!-- Tool exchanger robotside attached to arm mount (not camera) -->

File: src/custom-ur-descriptions/ur5e_robot_description/urdf/ur_with_zivid_epick.xacro (robot description, xacro)
@@ -103,5 +103,5 @@
     parent_link="$(arg tf_prefix)tool0"
     xyz="0 0 0.005"
-    rpy="0 0 3.14159"
+    rpy="0 0 0"
     zivid_model="ZIVID_2_PLUS_MR60"/>
   <!-- Tool block attached to the Zivid arm mount (not the camera) -->

File: src/custom-ur-descriptions/ur5e_robot_description/urdf/ur_with_zivid_hande.xacro (robot description, xacro)
@@ -101,6 +101,6 @@
   <xacro:zivid_camera_mount
     parent_link="$(arg tf_prefix)tool0"
-    xyz="0.00000 0.00000 0.00500"
-    rpy="0.00000 0.00000 3.14159"
+    xyz="0 0 0.005"
+    rpy="0 0 0"
     zivid_model="ZIVID_2_PLUS_MR60"/>
   <!-- Tool block attached to the Zivid arm mount (not the camera) -->

File: src/custom-ur-descriptions/ur5e_robot_description/urdf/ur_with_zivid_pipettor.xacro (robot description, xacro)
@@ -102,5 +102,5 @@
     parent_link="$(arg tf_prefix)tool0"
     xyz="0 0 0.005"
-    rpy="0 0 3.14159"
+    rpy="0 0 0"
     zivid_model="ZIVID_2_PLUS_MR60"/>
   <!-- Tool block attached to the Zivid arm mount (not the camera) -->

File: src/custom-ur-descriptions/ur5e_robot_description/urdf/zivid_camera_mount.xacro (robot description, xacro)
@@ -9,7 +9,8 @@
         <origin xyz="0 0 0" rpy="0 0 0"/>
         <geometry>
-          <!-- MOUNT MESH - Updated with custom mount from Zivid -->
-          <mesh filename="package://ur5e_robot_description/meshes/zivid/zivid_custom_mount.dae"
-                scale="1.0 1.0 1.0"/>
+          <!-- Official Zivid On-Arm Mount (from zivid.com/downloads) -->
+          <!-- Scale 0.001 if STL is in mm (from STEP), 1.0 if already in meters -->
+          <mesh filename="package://ur5e_robot_description/meshes/zivid/zivid_onarm_mount.stl"
+                scale="0.001 0.001 0.001"/>
         </geometry>
         <material name="mount_dark">
@@ -20,6 +21,6 @@
         <origin xyz="0 0 0" rpy="0 0 0"/>
         <geometry>
-          <mesh filename="package://ur5e_robot_description/meshes/zivid/zivid_custom_mount.dae"
-                scale="1.0 1.0 1.0"/>
+          <mesh filename="package://ur5e_robot_description/meshes/zivid/zivid_onarm_mount.stl"
+                scale="0.001 0.001 0.001"/>
         </geometry>
       </collision>
@@ -48,5 +49,5 @@
       <parent link="zivid_arm_mount"/>
       <child link="zivid_base_link"/>
-      <origin xyz="0.02803 0.07664 -0.04577"
+      <origin xyz="0.02803 0.07664 0.0"
               rpy="0.53964 -1.53712 -2.13794"/>
     </joint>

Commit message: jazzy: refactor ur_standalone.xacro to use separate ur_ros2_control macro
In Jazzy, ur_robot (kinematic) and ur_ros2_control (hardware interface) are
separate macros. All hardware driver params (robot_ip, script files, tool comm,
mock hardware) moved from xacro:ur_robot to xacro:ur_ros2_control, which is
included from ur_robot_driver.

File: src/custom-ur-descriptions/ur5e_robot_description/urdf/ur_standalone.xacro (robot description, xacro)
@@ -1,15 +1,15 @@
 <?xml version="1.0"?>
 <robot xmlns:xacro="http://wiki.ros.org/xacro" name="$(arg name)">
-<!--Based on same file and version as https://github.com/UniversalRobots/Universal_Robots_ROS2_Description/blob/29e90d5095fdf4af99eba3c3eae153d7d5d769c0/urdf/ur.urdf.xacro-->
+<!--Jazzy-compatible version: ur_robot (kinematic) and ur_ros2_control (hardware) are now separate macros-->
    <!-- robot name parameter -->
    <xacro:arg name="name" default="ur5e"/>
    <!-- import main macro -->
    <xacro:include filename="$(find ur_description)/urdf/ur_macro.xacro"/>
+   <xacro:include filename="$(find ur_robot_driver)/urdf/ur.ros2_control.xacro"/>
    <xacro:include filename="$(find ur5e_robot_description)/urdf/zivid_camera_mount.xacro"/>
    <xacro:include filename="$(find ur5e_robot_description)/urdf/te_robotside.xacro"/>
    <!-- possible 'ur_type' values: ur3, ur5e, ur5, ur5e, ur10, ur10e, ur16e, ur20 -->
-   <!-- the default value should raise an error in case this was called without defining the type -->
    <xacro:arg name="ur_type" default="ur5e"/>
-   <!-- These parameters are from https://github.com/UniversalRobots/Universal_Robots_ROS2_Description/blob/29e90d5095fdf4af99eba3c3eae153d7d5d769c0/urdf/ur.urdf.xacro-->
+   <!-- Kinematic parameters -->
    <xacro:arg name="tf_prefix" default="" />
    <xacro:arg name="joint_limit_params" default="$(find ur_description)/config/$(arg ur_type)/joint_limits.yaml"/>
@@ -20,10 +20,10 @@
    <xacro:arg name="safety_pos_margin" default="0.15"/>
    <xacro:arg name="safety_k_position" default="20"/>
-   <!-- ros2_control related parameters -->
+   <!-- ros2_control / hardware driver parameters -->
    <xacro:arg name="headless_mode" default="false" />
    <xacro:arg name="robot_ip" default="0.0.0.0" />
-   <xacro:arg name="script_filename" default=""/>
-   <xacro:arg name="output_recipe_filename" default=""/>
-   <xacro:arg name="input_recipe_filename" default=""/>
+   <xacro:arg name="script_filename" default="$(find ur_client_library)/resources/external_control.urscript"/>
+   <xacro:arg name="output_recipe_filename" default="$(find ur_robot_driver)/resources/rtde_output_recipe.txt"/>
+   <xacro:arg name="input_recipe_filename" default="$(find ur_robot_driver)/resources/rtde_input_recipe.txt"/>
    <xacro:arg name="reverse_ip" default="0.0.0.0"/>
    <xacro:arg name="script_command_port" default="50004"/>
@@ -31,7 +31,6 @@
    <xacro:arg name="script_sender_port" default="50002"/>
    <xacro:arg name="trajectory_port" default="50003"/>
-   <!-- Keep-alive: number of 20ms cycles without response before disconnect (10 = 200ms timeout) -->
    <xacro:arg name="robot_receive_timeout" default="0.2"/>
-   <!--   tool communication related parameters-->
+   <!-- Tool communication parameters -->
    <xacro:arg name="use_tool_communication" default="false" />
    <xacro:arg name="tool_voltage" default="0" />
@@ -43,17 +42,13 @@
    <xacro:arg name="tool_device_name" default="/tmp/ttyUR" />
    <xacro:arg name="tool_tcp_port" default="54321" />
-     <!-- Simulation parameters -->
+   <!-- Simulation parameters -->
+   <xacro:arg name="use_mock_hardware" default="false" />
    <xacro:arg name="mock_sensor_commands" default="false" />
-   <xacro:arg name="sim_gazebo" default="false" />
-   <xacro:arg name="sim_ignition" default="false" />
-   <xacro:arg name="simulation_controllers" default="" />
-   <xacro:arg name="mock_hardware" default="true" />
-   <!-- initial position for simulations (Fake Hardware, Gazebo, Ignition) -->
+   <!-- initial position for simulations -->
    <xacro:arg name="initial_positions_file" default="$(find ur_standalone_moveit_config)/config/initial_positions.yaml"/>
-   <!-- convert to property to use substitution in function -->
    <xacro:property name="initial_positions_file" default="$(arg initial_positions_file)"/>
    <!-- create link fixed to the "map" -->
    <link name="map" />
-   <!-- arm -->
+   <!-- Kinematic model (Jazzy: no hardware params here) -->
    <xacro:ur_robot
      name="$(arg name)"
@@ -67,7 +62,18 @@
      safety_pos_margin="$(arg safety_pos_margin)"
      safety_k_position="$(arg safety_k_position)"
+     >
+     <origin xyz="0 0 0" rpy="0 0 0" />
+   </xacro:ur_robot>
+   <!-- ros2_control hardware interface (Jazzy: separate from kinematic macro) -->
+   <xacro:ur_ros2_control
+     name="$(arg name)"
+     tf_prefix="$(arg tf_prefix)"
+     kinematics_parameters_file="$(arg kinematics_params)"
+     robot_ip="$(arg robot_ip)"
+     script_filename="$(arg script_filename)"
+     input_recipe_filename="$(arg input_recipe_filename)"
+     output_recipe_filename="$(arg output_recipe_filename)"
+     use_mock_hardware="$(arg use_mock_hardware)"
      mock_sensor_commands="$(arg mock_sensor_commands)"
-     sim_gazebo="$(arg sim_gazebo)"
-     sim_ignition="$(arg sim_ignition)"
      headless_mode="$(arg headless_mode)"
      initial_positions="${xacro.load_yaml(initial_positions_file)}"
@@ -81,8 +87,4 @@
      tool_device_name="$(arg tool_device_name)"
      tool_tcp_port="$(arg tool_tcp_port)"
-     robot_ip="$(arg robot_ip)"
-     script_filename="$(arg script_filename)"
-     output_recipe_filename="$(arg output_recipe_filename)"
-     input_recipe_filename="$(arg input_recipe_filename)"
      reverse_ip="$(arg reverse_ip)"
      script_command_port="$(arg script_command_port)"
@@ -91,9 +93,6 @@
      trajectory_port="$(arg trajectory_port)"
      robot_receive_timeout="$(arg robot_receive_timeout)"
-     >
-     <origin xyz="0 0 0" rpy="0 0 0" />          <!-- position robot in the map -->
-   </xacro:ur_robot>
+   />
   <!-- Modular Zivid: Arm Mount + Camera (with calibrated camera position) -->
-  <!-- Using tool0 instead of flange - Zivid calibration uses tool0 frame -->
   <xacro:zivid_camera_mount
     parent_link="$(arg tf_prefix)tool0"
