Commit message: Fix ePick URDF geometry to match physical hardware (#28)
Measured full kinematic chain and corrected URDF offsets that were
causing epick_tip TF frame to be ~19mm off from the physical tip.
Previously compensated by software z_offsets in vision stages.

URDF fixes:
- tool_block Z offset: 55mm → 51mm (all 3 gripper xacros)
- tool_block → gripper mounting offset: 20mm → 32.35mm (epick + hande)
- Added extension nozzle: 37mm × ø2mm (was missing)
- Corrected suction cup: 2mm × ø7mm (was 20mm × ø24mm)

Software z_offset cleanup:
- vision_stages auto-detect: 23mm → 2mm
- vision_stages fallback: 100mm → 2mm
- vision_pick_place default: 20mm → 2mm
- Remaining 2mm compensates for ~2mm residual URDF error

Added kinematic chain reference to ur5e_robot_description README.

File: src/custom-ur-descriptions/ur5e_robot_description/urdf/ur_with_zivid_epick.urdf (robot description, URDF)
Before this commit: robot ur5e, 23 links, 22 joints
Links:
- added link epick_extension; collision cylinder length=0.037 radius=0.001; visual cylinder length=0.037 radius=0.001
- link epick_suction_cup: geometry collision cylinder length=0.002 radius=0.0035; visual cylinder length=0.002 radius=0.0035
- link zivid_arm_mount: geometry collision mesh filename=package://ur5e_robot_description/meshes/zivid/zivid_onarm_m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 scale=0.001 0.001 0.001; visual mesh filename=package://ur5e_robot_description/meshes/zivid/zivid_onarm_m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 scale=0.001 0.001 0.001
Joints:
- removed joint epick_body_to_epick_suction_cup
- removed joint mount_to_camera_joint
- removed joint zivid_uncalibrated_optical_joint
- added joint epick_body_to_epick_extension: type fixed, parent epick_body, child epick_extension, origin xyz=0 0 0.06965 rpy=0 0 0
- added joint epick_extension_to_epick_suction_cup: type fixed, parent epick_extension, child epick_suction_cup, origin xyz=0 0 0.0195 rpy=0 0 0
- added joint optical_to_base_link: type fixed, parent zivid_optical_frame, child zivid_base_link, origin xyz=0.03413 0.02950 -0.04756 rpy=-1.57080 -1.52716 3.14159
- added joint tool0_to_zivid_optical: type fixed, parent tool0, child zivid_optical_frame, origin xyz=0.05675 0.10322 0.05489 rpy=-0.00615 0.04362 3.13541
- joint epick_suction_cup_to_epick_tip: origin xyz=0 0 0.01 rpy=0 0 0 -> xyz=0 0 0.001 rpy=0 0 0
- joint tool_block_joint: origin xyz=0 0 0.055 rpy=-1.5708 0 3.14159 -> xyz=0 0 0.051 rpy=-1.5708 0 3.14159
- joint tool_block_to_epick_base_link: origin xyz=0 -0.02 0 rpy=-1.5708 0 3.1416 -> xyz=0 -0.03235 0 rpy=-1.5708 0 3.1416
- joint zivid_arm_mount_joint: origin xyz=0 0 0.005 rpy=0 0 3.14159 -> xyz=0 0 0.005 rpy=0 0 0

File: src/custom-ur-descriptions/ur5e_robot_description/urdf/ur_with_zivid_epick.xacro (robot description, xacro)
@@ -106,8 +106,8 @@
     zivid_model="ZIVID_2_PLUS_MR60"/>
   <!-- Tool block attached to the Zivid arm mount (not the camera) -->
-  <xacro:tool_block parent_link="zivid_arm_mount" xyz="0 0 0.055" rpy="-1.5708 0 3.14159"/>
+  <xacro:tool_block parent_link="zivid_arm_mount" xyz="0 0 0.051" rpy="-1.5708 0 3.14159"/>
   <!-- Epick Gripper -->
   <xacro:epick_overlay use_fake_hardware="$(arg use_fake_hardware)" parent="tool_block"
-                  origin_xyz="0 -0.02 0"
+                  origin_xyz="0 -0.03235 0"
                   origin_rpy="-1.5708 0 3.1416"/>
 </robot>

File: src/custom-ur-descriptions/ur5e_robot_description/urdf/ur_with_zivid_hande.xacro (robot description, xacro)
@@ -105,5 +105,5 @@
     zivid_model="ZIVID_2_PLUS_MR60"/>
   <!-- Tool block attached to the Zivid arm mount (not the camera) -->
-  <xacro:tool_block parent_link="zivid_arm_mount" xyz="0 0 0.055" rpy="-1.5708 0 3.14159"/>
+  <xacro:tool_block parent_link="zivid_arm_mount" xyz="0 0 0.051" rpy="-1.5708 0 3.14159"/>
   <!-- gripper pos wrt camera    -->
   <xacro:arg name="grip_pos_min" default="0"/>
@@ -118,4 +118,5 @@
   <xacro:arg name="socat_ip_address" default="$(arg robot_ip)"/>
   <xacro:arg name="socat_port" default="54321"/>
+  <!-- Hand-E xyz previously "0 -0.02 0" — updated based on physical measurement -->
   <xacro:robotiq_hande_gripper
     name="robotiq_hande_gripper"
@@ -131,5 +132,5 @@
     slave_id="$(arg slave_id)"
     use_fake_hardware="$(arg use_fake_hardware)"
-    xyz="0 -0.02 0"
+    xyz="0 -0.03235 0"
     rpy="-1.5708 0 3.1416"
     create_socat_tty="$(arg create_socat_tty)"

File: src/custom-ur-descriptions/ur5e_robot_description/urdf/ur_with_zivid_pipettor.xacro (robot description, xacro)
@@ -105,5 +105,5 @@
     zivid_model="ZIVID_2_PLUS_MR60"/>
   <!-- Tool block attached to the Zivid arm mount (not the camera) -->
-  <xacro:tool_block parent_link="zivid_arm_mount" xyz="0 0 0.055" rpy="-1.5708 0 3.14159"/>
+  <xacro:tool_block parent_link="zivid_arm_mount" xyz="0 0 0.051" rpy="-1.5708 0 3.14159"/>
   <!-- Pipettor attached to tool block -->
   <xacro:pipette

File: src/end_effectors/epick_config/urdf/epick_overlay.xacro (robot description, xacro)
@@ -5,7 +5,10 @@
   <!-- Arguments for parent link and optional prefix -->
   <xacro:macro name="epick_overlay" params="parent prefix:=''
-                                 origin_xyz:='0 -0.019 0'
+                                 origin_xyz:='0 -0.03235 0'
                                  origin_rpy:='1.5708 0 0'
-                                 suction_cup_height:=0.020
+                                 suction_cup_height:=0.002
+                                 suction_cup_radius:=0.0035
+                                 extension_length:=0.037
+                                 extension_radius:=0.001
                                  use_fake_hardware:=false
                                  usb_port:=/tmp/ttyUR">
@@ -16,4 +19,7 @@
       origin_rpy="${origin_rpy}"
       suction_cup_height="${suction_cup_height}"
+      suction_cup_radius="${suction_cup_radius}"
+      extension_length="${extension_length}"
+      extension_radius="${extension_radius}"
       use_fake_hardware="${use_fake_hardware}"
       usb_port="${usb_port}"/>

Commit message: Fine-tune URDF offsets and remove all software z_offset compensation
Calibrated arm_mount → tool_block offset (51→49mm) and cup dimensions
by testing both pen_vacuum and 7mm_dia profiles against physical hardware.
Tip now lands exactly at the target with zero software z_offset.

Offset changes:
- arm_mount → tool_block: 51mm → 49mm (all 3 gripper xacros)
- pen_vacuum extension: 37mm → 34.5mm
- 7mm_dia extension: 19mm → 18mm, cup height: 7mm → 6mm

z_offset removal:
- default_beamline.yaml: 0.002 → 0.0
- vision_stages.py auto-detect: 0.002 → 0.0
- vision_stages.py fallback: 0.002 → 0.0
- vision_pick_place_stages.py: uses goal z_offset directly (no default)
- CLAUDE.md: updated cup dimensions and z_offset docs

File: src/custom-ur-descriptions/ur5e_robot_description/urdf/ur_with_zivid_epick.urdf (robot description, URDF)
Before this commit: robot ur5e, 24 links, 23 joints
Links:
- link epick_extension: geometry collision cylinder length=0.0345 radius=0.001; visual cylinder length=0.0345 radius=0.001
Joints:
- joint epick_body_to_epick_extension: origin xyz=0 0 0.06965 rpy=0 0 0 -> xyz=0 0 0.0684 rpy=0 0 0
- joint epick_extension_to_epick_suction_cup: origin xyz=0 0 0.0195 rpy=0 0 0 -> xyz=0 0 0.018250000000000002 rpy=0 0 0
- joint tool_block_joint: origin xyz=0 0 0.051 rpy=-1.5708 0 3.14159 -> xyz=0 0 0.049 rpy=-1.5708 0 3.14159

File: src/custom-ur-descriptions/ur5e_robot_description/urdf/ur_with_zivid_epick.xacro (robot description, xacro)
@@ -106,7 +106,7 @@
     zivid_model="ZIVID_2_PLUS_MR60"/>
   <!-- Tool block attached to the Zivid arm mount (not the camera) -->
-  <xacro:tool_block parent_link="zivid_arm_mount" xyz="0 0 0.051" rpy="-1.5708 0 3.14159"/>
+  <xacro:tool_block parent_link="zivid_arm_mount" xyz="0 0 0.049" rpy="-1.5708 0 3.14159"/>
   <!-- Suction cup dimensions (passed from launch file via cup profile) -->
-  <xacro:arg name="extension_length" default="0.037"/>
+  <xacro:arg name="extension_length" default="0.0345"/>
   <xacro:arg name="extension_radius" default="0.001"/>
   <xacro:arg name="suction_cup_height" default="0.002"/>

File: src/custom-ur-descriptions/ur5e_robot_description/urdf/ur_with_zivid_hande.xacro (robot description, xacro)
@@ -105,5 +105,5 @@
     zivid_model="ZIVID_2_PLUS_MR60"/>
   <!-- Tool block attached to the Zivid arm mount (not the camera) -->
-  <xacro:tool_block parent_link="zivid_arm_mount" xyz="0 0 0.051" rpy="-1.5708 0 3.14159"/>
+  <xacro:tool_block parent_link="zivid_arm_mount" xyz="0 0 0.049" rpy="-1.5708 0 3.14159"/>
   <!-- gripper pos wrt camera    -->
   <xacro:arg name="grip_pos_min" default="0"/>

File: src/custom-ur-descriptions/ur5e_robot_description/urdf/ur_with_zivid_pipettor.xacro (robot description, xacro)
@@ -105,5 +105,5 @@
     zivid_model="ZIVID_2_PLUS_MR60"/>
   <!-- Tool block attached to the Zivid arm mount (not the camera) -->
-  <xacro:tool_block parent_link="zivid_arm_mount" xyz="0 0 0.051" rpy="-1.5708 0 3.14159"/>
+  <xacro:tool_block parent_link="zivid_arm_mount" xyz="0 0 0.049" rpy="-1.5708 0 3.14159"/>
   <!-- Pipettor attached to tool block -->
   <xacro:pipette

Commit message: Re-calibrate Zivid hand-eye (2026-03-25)
New calibration after URDF chain changes (tool_block, epick mounting).
Residuals: rot < 0.15°, trans < 1.0mm. XY accuracy improved ~1cm.

File: src/custom-ur-descriptions/ur5e_robot_description/urdf/ur_with_zivid_epick.urdf (robot description, URDF)
Before this commit: robot ur5e, 24 links, 23 joints
Joints:
- joint tool0_to_zivid_optical: origin xyz=0.05675 0.10322 0.05489 rpy=-0.00615 0.04362 3.13541 -> xyz=0.05475 0.10491 0.06013 rpy=-0.03489 0.05317 3.13637

File: src/custom-ur-descriptions/ur5e_robot_description/urdf/zivid_camera_mount.xacro (robot description, xacro)
@@ -21,7 +21,10 @@
       <!-- Hand-eye calibration: tool0 -> optical_frame -->
       <!-- Rotation: Euler XYZ extrinsic, radians | Translation: meters -->
-      <!-- Calibration (2026-01-15): Residuals: rot < 0.22°, trans < 0.47mm -->
+      <!-- Calibration (2026-03-25): Residuals: rot < 0.15°, trans < 1.0mm -->
+      <origin xyz="0.05475 0.10491 0.06013"
+              rpy="-0.03489 0.05317 3.13637"/>
+      <!-- Calibration (2026-01-15): Residuals: rot < 0.22°, trans < 0.47mm
       <origin xyz="0.05675 0.10322 0.05489"
-              rpy="-0.00615 0.04362 3.13541"/>
+              rpy="-0.00615 0.04362 3.13541"/> -->
       <!-- TEST (2026-01-22): Zero roll/pitch - did NOT help Y variance
       <origin xyz="0.05675 0.10322 0.05489"
