Commit message: Recalibrate Zivid hand-eye, fix 12mm vision Z error, tighten controller tolerances
- Recalibrate hand-eye for beamline move (2026-03-27, 12 poses, pose 4 outlier excluded)
- Fix 12mm systematic Z error in vision_moveto caused by ePick cup profile mismatch:
  baked URDF had pen_vacuum (138.8mm chain) while MoveIt launched with 7mm_dia (126.3mm).
  Aligned all defaults (xacro, launch, overlay) to 7mm_dia and regenerated baked URDFs.
- Fix bimodal Z error in vision_moveto: use fixed roll=180°/pitch=0° for stable flat
  approach with marker-derived yaw (via 180° Z rotation) for minimal wrist motion
- Tighten trajectory controller goal tolerance from 0.1 to 0.01 rad across all configs
  (was allowing ~14mm positional error at gripper tip)

File: src/custom-ur-descriptions/ur5e_robot_description/urdf/ur_standalone.urdf (robot description, URDF)
Before this commit: robot ur5e, 17 links, 16 joints
Links:
- link zivid_arm_mount: geometry collision mesh filename=package://ur5e_robot_description/meshes/zivid/zivid_onarm_m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 scale=0.001 0.001 0.001; visual mesh filename=package://ur5e_robot_description/meshes/zivid/zivid_onarm_m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 scale=0.001 0.001 0.001
Joints:
- removed joint mount_to_camera_joint
- removed joint zivid_uncalibrated_optical_joint
- added joint optical_to_base_link: type fixed, parent zivid_optical_frame, child zivid_base_link, origin xyz=0.03413 0.02950 -0.04756 rpy=-1.57080 -1.52716 3.14159
- added joint tool0_to_zivid_optical: type fixed, parent tool0, child zivid_optical_frame, origin xyz=0.05635 0.10228 0.06025 rpy=-0.03622 0.05218 3.13437
- joint zivid_arm_mount_joint: origin xyz=0 0 0.005 rpy=0 0 3.14159 -> xyz=0 0 0.005 rpy=0 0 0

File: src/custom-ur-descriptions/ur5e_robot_description/urdf/ur_standalone_isaac.urdf (robot description, URDF)
Before this commit: robot ur5e, 17 links, 16 joints
Links:
- link base_link_inertia: geometry collision mesh filename=package://ur_description/meshes/ur5e/collision/base.stl; visual mesh filename=package://ur_description/meshes/ur5e/visual/base.dae
- link forearm_link: geometry collision mesh filename=package://ur_description/meshes/ur5e/collision/forearm.stl; visual mesh filename=package://ur_description/meshes/ur5e/visual/forearm.dae
- link map: mass 0.0 -> None
- link shoulder_link: geometry collision mesh filename=package://ur_description/meshes/ur5e/collision/shoulder.stl; visual mesh filename=package://ur_description/meshes/ur5e/visual/shoulder.dae
- link te_robotside: geometry collision mesh filename=package://ur5e_robot_description/meshes/tool_exchanger/Tool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 scale=0.001 0.001 0.001; visual mesh filename=package://ur5e_robot_description/meshes/tool_exchanger/Tool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 scale=0.001 0.001 0.001
- link upper_arm_link: geometry collision mesh filename=package://ur_description/meshes/ur5e/collision/upperarm.stl; visual mesh filename=package://ur_description/meshes/ur5e/visual/upperarm.dae
- link wrist_1_link: geometry collision mesh filename=package://ur_description/meshes/ur5e/collision/wrist1.stl; visual mesh filename=package://ur_description/meshes/ur5e/visual/wrist1.dae
- link wrist_2_link: geometry collision mesh filename=package://ur_description/meshes/ur5e/collision/wrist2.stl; visual mesh filename=package://ur_description/meshes/ur5e/visual/wrist2.dae
- link wrist_3_link: geometry collision mesh filename=package://ur_description/meshes/ur5e/collision/wrist3.stl; visual mesh filename=package://ur_description/meshes/ur5e/visual/wrist3.dae
- link zivid_arm_mount: geometry collision mesh filename=package://ur5e_robot_description/meshes/zivid/zivid_onarm_m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 scale=0.001 0.001 0.001; visual mesh filename=package://ur5e_robot_description/meshes/zivid/zivid_onarm_m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 scale=0.001 0.001 0.001
- link zivid_base_link: geometry collision mesh filename=package://zivid_description/meshes/collision/zivid_2_plus_c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; visual mesh filename=package://zivid_description/meshes/visual/zivid_2_plus.stl
Joints:
- removed joint mount_to_camera_joint
- removed joint zivid_uncalibrated_optical_joint
- added joint optical_to_base_link: type fixed, parent zivid_optical_frame, child zivid_base_link, origin xyz=0.03413 0.02950 -0.04756 rpy=-1.57080 -1.52716 3.14159
- added joint tool0_to_zivid_optical: type fixed, parent tool0, child zivid_optical_frame, origin xyz=0.05635 0.10228 0.06025 rpy=-0.03622 0.05218 3.13437
- joint zivid_arm_mount_joint: origin xyz=0 0 0.005 rpy=0 0 3.14159 -> xyz=0 0 0.005 rpy=0 0 0

File: src/custom-ur-descriptions/ur5e_robot_description/urdf/ur_with_zivid_epick.urdf (robot description, URDF)
Before this commit: robot ur5e, 24 links, 23 joints
Links:
- link epick_extension: geometry collision cylinder length=0.018 radius=0.006; visual cylinder length=0.018 radius=0.006
- link epick_suction_cup: geometry collision cylinder length=0.006 radius=0.0035; visual cylinder length=0.006 radius=0.0035
Joints:
- joint epick_body_to_epick_extension: origin xyz=0 0 0.0684 rpy=0 0 0 -> xyz=0 0 0.06015 rpy=0 0 0
- joint epick_extension_to_epick_suction_cup: origin xyz=0 0 0.018250000000000002 rpy=0 0 0 -> xyz=0 0 0.012 rpy=0 0 0
- joint epick_suction_cup_to_epick_tip: origin xyz=0 0 0.001 rpy=0 0 0 -> xyz=0 0 0.003 rpy=0 0 0
- joint tool0_to_zivid_optical: origin xyz=0.05475 0.10491 0.06013 rpy=-0.03489 0.05317 3.13637 -> xyz=0.05635 0.10228 0.06025 rpy=-0.03622 0.05218 3.13437

File: src/custom-ur-descriptions/ur5e_robot_description/urdf/ur_with_zivid_epick.xacro (robot description, xacro)
@@ -108,7 +108,7 @@
   <xacro:tool_block parent_link="zivid_arm_mount" xyz="0 0 0.049" rpy="-1.5708 0 3.14159"/>
   <!-- Suction cup dimensions (passed from launch file via cup profile) -->
-  <xacro:arg name="extension_length" default="0.0345"/>
-  <xacro:arg name="extension_radius" default="0.001"/>
-  <xacro:arg name="suction_cup_height" default="0.002"/>
+  <xacro:arg name="extension_length" default="0.018"/>
+  <xacro:arg name="extension_radius" default="0.006"/>
+  <xacro:arg name="suction_cup_height" default="0.006"/>
   <xacro:arg name="suction_cup_radius" default="0.0035"/>
   <!-- Epick Gripper -->

File: src/custom-ur-descriptions/ur5e_robot_description/urdf/ur_with_zivid_epick_isaac.urdf (robot description, URDF)
Before this commit: robot ur5e, 23 links, 22 joints
Links:
- added link epick_extension; collision cylinder length=0.018 radius=0.006; visual cylinder length=0.018 radius=0.006
- link base_link_inertia: geometry collision mesh filename=package://ur_description/meshes/ur5e/collision/base.stl; visual mesh filename=package://ur_description/meshes/ur5e/visual/base.dae
- link epick_body: geometry collision cylinder length=0.1023 radius=0.044; visual mesh filename=package://epick_description/meshes/visual/epick_body.stl scale=0.001 0.001 0.001
- link epick_suction_cup: geometry collision cylinder length=0.006 radius=0.0035; visual cylinder length=0.006 radius=0.0035
- link forearm_link: geometry collision mesh filename=package://ur_description/meshes/ur5e/collision/forearm.stl; visual mesh filename=package://ur_description/meshes/ur5e/visual/forearm.dae
- link map: mass 0.0 -> None
- link shoulder_link: geometry collision mesh filename=package://ur_description/meshes/ur5e/collision/shoulder.stl; visual mesh filename=package://ur_description/meshes/ur5e/visual/shoulder.dae
- link tool_block: geometry collision mesh filename=package://ur5e_robot_description/meshes/tool_exchanger/Tool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 scale=0.001 0.001 0.001; visual mesh filename=package://ur5e_robot_description/meshes/tool_exchanger/Tool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 scale=0.001 0.001 0.001
- link upper_arm_link: geometry collision mesh filename=package://ur_description/meshes/ur5e/collision/upperarm.stl; visual mesh filename=package://ur_description/meshes/ur5e/visual/upperarm.dae
- link wrist_1_link: geometry collision mesh filename=package://ur_description/meshes/ur5e/collision/wrist1.stl; visual mesh filename=package://ur_description/meshes/ur5e/visual/wrist1.dae
- link wrist_2_link: geometry collision mesh filename=package://ur_description/meshes/ur5e/collision/wrist2.stl; visual mesh filename=package://ur_description/meshes/ur5e/visual/wrist2.dae
- link wrist_3_link: geometry collision mesh filename=package://ur_description/meshes/ur5e/collision/wrist3.stl; visual mesh filename=package://ur_description/meshes/ur5e/visual/wrist3.dae
- link zivid_arm_mount: geometry collision mesh filename=package://ur5e_robot_description/meshes/zivid/zivid_onarm_m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 scale=0.001 0.001 0.001; visual mesh filename=package://ur5e_robot_description/meshes/zivid/zivid_onarm_m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 scale=0.001 0.001 0.001
- link zivid_base_link: geometry collision mesh filename=package://zivid_description/meshes/collision/zivid_2_plus_c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; visual mesh filename=package://zivid_description/meshes/visual/zivid_2_plus.stl
Joints:
- removed joint epick_body_to_epick_suction_cup
- removed joint mount_to_camera_joint
- removed joint zivid_uncalibrated_optical_joint
- added joint epick_body_to_epick_extension: type fixed, parent epick_body, child epick_extension, origin xyz=0 0 0.06015 rpy=0 0 0
- added joint epick_extension_to_epick_suction_cup: type fixed, parent epick_extension, child epick_suction_cup, origin xyz=0 0 0.012 rpy=0 0 0
- added joint optical_to_base_link: type fixed, parent zivid_optical_frame, child zivid_base_link, origin xyz=0.03413 0.02950 -0.04756 rpy=-1.57080 -1.52716 3.14159
- added joint tool0_to_zivid_optical: type fixed, parent tool0, child zivid_optical_frame, origin xyz=0.05635 0.10228 0.06025 rpy=-0.03622 0.05218 3.13437
- joint epick_suction_cup_to_epick_tip: origin xyz=0 0 0.01 rpy=0 0 0 -> xyz=0 0 0.003 rpy=0 0 0
- joint tool_block_joint: origin xyz=0 0 0.055 rpy=-1.5708 0 3.14159 -> xyz=0 0 0.049 rpy=-1.5708 0 3.14159
- joint tool_block_to_epick_base_link: origin xyz=0 -0.02 0 rpy=-1.5708 0 3.1416 -> xyz=0 -0.03235 0 rpy=-1.5708 0 3.1416
- joint zivid_arm_mount_joint: origin xyz=0 0 0.005 rpy=0 0 3.14159 -> xyz=0 0 0.005 rpy=0 0 0

File: src/custom-ur-descriptions/ur5e_robot_description/urdf/ur_with_zivid_hande.urdf (robot description, URDF)
Before this commit: robot ur5e, 22 links, 21 joints
Links:
- link zivid_arm_mount: geometry collision mesh filename=package://ur5e_robot_description/meshes/zivid/zivid_onarm_m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 scale=0.001 0.001 0.001; visual mesh filename=package://ur5e_robot_description/meshes/zivid/zivid_onarm_m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 scale=0.001 0.001 0.001
Joints:
- removed joint mount_to_camera_joint
- removed joint zivid_uncalibrated_optical_joint
- added joint optical_to_base_link: type fixed, parent zivid_optical_frame, child zivid_base_link, origin xyz=0.03413 0.02950 -0.04756 rpy=-1.57080 -1.52716 3.14159
- added joint tool0_to_zivid_optical: type fixed, parent tool0, child zivid_optical_frame, origin xyz=0.05635 0.10228 0.06025 rpy=-0.03622 0.05218 3.13437
- joint robotiq_hande_coupler_joint: origin xyz=0 -0.02 0 rpy=-1.5708 0 3.1416 -> xyz=0 -0.03235 0 rpy=-1.5708 0 3.1416
- joint tool_block_joint: origin xyz=0 0 0.055 rpy=-1.5708 0 3.14159 -> xyz=0 0 0.049 rpy=-1.5708 0 3.14159
- joint zivid_arm_mount_joint: origin xyz=0.00000 0.00000 0.00500 rpy=0.00000 0.00000 3.14159 -> xyz=0 0 0.005 rpy=0 0 0

File: src/custom-ur-descriptions/ur5e_robot_description/urdf/ur_with_zivid_hande_isaac.urdf (robot description, URDF)
Before this commit: robot ur5e, 22 links, 21 joints
Links:
- link base_link_inertia: geometry collision mesh filename=package://ur_description/meshes/ur5e/collision/base.stl; visual mesh filename=package://ur_description/meshes/ur5e/visual/base.dae
- link forearm_link: geometry collision mesh filename=package://ur_description/meshes/ur5e/collision/forearm.stl; visual mesh filename=package://ur_description/meshes/ur5e/visual/forearm.dae
- link map: mass 0.0 -> None
- link robotiq_hande_coupler: geometry collision cylinder length=0.0169 radius=0.0385; visual mesh filename=package://robotiq_hande_description/meshes/io_coupler.dae
- link robotiq_hande_left_finger: geometry collision mesh filename=package://robotiq_hande_description/meshes/finger_collision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 scale=1.0 1.0 1.0; visual mesh filename=package://robotiq_hande_description/meshes/finger.dae scale=1.0 1.0 1.0
- link robotiq_hande_link: geometry collision cylinder length=0.10690000000000001 radius=0.0385; visual mesh filename=package://robotiq_hande_description/meshes/hande.dae scale=1.0 1.0 1.0
- link robotiq_hande_right_finger: geometry collision mesh filename=package://robotiq_hande_description/meshes/finger_collision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 scale=1.0 1.0 1.0; visual mesh filename=package://robotiq_hande_description/meshes/finger.dae scale=1.0 1.0 1.0
- link shoulder_link: geometry collision mesh filename=package://ur_description/meshes/ur5e/collision/shoulder.stl; visual mesh filename=package://ur_description/meshes/ur5e/visual/shoulder.dae
- link tool_block: geometry collision mesh filename=package://ur5e_robot_description/meshes/tool_exchanger/Tool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 scale=0.001 0.001 0.001; visual mesh filename=package://ur5e_robot_description/meshes/tool_exchanger/Tool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 scale=0.001 0.001 0.001
- link upper_arm_link: geometry collision mesh filename=package://ur_description/meshes/ur5e/collision/upperarm.stl; visual mesh filename=package://ur_description/meshes/ur5e/visual/upperarm.dae
- link wrist_1_link: geometry collision mesh filename=package://ur_description/meshes/ur5e/collision/wrist1.stl; visual mesh filename=package://ur_description/meshes/ur5e/visual/wrist1.dae
- link wrist_2_link: geometry collision mesh filename=package://ur_description/meshes/ur5e/collision/wrist2.stl; visual mesh filename=package://ur_description/meshes/ur5e/visual/wrist2.dae
- link wrist_3_link: geometry collision mesh filename=package://ur_description/meshes/ur5e/collision/wrist3.stl; visual mesh filename=package://ur_description/meshes/ur5e/visual/wrist3.dae
- link zivid_arm_mount: geometry collision mesh filename=package://ur5e_robot_description/meshes/zivid/zivid_onarm_m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 scale=0.001 0.001 0.001; visual mesh filename=package://ur5e_robot_description/meshes/zivid/zivid_onarm_m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 scale=0.001 0.001 0.001
- link zivid_base_link: geometry collision mesh filename=package://zivid_description/meshes/collision/zivid_2_plus_c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; visual mesh filename=package://zivid_description/meshes/visual/zivid_2_plus.stl
Joints:
- removed joint mount_to_camera_joint
- removed joint zivid_uncalibrated_optical_joint
- added joint optical_to_base_link: type fixed, parent zivid_optical_frame, child zivid_base_link, origin xyz=0.03413 0.02950 -0.04756 rpy=-1.57080 -1.52716 3.14159
- added joint tool0_to_zivid_optical: type fixed, parent tool0, child zivid_optical_frame, origin xyz=0.05635 0.10228 0.06025 rpy=-0.03622 0.05218 3.13437
- joint robotiq_hande_coupler_joint: origin xyz=0 -0.02 0 rpy=-1.5708 0 3.1416 -> xyz=0 -0.03235 0 rpy=-1.5708 0 3.1416
- joint tool_block_joint: origin xyz=0 0 0.055 rpy=-1.5708 0 3.14159 -> xyz=0 0 0.049 rpy=-1.5708 0 3.14159
- joint zivid_arm_mount_joint: origin xyz=0.00000 0.00000 0.00500 rpy=0.00000 0.00000 3.14159 -> xyz=0 0 0.005 rpy=0 0 0

File: src/custom-ur-descriptions/ur5e_robot_description/urdf/ur_with_zivid_pipettor.urdf (robot description, URDF)
Before this commit: robot ur5e, 21 links, 20 joints
Links:
- link zivid_arm_mount: geometry collision mesh filename=package://ur5e_robot_description/meshes/zivid/zivid_onarm_m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 scale=0.001 0.001 0.001; visual mesh filename=package://ur5e_robot_description/meshes/zivid/zivid_onarm_m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 scale=0.001 0.001 0.001
Joints:
- removed joint mount_to_camera_joint
- removed joint zivid_uncalibrated_optical_joint
- added joint optical_to_base_link: type fixed, parent zivid_optical_frame, child zivid_base_link, origin xyz=0.03413 0.02950 -0.04756 rpy=-1.57080 -1.52716 3.14159
- added joint tool0_to_zivid_optical: type fixed, parent tool0, child zivid_optical_frame, origin xyz=0.05635 0.10228 0.06025 rpy=-0.03622 0.05218 3.13437
- joint tool_block_joint: origin xyz=0 0 0.055 rpy=-1.5708 0 3.14159 -> xyz=0 0 0.049 rpy=-1.5708 0 3.14159
- joint zivid_arm_mount_joint: origin xyz=0 0 0.005 rpy=0 0 3.14159 -> xyz=0 0 0.005 rpy=0 0 0

File: src/custom-ur-descriptions/ur5e_robot_description/urdf/ur_with_zivid_pipettor_isaac.urdf (robot description, URDF)
Before this commit: robot ur5e, 21 links, 20 joints
Links:
- link base_link_inertia: geometry collision mesh filename=package://ur_description/meshes/ur5e/collision/base.stl; visual mesh filename=package://ur_description/meshes/ur5e/visual/base.dae
- link forearm_link: geometry collision mesh filename=package://ur_description/meshes/ur5e/collision/forearm.stl; visual mesh filename=package://ur_description/meshes/ur5e/visual/forearm.dae
- link map: mass 0.0 -> None
- link pipette_body_link: geometry collision mesh filename=package://pipette_description/meshes/collision/pipettor_col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 scale=0.001 0.001 0.001; visual mesh filename=package://pipette_description/meshes/visual/pipettor_visual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 scale=0.001 0.001 0.001
- link shoulder_link: geometry collision mesh filename=package://ur_description/meshes/ur5e/collision/shoulder.stl; visual mesh filename=package://ur_description/meshes/ur5e/visual/shoulder.dae
- link tool_block: geometry collision mesh filename=package://ur5e_robot_description/meshes/tool_exchanger/Tool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 scale=0.001 0.001 0.001; visual mesh filename=package://ur5e_robot_description/meshes/tool_exchanger/Tool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 scale=0.001 0.001 0.001
- link upper_arm_link: geometry collision mesh filename=package://ur_description/meshes/ur5e/collision/upperarm.stl; visual mesh filename=package://ur_description/meshes/ur5e/visual/upperarm.dae
- link wrist_1_link: geometry collision mesh filename=package://ur_description/meshes/ur5e/collision/wrist1.stl; visual mesh filename=package://ur_description/meshes/ur5e/visual/wrist1.dae
- link wrist_2_link: geometry collision mesh filename=package://ur_description/meshes/ur5e/collision/wrist2.stl; visual mesh filename=package://ur_description/meshes/ur5e/visual/wrist2.dae
- link wrist_3_link: geometry collision mesh filename=package://ur_description/meshes/ur5e/collision/wrist3.stl; visual mesh filename=package://ur_description/meshes/ur5e/visual/wrist3.dae
- link zivid_arm_mount: geometry collision mesh filename=package://ur5e_robot_description/meshes/zivid/zivid_onarm_m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 scale=0.001 0.001 0.001; visual mesh filename=package://ur5e_robot_description/meshes/zivid/zivid_onarm_m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 scale=0.001 0.001 0.001
- link zivid_base_link: geometry collision mesh filename=package://zivid_description/meshes/collision/zivid_2_plus_c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; visual mesh filename=package://zivid_description/meshes/visual/zivid_2_plus.stl
Joints:
- removed joint mount_to_camera_joint
- removed joint zivid_uncalibrated_optical_joint
- added joint optical_to_base_link: type fixed, parent zivid_optical_frame, child zivid_base_link, origin xyz=0.03413 0.02950 -0.04756 rpy=-1.57080 -1.52716 3.14159
- added joint tool0_to_zivid_optical: type fixed, parent tool0, child zivid_optical_frame, origin xyz=0.05635 0.10228 0.06025 rpy=-0.03622 0.05218 3.13437
- joint tool_block_joint: origin xyz=0 0 0.055 rpy=-1.5708 0 3.14159 -> xyz=0 0 0.049 rpy=-1.5708 0 3.14159
- joint zivid_arm_mount_joint: origin xyz=0 0 0.005 rpy=0 0 3.14159 -> xyz=0 0 0.005 rpy=0 0 0

File: src/custom-ur-descriptions/ur5e_robot_description/urdf/zivid_camera_mount.xacro (robot description, xacro)
@@ -21,7 +21,10 @@
       <!-- Hand-eye calibration: tool0 -> optical_frame -->
       <!-- Rotation: Euler XYZ extrinsic, radians | Translation: meters -->
-      <!-- Calibration (2026-03-25): Residuals: rot < 0.15°, trans < 1.0mm -->
+      <!-- Calibration (2026-03-27): 12 poses (pose 4 excluded as outlier). Residuals: rot < 0.33°, trans < 1.53mm -->
+      <origin xyz="0.05635 0.10228 0.06025"
+              rpy="-0.03622 0.05218 3.13437"/>
+      <!-- Calibration (2026-03-25): Residuals: rot < 0.15°, trans < 1.0mm
       <origin xyz="0.05475 0.10491 0.06013"
-              rpy="-0.03489 0.05317 3.13637"/>
+              rpy="-0.03489 0.05317 3.13637"/> -->
       <!-- Calibration (2026-01-15): Residuals: rot < 0.22°, trans < 0.47mm
       <origin xyz="0.05675 0.10322 0.05489"

File: src/end_effectors/epick_config/urdf/epick_overlay.xacro (robot description, xacro)
@@ -7,8 +7,8 @@
                                  origin_xyz:='0 -0.03235 0'
                                  origin_rpy:='1.5708 0 0'
-                                 suction_cup_height:=0.002
+                                 suction_cup_height:=0.006
                                  suction_cup_radius:=0.0035
-                                 extension_length:=0.037
-                                 extension_radius:=0.001
+                                 extension_length:=0.018
+                                 extension_radius:=0.006
                                  use_fake_hardware:=false
                                  usb_port:=/tmp/ttyUR">
