Commit message: chore: regenerate static URDFs from Jazzy-fixed xacros
Regenerated ur_standalone.urdf, ur_with_zivid_hande.urdf,
ur_with_zivid_epick.urdf, and ur_with_zivid_pipettor.urdf
using the corrected Jazzy xacro architecture (split ur_robot +
ur_ros2_control macros).

Co-Authored-By: Claude Opus 4.6 (1M context) <noreply@anthropic.com>

File: src/custom-ur-descriptions/ur5e_robot_description/urdf/ur_standalone.urdf (robot description, URDF)
Before this commit: robot ur5e, 17 links, 16 joints
Links:
- link zivid_arm_mount: geometry collision mesh filename=package://ur5e_robot_description/meshes/zivid/zivid_onarm_m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 scale=0.001 0.001 0.001; visual mesh filename=package://ur5e_robot_description/meshes/zivid/zivid_onarm_m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 scale=0.001 0.001 0.001
Joints:
- removed joint mount_to_camera_joint
- removed joint zivid_uncalibrated_optical_joint
- added joint optical_to_base_link: type fixed, parent zivid_optical_frame, child zivid_base_link, origin xyz=0.03413 0.02950 -0.04756 rpy=-1.57080 -1.52716 3.14159
- added joint tool0_to_zivid_optical: type fixed, parent tool0, child zivid_optical_frame, origin xyz=0.05635 0.10228 0.06025 rpy=-0.03622 0.05218 3.13437
- joint zivid_arm_mount_joint: origin xyz=0 0 0.005 rpy=0 0 3.14159 -> xyz=0 0 0.005 rpy=0 0 0

File: src/custom-ur-descriptions/ur5e_robot_description/urdf/ur_with_zivid_epick.urdf (robot description, URDF)
Before this commit: robot ur5e, 23 links, 22 joints
Links:
- added link epick_extension; collision cylinder length=0.018 radius=0.006; visual cylinder length=0.018 radius=0.006
- link epick_suction_cup: geometry collision cylinder length=0.006 radius=0.0035; visual cylinder length=0.006 radius=0.0035
- link zivid_arm_mount: geometry collision mesh filename=package://ur5e_robot_description/meshes/zivid/zivid_onarm_m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 scale=0.001 0.001 0.001; visual mesh filename=package://ur5e_robot_description/meshes/zivid/zivid_onarm_m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 scale=0.001 0.001 0.001
Joints:
- removed joint epick_body_to_epick_suction_cup
- removed joint mount_to_camera_joint
- removed joint zivid_uncalibrated_optical_joint
- added joint epick_body_to_epick_extension: type fixed, parent epick_body, child epick_extension, origin xyz=0 0 0.06015 rpy=0 0 0
- added joint epick_extension_to_epick_suction_cup: type fixed, parent epick_extension, child epick_suction_cup, origin xyz=0 0 0.012 rpy=0 0 0
- added joint optical_to_base_link: type fixed, parent zivid_optical_frame, child zivid_base_link, origin xyz=0.03413 0.02950 -0.04756 rpy=-1.57080 -1.52716 3.14159
- added joint tool0_to_zivid_optical: type fixed, parent tool0, child zivid_optical_frame, origin xyz=0.05635 0.10228 0.06025 rpy=-0.03622 0.05218 3.13437
- joint epick_suction_cup_to_epick_tip: origin xyz=0 0 0.01 rpy=0 0 0 -> xyz=0 0 0.003 rpy=0 0 0
- joint zivid_arm_mount_joint: origin xyz=0 0 0.005 rpy=0 0 3.14159 -> xyz=0 0 0.005 rpy=0 0 0

File: src/custom-ur-descriptions/ur5e_robot_description/urdf/ur_with_zivid_hande.urdf (robot description, URDF)
Before this commit: robot ur5e, 22 links, 21 joints
Links:
- link zivid_arm_mount: geometry collision mesh filename=package://ur5e_robot_description/meshes/zivid/zivid_onarm_m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 scale=0.001 0.001 0.001; visual mesh filename=package://ur5e_robot_description/meshes/zivid/zivid_onarm_m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 scale=0.001 0.001 0.001
Joints:
- removed joint mount_to_camera_joint
- removed joint zivid_uncalibrated_optical_joint
- added joint optical_to_base_link: type fixed, parent zivid_optical_frame, child zivid_base_link, origin xyz=0.03413 0.02950 -0.04756 rpy=-1.57080 -1.52716 3.14159
- added joint tool0_to_zivid_optical: type fixed, parent tool0, child zivid_optical_frame, origin xyz=0.05635 0.10228 0.06025 rpy=-0.03622 0.05218 3.13437
- joint zivid_arm_mount_joint: origin xyz=0.00000 0.00000 0.00500 rpy=0.00000 0.00000 3.14159 -> xyz=0 0 0.005 rpy=0 0 0

File: src/custom-ur-descriptions/ur5e_robot_description/urdf/ur_with_zivid_pipettor.urdf (robot description, URDF)
Before this commit: robot ur5e, 21 links, 20 joints
Links:
- link zivid_arm_mount: geometry collision mesh filename=package://ur5e_robot_description/meshes/zivid/zivid_onarm_m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 scale=0.001 0.001 0.001; visual mesh filename=package://ur5e_robot_description/meshes/zivid/zivid_onarm_m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 scale=0.001 0.001 0.001
Joints:
- removed joint mount_to_camera_joint
- removed joint zivid_uncalibrated_optical_joint
- added joint optical_to_base_link: type fixed, parent zivid_optical_frame, child zivid_base_link, origin xyz=0.03413 0.02950 -0.04756 rpy=-1.57080 -1.52716 3.14159
- added joint tool0_to_zivid_optical: type fixed, parent tool0, child zivid_optical_frame, origin xyz=0.05635 0.10228 0.06025 rpy=-0.03622 0.05218 3.13437
- joint tool_block_joint: origin xyz=0 0 0.055 rpy=-1.5708 0 3.14159 -> xyz=0 0 0.049 rpy=-1.5708 0 3.14159
- joint zivid_arm_mount_joint: origin xyz=0 0 0.005 rpy=0 0 3.14159 -> xyz=0 0 0.005 rpy=0 0 0
