Commit message: fix: split ur_robot/ur_ros2_control in gripper xacros for Jazzy
Jazzy ur_description splits the UR robot into a kinematic-only
ur_robot macro and a separate ur_ros2_control macro for hardware
interface. The 4 gripper xacros were still using the Humble
single-macro pattern, passing hardware params to ur_robot which
now rejects them.

Split each into:
1. ur_robot — kinematic model only
2. ur_ros2_control — hardware interface (mock_hardware, robot_ip, etc.)

Also remove obsolete sim_gazebo/sim_ignition/simulation_controllers
args (Gazebo Classic removed in Jazzy).

Co-Authored-By: Claude Opus 4.6 (1M context) <noreply@anthropic.com>

File: src/custom-ur-descriptions/ur5e_robot_description/urdf/ur_with_zivid_2fg7.xacro (robot description, xacro)
@@ -6,4 +6,5 @@
   <!-- import main macros -->
   <xacro:include filename="$(find ur_description)/urdf/ur_macro.xacro"/>
+  <xacro:include filename="$(find ur_robot_driver)/urdf/ur.ros2_control.xacro"/>
   <xacro:include filename="$(find ur5e_robot_description)/urdf/zivid_camera_mount.xacro"/>
   <xacro:include filename="$(find ur5e_robot_description)/urdf/tool_block.xacro"/>
@@ -45,7 +46,4 @@
   <!-- Simulation parameters -->
   <xacro:arg name="mock_sensor_commands" default="false" />
-  <xacro:arg name="sim_gazebo" default="false" />
-  <xacro:arg name="sim_ignition" default="false" />
-  <xacro:arg name="simulation_controllers" default="" />
   <xacro:arg name="mock_hardware" default="true" />
   <!-- initial position for simulations (Fake Hardware, Gazebo, Ignition) -->
@@ -54,5 +52,5 @@
   <!-- create link fixed to the "map" -->
   <link name="map" />
-  <!-- UR arm -->
+  <!-- Kinematic model (Jazzy: no hardware params here) -->
   <xacro:ur_robot
     name="$(arg name)"
@@ -66,7 +64,18 @@
     safety_pos_margin="$(arg safety_pos_margin)"
     safety_k_position="$(arg safety_k_position)"
+    >
+    <origin xyz="0 0 0" rpy="0 0 0" />
+  </xacro:ur_robot>
+  <!-- ros2_control hardware interface (Jazzy: separate from kinematic macro) -->
+  <xacro:ur_ros2_control
+    name="$(arg name)"
+    tf_prefix="$(arg tf_prefix)"
+    kinematics_parameters_file="$(arg kinematics_params)"
+    robot_ip="$(arg robot_ip)"
+    script_filename="$(arg script_filename)"
+    input_recipe_filename="$(arg input_recipe_filename)"
+    output_recipe_filename="$(arg output_recipe_filename)"
+    use_mock_hardware="$(arg mock_hardware)"
     mock_sensor_commands="$(arg mock_sensor_commands)"
-    sim_gazebo="$(arg sim_gazebo)"
-    sim_ignition="$(arg sim_ignition)"
     headless_mode="$(arg headless_mode)"
     initial_positions="${xacro.load_yaml(initial_positions_file)}"
@@ -80,8 +89,4 @@
     tool_device_name="$(arg tool_device_name)"
     tool_tcp_port="$(arg tool_tcp_port)"
-    robot_ip="$(arg robot_ip)"
-    script_filename="$(arg script_filename)"
-    output_recipe_filename="$(arg output_recipe_filename)"
-    input_recipe_filename="$(arg input_recipe_filename)"
     reverse_ip="$(arg reverse_ip)"
     script_command_port="$(arg script_command_port)"
@@ -90,7 +95,5 @@
     trajectory_port="$(arg trajectory_port)"
     robot_receive_timeout="$(arg robot_receive_timeout)"
-    >
-    <origin xyz="0 0 0" rpy="0 0 0" />
-  </xacro:ur_robot>
+  />
   <!-- Modular Zivid: Arm Mount + Camera (with calibrated camera position) -->
   <!-- Using tool0 instead of flange - Zivid calibration uses tool0 frame -->

File: src/custom-ur-descriptions/ur5e_robot_description/urdf/ur_with_zivid_epick.xacro (robot description, xacro)
@@ -6,4 +6,5 @@
   <!-- import main macros -->
   <xacro:include filename="$(find ur_description)/urdf/ur_macro.xacro"/>
+  <xacro:include filename="$(find ur_robot_driver)/urdf/ur.ros2_control.xacro"/>
   <xacro:include filename="$(find ur5e_robot_description)/urdf/zivid_camera_mount.xacro"/>
   <xacro:include filename="$(find ur5e_robot_description)/urdf/tool_block.xacro"/>
@@ -46,7 +47,4 @@
   <!-- Simulation parameters -->
   <xacro:arg name="mock_sensor_commands" default="false" />
-  <xacro:arg name="sim_gazebo" default="false" />
-  <xacro:arg name="sim_ignition" default="false" />
-  <xacro:arg name="simulation_controllers" default="" />
   <xacro:arg name="mock_hardware" default="true" />
   <!-- initial position for simulations (Fake Hardware, Gazebo, Ignition) -->
@@ -55,5 +53,5 @@
   <!-- create link fixed to the "map" -->
   <link name="map" />
-  <!-- UR arm -->
+  <!-- Kinematic model (Jazzy: no hardware params here) -->
   <xacro:ur_robot
     name="$(arg name)"
@@ -67,7 +65,18 @@
     safety_pos_margin="$(arg safety_pos_margin)"
     safety_k_position="$(arg safety_k_position)"
+    >
+    <origin xyz="0 0 0" rpy="0 0 0" />
+  </xacro:ur_robot>
+  <!-- ros2_control hardware interface (Jazzy: separate from kinematic macro) -->
+  <xacro:ur_ros2_control
+    name="$(arg name)"
+    tf_prefix="$(arg tf_prefix)"
+    kinematics_parameters_file="$(arg kinematics_params)"
+    robot_ip="$(arg robot_ip)"
+    script_filename="$(arg script_filename)"
+    input_recipe_filename="$(arg input_recipe_filename)"
+    output_recipe_filename="$(arg output_recipe_filename)"
+    use_mock_hardware="$(arg mock_hardware)"
     mock_sensor_commands="$(arg mock_sensor_commands)"
-    sim_gazebo="$(arg sim_gazebo)"
-    sim_ignition="$(arg sim_ignition)"
     headless_mode="$(arg headless_mode)"
     initial_positions="${xacro.load_yaml(initial_positions_file)}"
@@ -81,8 +90,4 @@
     tool_device_name="$(arg tool_device_name)"
     tool_tcp_port="$(arg tool_tcp_port)"
-    robot_ip="$(arg robot_ip)"
-    script_filename="$(arg script_filename)"
-    output_recipe_filename="$(arg output_recipe_filename)"
-    input_recipe_filename="$(arg input_recipe_filename)"
     reverse_ip="$(arg reverse_ip)"
     script_command_port="$(arg script_command_port)"
@@ -91,7 +96,5 @@
     trajectory_port="$(arg trajectory_port)"
     robot_receive_timeout="$(arg robot_receive_timeout)"
-    >
-    <origin xyz="0 0 0" rpy="0 0 0" />
-  </xacro:ur_robot>
+  />
   <!-- Modular Zivid: Arm Mount + Camera (with calibrated camera position) -->
   <!-- Using tool0 instead of flange - Zivid calibration uses tool0 frame -->

File: src/custom-ur-descriptions/ur5e_robot_description/urdf/ur_with_zivid_hande.xacro (robot description, xacro)
@@ -6,4 +6,5 @@
   <!-- import main macros -->
   <xacro:include filename="$(find ur_description)/urdf/ur_macro.xacro"/>
+  <xacro:include filename="$(find ur_robot_driver)/urdf/ur.ros2_control.xacro"/>
   <xacro:include filename="$(find ur5e_robot_description)/urdf/zivid_camera_mount.xacro"/>
   <xacro:include filename="$(find ur5e_robot_description)/urdf/tool_block.xacro"/>
@@ -45,7 +46,4 @@
   <!-- Simulation parameters -->
   <xacro:arg name="mock_sensor_commands" default="false" />
-  <xacro:arg name="sim_gazebo" default="false" />
-  <xacro:arg name="sim_ignition" default="false" />
-  <xacro:arg name="simulation_controllers" default="" />
   <xacro:arg name="mock_hardware" default="true" />
   <!-- initial position for simulations (Fake Hardware, Gazebo, Ignition) -->
@@ -54,5 +52,5 @@
   <!-- create link fixed to the "map" -->
   <link name="map" />
-  <!-- UR arm -->
+  <!-- Kinematic model (Jazzy: no hardware params here) -->
   <xacro:ur_robot
     name="$(arg name)"
@@ -66,7 +64,18 @@
     safety_pos_margin="$(arg safety_pos_margin)"
     safety_k_position="$(arg safety_k_position)"
+    >
+    <origin xyz="0 0 0" rpy="0 0 0" />
+  </xacro:ur_robot>
+  <!-- ros2_control hardware interface (Jazzy: separate from kinematic macro) -->
+  <xacro:ur_ros2_control
+    name="$(arg name)"
+    tf_prefix="$(arg tf_prefix)"
+    kinematics_parameters_file="$(arg kinematics_params)"
+    robot_ip="$(arg robot_ip)"
+    script_filename="$(arg script_filename)"
+    input_recipe_filename="$(arg input_recipe_filename)"
+    output_recipe_filename="$(arg output_recipe_filename)"
+    use_mock_hardware="$(arg mock_hardware)"
     mock_sensor_commands="$(arg mock_sensor_commands)"
-    sim_gazebo="$(arg sim_gazebo)"
-    sim_ignition="$(arg sim_ignition)"
     headless_mode="$(arg headless_mode)"
     initial_positions="${xacro.load_yaml(initial_positions_file)}"
@@ -80,8 +89,4 @@
     tool_device_name="$(arg tool_device_name)"
     tool_tcp_port="$(arg tool_tcp_port)"
-    robot_ip="$(arg robot_ip)"
-    script_filename="$(arg script_filename)"
-    output_recipe_filename="$(arg output_recipe_filename)"
-    input_recipe_filename="$(arg input_recipe_filename)"
     reverse_ip="$(arg reverse_ip)"
     script_command_port="$(arg script_command_port)"
@@ -90,7 +95,5 @@
     trajectory_port="$(arg trajectory_port)"
     robot_receive_timeout="$(arg robot_receive_timeout)"
-    >
-    <origin xyz="0 0 0" rpy="0 0 0" />
-  </xacro:ur_robot>
+  />
   <!-- Modular Zivid: Arm Mount + Camera (with calibrated camera position) -->
   <!-- Using tool0 instead of flange - Zivid calibration uses tool0 frame -->

File: src/custom-ur-descriptions/ur5e_robot_description/urdf/ur_with_zivid_pipettor.xacro (robot description, xacro)
@@ -6,4 +6,5 @@
   <!-- import main macros -->
   <xacro:include filename="$(find ur_description)/urdf/ur_macro.xacro"/>
+  <xacro:include filename="$(find ur_robot_driver)/urdf/ur.ros2_control.xacro"/>
   <xacro:include filename="$(find ur5e_robot_description)/urdf/zivid_camera_mount.xacro"/>
   <xacro:include filename="$(find ur5e_robot_description)/urdf/tool_block.xacro"/>
@@ -45,7 +46,4 @@
   <!-- Simulation parameters -->
   <xacro:arg name="mock_sensor_commands" default="false" />
-  <xacro:arg name="sim_gazebo" default="false" />
-  <xacro:arg name="sim_ignition" default="false" />
-  <xacro:arg name="simulation_controllers" default="" />
   <xacro:arg name="mock_hardware" default="true" />
   <!-- initial position for simulations (Fake Hardware, Gazebo, Ignition) -->
@@ -54,5 +52,5 @@
   <!-- create link fixed to the "map" -->
   <link name="map" />
-  <!-- UR arm -->
+  <!-- Kinematic model (Jazzy: no hardware params here) -->
   <xacro:ur_robot
     name="$(arg name)"
@@ -66,7 +64,18 @@
     safety_pos_margin="$(arg safety_pos_margin)"
     safety_k_position="$(arg safety_k_position)"
+    >
+    <origin xyz="0 0 0" rpy="0 0 0" />
+  </xacro:ur_robot>
+  <!-- ros2_control hardware interface (Jazzy: separate from kinematic macro) -->
+  <xacro:ur_ros2_control
+    name="$(arg name)"
+    tf_prefix="$(arg tf_prefix)"
+    kinematics_parameters_file="$(arg kinematics_params)"
+    robot_ip="$(arg robot_ip)"
+    script_filename="$(arg script_filename)"
+    input_recipe_filename="$(arg input_recipe_filename)"
+    output_recipe_filename="$(arg output_recipe_filename)"
+    use_mock_hardware="$(arg mock_hardware)"
     mock_sensor_commands="$(arg mock_sensor_commands)"
-    sim_gazebo="$(arg sim_gazebo)"
-    sim_ignition="$(arg sim_ignition)"
     headless_mode="$(arg headless_mode)"
     initial_positions="${xacro.load_yaml(initial_positions_file)}"
@@ -80,8 +89,4 @@
     tool_device_name="$(arg tool_device_name)"
     tool_tcp_port="$(arg tool_tcp_port)"
-    robot_ip="$(arg robot_ip)"
-    script_filename="$(arg script_filename)"
-    output_recipe_filename="$(arg output_recipe_filename)"
-    input_recipe_filename="$(arg input_recipe_filename)"
     reverse_ip="$(arg reverse_ip)"
     script_command_port="$(arg script_command_port)"
@@ -90,7 +95,5 @@
     trajectory_port="$(arg trajectory_port)"
     robot_receive_timeout="$(arg robot_receive_timeout)"
-    >
-    <origin xyz="0 0 0" rpy="0 0 0" />
-  </xacro:ur_robot>
+  />
   <!-- Modular Zivid: Arm Mount + Camera (with calibrated camera position) -->
   <!-- Using tool0 instead of flange - Zivid calibration uses tool0 frame -->
