Commit message: jazzy: update Isaac URDF mesh paths from humble to jazzy
Updated 4 Isaac URDF files and convert_urdf_for_isaac.sh to reference
/opt/ros/jazzy/ instead of /opt/ros/humble/ for mesh file paths.

Co-Authored-By: Claude Opus 4.6 <noreply@anthropic.com>

File: src/custom-ur-descriptions/ur5e_robot_description/urdf/ur_standalone_isaac.urdf (robot description, URDF)
Before this commit: robot ur5e, 17 links, 16 joints
Links:
- link base_link_inertia: geometry collision mesh filename=/opt/ros/jazzy/share/ur_description/meshes/ur5e/collision/b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; visual mesh filename=/opt/ros/jazzy/share/ur_description/meshes/ur5e/visual/base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
- link forearm_link: geometry collision mesh filename=/opt/ros/jazzy/share/ur_description/meshes/ur5e/collision/f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; visual mesh filename=/opt/ros/jazzy/share/ur_description/meshes/ur5e/visual/fore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
- link shoulder_link: geometry collision mesh filename=/opt/ros/jazzy/share/ur_description/meshes/ur5e/collision/s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; visual mesh filename=/opt/ros/jazzy/share/ur_description/meshes/ur5e/visual/shou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
- link upper_arm_link: geometry collision mesh filename=/opt/ros/jazzy/share/ur_description/meshes/ur5e/collision/u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; visual mesh filename=/opt/ros/jazzy/share/ur_description/meshes/ur5e/visual/uppe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
- link wrist_1_link: geometry collision mesh filename=/opt/ros/jazzy/share/ur_description/meshes/ur5e/collision/w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; visual mesh filename=/opt/ros/jazzy/share/ur_description/meshes/ur5e/visual/wris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
- link wrist_2_link: geometry collision mesh filename=/opt/ros/jazzy/share/ur_description/meshes/ur5e/collision/w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; visual mesh filename=/opt/ros/jazzy/share/ur_description/meshes/ur5e/visual/wris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
- link wrist_3_link: geometry collision mesh filename=/opt/ros/jazzy/share/ur_description/meshes/ur5e/collision/w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; visual mesh filename=/opt/ros/jazzy/share/ur_description/meshes/ur5e/visual/wris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

File: src/custom-ur-descriptions/ur5e_robot_description/urdf/ur_with_zivid_epick_isaac.urdf (robot description, URDF)
Before this commit: robot ur5e, 23 links, 22 joints
Links:
- link base_link_inertia: geometry collision mesh filename=/opt/ros/jazzy/share/ur_description/meshes/ur5e/collision/b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; visual mesh filename=/opt/ros/jazzy/share/ur_description/meshes/ur5e/visual/base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
- link forearm_link: geometry collision mesh filename=/opt/ros/jazzy/share/ur_description/meshes/ur5e/collision/f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; visual mesh filename=/opt/ros/jazzy/share/ur_description/meshes/ur5e/visual/fore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
- link shoulder_link: geometry collision mesh filename=/opt/ros/jazzy/share/ur_description/meshes/ur5e/collision/s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; visual mesh filename=/opt/ros/jazzy/share/ur_description/meshes/ur5e/visual/shou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
- link upper_arm_link: geometry collision mesh filename=/opt/ros/jazzy/share/ur_description/meshes/ur5e/collision/u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; visual mesh filename=/opt/ros/jazzy/share/ur_description/meshes/ur5e/visual/uppe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
- link wrist_1_link: geometry collision mesh filename=/opt/ros/jazzy/share/ur_description/meshes/ur5e/collision/w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; visual mesh filename=/opt/ros/jazzy/share/ur_description/meshes/ur5e/visual/wris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
- link wrist_2_link: geometry collision mesh filename=/opt/ros/jazzy/share/ur_description/meshes/ur5e/collision/w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; visual mesh filename=/opt/ros/jazzy/share/ur_description/meshes/ur5e/visual/wris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
- link wrist_3_link: geometry collision mesh filename=/opt/ros/jazzy/share/ur_description/meshes/ur5e/collision/w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; visual mesh filename=/opt/ros/jazzy/share/ur_description/meshes/ur5e/visual/wris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

File: src/custom-ur-descriptions/ur5e_robot_description/urdf/ur_with_zivid_hande_isaac.urdf (robot description, URDF)
Before this commit: robot ur5e, 22 links, 21 joints
Links:
- link base_link_inertia: geometry collision mesh filename=/opt/ros/jazzy/share/ur_description/meshes/ur5e/collision/b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; visual mesh filename=/opt/ros/jazzy/share/ur_description/meshes/ur5e/visual/base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
- link forearm_link: geometry collision mesh filename=/opt/ros/jazzy/share/ur_description/meshes/ur5e/collision/f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; visual mesh filename=/opt/ros/jazzy/share/ur_description/meshes/ur5e/visual/fore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
- link shoulder_link: geometry collision mesh filename=/opt/ros/jazzy/share/ur_description/meshes/ur5e/collision/s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; visual mesh filename=/opt/ros/jazzy/share/ur_description/meshes/ur5e/visual/shou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
- link upper_arm_link: geometry collision mesh filename=/opt/ros/jazzy/share/ur_description/meshes/ur5e/collision/u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; visual mesh filename=/opt/ros/jazzy/share/ur_description/meshes/ur5e/visual/uppe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
- link wrist_1_link: geometry collision mesh filename=/opt/ros/jazzy/share/ur_description/meshes/ur5e/collision/w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; visual mesh filename=/opt/ros/jazzy/share/ur_description/meshes/ur5e/visual/wris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
- link wrist_2_link: geometry collision mesh filename=/opt/ros/jazzy/share/ur_description/meshes/ur5e/collision/w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; visual mesh filename=/opt/ros/jazzy/share/ur_description/meshes/ur5e/visual/wris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
- link wrist_3_link: geometry collision mesh filename=/opt/ros/jazzy/share/ur_description/meshes/ur5e/collision/w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; visual mesh filename=/opt/ros/jazzy/share/ur_description/meshes/ur5e/visual/wris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

File: src/custom-ur-descriptions/ur5e_robot_description/urdf/ur_with_zivid_pipettor_isaac.urdf (robot description, URDF)
Before this commit: robot ur5e, 21 links, 20 joints
Links:
- link base_link_inertia: geometry collision mesh filename=/opt/ros/jazzy/share/ur_description/meshes/ur5e/collision/b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; visual mesh filename=/opt/ros/jazzy/share/ur_description/meshes/ur5e/visual/base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
- link forearm_link: geometry collision mesh filename=/opt/ros/jazzy/share/ur_description/meshes/ur5e/collision/f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; visual mesh filename=/opt/ros/jazzy/share/ur_description/meshes/ur5e/visual/fore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
- link shoulder_link: geometry collision mesh filename=/opt/ros/jazzy/share/ur_description/meshes/ur5e/collision/s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; visual mesh filename=/opt/ros/jazzy/share/ur_description/meshes/ur5e/visual/shou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
- link upper_arm_link: geometry collision mesh filename=/opt/ros/jazzy/share/ur_description/meshes/ur5e/collision/u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; visual mesh filename=/opt/ros/jazzy/share/ur_description/meshes/ur5e/visual/uppe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
- link wrist_1_link: geometry collision mesh filename=/opt/ros/jazzy/share/ur_description/meshes/ur5e/collision/w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; visual mesh filename=/opt/ros/jazzy/share/ur_description/meshes/ur5e/visual/wris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
- link wrist_2_link: geometry collision mesh filename=/opt/ros/jazzy/share/ur_description/meshes/ur5e/collision/w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; visual mesh filename=/opt/ros/jazzy/share/ur_description/meshes/ur5e/visual/wris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
- link wrist_3_link: geometry collision mesh filename=/opt/ros/jazzy/share/ur_description/meshes/ur5e/collision/w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; visual mesh filename=/opt/ros/jazzy/share/ur_description/meshes/ur5e/visual/wris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

Commit message: chore: fix Isaac URDF converter paths, regenerate Isaac URDFs
Update convert_urdf_for_isaac.sh paths from stale github_ws to
current erobs workspace. Add onrobot_2fg7_description mapping.
Regenerate all 4 Isaac URDFs from Jazzy-updated base URDFs.

Co-Authored-By: Claude Opus 4.6 (1M context) <noreply@anthropic.com>

File: src/custom-ur-descriptions/ur5e_robot_description/urdf/ur_standalone_isaac.urdf (robot description, URDF)
Before this commit: robot ur5e, 17 links, 16 joints
Links:
- link map: mass 0.0 -> None
- link te_robotside: geometry collision mesh filename=/home/aditya/work/erobs/src/custom-ur-descriptions/ur5e_rob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 scale=0.001 0.001 0.001; visual mesh filename=/home/aditya/work/erobs/src/custom-ur-descriptions/ur5e_rob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 scale=0.001 0.001 0.001
- link zivid_arm_mount: geometry collision mesh filename=/home/aditya/work/erobs/src/custom-ur-descriptions/ur5e_rob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 scale=0.001 0.001 0.001; visual mesh filename=/home/aditya/work/erobs/src/custom-ur-descriptions/ur5e_rob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 scale=0.001 0.001 0.001
- link zivid_base_link: geometry collision mesh filename=/home/aditya/work/erobs/src/vision/zivid-ros/zivid_descript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; visual mesh filename=/home/aditya/work/erobs/src/vision/zivid-ros/zivid_descript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
Joints:
- removed joint mount_to_camera_joint
- removed joint zivid_uncalibrated_optical_joint
- added joint optical_to_base_link: type fixed, parent zivid_optical_frame, child zivid_base_link, origin xyz=0.03413 0.02950 -0.04756 rpy=-1.57080 -1.52716 3.14159
- added joint tool0_to_zivid_optical: type fixed, parent tool0, child zivid_optical_frame, origin xyz=0.05635 0.10228 0.06025 rpy=-0.03622 0.05218 3.13437
- joint zivid_arm_mount_joint: origin xyz=0 0 0.005 rpy=0 0 3.14159 -> xyz=0 0 0.005 rpy=0 0 0

File: src/custom-ur-descriptions/ur5e_robot_description/urdf/ur_with_zivid_epick_isaac.urdf (robot description, URDF)
Before this commit: robot ur5e, 23 links, 22 joints
Links:
- added link epick_extension; collision cylinder length=0.018 radius=0.006; visual cylinder length=0.018 radius=0.006
- link epick_body: geometry collision cylinder length=0.1023 radius=0.044; visual mesh filename=/home/aditya/work/erobs/src/end_effectors/ros2_epick_grippe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 scale=0.001 0.001 0.001
- link epick_suction_cup: geometry collision cylinder length=0.006 radius=0.0035; visual cylinder length=0.006 radius=0.0035
- link map: mass 0.0 -> None
- link tool_block: geometry collision mesh filename=/home/aditya/work/erobs/src/custom-ur-descriptions/ur5e_rob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 scale=0.001 0.001 0.001; visual mesh filename=/home/aditya/work/erobs/src/custom-ur-descriptions/ur5e_rob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 scale=0.001 0.001 0.001
- link zivid_arm_mount: geometry collision mesh filename=/home/aditya/work/erobs/src/custom-ur-descriptions/ur5e_rob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 scale=0.001 0.001 0.001; visual mesh filename=/home/aditya/work/erobs/src/custom-ur-descriptions/ur5e_rob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 scale=0.001 0.001 0.001
- link zivid_base_link: geometry collision mesh filename=/home/aditya/work/erobs/src/vision/zivid-ros/zivid_descript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; visual mesh filename=/home/aditya/work/erobs/src/vision/zivid-ros/zivid_descript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
Joints:
- removed joint epick_body_to_epick_suction_cup
- removed joint mount_to_camera_joint
- removed joint zivid_uncalibrated_optical_joint
- added joint epick_body_to_epick_extension: type fixed, parent epick_body, child epick_extension, origin xyz=0 0 0.06015 rpy=0 0 0
- added joint epick_extension_to_epick_suction_cup: type fixed, parent epick_extension, child epick_suction_cup, origin xyz=0 0 0.012 rpy=0 0 0
- added joint optical_to_base_link: type fixed, parent zivid_optical_frame, child zivid_base_link, origin xyz=0.03413 0.02950 -0.04756 rpy=-1.57080 -1.52716 3.14159
- added joint tool0_to_zivid_optical: type fixed, parent tool0, child zivid_optical_frame, origin xyz=0.05635 0.10228 0.06025 rpy=-0.03622 0.05218 3.13437
- joint epick_suction_cup_to_epick_tip: origin xyz=0 0 0.01 rpy=0 0 0 -> xyz=0 0 0.003 rpy=0 0 0
- joint zivid_arm_mount_joint: origin xyz=0 0 0.005 rpy=0 0 3.14159 -> xyz=0 0 0.005 rpy=0 0 0

File: src/custom-ur-descriptions/ur5e_robot_description/urdf/ur_with_zivid_hande_isaac.urdf (robot description, URDF)
Before this commit: robot ur5e, 22 links, 21 joints
Links:
- link map: mass 0.0 -> None
- link robotiq_hande_coupler: geometry collision cylinder length=0.0169 radius=0.0385; visual mesh filename=/home/aditya/work/erobs/src/end_effectors/robotiq_hande_des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
- link robotiq_hande_left_finger: geometry collision mesh filename=/home/aditya/work/erobs/src/end_effectors/robotiq_hande_des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 scale=1.0 1.0 1.0; visual mesh filename=/home/aditya/work/erobs/src/end_effectors/robotiq_hande_des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 scale=1.0 1.0 1.0
- link robotiq_hande_link: geometry collision cylinder length=0.10690000000000001 radius=0.0385; visual mesh filename=/home/aditya/work/erobs/src/end_effectors/robotiq_hande_des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 scale=1.0 1.0 1.0
- link robotiq_hande_right_finger: geometry collision mesh filename=/home/aditya/work/erobs/src/end_effectors/robotiq_hande_des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 scale=1.0 1.0 1.0; visual mesh filename=/home/aditya/work/erobs/src/end_effectors/robotiq_hande_des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 scale=1.0 1.0 1.0
- link tool_block: geometry collision mesh filename=/home/aditya/work/erobs/src/custom-ur-descriptions/ur5e_rob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 scale=0.001 0.001 0.001; visual mesh filename=/home/aditya/work/erobs/src/custom-ur-descriptions/ur5e_rob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 scale=0.001 0.001 0.001
- link zivid_arm_mount: geometry collision mesh filename=/home/aditya/work/erobs/src/custom-ur-descriptions/ur5e_rob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 scale=0.001 0.001 0.001; visual mesh filename=/home/aditya/work/erobs/src/custom-ur-descriptions/ur5e_rob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 scale=0.001 0.001 0.001
- link zivid_base_link: geometry collision mesh filename=/home/aditya/work/erobs/src/vision/zivid-ros/zivid_descript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; visual mesh filename=/home/aditya/work/erobs/src/vision/zivid-ros/zivid_descript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
Joints:
- removed joint mount_to_camera_joint
- removed joint zivid_uncalibrated_optical_joint
- added joint optical_to_base_link: type fixed, parent zivid_optical_frame, child zivid_base_link, origin xyz=0.03413 0.02950 -0.04756 rpy=-1.57080 -1.52716 3.14159
- added joint tool0_to_zivid_optical: type fixed, parent tool0, child zivid_optical_frame, origin xyz=0.05635 0.10228 0.06025 rpy=-0.03622 0.05218 3.13437
- joint zivid_arm_mount_joint: origin xyz=0.00000 0.00000 0.00500 rpy=0.00000 0.00000 3.14159 -> xyz=0 0 0.005 rpy=0 0 0

File: src/custom-ur-descriptions/ur5e_robot_description/urdf/ur_with_zivid_pipettor_isaac.urdf (robot description, URDF)
Before this commit: robot ur5e, 21 links, 20 joints
Links:
- link map: mass 0.0 -> None
- link pipette_body_link: geometry collision mesh filename=/home/aditya/work/erobs/src/end_effectors/pipettor/pipette_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 scale=0.001 0.001 0.001; visual mesh filename=/home/aditya/work/erobs/src/end_effectors/pipettor/pipette_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 scale=0.001 0.001 0.001
- link tool_block: geometry collision mesh filename=/home/aditya/work/erobs/src/custom-ur-descriptions/ur5e_rob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 scale=0.001 0.001 0.001; visual mesh filename=/home/aditya/work/erobs/src/custom-ur-descriptions/ur5e_rob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 scale=0.001 0.001 0.001
- link zivid_arm_mount: geometry collision mesh filename=/home/aditya/work/erobs/src/custom-ur-descriptions/ur5e_rob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 scale=0.001 0.001 0.001; visual mesh filename=/home/aditya/work/erobs/src/custom-ur-descriptions/ur5e_rob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 scale=0.001 0.001 0.001
- link zivid_base_link: geometry collision mesh filename=/home/aditya/work/erobs/src/vision/zivid-ros/zivid_descript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; visual mesh filename=/home/aditya/work/erobs/src/vision/zivid-ros/zivid_descript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
Joints:
- removed joint mount_to_camera_joint
- removed joint zivid_uncalibrated_optical_joint
- added joint optical_to_base_link: type fixed, parent zivid_optical_frame, child zivid_base_link, origin xyz=0.03413 0.02950 -0.04756 rpy=-1.57080 -1.52716 3.14159
- added joint tool0_to_zivid_optical: type fixed, parent tool0, child zivid_optical_frame, origin xyz=0.05635 0.10228 0.06025 rpy=-0.03622 0.05218 3.13437
- joint tool_block_joint: origin xyz=0 0 0.055 rpy=-1.5708 0 3.14159 -> xyz=0 0 0.049 rpy=-1.5708 0 3.14159
- joint zivid_arm_mount_joint: origin xyz=0 0 0.005 rpy=0 0 3.14159 -> xyz=0 0 0.005 rpy=0 0 0
