Commit message: Single source of truth for ePick suction cup profile (#53)
Replace 4 hardcoded numeric xacro args with xacro.load_yaml() that
resolves cup dimensions from suction_cups.yaml at URDF generation time.
Changing cups now requires updating 1 profile name string in 2 files
instead of 4 numeric floats across 3 files.

- ur_with_zivid_epick.xacro: load_yaml + cup_profile arg replaces
  extension_length/radius/suction_cup_height/radius args
- robot_bringup.launch.py: 4 numeric DeclareLaunchArguments → 1 string
- moveit_lifecycle_manager.py: passes profile name, not dimensions
- epick_overlay.xacro: zero stale 7mm_dia defaults
- package.xml: add missing epick_config exec_depend
- CLAUDE.md: fix stale 7mm_dia → 3mm_dia default references
- README.md: document new cup-change workflow

File: src/custom-ur-descriptions/ur5e_robot_description/urdf/ur_with_zivid_epick.xacro (robot description, xacro)
@@ -107,22 +107,21 @@
   <!-- Tool block attached to the Zivid arm mount (not the camera) -->
   <xacro:tool_block parent_link="zivid_arm_mount" xyz="0 0 0.049" rpy="-1.5708 0 3.14159"/>
-  <!-- Suction cup dimensions (passed from launch file via cup profile).
-       IMPORTANT: These defaults are used by the UR driver's robot_state_publisher
-       (which doesn't receive cup profile args from the orchestrator). They MUST
-       match the physically attached cup. When changing cups, update both this file
-       AND default_beamline.yaml grippers.epick.cup_profile.
-       See: epick_config/config/suction_cups.yaml for available profiles. -->
-  <!-- Current physical cup: 3mm_dia -->
-  <xacro:arg name="extension_length" default="0.013"/>
-  <xacro:arg name="extension_radius" default="0.004"/>
-  <xacro:arg name="suction_cup_height" default="0.003"/>
-  <xacro:arg name="suction_cup_radius" default="0.0015"/>
+  <!-- Suction cup profile: dimensions loaded from suction_cups.yaml (single source of truth).
+       The cup_profile default MUST match the physically attached cup — the UR driver's
+       robot_state_publisher uses this default (it can't receive args from the orchestrator).
+       When changing cups, update this default AND default_beamline.yaml grippers.epick.cup_profile.
+       Available profiles: see epick_config/config/suction_cups.yaml -->
+  <xacro:property name="cups_yaml_path" value="$(find epick_config)/config/suction_cups.yaml"/>
+  <xacro:property name="cups_config" value="${xacro.load_yaml(cups_yaml_path)}"/>
+  <xacro:arg name="cup_profile" default="3mm_dia"/>
+  <xacro:property name="cup_profile_name" value="$(arg cup_profile)"/>
+  <xacro:property name="cup" value="${cups_config['cups'][cup_profile_name]}"/>
   <!-- Epick Gripper -->
   <xacro:epick_overlay use_fake_hardware="$(arg use_fake_hardware)" parent="tool_block"
                   origin_xyz="0 -0.03235 0"
                   origin_rpy="-1.5708 0 3.1416"
-                  extension_length="$(arg extension_length)"
-                  extension_radius="$(arg extension_radius)"
-                  suction_cup_height="$(arg suction_cup_height)"
-                  suction_cup_radius="$(arg suction_cup_radius)"/>
+                  extension_length="${cup['extension_length']}"
+                  extension_radius="${cup['extension_radius']}"
+                  suction_cup_height="${cup['suction_cup_height']}"
+                  suction_cup_radius="${cup['suction_cup_radius']}"/>
 </robot>

File: src/end_effectors/epick_config/urdf/epick_overlay.xacro (robot description, xacro)
@@ -4,11 +4,13 @@
   <xacro:include filename="$(find epick_description)/urdf/epick_single_suction_cup.xacro"/>
   <!-- Arguments for parent link and optional prefix -->
+  <!-- Dimension defaults are zeroed — callers must pass actual values from cup profile.
+       Zero geometry makes it obvious if a caller forgets to pass dimensions. -->
   <xacro:macro name="epick_overlay" params="parent prefix:=''
                                  origin_xyz:='0 -0.03235 0'
                                  origin_rpy:='1.5708 0 0'
-                                 suction_cup_height:=0.006
-                                 suction_cup_radius:=0.0035
-                                 extension_length:=0.018
-                                 extension_radius:=0.006
+                                 suction_cup_height:=0.0
+                                 suction_cup_radius:=0.0
+                                 extension_length:=0.0
+                                 extension_radius:=0.0
                                  use_fake_hardware:=false
                                  usb_port:=/tmp/ttyUR">
