Commit message: jazzy: adapt all merged humble code for ROS2 Jazzy
Python:
- Fix 17 remaining warn() → warning() calls across orchestrator,
  zed.py, move_to_stages, vision_stages, mcp_server

MoveIt/URDF:
- Fully adapt ur_zivid_2fg7_moveit_config for Jazzy
  (ompl request_adapters format, joint names, kinematics, rviz)
- Fix ur_with_zivid_2fg7.xacro: use_mock_hardware,
  robot_receive_timeout, remove transmission_hw_interface

End Effectors:
- Fix 2FG7 driver: mock_hardware, pymodbus 3.x cleanup,
  Python 3.12 install path, launch_ros dependency
- Fix ePick: use_mock_hardware in overlay xacro, clean package.xml
- Update end_effectors.repos: hande_description → jazzy-devel

Infrastructure:
- Update 4 Dockerfiles: jazzy base images, Ubuntu 24.04 SDK URLs,
  Python 3.12, branch refs
- Update super-linter default branch to jazzy_dev

Co-Authored-By: Claude Opus 4.6 (1M context) <noreply@anthropic.com>

File: src/custom-ur-descriptions/ur5e_moveit_configs/ur_zivid_2fg7_moveit_config/config/ur.ros2_control.xacro (robot description, xacro)
@@ -50,8 +50,8 @@
                 <state_interface name="velocity"/>
             </joint>
-            <joint name="robotiq_hande_left_finger_joint">
+            <joint name="2fg7_left_finger_joint">
                 <command_interface name="position"/>
                 <state_interface name="position">
-                  <param name="initial_value">${initial_positions['robotiq_hande_left_finger_joint']}</param>
+                  <param name="initial_value">${initial_positions['2fg7_left_finger_joint']}</param>
                 </state_interface>
                 <state_interface name="velocity"/>

File: src/custom-ur-descriptions/ur5e_robot_description/urdf/ur_with_zivid_2fg7.xacro (robot description, xacro)
@@ -17,5 +17,4 @@
   <xacro:arg name="physical_params" default="$(find ur_description)/config/$(arg ur_type)/physical_parameters.yaml"/>
   <xacro:arg name="visual_params" default="$(find ur_description)/config/$(arg ur_type)/visual_parameters.yaml"/>
-  <xacro:arg name="transmission_hw_interface" default=""/>
   <xacro:arg name="safety_limits" default="false"/>
   <xacro:arg name="safety_pos_margin" default="0.15"/>
@@ -33,5 +32,5 @@
   <xacro:arg name="trajectory_port" default="50003"/>
   <!-- Keep-alive: number of 20ms cycles without response before disconnect (10 = 200ms timeout) -->
-  <xacro:arg name="keep_alive_count" default="10"/>
+  <xacro:arg name="robot_receive_timeout" default="0.2"/>
   <!-- tool communication related parameters (2FG7 defaults: 1Mbps, Even parity) -->
   <xacro:arg name="use_tool_communication" default="true" />
@@ -45,6 +44,5 @@
   <xacro:arg name="tool_tcp_port" default="54321" />
   <!-- Simulation parameters -->
-  <xacro:arg name="use_fake_hardware" default="false" />
-  <xacro:arg name="fake_sensor_commands" default="false" />
+  <xacro:arg name="mock_sensor_commands" default="false" />
   <xacro:arg name="sim_gazebo" default="false" />
   <xacro:arg name="sim_ignition" default="false" />
@@ -65,10 +63,8 @@
     physical_parameters_file="$(arg physical_params)"
     visual_parameters_file="$(arg visual_params)"
-    transmission_hw_interface="$(arg transmission_hw_interface)"
     safety_limits="$(arg safety_limits)"
     safety_pos_margin="$(arg safety_pos_margin)"
     safety_k_position="$(arg safety_k_position)"
-    use_fake_hardware="$(arg use_fake_hardware)"
-    fake_sensor_commands="$(arg fake_sensor_commands)"
+    mock_sensor_commands="$(arg mock_sensor_commands)"
     sim_gazebo="$(arg sim_gazebo)"
     sim_ignition="$(arg sim_ignition)"
@@ -93,5 +89,5 @@
     script_sender_port="$(arg script_sender_port)"
     trajectory_port="$(arg trajectory_port)"
-    keep_alive_count="$(arg keep_alive_count)"
+    robot_receive_timeout="$(arg robot_receive_timeout)"
     >
     <origin xyz="0 0 0" rpy="0 0 0" />

File: src/end_effectors/epick_config/urdf/epick_overlay.xacro (robot description, xacro)
@@ -11,5 +11,5 @@
                                  extension_length:=0.018
                                  extension_radius:=0.006
-                                 use_fake_hardware:=false
+                                 use_mock_hardware:=false
                                  usb_port:=/tmp/ttyUR">
     <xacro:epick_single_suction_cup
@@ -22,5 +22,5 @@
       extension_length="${extension_length}"
       extension_radius="${extension_radius}"
-      use_fake_hardware="${use_fake_hardware}"
+      use_mock_hardware="${use_mock_hardware}"
       usb_port="${usb_port}"/>
   </xacro:macro>
