Commit message: rename 2fg7 finger joints to twofg7_* for ROS 2 param compliance
Joint names starting with a digit violate the ROS 2 parameter regex
[a-zA-Z_][a-zA-Z0-9_]*, which blocked -p override injection and forced
beambot_mtc to skip these joints when aggregating TOTG limits.

Rename 2fg7_{left,right}_finger_joint -> twofg7_{left,right}_finger_joint
across URDF, SRDF, joint_limits, controllers, and the Python driver.
Link names, group names, and group_state names (2fg7_open/closed) are
unchanged -- only parameter names had the regex constraint. Drop the
now-obsolete ros_param_name filter and re import in base_stages.py.

Validated end-to-end with hardware: 2fg7 loaded via tool_exchange from
dock, driver advertises gripper_action_controller/gripper_cmd, and
open/close transitions execute on real hardware. Closes #71.

File: src/custom-ur-descriptions/ur5e_moveit_config/config/2fg7/ur.ros2_control.xacro (robot description, xacro)
@@ -50,8 +50,8 @@
                 <state_interface name="velocity"/>
             </joint>
-            <joint name="2fg7_left_finger_joint">
+            <joint name="twofg7_left_finger_joint">
                 <command_interface name="position"/>
                 <state_interface name="position">
-                  <param name="initial_value">${initial_positions['2fg7_left_finger_joint']}</param>
+                  <param name="initial_value">${initial_positions['twofg7_left_finger_joint']}</param>
                 </state_interface>
                 <state_interface name="velocity"/>

File: src/custom-ur-descriptions/ur5e_moveit_config/srdf/2fg7.srdf.xacro (robot description, xacro)
@@ -8,12 +8,12 @@
         <link name="2fg7_right_finger"/>
         <link name="2fg7_tip"/>
-        <joint name="2fg7_left_finger_joint"/>
-        <joint name="2fg7_right_finger_joint"/>
+        <joint name="twofg7_left_finger_joint"/>
+        <joint name="twofg7_right_finger_joint"/>
     </group>
     <group_state name="2fg7_open" group="2fg7_gripper">
-        <joint name="2fg7_left_finger_joint" value="0.035"/>
+        <joint name="twofg7_left_finger_joint" value="0.035"/>
     </group_state>
     <group_state name="2fg7_closed" group="2fg7_gripper">
-        <joint name="2fg7_left_finger_joint" value="0"/>
+        <joint name="twofg7_left_finger_joint" value="0"/>
     </group_state>
     <end_effector name="2fg7_gripper" parent_link="flange" group="2fg7_gripper"/>

File: src/end_effectors/onrobot_2fg7_description/urdf/onrobot_2fg7.xacro (robot description, xacro)
@@ -91,5 +91,5 @@
     </link>
     <!-- Left finger (prismatic, moves in +X direction) -->
-    <joint name="${prefix}2fg7_left_finger_joint" type="prismatic">
+    <joint name="${prefix}twofg7_left_finger_joint" type="prismatic">
       <origin xyz="${finger_base_offset} 0 ${body_height}" rpy="0 0 0"/>
       <parent link="${prefix}2fg7_body"/>
@@ -121,5 +121,5 @@
     </link>
     <!-- Right finger (mimic of left, moves in -X direction) -->
-    <joint name="${prefix}2fg7_right_finger_joint" type="prismatic">
+    <joint name="${prefix}twofg7_right_finger_joint" type="prismatic">
       <origin xyz="${-finger_base_offset} 0 ${body_height}" rpy="0 0 0"/>
       <parent link="${prefix}2fg7_body"/>
@@ -127,5 +127,5 @@
       <axis xyz="-1 0 0"/>
       <limit effort="140" lower="${grip_pos_min}" upper="${grip_pos_max}" velocity="0.450"/>
-      <mimic joint="${prefix}2fg7_left_finger_joint" multiplier="1" offset="0"/>
+      <mimic joint="${prefix}twofg7_left_finger_joint" multiplier="1" offset="0"/>
     </joint>
     <link name="${prefix}2fg7_right_finger">
