Commit message: refactor: rename ur5e_moveit_config → cms_moveit_config, ur5e_robot_description → cms_robot_description
These packages are CMS beamline-specific (gripper configs, URDF meshes,
controller params) but were named generically after the robot model. Since
multiple beamlines will each have their own UR5e, the generic name was
ambiguous. Beamline-prefixed names make ownership clear and let new beamlines
create their own packages (e.g. chx_moveit_config) without confusion.

Updated: package.xml, CMakeLists.txt, launch files, xacro includes, SRDF,
beamline YAML, docs, and all generated URDFs.

File: src/custom-ur-descriptions/cms_moveit_config/srdf/ur.srdf.xacro (robot description, xacro)
@@ -5,20 +5,20 @@
     <xacro:arg name="gripper" default="none"/>
     <!-- Common: ur_arm group, moveit_home, virtual_joint, arm self-collisions -->
-    <xacro:include filename="$(find ur5e_moveit_config)/srdf/common.srdf.xacro"/>
+    <xacro:include filename="$(find cms_moveit_config)/srdf/common.srdf.xacro"/>
     <!-- Gripper-specific: group, states, end_effector, collision pairs -->
     <xacro:if value="${'$(arg gripper)' == 'none'}">
-        <xacro:include filename="$(find ur5e_moveit_config)/srdf/none.srdf.xacro"/>
+        <xacro:include filename="$(find cms_moveit_config)/srdf/none.srdf.xacro"/>
     </xacro:if>
     <xacro:if value="${'$(arg gripper)' == 'epick'}">
-        <xacro:include filename="$(find ur5e_moveit_config)/srdf/epick.srdf.xacro"/>
+        <xacro:include filename="$(find cms_moveit_config)/srdf/epick.srdf.xacro"/>
     </xacro:if>
     <xacro:if value="${'$(arg gripper)' == 'hande'}">
-        <xacro:include filename="$(find ur5e_moveit_config)/srdf/hande.srdf.xacro"/>
+        <xacro:include filename="$(find cms_moveit_config)/srdf/hande.srdf.xacro"/>
     </xacro:if>
     <xacro:if value="${'$(arg gripper)' == '2fg7'}">
-        <xacro:include filename="$(find ur5e_moveit_config)/srdf/2fg7.srdf.xacro"/>
+        <xacro:include filename="$(find cms_moveit_config)/srdf/2fg7.srdf.xacro"/>
     </xacro:if>
     <xacro:if value="${'$(arg gripper)' == 'pipettor'}">
-        <xacro:include filename="$(find ur5e_moveit_config)/srdf/pipettor.srdf.xacro"/>
+        <xacro:include filename="$(find cms_moveit_config)/srdf/pipettor.srdf.xacro"/>
     </xacro:if>
 </robot>

File: src/custom-ur-descriptions/cms_robot_description/urdf/te_robotside.xacro (robot description, xacro)
@@ -6,5 +6,5 @@
         <origin xyz="0 0 0" rpy="0 0 0"/>
         <geometry>
-          <mesh filename="package://ur5e_robot_description/meshes/tool_exchanger/Tool_block_robotside.stl"
+          <mesh filename="package://cms_robot_description/meshes/tool_exchanger/Tool_block_robotside.stl"
                 scale="${scale} ${scale} ${scale}"/>
         </geometry>
@@ -16,5 +16,5 @@
         <origin xyz="0 0 0" rpy="0 0 0"/>
         <geometry>
-          <mesh filename="package://ur5e_robot_description/meshes/tool_exchanger/Tool_block_robotside.stl"
+          <mesh filename="package://cms_robot_description/meshes/tool_exchanger/Tool_block_robotside.stl"
                 scale="${scale} ${scale} ${scale}"/>
         </geometry>

File: src/custom-ur-descriptions/cms_robot_description/urdf/tool_block.xacro (robot description, xacro)
@@ -6,5 +6,5 @@
         <origin xyz="0 0 0" rpy="0 0 0"/>
         <geometry>
-          <mesh filename="package://ur5e_robot_description/meshes/tool_exchanger/Tool_block.stl"
+          <mesh filename="package://cms_robot_description/meshes/tool_exchanger/Tool_block.stl"
                 scale="${scale} ${scale} ${scale}"/>
         </geometry>
@@ -16,5 +16,5 @@
         <origin xyz="0 0 0" rpy="0 0 0"/>
         <geometry>
-          <mesh filename="package://ur5e_robot_description/meshes/tool_exchanger/Tool_block.stl"
+          <mesh filename="package://cms_robot_description/meshes/tool_exchanger/Tool_block.stl"
                 scale="${scale} ${scale} ${scale}"/>
         </geometry>

File: src/custom-ur-descriptions/cms_robot_description/urdf/ur_standalone.urdf (robot description, URDF)
Before this commit: robot ur5e, 17 links, 16 joints
Links:
- link te_robotside: geometry collision mesh filename=package://cms_robot_description/meshes/tool_exchanger/Tool_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 scale=0.001 0.001 0.001; visual mesh filename=package://cms_robot_description/meshes/tool_exchanger/Tool_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 scale=0.001 0.001 0.001
- link zivid_arm_mount: geometry collision mesh filename=package://cms_robot_description/meshes/zivid/zivid_onarm_mo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 scale=0.001 0.001 0.001; visual mesh filename=package://cms_robot_description/meshes/zivid/zivid_onarm_mo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 scale=0.001 0.001 0.001

File: src/custom-ur-descriptions/cms_robot_description/urdf/ur_standalone.xacro (robot description, xacro)
@@ -6,6 +6,6 @@
    <!-- import main macro -->
    <xacro:include filename="$(find ur_description)/urdf/ur_macro.xacro"/>
-   <xacro:include filename="$(find ur5e_robot_description)/urdf/zivid_camera_mount.xacro"/>
-   <xacro:include filename="$(find ur5e_robot_description)/urdf/te_robotside.xacro"/>
+   <xacro:include filename="$(find cms_robot_description)/urdf/zivid_camera_mount.xacro"/>
+   <xacro:include filename="$(find cms_robot_description)/urdf/te_robotside.xacro"/>
    <!-- possible 'ur_type' values: ur3, ur5e, ur5, ur5e, ur10, ur10e, ur16e, ur20 -->
    <!-- the default value should raise an error in case this was called without defining the type -->
@@ -52,5 +52,5 @@
    <xacro:arg name="mock_hardware" default="true" />
    <!-- initial position for simulations (Fake Hardware, Gazebo, Ignition) -->
-   <xacro:arg name="initial_positions_file" default="$(find ur5e_moveit_config)/config/none/initial_positions.yaml"/>
+   <xacro:arg name="initial_positions_file" default="$(find cms_moveit_config)/config/none/initial_positions.yaml"/>
    <!-- convert to property to use substitution in function -->
    <xacro:property name="initial_positions_file" default="$(arg initial_positions_file)"/>

File: src/custom-ur-descriptions/cms_robot_description/urdf/ur_standalone_isaac.urdf (robot description, URDF)
Before this commit: robot ur5e, 24 links, 23 joints
Links:
- removed link epick_base_link
- removed link epick_body
- removed link epick_extension
- removed link epick_suction_cup
- removed link epick_tcp
- removed link epick_tip
- removed link epick_vacuum_state
- removed link tool_block
- added link te_robotside, mass 0.5; collision mesh filename=package://cms_robot_description/meshes/tool_exchanger/Tool_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 scale=0.001 0.001 0.001; visual mesh filename=package://cms_robot_description/meshes/tool_exchanger/Tool_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 scale=0.001 0.001 0.001
- link zivid_arm_mount: geometry collision mesh filename=package://cms_robot_description/meshes/zivid/zivid_onarm_mo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 scale=0.001 0.001 0.001; visual mesh filename=package://cms_robot_description/meshes/zivid/zivid_onarm_mo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 scale=0.001 0.001 0.001
Joints:
- removed joint epick_base_link_to_epick_body
- removed joint epick_body_to_epick_extension
- removed joint epick_extension_to_epick_suction_cup
- removed joint epick_suction_cup_to_epick_tip
- removed joint epick_tip_to_epick_tcp
- removed joint gripper
- removed joint tool_block_joint
- removed joint tool_block_to_epick_base_link
- added joint te_robotside_joint: type fixed, parent zivid_arm_mount, child te_robotside, origin xyz=0 0 0.055 rpy=-1.5708 0 3.14159

File: src/custom-ur-descriptions/cms_robot_description/urdf/ur_with_zivid_2fg7.xacro (robot description, xacro)
@@ -1,12 +1,12 @@
 <?xml version="1.0"?>
 <robot xmlns:xacro="http://wiki.ros.org/xacro" name="$(arg name)">
-<!--Chain: map -> UR -> flange -> zivid_camera_mount -> zivid_camera -> HandE gripper -->
+<!--Chain: map -> UR -> flange -> zivid_camera_mount -> zivid_camera -> 2FG7 gripper -->
   <!-- robot name parameter -->
   <xacro:arg name="name" default="ur5e"/>
   <!-- import main macros -->
   <xacro:include filename="$(find ur_description)/urdf/ur_macro.xacro"/>
-  <xacro:include filename="$(find ur5e_robot_description)/urdf/zivid_camera_mount.xacro"/>
-  <xacro:include filename="$(find ur5e_robot_description)/urdf/tool_block.xacro"/>
-  <xacro:include filename="$(find robotiq_hande_description)/urdf/robotiq_hande_gripper.xacro"/>
+  <xacro:include filename="$(find cms_robot_description)/urdf/zivid_camera_mount.xacro"/>
+  <xacro:include filename="$(find cms_robot_description)/urdf/tool_block.xacro"/>
+  <xacro:include filename="$(find onrobot_2fg7_description)/urdf/onrobot_2fg7.xacro"/>
   <!-- possible 'ur_type' values: ur3, ur5e, ur5, ur10, ur10e, ur16e, ur20 -->
   <xacro:arg name="ur_type" default="ur5e"/>
@@ -34,9 +34,9 @@
   <!-- Keep-alive: number of 20ms cycles without response before disconnect (10 = 200ms timeout) -->
   <xacro:arg name="keep_alive_count" default="10"/>
-  <!-- tool communication related parameters -->
-  <xacro:arg name="use_tool_communication" default="false" />
-  <xacro:arg name="tool_voltage" default="0" />
-  <xacro:arg name="tool_parity" default="0" />
-  <xacro:arg name="tool_baud_rate" default="115200" />
+  <!-- tool communication related parameters (2FG7 defaults: 1Mbps, Even parity) -->
+  <xacro:arg name="use_tool_communication" default="true" />
+  <xacro:arg name="tool_voltage" default="24" />
+  <xacro:arg name="tool_parity" default="2" />
+  <xacro:arg name="tool_baud_rate" default="1000000" />
   <xacro:arg name="tool_stop_bits" default="1" />
   <xacro:arg name="tool_rx_idle_chars" default="1.5" />
@@ -52,5 +52,5 @@
   <xacro:arg name="mock_hardware" default="true" />
   <!-- initial position for simulations (Fake Hardware, Gazebo, Ignition) -->
-  <xacro:arg name="initial_positions_file" default="$(find ur5e_moveit_config)/config/hande/initial_positions.yaml"/>
+  <xacro:arg name="initial_positions_file" default="$(find cms_moveit_config)/config/2fg7/initial_positions.yaml"/>
   <xacro:property name="initial_positions_file" default="$(arg initial_positions_file)"/>
   <!-- create link fixed to the "map" -->
@@ -106,35 +106,8 @@
   <!-- Tool block attached to the Zivid arm mount (not the camera) -->
   <xacro:tool_block parent_link="zivid_arm_mount" xyz="0 0 0.049" rpy="-1.5708 0 3.14159"/>
-  <!-- gripper pos wrt camera    -->
-  <xacro:arg name="grip_pos_min" default="0"/>
-  <xacro:arg name="grip_pos_max" default="0.025"/>
-  <xacro:arg name="tty_port" default="/tmp/ttyUR"/>
-  <xacro:arg name="baudrate" default="115200"/>
-  <xacro:arg name="parity" default="N"/>
-  <xacro:arg name="data_bits" default="8"/>
-  <xacro:arg name="stop_bit" default="1"/>
-  <xacro:arg name="slave_id" default="9"/>
-  <xacro:arg name="create_socat_tty" default="true"/>
-  <xacro:arg name="socat_ip_address" default="$(arg robot_ip)"/>
-  <xacro:arg name="socat_port" default="54321"/>
-  <!-- Hand-E xyz previously "0 -0.02 0" — updated based on physical measurement -->
-  <xacro:robotiq_hande_gripper
-    name="robotiq_hande_gripper"
-    prefix="$(arg tf_prefix)"
+  <!-- OnRobot 2FG7 gripper — same mounting offset as ePick/Hand-E (same bolt pattern) -->
+  <xacro:onrobot_2fg7
     parent="tool_block"
-    grip_pos_min="$(arg grip_pos_min)"
-    grip_pos_max="$(arg grip_pos_max)"
-    tty_port="$(arg tty_port)"
-    baudrate="$(arg baudrate)"
-    parity="$(arg parity)"
-    data_bits="$(arg data_bits)"
-    stop_bit="$(arg stop_bit)"
-    slave_id="$(arg slave_id)"
-    use_fake_hardware="$(arg use_fake_hardware)"
     xyz="0 -0.03235 0"
-    rpy="-1.5708 0 3.1416"
-    create_socat_tty="$(arg create_socat_tty)"
-    socat_ip_address="$(arg socat_ip_address)"
-    socat_port="$(arg socat_port)"
-  />
+    rpy="-1.5708 0 3.1416"/>
 </robot>

File: src/custom-ur-descriptions/cms_robot_description/urdf/ur_with_zivid_epick.urdf (robot description, URDF)
Before this commit: robot ur5e, 22 links, 21 joints
Links:
- removed link robotiq_hande_coupler
- removed link robotiq_hande_end
- removed link robotiq_hande_left_finger
- removed link robotiq_hande_link
- removed link robotiq_hande_right_finger
- added link epick_base_link
- added link epick_body; collision cylinder length=0.1023 radius=0.044; visual mesh filename=package://epick_description/meshes/visual/epick_body.stl scale=0.001 0.001 0.001
- added link epick_extension; collision cylinder length=0.018 radius=0.006; visual cylinder length=0.018 radius=0.006
- added link epick_suction_cup; collision cylinder length=0.006 radius=0.0035; visual cylinder length=0.006 radius=0.0035
- added link epick_tcp
- added link epick_tip
- added link epick_vacuum_state
- link tool_block: geometry collision mesh filename=package://cms_robot_description/meshes/tool_exchanger/Tool_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 scale=0.001 0.001 0.001; visual mesh filename=package://cms_robot_description/meshes/tool_exchanger/Tool_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 scale=0.001 0.001 0.001
- link zivid_arm_mount: geometry collision mesh filename=package://cms_robot_description/meshes/zivid/zivid_onarm_mo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 scale=0.001 0.001 0.001; visual mesh filename=package://cms_robot_description/meshes/zivid/zivid_onarm_mo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 scale=0.001 0.001 0.001
Joints:
- removed joint robotiq_hande_base_joint
- removed joint robotiq_hande_coupler_joint
- removed joint robotiq_hande_end_joint
- removed joint robotiq_hande_left_finger_joint
- removed joint robotiq_hande_right_finger_joint
- added joint epick_base_link_to_epick_body: type fixed, parent epick_base_link, child epick_body, origin xyz=0 0 0.05115 rpy=0 0 0
- added joint epick_body_to_epick_extension: type fixed, parent epick_body, child epick_extension, origin xyz=0 0 0.06015 rpy=0 0 0
- added joint epick_extension_to_epick_suction_cup: type fixed, parent epick_extension, child epick_suction_cup, origin xyz=0 0 0.012 rpy=0 0 0
- added joint epick_suction_cup_to_epick_tip: type fixed, parent epick_suction_cup, child epick_tip, origin xyz=0 0 0.003 rpy=0 0 0
- added joint epick_tip_to_epick_tcp: type fixed, parent epick_tip, child epick_tcp, origin xyz=0 0 -0.0 rpy=0 0 0
- added joint gripper: type revolute, parent epick_tcp, child epick_vacuum_state, origin xyz=0 0 0 rpy=0 0 0, limit lower=0.0 upper=1.0 effort=30 velocity=1.0
- added joint tool_block_to_epick_base_link: type fixed, parent tool_block, child epick_base_link, origin xyz=0 -0.03235 0 rpy=-1.5708 0 3.1416

File: src/custom-ur-descriptions/cms_robot_description/urdf/ur_with_zivid_epick.xacro (robot description, xacro)
@@ -6,6 +6,6 @@
   <!-- import main macros -->
   <xacro:include filename="$(find ur_description)/urdf/ur_macro.xacro"/>
-  <xacro:include filename="$(find ur5e_robot_description)/urdf/zivid_camera_mount.xacro"/>
-  <xacro:include filename="$(find ur5e_robot_description)/urdf/tool_block.xacro"/>
+  <xacro:include filename="$(find cms_robot_description)/urdf/zivid_camera_mount.xacro"/>
+  <xacro:include filename="$(find cms_robot_description)/urdf/tool_block.xacro"/>
   <xacro:include filename="$(find epick_config)/urdf/epick_overlay.xacro"/>
   <!-- possible 'ur_type' values: ur3, ur5e, ur5, ur10, ur10e, ur16e, ur20 -->
@@ -53,5 +53,5 @@
   <xacro:arg name="mock_hardware" default="true" />
   <!-- initial position for simulations (Fake Hardware, Gazebo, Ignition) -->
-  <xacro:arg name="initial_positions_file" default="$(find ur5e_moveit_config)/config/epick/initial_positions.yaml"/>
+  <xacro:arg name="initial_positions_file" default="$(find cms_moveit_config)/config/epick/initial_positions.yaml"/>
   <xacro:property name="initial_positions_file" default="$(arg initial_positions_file)"/>
   <!-- create link fixed to the "map" -->

File: src/custom-ur-descriptions/cms_robot_description/urdf/ur_with_zivid_epick_isaac.urdf (robot description, URDF)
Before this commit: robot ur5e, 24 links, 23 joints
Links:
- link tool_block: geometry collision mesh filename=package://cms_robot_description/meshes/tool_exchanger/Tool_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 scale=0.001 0.001 0.001; visual mesh filename=package://cms_robot_description/meshes/tool_exchanger/Tool_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 scale=0.001 0.001 0.001
- link zivid_arm_mount: geometry collision mesh filename=package://cms_robot_description/meshes/zivid/zivid_onarm_mo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 scale=0.001 0.001 0.001; visual mesh filename=package://cms_robot_description/meshes/zivid/zivid_onarm_mo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 scale=0.001 0.001 0.001

File: src/custom-ur-descriptions/cms_robot_description/urdf/ur_with_zivid_hande.urdf (robot description, URDF)
Before this commit: robot ur5e, 22 links, 21 joints
Links:
- link tool_block: geometry collision mesh filename=package://cms_robot_description/meshes/tool_exchanger/Tool_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 scale=0.001 0.001 0.001; visual mesh filename=package://cms_robot_description/meshes/tool_exchanger/Tool_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 scale=0.001 0.001 0.001
- link zivid_arm_mount: geometry collision mesh filename=package://cms_robot_description/meshes/zivid/zivid_onarm_mo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 scale=0.001 0.001 0.001; visual mesh filename=package://cms_robot_description/meshes/zivid/zivid_onarm_mo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 scale=0.001 0.001 0.001

File: src/custom-ur-descriptions/cms_robot_description/urdf/ur_with_zivid_hande.xacro (robot description, xacro)
@@ -1,12 +1,12 @@
 <?xml version="1.0"?>
 <robot xmlns:xacro="http://wiki.ros.org/xacro" name="$(arg name)">
-<!--Chain: map -> UR -> flange -> zivid_camera_mount -> zivid_camera -> 2FG7 gripper -->
+<!--Chain: map -> UR -> flange -> zivid_camera_mount -> zivid_camera -> HandE gripper -->
   <!-- robot name parameter -->
   <xacro:arg name="name" default="ur5e"/>
   <!-- import main macros -->
   <xacro:include filename="$(find ur_description)/urdf/ur_macro.xacro"/>
-  <xacro:include filename="$(find ur5e_robot_description)/urdf/zivid_camera_mount.xacro"/>
-  <xacro:include filename="$(find ur5e_robot_description)/urdf/tool_block.xacro"/>
-  <xacro:include filename="$(find onrobot_2fg7_description)/urdf/onrobot_2fg7.xacro"/>
+  <xacro:include filename="$(find cms_robot_description)/urdf/zivid_camera_mount.xacro"/>
+  <xacro:include filename="$(find cms_robot_description)/urdf/tool_block.xacro"/>
+  <xacro:include filename="$(find robotiq_hande_description)/urdf/robotiq_hande_gripper.xacro"/>
   <!-- possible 'ur_type' values: ur3, ur5e, ur5, ur10, ur10e, ur16e, ur20 -->
   <xacro:arg name="ur_type" default="ur5e"/>
@@ -34,9 +34,9 @@
   <!-- Keep-alive: number of 20ms cycles without response before disconnect (10 = 200ms timeout) -->
   <xacro:arg name="keep_alive_count" default="10"/>
-  <!-- tool communication related parameters (2FG7 defaults: 1Mbps, Even parity) -->
-  <xacro:arg name="use_tool_communication" default="true" />
-  <xacro:arg name="tool_voltage" default="24" />
-  <xacro:arg name="tool_parity" default="2" />
-  <xacro:arg name="tool_baud_rate" default="1000000" />
+  <!-- tool communication related parameters -->
+  <xacro:arg name="use_tool_communication" default="false" />
+  <xacro:arg name="tool_voltage" default="0" />
+  <xacro:arg name="tool_parity" default="0" />
+  <xacro:arg name="tool_baud_rate" default="115200" />
   <xacro:arg name="tool_stop_bits" default="1" />
   <xacro:arg name="tool_rx_idle_chars" default="1.5" />
@@ -52,5 +52,5 @@
   <xacro:arg name="mock_hardware" default="true" />
   <!-- initial position for simulations (Fake Hardware, Gazebo, Ignition) -->
-  <xacro:arg name="initial_positions_file" default="$(find ur5e_moveit_config)/config/2fg7/initial_positions.yaml"/>
+  <xacro:arg name="initial_positions_file" default="$(find cms_moveit_config)/config/hande/initial_positions.yaml"/>
   <xacro:property name="initial_positions_file" default="$(arg initial_positions_file)"/>
   <!-- create link fixed to the "map" -->
@@ -106,8 +106,35 @@
   <!-- Tool block attached to the Zivid arm mount (not the camera) -->
   <xacro:tool_block parent_link="zivid_arm_mount" xyz="0 0 0.049" rpy="-1.5708 0 3.14159"/>
-  <!-- OnRobot 2FG7 gripper — same mounting offset as ePick/Hand-E (same bolt pattern) -->
-  <xacro:onrobot_2fg7
+  <!-- gripper pos wrt camera    -->
+  <xacro:arg name="grip_pos_min" default="0"/>
+  <xacro:arg name="grip_pos_max" default="0.025"/>
+  <xacro:arg name="tty_port" default="/tmp/ttyUR"/>
+  <xacro:arg name="baudrate" default="115200"/>
+  <xacro:arg name="parity" default="N"/>
+  <xacro:arg name="data_bits" default="8"/>
+  <xacro:arg name="stop_bit" default="1"/>
+  <xacro:arg name="slave_id" default="9"/>
+  <xacro:arg name="create_socat_tty" default="true"/>
+  <xacro:arg name="socat_ip_address" default="$(arg robot_ip)"/>
+  <xacro:arg name="socat_port" default="54321"/>
+  <!-- Hand-E xyz previously "0 -0.02 0" — updated based on physical measurement -->
+  <xacro:robotiq_hande_gripper
+    name="robotiq_hande_gripper"
+    prefix="$(arg tf_prefix)"
     parent="tool_block"
+    grip_pos_min="$(arg grip_pos_min)"
+    grip_pos_max="$(arg grip_pos_max)"
+    tty_port="$(arg tty_port)"
+    baudrate="$(arg baudrate)"
+    parity="$(arg parity)"
+    data_bits="$(arg data_bits)"
+    stop_bit="$(arg stop_bit)"
+    slave_id="$(arg slave_id)"
+    use_fake_hardware="$(arg use_fake_hardware)"
     xyz="0 -0.03235 0"
-    rpy="-1.5708 0 3.1416"/>
+    rpy="-1.5708 0 3.1416"
+    create_socat_tty="$(arg create_socat_tty)"
+    socat_ip_address="$(arg socat_ip_address)"
+    socat_port="$(arg socat_port)"
+  />
 </robot>
