Commit message: refactor: rename ur5e_moveit_config → cms_moveit_config, ur5e_robot_description → cms_robot_description
These packages are CMS beamline-specific (gripper configs, URDF meshes,
controller params) but were named generically after the robot model. Since
multiple beamlines will each have their own UR5e, the generic name was
ambiguous. Beamline-prefixed names make ownership clear and let new beamlines
create their own packages (e.g. chx_moveit_config) without confusion.

Updated: package.xml, CMakeLists.txt, launch files, xacro includes, SRDF,
beamline YAML, docs, and all generated URDFs.

File: src/custom-ur-descriptions/cms_robot_description/urdf/ur_with_zivid_hande_isaac.urdf (robot description, URDF)
Before this commit: robot ur5e, 21 links, 20 joints
Links:
- removed link led_strip_link
- removed link pipette_base_link
- removed link pipette_body_link
- removed link pipette_tip_link
- added link robotiq_hande_coupler, mass 0.119; collision cylinder length=0.0169 radius=0.0385; visual mesh filename=package://robotiq_hande_description/meshes/io_coupler.dae
- added link robotiq_hande_end
- added link robotiq_hande_left_finger, mass 0.03804; collision mesh filename=package://robotiq_hande_description/meshes/finger_collision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 scale=1.0 1.0 1.0; visual mesh filename=package://robotiq_hande_description/meshes/finger.dae scale=1.0 1.0 1.0
- added link robotiq_hande_link, mass 0.86387; collision cylinder length=0.10690000000000001 radius=0.0385; visual mesh filename=package://robotiq_hande_description/meshes/hande.dae scale=1.0 1.0 1.0
- added link robotiq_hande_right_finger, mass 0.03804; collision mesh filename=package://robotiq_hande_description/meshes/finger_collision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 scale=1.0 1.0 1.0; visual mesh filename=package://robotiq_hande_description/meshes/finger.dae scale=1.0 1.0 1.0
- link tool_block: geometry collision mesh filename=package://cms_robot_description/meshes/tool_exchanger/Tool_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 scale=0.001 0.001 0.001; visual mesh filename=package://cms_robot_description/meshes/tool_exchanger/Tool_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 scale=0.001 0.001 0.001
- link zivid_arm_mount: geometry collision mesh filename=package://cms_robot_description/meshes/zivid/zivid_onarm_mo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 scale=0.001 0.001 0.001; visual mesh filename=package://cms_robot_description/meshes/zivid/zivid_onarm_mo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 scale=0.001 0.001 0.001
Joints:
- removed joint led_strip_joint
- removed joint pipette_attachment_joint
- removed joint pipette_orientation_joint
- removed joint pipette_tip_joint
- added joint robotiq_hande_base_joint: type fixed, parent robotiq_hande_coupler, child robotiq_hande_link, origin xyz=0 0 0.011 rpy=0 0 0
- added joint robotiq_hande_coupler_joint: type fixed, parent tool_block, child robotiq_hande_coupler, origin xyz=0 -0.03235 0 rpy=-1.5708 0 3.1416
- added joint robotiq_hande_end_joint: type fixed, parent robotiq_hande_link, child robotiq_hande_end, origin xyz=0 0 0.14550000000000002 rpy=0 0 0
- added joint robotiq_hande_left_finger_joint: type prismatic, parent robotiq_hande_link, child robotiq_hande_left_finger, origin xyz=0 0 0.099 rpy=0 0 0, axis 1 0 0, limit lower=0 upper=0.025 effort=130 velocity=0.15
- added joint robotiq_hande_right_finger_joint: type prismatic, parent robotiq_hande_link, child robotiq_hande_right_finger, origin xyz=0 0 0.099 rpy=0 0 0, axis -1 0 0, limit lower=0 upper=0.025 effort=130 velocity=0.15, mimic joint=robotiq_hande_left_finger_joint multiplier=1 offset=0

File: src/custom-ur-descriptions/cms_robot_description/urdf/ur_with_zivid_pipettor.urdf (robot description, URDF)
Before this commit: robot ur5e, 21 links, 20 joints
Links:
- link tool_block: geometry collision mesh filename=package://cms_robot_description/meshes/tool_exchanger/Tool_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 scale=0.001 0.001 0.001; visual mesh filename=package://cms_robot_description/meshes/tool_exchanger/Tool_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 scale=0.001 0.001 0.001
- link zivid_arm_mount: geometry collision mesh filename=package://cms_robot_description/meshes/zivid/zivid_onarm_mo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 scale=0.001 0.001 0.001; visual mesh filename=package://cms_robot_description/meshes/zivid/zivid_onarm_mo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 scale=0.001 0.001 0.001

File: src/custom-ur-descriptions/cms_robot_description/urdf/ur_with_zivid_pipettor.xacro (robot description, xacro)
@@ -6,6 +6,6 @@
   <!-- import main macros -->
   <xacro:include filename="$(find ur_description)/urdf/ur_macro.xacro"/>
-  <xacro:include filename="$(find ur5e_robot_description)/urdf/zivid_camera_mount.xacro"/>
-  <xacro:include filename="$(find ur5e_robot_description)/urdf/tool_block.xacro"/>
+  <xacro:include filename="$(find cms_robot_description)/urdf/zivid_camera_mount.xacro"/>
+  <xacro:include filename="$(find cms_robot_description)/urdf/tool_block.xacro"/>
   <xacro:include filename="$(find pipette_description)/urdf/pipette_macro.urdf.xacro"/>
   <!-- possible 'ur_type' values: ur3, ur5e, ur5, ur10, ur10e, ur16e, ur20 -->
@@ -52,5 +52,5 @@
   <xacro:arg name="mock_hardware" default="true" />
   <!-- initial position for simulations (Fake Hardware, Gazebo, Ignition) -->
-  <xacro:arg name="initial_positions_file" default="$(find ur5e_moveit_config)/config/pipettor/initial_positions.yaml"/>
+  <xacro:arg name="initial_positions_file" default="$(find cms_moveit_config)/config/pipettor/initial_positions.yaml"/>
   <xacro:property name="initial_positions_file" default="$(arg initial_positions_file)"/>
   <!-- create link fixed to the "map" -->

File: src/custom-ur-descriptions/cms_robot_description/urdf/ur_with_zivid_pipettor_isaac.urdf (robot description, URDF)
Before this commit: robot ur5e, 17 links, 16 joints
Links:
- removed link te_robotside
- added link led_strip_link; visual box size=0.002 0.001 0.02
- added link pipette_base_link
- added link pipette_body_link, mass 0.2; collision mesh filename=package://pipette_description/meshes/collision/pipettor_col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 scale=0.001 0.001 0.001; visual mesh filename=package://pipette_description/meshes/visual/pipettor_visual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 scale=0.001 0.001 0.001
- added link pipette_tip_link
- added link tool_block, mass 0.2; collision mesh filename=package://cms_robot_description/meshes/tool_exchanger/Tool_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 scale=0.001 0.001 0.001; visual mesh filename=package://cms_robot_description/meshes/tool_exchanger/Tool_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 scale=0.001 0.001 0.001
- link zivid_arm_mount: geometry collision mesh filename=package://cms_robot_description/meshes/zivid/zivid_onarm_mo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 scale=0.001 0.001 0.001; visual mesh filename=package://cms_robot_description/meshes/zivid/zivid_onarm_mo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 scale=0.001 0.001 0.001
Joints:
- removed joint te_robotside_joint
- added joint led_strip_joint: type fixed, parent pipette_base_link, child led_strip_link, origin xyz=0 0.025 0.238 rpy=0 0 0
- added joint pipette_attachment_joint: type fixed, parent tool_block, child pipette_base_link, origin xyz=-0.005 -0.015 0 rpy=-1.5708 0 3.1416
- added joint pipette_orientation_joint: type fixed, parent pipette_base_link, child pipette_body_link, origin xyz=-0.09 -0.055 0.34 rpy=-1.5708 0 0
- added joint pipette_tip_joint: type fixed, parent pipette_base_link, child pipette_tip_link, origin xyz=0 0 0.34 rpy=0 0 0
- added joint tool_block_joint: type fixed, parent zivid_arm_mount, child tool_block, origin xyz=0 0 0.049 rpy=-1.5708 0 3.14159

File: src/custom-ur-descriptions/cms_robot_description/urdf/zivid_camera_mount.xacro (robot description, xacro)
@@ -51,5 +51,5 @@
         <geometry>
           <!-- Official Zivid On-Arm Mount (from zivid.com/downloads) -->
-          <mesh filename="package://ur5e_robot_description/meshes/zivid/zivid_onarm_mount.stl"
+          <mesh filename="package://cms_robot_description/meshes/zivid/zivid_onarm_mount.stl"
                 scale="0.001 0.001 0.001"/>
         </geometry>
@@ -61,5 +61,5 @@
         <origin xyz="0 0 0" rpy="0 0 0"/>
         <geometry>
-          <mesh filename="package://ur5e_robot_description/meshes/zivid/zivid_onarm_mount.stl"
+          <mesh filename="package://cms_robot_description/meshes/zivid/zivid_onarm_mount.stl"
                 scale="0.001 0.001 0.001"/>
         </geometry>
