Commit message: replace makeshift tool block with EX-50-35 wrist extension + Wingman plates
Replaces the old 2-spacer makeshift tool block with a proper setup:
- EX-50-35 wrist extension (35mm, bolts to flange)
- Wingman WM1 robot-side plate (te_robotside)
- Wingman WM1 tool-side plate (te_toolside, per-gripper)

New kinematic chain: tool0 → wrist_extension → te_robotside → te_toolside → gripper
"none" config ends at te_robotside (no tool plate, no gripper).

Updated all 5 CMS gripper configs (none, epick, hande, 2fg7, pipettor),
their SRDFs, and regenerated pre-built URDF files.

File: src/custom-ur-descriptions/cms_moveit_config/srdf/2fg7.srdf.xacro (robot description, xacro)
@@ -22,5 +22,7 @@
     <disable_collisions link1="2fg7_base_link" link2="2fg7_left_finger" reason="Never"/>
     <disable_collisions link1="2fg7_base_link" link2="2fg7_right_finger" reason="Never"/>
-    <disable_collisions link1="2fg7_base_link" link2="tool_block" reason="Adjacent"/>
+    <disable_collisions link1="2fg7_base_link" link2="te_toolside" reason="Adjacent"/>
+    <disable_collisions link1="2fg7_base_link" link2="te_robotside" reason="Never"/>
+    <disable_collisions link1="2fg7_base_link" link2="wrist_extension" reason="Never"/>
     <disable_collisions link1="2fg7_base_link" link2="wrist_1_link" reason="Never"/>
     <disable_collisions link1="2fg7_base_link" link2="wrist_2_link" reason="Never"/>
@@ -30,5 +32,5 @@
     <disable_collisions link1="2fg7_body" link2="2fg7_left_finger" reason="Adjacent"/>
     <disable_collisions link1="2fg7_body" link2="2fg7_right_finger" reason="Adjacent"/>
-    <disable_collisions link1="2fg7_body" link2="tool_block" reason="Never"/>
+    <disable_collisions link1="2fg7_body" link2="te_toolside" reason="Never"/>
     <disable_collisions link1="2fg7_body" link2="wrist_1_link" reason="Never"/>
     <disable_collisions link1="2fg7_body" link2="wrist_2_link" reason="Never"/>
@@ -37,5 +39,5 @@
     <disable_collisions link1="2fg7_body" link2="zivid_base_link" reason="Never"/>
     <disable_collisions link1="2fg7_left_finger" link2="2fg7_right_finger" reason="Default"/>
-    <disable_collisions link1="2fg7_left_finger" link2="tool_block" reason="Never"/>
+    <disable_collisions link1="2fg7_left_finger" link2="te_toolside" reason="Never"/>
     <disable_collisions link1="2fg7_left_finger" link2="wrist_1_link" reason="Never"/>
     <disable_collisions link1="2fg7_left_finger" link2="wrist_2_link" reason="Never"/>
@@ -43,5 +45,5 @@
     <disable_collisions link1="2fg7_left_finger" link2="zivid_arm_mount" reason="Never"/>
     <disable_collisions link1="2fg7_left_finger" link2="zivid_base_link" reason="Never"/>
-    <disable_collisions link1="2fg7_right_finger" link2="tool_block" reason="Never"/>
+    <disable_collisions link1="2fg7_right_finger" link2="te_toolside" reason="Never"/>
     <disable_collisions link1="2fg7_right_finger" link2="wrist_1_link" reason="Never"/>
     <disable_collisions link1="2fg7_right_finger" link2="wrist_2_link" reason="Never"/>
@@ -49,10 +51,24 @@
     <disable_collisions link1="2fg7_right_finger" link2="zivid_arm_mount" reason="Never"/>
     <disable_collisions link1="2fg7_right_finger" link2="zivid_base_link" reason="Never"/>
-    <!-- Shared tool_block + camera collision rules -->
-    <disable_collisions link1="tool_block" link2="wrist_1_link" reason="Never"/>
-    <disable_collisions link1="tool_block" link2="wrist_2_link" reason="Never"/>
-    <disable_collisions link1="tool_block" link2="wrist_3_link" reason="Never"/>
-    <disable_collisions link1="tool_block" link2="zivid_arm_mount" reason="Adjacent"/>
-    <disable_collisions link1="tool_block" link2="zivid_base_link" reason="Never"/>
+    <!-- Wrist extension + tool exchanger + camera collision rules -->
+    <disable_collisions link1="wrist_extension" link2="wrist_1_link" reason="Never"/>
+    <disable_collisions link1="wrist_extension" link2="wrist_2_link" reason="Never"/>
+    <disable_collisions link1="wrist_extension" link2="wrist_3_link" reason="Never"/>
+    <disable_collisions link1="wrist_extension" link2="flange" reason="Adjacent"/>
+    <disable_collisions link1="wrist_extension" link2="zivid_arm_mount" reason="Adjacent"/>
+    <disable_collisions link1="wrist_extension" link2="zivid_base_link" reason="Never"/>
+    <disable_collisions link1="te_robotside" link2="wrist_extension" reason="Adjacent"/>
+    <disable_collisions link1="te_robotside" link2="wrist_1_link" reason="Never"/>
+    <disable_collisions link1="te_robotside" link2="wrist_2_link" reason="Never"/>
+    <disable_collisions link1="te_robotside" link2="wrist_3_link" reason="Never"/>
+    <disable_collisions link1="te_robotside" link2="zivid_arm_mount" reason="Never"/>
+    <disable_collisions link1="te_robotside" link2="zivid_base_link" reason="Never"/>
+    <disable_collisions link1="te_toolside" link2="te_robotside" reason="Adjacent"/>
+    <disable_collisions link1="te_toolside" link2="wrist_extension" reason="Never"/>
+    <disable_collisions link1="te_toolside" link2="wrist_1_link" reason="Never"/>
+    <disable_collisions link1="te_toolside" link2="wrist_2_link" reason="Never"/>
+    <disable_collisions link1="te_toolside" link2="wrist_3_link" reason="Never"/>
+    <disable_collisions link1="te_toolside" link2="zivid_arm_mount" reason="Never"/>
+    <disable_collisions link1="te_toolside" link2="zivid_base_link" reason="Never"/>
     <disable_collisions link1="wrist_2_link" link2="zivid_arm_mount" reason="Never"/>
     <disable_collisions link1="wrist_2_link" link2="zivid_base_link" reason="Never"/>
@@ -61,4 +77,3 @@
     <disable_collisions link1="zivid_arm_mount" link2="zivid_base_link" reason="Adjacent"/>
     <disable_collisions link1="flange" link2="zivid_arm_mount" reason="Adjacent"/>
-    <disable_collisions link1="flange" link2="tool_block" reason="Never"/>
 </robot>

File: src/custom-ur-descriptions/cms_moveit_config/srdf/epick.srdf.xacro (robot description, xacro)
@@ -3,5 +3,5 @@
 <robot xmlns:xacro="http://www.ros.org/wiki/xacro">
     <group name="epick_gripper">
-        <link name="tool_block"/>
+        <link name="te_toolside"/>
         <link name="epick_base_link"/>
         <link name="epick_body"/>
@@ -22,7 +22,9 @@
     <disable_collisions link1="epick_body" link2="epick_extension" reason="Adjacent"/>
     <disable_collisions link1="epick_body" link2="epick_suction_cup" reason="Never"/>
-    <disable_collisions link1="epick_body" link2="tool_block" reason="Adjacent"/>
+    <disable_collisions link1="epick_body" link2="te_toolside" reason="Adjacent"/>
+    <disable_collisions link1="epick_body" link2="te_robotside" reason="Never"/>
+    <disable_collisions link1="epick_body" link2="wrist_extension" reason="Never"/>
     <disable_collisions link1="epick_extension" link2="epick_suction_cup" reason="Adjacent"/>
-    <disable_collisions link1="epick_extension" link2="tool_block" reason="Never"/>
+    <disable_collisions link1="epick_extension" link2="te_toolside" reason="Never"/>
     <disable_collisions link1="epick_extension" link2="wrist_1_link" reason="Never"/>
     <disable_collisions link1="epick_extension" link2="wrist_2_link" reason="Never"/>
@@ -35,5 +37,5 @@
     <disable_collisions link1="epick_body" link2="zivid_arm_mount" reason="Never"/>
     <disable_collisions link1="epick_body" link2="zivid_base_link" reason="Never"/>
-    <disable_collisions link1="epick_suction_cup" link2="tool_block" reason="Never"/>
+    <disable_collisions link1="epick_suction_cup" link2="te_toolside" reason="Never"/>
     <disable_collisions link1="epick_suction_cup" link2="wrist_1_link" reason="Never"/>
     <disable_collisions link1="epick_suction_cup" link2="wrist_2_link" reason="Never"/>
@@ -41,10 +43,24 @@
     <disable_collisions link1="epick_suction_cup" link2="zivid_arm_mount" reason="Never"/>
     <disable_collisions link1="epick_suction_cup" link2="zivid_base_link" reason="Never"/>
-    <!-- Shared tool_block + camera collision rules -->
-    <disable_collisions link1="tool_block" link2="wrist_1_link" reason="Never"/>
-    <disable_collisions link1="tool_block" link2="wrist_2_link" reason="Never"/>
-    <disable_collisions link1="tool_block" link2="wrist_3_link" reason="Never"/>
-    <disable_collisions link1="tool_block" link2="zivid_arm_mount" reason="Adjacent"/>
-    <disable_collisions link1="tool_block" link2="zivid_base_link" reason="Never"/>
+    <!-- Wrist extension + tool exchanger + camera collision rules -->
+    <disable_collisions link1="wrist_extension" link2="wrist_1_link" reason="Never"/>
+    <disable_collisions link1="wrist_extension" link2="wrist_2_link" reason="Never"/>
+    <disable_collisions link1="wrist_extension" link2="wrist_3_link" reason="Never"/>
+    <disable_collisions link1="wrist_extension" link2="flange" reason="Adjacent"/>
+    <disable_collisions link1="wrist_extension" link2="zivid_arm_mount" reason="Adjacent"/>
+    <disable_collisions link1="wrist_extension" link2="zivid_base_link" reason="Never"/>
+    <disable_collisions link1="te_robotside" link2="wrist_extension" reason="Adjacent"/>
+    <disable_collisions link1="te_robotside" link2="wrist_1_link" reason="Never"/>
+    <disable_collisions link1="te_robotside" link2="wrist_2_link" reason="Never"/>
+    <disable_collisions link1="te_robotside" link2="wrist_3_link" reason="Never"/>
+    <disable_collisions link1="te_robotside" link2="zivid_arm_mount" reason="Never"/>
+    <disable_collisions link1="te_robotside" link2="zivid_base_link" reason="Never"/>
+    <disable_collisions link1="te_toolside" link2="te_robotside" reason="Adjacent"/>
+    <disable_collisions link1="te_toolside" link2="wrist_extension" reason="Never"/>
+    <disable_collisions link1="te_toolside" link2="wrist_1_link" reason="Never"/>
+    <disable_collisions link1="te_toolside" link2="wrist_2_link" reason="Never"/>
+    <disable_collisions link1="te_toolside" link2="wrist_3_link" reason="Never"/>
+    <disable_collisions link1="te_toolside" link2="zivid_arm_mount" reason="Never"/>
+    <disable_collisions link1="te_toolside" link2="zivid_base_link" reason="Never"/>
     <disable_collisions link1="wrist_2_link" link2="zivid_arm_mount" reason="Never"/>
     <disable_collisions link1="wrist_2_link" link2="zivid_base_link" reason="Never"/>

File: src/custom-ur-descriptions/cms_moveit_config/srdf/hande.srdf.xacro (robot description, xacro)
@@ -22,5 +22,7 @@
     <disable_collisions link1="robotiq_hande_coupler" link2="robotiq_hande_link" reason="Adjacent"/>
     <disable_collisions link1="robotiq_hande_coupler" link2="robotiq_hande_right_finger" reason="Never"/>
-    <disable_collisions link1="robotiq_hande_coupler" link2="tool_block" reason="Adjacent"/>
+    <disable_collisions link1="robotiq_hande_coupler" link2="te_toolside" reason="Adjacent"/>
+    <disable_collisions link1="robotiq_hande_coupler" link2="te_robotside" reason="Never"/>
+    <disable_collisions link1="robotiq_hande_coupler" link2="wrist_extension" reason="Never"/>
     <disable_collisions link1="robotiq_hande_coupler" link2="wrist_1_link" reason="Never"/>
     <disable_collisions link1="robotiq_hande_coupler" link2="wrist_2_link" reason="Never"/>
@@ -30,5 +32,5 @@
     <disable_collisions link1="robotiq_hande_left_finger" link2="robotiq_hande_link" reason="Adjacent"/>
     <disable_collisions link1="robotiq_hande_left_finger" link2="robotiq_hande_right_finger" reason="Default"/>
-    <disable_collisions link1="robotiq_hande_left_finger" link2="tool_block" reason="Never"/>
+    <disable_collisions link1="robotiq_hande_left_finger" link2="te_toolside" reason="Never"/>
     <disable_collisions link1="robotiq_hande_left_finger" link2="wrist_1_link" reason="Never"/>
     <disable_collisions link1="robotiq_hande_left_finger" link2="wrist_2_link" reason="Never"/>
@@ -37,5 +39,5 @@
     <disable_collisions link1="robotiq_hande_left_finger" link2="zivid_base_link" reason="Never"/>
     <disable_collisions link1="robotiq_hande_link" link2="robotiq_hande_right_finger" reason="Adjacent"/>
-    <disable_collisions link1="robotiq_hande_link" link2="tool_block" reason="Never"/>
+    <disable_collisions link1="robotiq_hande_link" link2="te_toolside" reason="Never"/>
     <disable_collisions link1="robotiq_hande_link" link2="wrist_1_link" reason="Never"/>
     <disable_collisions link1="robotiq_hande_link" link2="wrist_2_link" reason="Never"/>
@@ -43,5 +45,5 @@
     <disable_collisions link1="robotiq_hande_link" link2="zivid_arm_mount" reason="Never"/>
     <disable_collisions link1="robotiq_hande_link" link2="zivid_base_link" reason="Never"/>
-    <disable_collisions link1="robotiq_hande_right_finger" link2="tool_block" reason="Never"/>
+    <disable_collisions link1="robotiq_hande_right_finger" link2="te_toolside" reason="Never"/>
     <disable_collisions link1="robotiq_hande_right_finger" link2="wrist_1_link" reason="Never"/>
     <disable_collisions link1="robotiq_hande_right_finger" link2="wrist_2_link" reason="Never"/>
@@ -49,10 +51,24 @@
     <disable_collisions link1="robotiq_hande_right_finger" link2="zivid_arm_mount" reason="Never"/>
     <disable_collisions link1="robotiq_hande_right_finger" link2="zivid_base_link" reason="Never"/>
-    <!-- Shared tool_block + camera collision rules -->
-    <disable_collisions link1="tool_block" link2="wrist_1_link" reason="Never"/>
-    <disable_collisions link1="tool_block" link2="wrist_2_link" reason="Never"/>
-    <disable_collisions link1="tool_block" link2="wrist_3_link" reason="Never"/>
-    <disable_collisions link1="tool_block" link2="zivid_arm_mount" reason="Adjacent"/>
-    <disable_collisions link1="tool_block" link2="zivid_base_link" reason="Never"/>
+    <!-- Wrist extension + tool exchanger + camera collision rules -->
+    <disable_collisions link1="wrist_extension" link2="wrist_1_link" reason="Never"/>
+    <disable_collisions link1="wrist_extension" link2="wrist_2_link" reason="Never"/>
+    <disable_collisions link1="wrist_extension" link2="wrist_3_link" reason="Never"/>
+    <disable_collisions link1="wrist_extension" link2="flange" reason="Adjacent"/>
+    <disable_collisions link1="wrist_extension" link2="zivid_arm_mount" reason="Adjacent"/>
+    <disable_collisions link1="wrist_extension" link2="zivid_base_link" reason="Never"/>
+    <disable_collisions link1="te_robotside" link2="wrist_extension" reason="Adjacent"/>
+    <disable_collisions link1="te_robotside" link2="wrist_1_link" reason="Never"/>
+    <disable_collisions link1="te_robotside" link2="wrist_2_link" reason="Never"/>
+    <disable_collisions link1="te_robotside" link2="wrist_3_link" reason="Never"/>
+    <disable_collisions link1="te_robotside" link2="zivid_arm_mount" reason="Never"/>
+    <disable_collisions link1="te_robotside" link2="zivid_base_link" reason="Never"/>
+    <disable_collisions link1="te_toolside" link2="te_robotside" reason="Adjacent"/>
+    <disable_collisions link1="te_toolside" link2="wrist_extension" reason="Never"/>
+    <disable_collisions link1="te_toolside" link2="wrist_1_link" reason="Never"/>
+    <disable_collisions link1="te_toolside" link2="wrist_2_link" reason="Never"/>
+    <disable_collisions link1="te_toolside" link2="wrist_3_link" reason="Never"/>
+    <disable_collisions link1="te_toolside" link2="zivid_arm_mount" reason="Never"/>
+    <disable_collisions link1="te_toolside" link2="zivid_base_link" reason="Never"/>
     <disable_collisions link1="wrist_2_link" link2="zivid_arm_mount" reason="Never"/>
     <disable_collisions link1="wrist_2_link" link2="zivid_base_link" reason="Never"/>
@@ -61,4 +77,3 @@
     <disable_collisions link1="zivid_arm_mount" link2="zivid_base_link" reason="Adjacent"/>
     <disable_collisions link1="flange" link2="zivid_arm_mount" reason="Adjacent"/>
-    <disable_collisions link1="flange" link2="tool_block" reason="Never"/>
 </robot>

File: src/custom-ur-descriptions/cms_moveit_config/srdf/none.srdf.xacro (robot description, xacro)
@@ -1,11 +1,19 @@
 <?xml version="1.0" ?>
-<!-- Standalone (no gripper) — tool exchanger robot-side plate only -->
+<!-- Standalone (no gripper) — EX-50-35 wrist extension only -->
 <robot xmlns:xacro="http://www.ros.org/wiki/xacro">
     <!-- No gripper group, no end_effector -->
-    <!-- Tool exchanger + camera collision rules -->
+    <!-- Wrist extension + tool exchanger robot plate + camera collision rules -->
+    <disable_collisions link1="wrist_extension" link2="wrist_1_link" reason="Never"/>
+    <disable_collisions link1="wrist_extension" link2="wrist_2_link" reason="Never"/>
+    <disable_collisions link1="wrist_extension" link2="wrist_3_link" reason="Never"/>
+    <disable_collisions link1="wrist_extension" link2="flange" reason="Adjacent"/>
+    <disable_collisions link1="wrist_extension" link2="zivid_arm_mount" reason="Adjacent"/>
+    <disable_collisions link1="wrist_extension" link2="zivid_base_link" reason="Never"/>
+    <disable_collisions link1="te_robotside" link2="wrist_extension" reason="Adjacent"/>
     <disable_collisions link1="te_robotside" link2="wrist_1_link" reason="Never"/>
     <disable_collisions link1="te_robotside" link2="wrist_2_link" reason="Never"/>
     <disable_collisions link1="te_robotside" link2="wrist_3_link" reason="Never"/>
-    <disable_collisions link1="te_robotside" link2="zivid_arm_mount" reason="Adjacent"/>
+    <disable_collisions link1="te_robotside" link2="flange" reason="Never"/>
+    <disable_collisions link1="te_robotside" link2="zivid_arm_mount" reason="Never"/>
     <disable_collisions link1="te_robotside" link2="zivid_base_link" reason="Never"/>
     <disable_collisions link1="wrist_2_link" link2="zivid_arm_mount" reason="Never"/>

File: src/custom-ur-descriptions/cms_moveit_config/srdf/pipettor.srdf.xacro (robot description, xacro)
@@ -3,15 +3,31 @@
 <robot xmlns:xacro="http://www.ros.org/wiki/xacro">
     <!-- No gripper group (pipettor is static), no end_effector -->
-    <!-- Camera and tool block collision rules -->
-    <disable_collisions link1="tool_block" link2="zivid_arm_mount" reason="Adjacent"/>
-    <disable_collisions link1="tool_block" link2="wrist_3_link" reason="Never"/>
+    <!-- Wrist extension + tool exchanger + camera collision rules -->
+    <disable_collisions link1="wrist_extension" link2="wrist_1_link" reason="Never"/>
+    <disable_collisions link1="wrist_extension" link2="wrist_2_link" reason="Never"/>
+    <disable_collisions link1="wrist_extension" link2="wrist_3_link" reason="Never"/>
+    <disable_collisions link1="wrist_extension" link2="flange" reason="Adjacent"/>
+    <disable_collisions link1="wrist_extension" link2="zivid_arm_mount" reason="Adjacent"/>
+    <disable_collisions link1="wrist_extension" link2="zivid_base_link" reason="Never"/>
+    <disable_collisions link1="te_robotside" link2="wrist_extension" reason="Adjacent"/>
+    <disable_collisions link1="te_robotside" link2="wrist_1_link" reason="Never"/>
+    <disable_collisions link1="te_robotside" link2="wrist_2_link" reason="Never"/>
+    <disable_collisions link1="te_robotside" link2="wrist_3_link" reason="Never"/>
+    <disable_collisions link1="te_robotside" link2="zivid_arm_mount" reason="Never"/>
+    <disable_collisions link1="te_robotside" link2="zivid_base_link" reason="Never"/>
+    <disable_collisions link1="te_toolside" link2="te_robotside" reason="Adjacent"/>
+    <disable_collisions link1="te_toolside" link2="wrist_extension" reason="Never"/>
+    <disable_collisions link1="te_toolside" link2="wrist_3_link" reason="Never"/>
+    <disable_collisions link1="te_toolside" link2="zivid_arm_mount" reason="Never"/>
+    <disable_collisions link1="te_toolside" link2="zivid_base_link" reason="Never"/>
     <disable_collisions link1="zivid_arm_mount" link2="wrist_3_link" reason="Never"/>
     <disable_collisions link1="zivid_arm_mount" link2="flange" reason="Adjacent"/>
     <disable_collisions link1="zivid_base_link" link2="zivid_arm_mount" reason="Adjacent"/>
     <disable_collisions link1="zivid_base_link" link2="wrist_3_link" reason="Never"/>
-    <disable_collisions link1="zivid_base_link" link2="tool_block" reason="Never"/>
     <!-- Pipettor collision rules -->
-    <disable_collisions link1="pipette_base_link" link2="tool_block" reason="Adjacent"/>
-    <disable_collisions link1="pipette_body_link" link2="tool_block" reason="Never"/>
+    <disable_collisions link1="pipette_base_link" link2="te_toolside" reason="Adjacent"/>
+    <disable_collisions link1="pipette_base_link" link2="te_robotside" reason="Never"/>
+    <disable_collisions link1="pipette_base_link" link2="wrist_extension" reason="Never"/>
+    <disable_collisions link1="pipette_body_link" link2="te_toolside" reason="Never"/>
     <disable_collisions link1="pipette_body_link" link2="pipette_base_link" reason="Adjacent"/>
     <disable_collisions link1="pipette_base_link" link2="wrist_3_link" reason="Never"/>

File: src/custom-ur-descriptions/cms_robot_description/urdf/te_robotside.xacro (robot description, xacro)
@@ -6,5 +6,5 @@
         <origin xyz="0 0 0" rpy="0 0 0"/>
         <geometry>
-          <mesh filename="package://cms_robot_description/meshes/tool_exchanger/Tool_block_robotside.stl"
+          <mesh filename="package://cms_robot_description/meshes/tool_exchanger/WM1_robot_plate.stl"
                 scale="${scale} ${scale} ${scale}"/>
         </geometry>
@@ -16,5 +16,5 @@
         <origin xyz="0 0 0" rpy="0 0 0"/>
         <geometry>
-          <mesh filename="package://cms_robot_description/meshes/tool_exchanger/Tool_block_robotside.stl"
+          <mesh filename="package://cms_robot_description/meshes/tool_exchanger/WM1_robot_plate.stl"
                 scale="${scale} ${scale} ${scale}"/>
         </geometry>

File: src/custom-ur-descriptions/cms_robot_description/urdf/ur_standalone.urdf (robot description, URDF)
Before this commit: robot ur5e, 17 links, 16 joints
Links:
- added link wrist_extension, mass 0.3; collision mesh filename=package://cms_robot_description/meshes/tool_exchanger/EX-50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 scale=0.001 0.001 0.001; visual mesh filename=package://cms_robot_description/meshes/tool_exchanger/EX-50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 scale=0.001 0.001 0.001
- link te_robotside: geometry collision mesh filename=package://cms_robot_description/meshes/tool_exchanger/WM1_r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 scale=0.001 0.001 0.001; visual mesh filename=package://cms_robot_description/meshes/tool_exchanger/WM1_r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 scale=0.001 0.001 0.001
Joints:
- added joint wrist_extension_joint: type fixed, parent tool0, child wrist_extension, origin xyz=0 0 0.016 rpy=1.5708 0 3.14159
- joint te_robotside_joint: origin xyz=0 0 0.055 rpy=-1.5708 0 3.14159 -> xyz=0 0.047 0 rpy=3.14159 0 0; parent zivid_arm_mount -> wrist_extension
