Commit message: replace makeshift tool block with EX-50-35 wrist extension + Wingman plates
Replaces the old 2-spacer makeshift tool block with a proper setup:
- EX-50-35 wrist extension (35mm, bolts to flange)
- Wingman WM1 robot-side plate (te_robotside)
- Wingman WM1 tool-side plate (te_toolside, per-gripper)

New kinematic chain: tool0 → wrist_extension → te_robotside → te_toolside → gripper
"none" config ends at te_robotside (no tool plate, no gripper).

Updated all 5 CMS gripper configs (none, epick, hande, 2fg7, pipettor),
their SRDFs, and regenerated pre-built URDF files.

File: src/custom-ur-descriptions/cms_robot_description/urdf/ur_standalone.xacro (robot description, xacro)
@@ -8,4 +8,5 @@
    <xacro:include filename="$(find ur_robot_driver)/urdf/ur.ros2_control.xacro"/>
    <xacro:include filename="$(find cms_robot_description)/urdf/zivid_camera_mount.xacro"/>
+   <xacro:include filename="$(find cms_robot_description)/urdf/wrist_extension.xacro"/>
    <xacro:include filename="$(find cms_robot_description)/urdf/te_robotside.xacro"/>
    <!-- possible 'ur_type' values: ur3, ur5e, ur5, ur5e, ur10, ur10e, ur16e, ur20 -->
@@ -94,4 +95,15 @@
      robot_receive_timeout="$(arg robot_receive_timeout)"
    />
+  <!-- Wrist extension (EX-50-35): bolts to flange, extends 35mm along tool-Z.
+       Replaces makeshift tool block spacer (was 55mm with 2 stacked spacers). -->
+  <xacro:wrist_extension
+    parent_link="$(arg tf_prefix)tool0"
+    xyz="0 0 0.016"
+    rpy="1.5708 0 3.14159"/>
+  <!-- Tool exchanger robot-side plate (Wingman WM1) at the tip of the extension -->
+  <xacro:te_robotside
+    parent_link="wrist_extension"
+    xyz="0 0.047 0"
+    rpy="3.14159 0 0"/>
   <!-- Modular Zivid: Arm Mount + Camera (with calibrated camera position) -->
   <xacro:zivid_camera_mount
@@ -100,5 +112,3 @@
     rpy="0 0 0"
     zivid_model="ZIVID_2_PLUS_MR60"/>
-  <!-- Tool exchanger robotside attached to arm mount (not camera) -->
-  <xacro:te_robotside parent_link="zivid_arm_mount" xyz="0 0 0.055" rpy="-1.5708 0 3.14159"/>
 </robot>

File: src/custom-ur-descriptions/cms_robot_description/urdf/ur_with_zivid_2fg7.xacro (robot description, xacro)
@@ -1,5 +1,5 @@
 <?xml version="1.0"?>
 <robot xmlns:xacro="http://wiki.ros.org/xacro" name="$(arg name)">
-<!--Chain: map -> UR -> flange -> zivid_camera_mount -> zivid_camera -> 2FG7 gripper -->
+<!--Chain: map -> UR -> flange -> wrist_extension -> te_robotside -> te_toolside -> 2FG7 gripper -->
   <!-- robot name parameter -->
   <xacro:arg name="name" default="ur5e"/>
@@ -8,5 +8,7 @@
   <xacro:include filename="$(find ur_robot_driver)/urdf/ur.ros2_control.xacro"/>
   <xacro:include filename="$(find cms_robot_description)/urdf/zivid_camera_mount.xacro"/>
-  <xacro:include filename="$(find cms_robot_description)/urdf/tool_block.xacro"/>
+  <xacro:include filename="$(find cms_robot_description)/urdf/wrist_extension.xacro"/>
+  <xacro:include filename="$(find cms_robot_description)/urdf/te_robotside.xacro"/>
+  <xacro:include filename="$(find cms_robot_description)/urdf/te_toolside.xacro"/>
   <xacro:include filename="$(find onrobot_2fg7_description)/urdf/onrobot_2fg7.xacro"/>
   <!-- possible 'ur_type' values: ur3, ur5e, ur5, ur10, ur10e, ur16e, ur20 -->
@@ -103,10 +105,23 @@
     rpy="0 0 0"
     zivid_model="ZIVID_2_PLUS_MR60"/>
-  <!-- Tool block attached to the Zivid arm mount (not the camera) -->
-  <xacro:tool_block parent_link="zivid_arm_mount" xyz="0 0 0.049" rpy="-1.5708 0 3.14159"/>
-  <!-- OnRobot 2FG7 gripper — same mounting offset as ePick/Hand-E (same bolt pattern) -->
+  <!-- Wrist extension (EX-50-35): bolts to flange, extends 35mm along tool-Z -->
+  <xacro:wrist_extension
+    parent_link="$(arg tf_prefix)tool0"
+    xyz="0 0 0.016"
+    rpy="1.5708 0 3.14159"/>
+  <!-- Tool exchanger robot-side plate (Wingman WM1) at the tip of the extension -->
+  <xacro:te_robotside
+    parent_link="wrist_extension"
+    xyz="0 0.047 0"
+    rpy="3.14159 0 0"/>
+  <!-- Tool exchanger tool-side plate (Wingman WM1) — comes with each gripper -->
+  <xacro:te_toolside
+    parent_link="te_robotside"
+    xyz="0 -0.011 0"
+    rpy="0 0 0"/>
+  <!-- OnRobot 2FG7 gripper -->
   <xacro:onrobot_2fg7
-    parent="tool_block"
-    xyz="0 -0.03235 0"
+    parent="te_toolside"
+    xyz="0 -0.005 0"
     rpy="-1.5708 0 3.1416"/>
 </robot>

File: src/custom-ur-descriptions/cms_robot_description/urdf/ur_with_zivid_epick.urdf (robot description, URDF)
Before this commit: robot ur5e, 24 links, 23 joints
Links:
- removed link tool_block
- added link te_robotside, mass 0.5; collision mesh filename=package://cms_robot_description/meshes/tool_exchanger/WM1_r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 scale=0.001 0.001 0.001; visual mesh filename=package://cms_robot_description/meshes/tool_exchanger/WM1_r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 scale=0.001 0.001 0.001
- added link te_toolside, mass 0.4; collision mesh filename=package://cms_robot_description/meshes/tool_exchanger/WM1_t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 scale=0.001 0.001 0.001; visual mesh filename=package://cms_robot_description/meshes/tool_exchanger/WM1_t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 scale=0.001 0.001 0.001
- added link wrist_extension, mass 0.3; collision mesh filename=package://cms_robot_description/meshes/tool_exchanger/EX-50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 scale=0.001 0.001 0.001; visual mesh filename=package://cms_robot_description/meshes/tool_exchanger/EX-50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 scale=0.001 0.001 0.001
- link epick_extension: geometry collision cylinder length=0.013 radius=0.004; visual cylinder length=0.013 radius=0.004
- link epick_suction_cup: geometry collision cylinder length=0.003 radius=0.0015; visual cylinder length=0.003 radius=0.0015
Joints:
- removed joint tool_block_joint
- removed joint tool_block_to_epick_base_link
- added joint te_robotside_joint: type fixed, parent wrist_extension, child te_robotside, origin xyz=0 0.047 0 rpy=3.14159 0 0
- added joint te_toolside_joint: type fixed, parent te_robotside, child te_toolside, origin xyz=0 -0.011 0 rpy=0 0 0
- added joint te_toolside_to_epick_base_link: type fixed, parent te_toolside, child epick_base_link, origin xyz=0 -0.005 0 rpy=-1.5708 0 3.1416
- added joint wrist_extension_joint: type fixed, parent tool0, child wrist_extension, origin xyz=0 0 0.016 rpy=1.5708 0 3.14159
- joint epick_body_to_epick_extension: origin xyz=0 0 0.06015 rpy=0 0 0 -> xyz=0 0 0.05765 rpy=0 0 0
- joint epick_extension_to_epick_suction_cup: origin xyz=0 0 0.012 rpy=0 0 0 -> xyz=0 0 0.008 rpy=0 0 0
- joint epick_suction_cup_to_epick_tip: origin xyz=0 0 0.003 rpy=0 0 0 -> xyz=0 0 0.0015 rpy=0 0 0

File: src/custom-ur-descriptions/cms_robot_description/urdf/ur_with_zivid_epick.xacro (robot description, xacro)
@@ -1,5 +1,5 @@
 <?xml version="1.0"?>
 <robot xmlns:xacro="http://wiki.ros.org/xacro" name="$(arg name)">
-<!--   Chain: map -> UR -> flange -> zivid_camera_mount -> zivid_camera -> EPick gripper -->
+<!--Chain: map -> UR -> flange -> wrist_extension -> te_robotside -> te_toolside -> EPick gripper -->
   <!-- robot name parameter -->
   <xacro:arg name="name" default="ur5e"/>
@@ -8,5 +8,7 @@
   <xacro:include filename="$(find ur_robot_driver)/urdf/ur.ros2_control.xacro"/>
   <xacro:include filename="$(find cms_robot_description)/urdf/zivid_camera_mount.xacro"/>
-  <xacro:include filename="$(find cms_robot_description)/urdf/tool_block.xacro"/>
+  <xacro:include filename="$(find cms_robot_description)/urdf/wrist_extension.xacro"/>
+  <xacro:include filename="$(find cms_robot_description)/urdf/te_robotside.xacro"/>
+  <xacro:include filename="$(find cms_robot_description)/urdf/te_toolside.xacro"/>
   <xacro:include filename="$(find epick_config)/urdf/epick_overlay.xacro"/>
   <!-- possible 'ur_type' values: ur3, ur5e, ur5, ur10, ur10e, ur16e, ur20 -->
@@ -104,6 +106,19 @@
     rpy="0 0 0"
     zivid_model="ZIVID_2_PLUS_MR60"/>
-  <!-- Tool block attached to the Zivid arm mount (not the camera) -->
-  <xacro:tool_block parent_link="zivid_arm_mount" xyz="0 0 0.049" rpy="-1.5708 0 3.14159"/>
+  <!-- Wrist extension (EX-50-35): bolts to flange, extends 35mm along tool-Z -->
+  <xacro:wrist_extension
+    parent_link="$(arg tf_prefix)tool0"
+    xyz="0 0 0.016"
+    rpy="1.5708 0 3.14159"/>
+  <!-- Tool exchanger robot-side plate (Wingman WM1) at the tip of the extension -->
+  <xacro:te_robotside
+    parent_link="wrist_extension"
+    xyz="0 0.047 0"
+    rpy="3.14159 0 0"/>
+  <!-- Tool exchanger tool-side plate (Wingman WM1) — comes with each gripper -->
+  <xacro:te_toolside
+    parent_link="te_robotside"
+    xyz="0 -0.011 0"
+    rpy="0 0 0"/>
   <!-- Suction cup profile: dimensions loaded from suction_cups.yaml (single source of truth).
        The cup_profile default MUST match the physically attached cup — the UR driver's
@@ -117,6 +132,6 @@
   <xacro:property name="cup" value="${cups_config['cups'][cup_profile_name]}"/>
   <!-- Epick Gripper -->
-  <xacro:epick_overlay use_mock_hardware="$(arg use_mock_hardware)" parent="tool_block"
-                  origin_xyz="0 -0.03235 0"
+  <xacro:epick_overlay use_mock_hardware="$(arg use_mock_hardware)" parent="te_toolside"
+                  origin_xyz="0 -0.005 0"
                   origin_rpy="-1.5708 0 3.1416"
                   extension_length="${cup['extension_length']}"

File: src/custom-ur-descriptions/cms_robot_description/urdf/ur_with_zivid_hande.urdf (robot description, URDF)
Before this commit: robot ur5e, 22 links, 21 joints
Links:
- removed link tool_block
- added link te_robotside, mass 0.5; collision mesh filename=package://cms_robot_description/meshes/tool_exchanger/WM1_r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 scale=0.001 0.001 0.001; visual mesh filename=package://cms_robot_description/meshes/tool_exchanger/WM1_r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 scale=0.001 0.001 0.001
- added link te_toolside, mass 0.4; collision mesh filename=package://cms_robot_description/meshes/tool_exchanger/WM1_t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 scale=0.001 0.001 0.001; visual mesh filename=package://cms_robot_description/meshes/tool_exchanger/WM1_t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 scale=0.001 0.001 0.001
- added link wrist_extension, mass 0.3; collision mesh filename=package://cms_robot_description/meshes/tool_exchanger/EX-50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 scale=0.001 0.001 0.001; visual mesh filename=package://cms_robot_description/meshes/tool_exchanger/EX-50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 scale=0.001 0.001 0.001
Joints:
- removed joint tool_block_joint
- added joint te_robotside_joint: type fixed, parent wrist_extension, child te_robotside, origin xyz=0 0.047 0 rpy=3.14159 0 0
- added joint te_toolside_joint: type fixed, parent te_robotside, child te_toolside, origin xyz=0 -0.011 0 rpy=0 0 0
- added joint wrist_extension_joint: type fixed, parent tool0, child wrist_extension, origin xyz=0 0 0.016 rpy=1.5708 0 3.14159
- joint robotiq_hande_coupler_joint: origin xyz=0 -0.02 0 rpy=-1.5708 0 3.1416 -> xyz=0 -0.005 0 rpy=-1.5708 0 3.1416; parent tool_block -> te_toolside

File: src/custom-ur-descriptions/cms_robot_description/urdf/ur_with_zivid_hande.xacro (robot description, xacro)
@@ -1,5 +1,5 @@
 <?xml version="1.0"?>
 <robot xmlns:xacro="http://wiki.ros.org/xacro" name="$(arg name)">
-<!--Chain: map -> UR -> flange -> zivid_camera_mount -> zivid_camera -> HandE gripper -->
+<!--Chain: map -> UR -> flange -> wrist_extension -> te_robotside -> te_toolside -> HandE gripper -->
   <!-- robot name parameter -->
   <xacro:arg name="name" default="ur5e"/>
@@ -8,5 +8,7 @@
   <xacro:include filename="$(find ur_robot_driver)/urdf/ur.ros2_control.xacro"/>
   <xacro:include filename="$(find cms_robot_description)/urdf/zivid_camera_mount.xacro"/>
-  <xacro:include filename="$(find cms_robot_description)/urdf/tool_block.xacro"/>
+  <xacro:include filename="$(find cms_robot_description)/urdf/wrist_extension.xacro"/>
+  <xacro:include filename="$(find cms_robot_description)/urdf/te_robotside.xacro"/>
+  <xacro:include filename="$(find cms_robot_description)/urdf/te_toolside.xacro"/>
   <xacro:include filename="$(find robotiq_hande_description)/urdf/robotiq_hande_gripper.xacro"/>
   <!-- possible 'ur_type' values: ur3, ur5e, ur5, ur10, ur10e, ur16e, ur20 -->
@@ -103,6 +105,19 @@
     rpy="0 0 0"
     zivid_model="ZIVID_2_PLUS_MR60"/>
-  <!-- Tool block attached to the Zivid arm mount (not the camera) -->
-  <xacro:tool_block parent_link="zivid_arm_mount" xyz="0 0 0.055" rpy="-1.5708 0 3.14159"/>
+  <!-- Wrist extension (EX-50-35): bolts to flange, extends 35mm along tool-Z -->
+  <xacro:wrist_extension
+    parent_link="$(arg tf_prefix)tool0"
+    xyz="0 0 0.016"
+    rpy="1.5708 0 3.14159"/>
+  <!-- Tool exchanger robot-side plate (Wingman WM1) at the tip of the extension -->
+  <xacro:te_robotside
+    parent_link="wrist_extension"
+    xyz="0 0.047 0"
+    rpy="3.14159 0 0"/>
+  <!-- Tool exchanger tool-side plate (Wingman WM1) — comes with each gripper -->
+  <xacro:te_toolside
+    parent_link="te_robotside"
+    xyz="0 -0.011 0"
+    rpy="0 0 0"/>
   <!-- gripper pos wrt camera    -->
   <xacro:arg name="grip_pos_min" default="0"/>
@@ -120,5 +135,5 @@
     name="robotiq_hande_gripper"
     prefix="$(arg tf_prefix)"
-    parent="tool_block"
+    parent="te_toolside"
     grip_pos_min="$(arg grip_pos_min)"
     grip_pos_max="$(arg grip_pos_max)"
@@ -130,5 +145,5 @@
     slave_id="$(arg slave_id)"
     use_fake_hardware="$(arg use_mock_hardware)"
-    xyz="0 -0.02 0"
+    xyz="0 -0.005 0"
     rpy="-1.5708 0 3.1416"
     create_socat_tty="$(arg create_socat_tty)"

File: src/custom-ur-descriptions/cms_robot_description/urdf/ur_with_zivid_pipettor.urdf (robot description, URDF)
Before this commit: robot ur5e, 21 links, 20 joints
Links:
- removed link tool_block
- added link te_robotside, mass 0.5; collision mesh filename=package://cms_robot_description/meshes/tool_exchanger/WM1_r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 scale=0.001 0.001 0.001; visual mesh filename=package://cms_robot_description/meshes/tool_exchanger/WM1_r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 scale=0.001 0.001 0.001
- added link te_toolside, mass 0.4; collision mesh filename=package://cms_robot_description/meshes/tool_exchanger/WM1_t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 scale=0.001 0.001 0.001; visual mesh filename=package://cms_robot_description/meshes/tool_exchanger/WM1_t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 scale=0.001 0.001 0.001
- added link wrist_extension, mass 0.3; collision mesh filename=package://cms_robot_description/meshes/tool_exchanger/EX-50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 scale=0.001 0.001 0.001; visual mesh filename=package://cms_robot_description/meshes/tool_exchanger/EX-50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 scale=0.001 0.001 0.001
Joints:
- removed joint tool_block_joint
- added joint te_robotside_joint: type fixed, parent wrist_extension, child te_robotside, origin xyz=0 0.047 0 rpy=3.14159 0 0
- added joint te_toolside_joint: type fixed, parent te_robotside, child te_toolside, origin xyz=0 -0.011 0 rpy=0 0 0
- added joint wrist_extension_joint: type fixed, parent tool0, child wrist_extension, origin xyz=0 0 0.016 rpy=1.5708 0 3.14159
- joint pipette_attachment_joint: origin xyz=-0.005 -0.015 0 rpy=-1.5708 0 3.1416 -> xyz=-0.005 -0.005 0 rpy=-1.5708 0 3.1416; parent tool_block -> te_toolside

File: src/custom-ur-descriptions/cms_robot_description/urdf/ur_with_zivid_pipettor.xacro (robot description, xacro)
@@ -1,5 +1,5 @@
 <?xml version="1.0"?>
 <robot xmlns:xacro="http://wiki.ros.org/xacro" name="$(arg name)">
-<!--Chain: map -> UR -> flange -> zivid_camera_mount -> zivid_camera -> tool_block -> pipettor -->
+<!--Chain: map -> UR -> flange -> wrist_extension -> te_robotside -> te_toolside -> pipettor -->
   <!-- robot name parameter -->
   <xacro:arg name="name" default="ur5e"/>
@@ -8,5 +8,7 @@
   <xacro:include filename="$(find ur_robot_driver)/urdf/ur.ros2_control.xacro"/>
   <xacro:include filename="$(find cms_robot_description)/urdf/zivid_camera_mount.xacro"/>
-  <xacro:include filename="$(find cms_robot_description)/urdf/tool_block.xacro"/>
+  <xacro:include filename="$(find cms_robot_description)/urdf/wrist_extension.xacro"/>
+  <xacro:include filename="$(find cms_robot_description)/urdf/te_robotside.xacro"/>
+  <xacro:include filename="$(find cms_robot_description)/urdf/te_toolside.xacro"/>
   <xacro:include filename="$(find pipette_description)/urdf/pipette_macro.urdf.xacro"/>
   <!-- possible 'ur_type' values: ur3, ur5e, ur5, ur10, ur10e, ur16e, ur20 -->
@@ -103,13 +105,26 @@
     rpy="0 0 0"
     zivid_model="ZIVID_2_PLUS_MR60"/>
-  <!-- Tool block attached to the Zivid arm mount (not the camera) -->
-  <xacro:tool_block parent_link="zivid_arm_mount" xyz="0 0 0.049" rpy="-1.5708 0 3.14159"/>
-  <!-- Pipettor attached to tool block -->
+  <!-- Wrist extension (EX-50-35): bolts to flange, extends 35mm along tool-Z -->
+  <xacro:wrist_extension
+    parent_link="$(arg tf_prefix)tool0"
+    xyz="0 0 0.016"
+    rpy="1.5708 0 3.14159"/>
+  <!-- Tool exchanger robot-side plate (Wingman WM1) at the tip of the extension -->
+  <xacro:te_robotside
+    parent_link="wrist_extension"
+    xyz="0 0.047 0"
+    rpy="3.14159 0 0"/>
+  <!-- Tool exchanger tool-side plate (Wingman WM1) — comes with each gripper -->
+  <xacro:te_toolside
+    parent_link="te_robotside"
+    xyz="0 -0.011 0"
+    rpy="0 0 0"/>
+  <!-- Pipettor attached to tool-side plate -->
   <xacro:pipette
     name="pipette"
     prefix="$(arg tf_prefix)"
-    parent="tool_block"
+    parent="te_toolside"
     pipette_mass="0.200"
-    xyz="-0.005 -0.015 0"
+    xyz="-0.005 -0.005 0"
     rpy="-1.5708 0 3.1416"
   />

File: src/custom-ur-descriptions/cms_robot_description/urdf/zivid_camera_mount.xacro (robot description, xacro)
@@ -44,5 +44,5 @@
     </joint>
     <!-- ============================================================ -->
-    <!-- ARM MOUNT (for attaching grippers via tool_block)            -->
+    <!-- ARM MOUNT (for attaching grippers via wrist_extension)       -->
     <!-- ============================================================ -->
     <link name="zivid_arm_mount">
