Commit message: fix epick coupling collisions + tip yaw flip; bandaid z_offset
Three fixes from hardware verification of the epick vision pickup:

- SRDF: add te_coupling to epick_gripper group + disable_collisions for it
  (was missing, blocked all planning with GOAL_IN_COLLISION on te_toolside).
- xacro: epick mounted on coupling with origin_rpy yaw=pi. The cylindrical
  coupling/spacer hid a 180deg yaw flip of epick_tip vs the validated frame;
  IK compensated by swinging wrist_3, driving the camera bracket into wrist_1.
  Restoring the yaw fixes the self-collision (verified: clean plan+execute).
- config: bandaid z_offset=-0.009 for epick. The W-010-B coupling axial length
  was over-counted (~9mm), so epick_tip sits ~9mm short of the real cup.
  Verified on tags 0 and 1; ROI/marker picks both inherit it via
  compute_approach_pose. Proper fix = correct te_coupling length in the xacro.

File: src/custom-ur-descriptions/cms_moveit_config/srdf/epick.srdf.xacro (robot description, xacro)
@@ -4,4 +4,5 @@
     <group name="epick_gripper">
         <link name="te_toolside"/>
+        <link name="te_coupling"/>
         <link name="epick_base_link"/>
         <link name="epick_body"/>
@@ -19,4 +20,17 @@
     </group_state>
     <end_effector name="epick_gripper" parent_link="flange" group="epick_gripper"/>
+    <!-- Tool-changer coupling (W-010-B) collision rules -->
+    <disable_collisions link1="te_coupling" link2="te_toolside" reason="Adjacent"/>
+    <disable_collisions link1="te_coupling" link2="epick_base_link" reason="Adjacent"/>
+    <disable_collisions link1="te_coupling" link2="epick_body" reason="Adjacent"/>
+    <disable_collisions link1="te_coupling" link2="te_robotside" reason="Never"/>
+    <disable_collisions link1="te_coupling" link2="wrist_extension" reason="Never"/>
+    <disable_collisions link1="te_coupling" link2="wrist_1_link" reason="Never"/>
+    <disable_collisions link1="te_coupling" link2="wrist_2_link" reason="Never"/>
+    <disable_collisions link1="te_coupling" link2="wrist_3_link" reason="Never"/>
+    <disable_collisions link1="te_coupling" link2="zivid_arm_mount" reason="Never"/>
+    <disable_collisions link1="te_coupling" link2="zivid_base_link" reason="Never"/>
+    <disable_collisions link1="te_coupling" link2="epick_extension" reason="Never"/>
+    <disable_collisions link1="te_coupling" link2="epick_suction_cup" reason="Never"/>
     <!-- ePick collision rules -->
     <disable_collisions link1="epick_body" link2="epick_extension" reason="Adjacent"/>

File: src/custom-ur-descriptions/cms_robot_description/urdf/ur_with_zivid_epick.urdf (robot description, URDF)
Before this commit: robot ur5e, 27 links, 26 joints
Joints:
- joint te_coupling_to_epick_base_link: origin xyz=0 0 0.0099 rpy=0 0 0 -> xyz=0 0 0.0099 rpy=0 0 3.14159

File: src/custom-ur-descriptions/cms_robot_description/urdf/ur_with_zivid_epick.xacro (robot description, xacro)
@@ -139,8 +139,11 @@
     xyz="0 -0.012 0"
     rpy="1.5708 0 0"/>
-  <!-- Epick Gripper — now mounted on the coupling far face -->
+  <!-- Epick Gripper — mounted on the coupling far face.
+       origin_rpy yaw=pi: the cylindrical coupling/spacer hid a 180 deg yaw flip
+       of epick_tip vs the validated pre-coupling frame; this restores it so the
+       IK target matches and wrist_3 doesn't swing the camera into wrist_1. -->
   <xacro:epick_overlay use_mock_hardware="$(arg use_mock_hardware)" parent="te_coupling"
                   origin_xyz="0 0 0.0099"
-                  origin_rpy="0 0 0"
+                  origin_rpy="0 0 3.14159"
                   extension_length="${cup['extension_length']}"
                   extension_radius="${cup['extension_radius']}"
