Commit message: refactor: rename ur5e_moveit_config → cms_moveit_config, ur5e_robot_description → cms_robot_description
These packages are CMS beamline-specific (gripper configs, URDF meshes,
controller params) but were named generically after the robot model. Since
multiple beamlines will each have their own UR5e, the generic name was
ambiguous. Beamline-prefixed names make ownership clear and let new beamlines
create their own packages (e.g. chx_moveit_config) without confusion.

Updated: package.xml, CMakeLists.txt, launch files, xacro includes, SRDF,
beamline YAML, visualization panel, docs, and all generated URDFs.

File: src/custom-ur-descriptions/cms_robot_description/urdf/ur_standalone.urdf (robot description, URDF)
Before this commit: robot ur5e, 24 links, 23 joints
Links:
- removed link epick_base_link
- removed link epick_body
- removed link epick_extension
- removed link epick_suction_cup
- removed link epick_tcp
- removed link epick_tip
- removed link epick_vacuum_state
- removed link tool_block
- added link te_robotside, mass 0.5; collision mesh filename=package://cms_robot_description/meshes/tool_exchanger/Tool_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 scale=0.001 0.001 0.001; visual mesh filename=package://cms_robot_description/meshes/tool_exchanger/Tool_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 scale=0.001 0.001 0.001
- link zivid_arm_mount: geometry collision mesh filename=package://cms_robot_description/meshes/zivid/zivid_onarm_mo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 scale=0.001 0.001 0.001; visual mesh filename=package://cms_robot_description/meshes/zivid/zivid_onarm_mo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 scale=0.001 0.001 0.001
Joints:
- removed joint epick_base_link_to_epick_body
- removed joint epick_body_to_epick_extension
- removed joint epick_extension_to_epick_suction_cup
- removed joint epick_suction_cup_to_epick_tip
- removed joint epick_tip_to_epick_tcp
- removed joint gripper
- removed joint tool_block_joint
- removed joint tool_block_to_epick_base_link
- added joint te_robotside_joint: type fixed, parent zivid_arm_mount, child te_robotside, origin xyz=0 0 0.055 rpy=-1.5708 0 3.14159

File: src/custom-ur-descriptions/cms_robot_description/urdf/ur_standalone.xacro (robot description, xacro)
@@ -7,6 +7,6 @@
    <xacro:include filename="$(find ur_description)/urdf/ur_macro.xacro"/>
    <xacro:include filename="$(find ur_robot_driver)/urdf/ur.ros2_control.xacro"/>
-   <xacro:include filename="$(find ur5e_robot_description)/urdf/zivid_camera_mount.xacro"/>
-   <xacro:include filename="$(find ur5e_robot_description)/urdf/te_robotside.xacro"/>
+   <xacro:include filename="$(find cms_robot_description)/urdf/zivid_camera_mount.xacro"/>
+   <xacro:include filename="$(find cms_robot_description)/urdf/te_robotside.xacro"/>
    <!-- possible 'ur_type' values: ur3, ur5e, ur5, ur5e, ur10, ur10e, ur16e, ur20 -->
    <xacro:arg name="ur_type" default="ur5e"/>
@@ -46,5 +46,5 @@
    <xacro:arg name="mock_sensor_commands" default="false" />
    <!-- initial position for simulations -->
-   <xacro:arg name="initial_positions_file" default="$(find ur5e_moveit_config)/config/none/initial_positions.yaml"/>
+   <xacro:arg name="initial_positions_file" default="$(find cms_moveit_config)/config/none/initial_positions.yaml"/>
    <xacro:property name="initial_positions_file" default="$(arg initial_positions_file)"/>
    <!-- create link fixed to the "map" -->

File: src/custom-ur-descriptions/cms_robot_description/urdf/ur_standalone_isaac.urdf (robot description, URDF)
Before this commit: robot ur5e, 21 links, 20 joints
Links:
- removed link led_strip_link
- removed link pipette_base_link
- removed link pipette_body_link
- removed link pipette_tip_link
- removed link tool_block
- added link te_robotside, mass 0.5; collision mesh filename=/home/aditya/work/erobs/src/custom-ur-descriptions/cms_robo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 scale=0.001 0.001 0.001; visual mesh filename=/home/aditya/work/erobs/src/custom-ur-descriptions/cms_robo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 scale=0.001 0.001 0.001
- link base_link_inertia: geometry collision mesh filename=/opt/ros/jazzy/share/ur_description/meshes/ur5e/collision/b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; visual mesh filename=/opt/ros/jazzy/share/ur_description/meshes/ur5e/visual/base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
- link forearm_link: geometry collision mesh filename=/opt/ros/jazzy/share/ur_description/meshes/ur5e/collision/f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; visual mesh filename=/opt/ros/jazzy/share/ur_description/meshes/ur5e/visual/fore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
- link shoulder_link: geometry collision mesh filename=/opt/ros/jazzy/share/ur_description/meshes/ur5e/collision/s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; visual mesh filename=/opt/ros/jazzy/share/ur_description/meshes/ur5e/visual/shou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
- link upper_arm_link: geometry collision mesh filename=/opt/ros/jazzy/share/ur_description/meshes/ur5e/collision/u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; visual mesh filename=/opt/ros/jazzy/share/ur_description/meshes/ur5e/visual/uppe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
- link wrist_1_link: geometry collision mesh filename=/opt/ros/jazzy/share/ur_description/meshes/ur5e/collision/w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; visual mesh filename=/opt/ros/jazzy/share/ur_description/meshes/ur5e/visual/wris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
- link wrist_2_link: geometry collision mesh filename=/opt/ros/jazzy/share/ur_description/meshes/ur5e/collision/w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; visual mesh filename=/opt/ros/jazzy/share/ur_description/meshes/ur5e/visual/wris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
- link wrist_3_link: geometry collision mesh filename=/opt/ros/jazzy/share/ur_description/meshes/ur5e/collision/w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; visual mesh filename=/opt/ros/jazzy/share/ur_description/meshes/ur5e/visual/wris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
- link zivid_arm_mount: geometry collision mesh filename=/home/aditya/work/erobs/src/custom-ur-descriptions/cms_robo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 scale=0.001 0.001 0.001; visual mesh filename=/home/aditya/work/erobs/src/custom-ur-descriptions/cms_robo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 scale=0.001 0.001 0.001
- link zivid_base_link: geometry collision mesh filename=/home/aditya/work/erobs/src/vision/zivid-ros/zivid_descript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; visual mesh filename=/home/aditya/work/erobs/src/vision/zivid-ros/zivid_descript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
Joints:
- removed joint led_strip_joint
- removed joint pipette_attachment_joint
- removed joint pipette_orientation_joint
- removed joint pipette_tip_joint
- removed joint tool_block_joint
- added joint te_robotside_joint: type fixed, parent zivid_arm_mount, child te_robotside, origin xyz=0 0 0.055 rpy=-1.5708 0 3.14159

File: src/custom-ur-descriptions/cms_robot_description/urdf/ur_with_zivid_2fg7.xacro (robot description, xacro)
@@ -1,5 +1,5 @@
 <?xml version="1.0"?>
 <robot xmlns:xacro="http://wiki.ros.org/xacro" name="$(arg name)">
-<!--Chain: map -> UR -> flange -> zivid_camera_mount -> zivid_camera -> tool_block -> pipettor -->
+<!--Chain: map -> UR -> flange -> zivid_camera_mount -> zivid_camera -> 2FG7 gripper -->
   <!-- robot name parameter -->
   <xacro:arg name="name" default="ur5e"/>
@@ -7,7 +7,7 @@
   <xacro:include filename="$(find ur_description)/urdf/ur_macro.xacro"/>
   <xacro:include filename="$(find ur_robot_driver)/urdf/ur.ros2_control.xacro"/>
-  <xacro:include filename="$(find ur5e_robot_description)/urdf/zivid_camera_mount.xacro"/>
-  <xacro:include filename="$(find ur5e_robot_description)/urdf/tool_block.xacro"/>
-  <xacro:include filename="$(find pipette_description)/urdf/pipette_macro.urdf.xacro"/>
+  <xacro:include filename="$(find cms_robot_description)/urdf/zivid_camera_mount.xacro"/>
+  <xacro:include filename="$(find cms_robot_description)/urdf/tool_block.xacro"/>
+  <xacro:include filename="$(find onrobot_2fg7_description)/urdf/onrobot_2fg7.xacro"/>
   <!-- possible 'ur_type' values: ur3, ur5e, ur5, ur10, ur10e, ur16e, ur20 -->
   <xacro:arg name="ur_type" default="ur5e"/>
@@ -34,9 +34,9 @@
   <!-- Keep-alive: number of 20ms cycles without response before disconnect (10 = 200ms timeout) -->
   <xacro:arg name="robot_receive_timeout" default="0.2"/>
-  <!-- tool communication related parameters -->
+  <!-- tool communication related parameters (2FG7 defaults: 1Mbps, Even parity) -->
   <xacro:arg name="use_tool_communication" default="true" />
   <xacro:arg name="tool_voltage" default="24" />
-  <xacro:arg name="tool_parity" default="0" />
-  <xacro:arg name="tool_baud_rate" default="115200" />
+  <xacro:arg name="tool_parity" default="2" />
+  <xacro:arg name="tool_baud_rate" default="1000000" />
   <xacro:arg name="tool_stop_bits" default="1" />
   <xacro:arg name="tool_rx_idle_chars" default="1.5" />
@@ -48,5 +48,5 @@
   <xacro:arg name="use_mock_hardware" default="false" />
   <!-- initial position for simulations (Fake Hardware, Gazebo, Ignition) -->
-  <xacro:arg name="initial_positions_file" default="$(find ur5e_moveit_config)/config/pipettor/initial_positions.yaml"/>
+  <xacro:arg name="initial_positions_file" default="$(find cms_moveit_config)/config/2fg7/initial_positions.yaml"/>
   <xacro:property name="initial_positions_file" default="$(arg initial_positions_file)"/>
   <!-- create link fixed to the "map" -->
@@ -105,12 +105,8 @@
   <!-- Tool block attached to the Zivid arm mount (not the camera) -->
   <xacro:tool_block parent_link="zivid_arm_mount" xyz="0 0 0.049" rpy="-1.5708 0 3.14159"/>
-  <!-- Pipettor attached to tool block -->
-  <xacro:pipette
-    name="pipette"
-    prefix="$(arg tf_prefix)"
+  <!-- OnRobot 2FG7 gripper — same mounting offset as ePick/Hand-E (same bolt pattern) -->
+  <xacro:onrobot_2fg7
     parent="tool_block"
-    pipette_mass="0.200"
-    xyz="-0.005 -0.015 0"
-    rpy="-1.5708 0 3.1416"
-  />
+    xyz="0 -0.03235 0"
+    rpy="-1.5708 0 3.1416"/>
 </robot>

File: src/custom-ur-descriptions/cms_robot_description/urdf/ur_with_zivid_epick.urdf (robot description, URDF)
Before this commit: robot ur5e, 24 links, 23 joints
Links:
- link base_link_inertia: geometry collision mesh filename=package://ur_description/meshes/ur5e/collision/base.stl; visual mesh filename=package://ur_description/meshes/ur5e/visual/base.dae
- link epick_body: geometry collision cylinder length=0.1023 radius=0.044; visual mesh filename=package://epick_description/meshes/visual/epick_body.stl scale=0.001 0.001 0.001
- link forearm_link: geometry collision mesh filename=package://ur_description/meshes/ur5e/collision/forearm.stl; visual mesh filename=package://ur_description/meshes/ur5e/visual/forearm.dae
- link shoulder_link: geometry collision mesh filename=package://ur_description/meshes/ur5e/collision/shoulder.stl; visual mesh filename=package://ur_description/meshes/ur5e/visual/shoulder.dae
- link tool_block: geometry collision mesh filename=package://cms_robot_description/meshes/tool_exchanger/Tool_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 scale=0.001 0.001 0.001; visual mesh filename=package://cms_robot_description/meshes/tool_exchanger/Tool_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 scale=0.001 0.001 0.001
- link upper_arm_link: geometry collision mesh filename=package://ur_description/meshes/ur5e/collision/upperarm.stl; visual mesh filename=package://ur_description/meshes/ur5e/visual/upperarm.dae
- link wrist_1_link: geometry collision mesh filename=package://ur_description/meshes/ur5e/collision/wrist1.stl; visual mesh filename=package://ur_description/meshes/ur5e/visual/wrist1.dae
- link wrist_2_link: geometry collision mesh filename=package://ur_description/meshes/ur5e/collision/wrist2.stl; visual mesh filename=package://ur_description/meshes/ur5e/visual/wrist2.dae
- link wrist_3_link: geometry collision mesh filename=package://ur_description/meshes/ur5e/collision/wrist3.stl; visual mesh filename=package://ur_description/meshes/ur5e/visual/wrist3.dae
- link zivid_arm_mount: geometry collision mesh filename=package://cms_robot_description/meshes/zivid/zivid_onarm_mo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 scale=0.001 0.001 0.001; visual mesh filename=package://cms_robot_description/meshes/zivid/zivid_onarm_mo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 scale=0.001 0.001 0.001
- link zivid_base_link: geometry collision mesh filename=package://zivid_description/meshes/collision/zivid_2_plus_c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; visual mesh filename=package://zivid_description/meshes/visual/zivid_2_plus.stl

File: src/custom-ur-descriptions/cms_robot_description/urdf/ur_with_zivid_epick.xacro (robot description, xacro)
@@ -1,5 +1,5 @@
 <?xml version="1.0"?>
 <robot xmlns:xacro="http://wiki.ros.org/xacro" name="$(arg name)">
-<!--Chain: map -> UR -> flange -> zivid_camera_mount -> zivid_camera -> 2FG7 gripper -->
+<!--   Chain: map -> UR -> flange -> zivid_camera_mount -> zivid_camera -> EPick gripper -->
   <!-- robot name parameter -->
   <xacro:arg name="name" default="ur5e"/>
@@ -7,9 +7,10 @@
   <xacro:include filename="$(find ur_description)/urdf/ur_macro.xacro"/>
   <xacro:include filename="$(find ur_robot_driver)/urdf/ur.ros2_control.xacro"/>
-  <xacro:include filename="$(find ur5e_robot_description)/urdf/zivid_camera_mount.xacro"/>
-  <xacro:include filename="$(find ur5e_robot_description)/urdf/tool_block.xacro"/>
-  <xacro:include filename="$(find onrobot_2fg7_description)/urdf/onrobot_2fg7.xacro"/>
+  <xacro:include filename="$(find cms_robot_description)/urdf/zivid_camera_mount.xacro"/>
+  <xacro:include filename="$(find cms_robot_description)/urdf/tool_block.xacro"/>
+  <xacro:include filename="$(find epick_config)/urdf/epick_overlay.xacro"/>
   <!-- possible 'ur_type' values: ur3, ur5e, ur5, ur10, ur10e, ur16e, ur20 -->
   <xacro:arg name="ur_type" default="ur5e"/>
+  <!--. -->
   <!-- Parameters from upstream UR description -->
   <xacro:arg name="tf_prefix" default="" />
@@ -34,9 +35,9 @@
   <!-- Keep-alive: number of 20ms cycles without response before disconnect (10 = 200ms timeout) -->
   <xacro:arg name="robot_receive_timeout" default="0.2"/>
-  <!-- tool communication related parameters (2FG7 defaults: 1Mbps, Even parity) -->
-  <xacro:arg name="use_tool_communication" default="true" />
-  <xacro:arg name="tool_voltage" default="24" />
-  <xacro:arg name="tool_parity" default="2" />
-  <xacro:arg name="tool_baud_rate" default="1000000" />
+  <!-- tool communication related parameters -->
+  <xacro:arg name="use_tool_communication" default="false" />
+  <xacro:arg name="tool_voltage" default="0" />
+  <xacro:arg name="tool_parity" default="0" />
+  <xacro:arg name="tool_baud_rate" default="115200" />
   <xacro:arg name="tool_stop_bits" default="1" />
   <xacro:arg name="tool_rx_idle_chars" default="1.5" />
@@ -48,5 +49,5 @@
   <xacro:arg name="use_mock_hardware" default="false" />
   <!-- initial position for simulations (Fake Hardware, Gazebo, Ignition) -->
-  <xacro:arg name="initial_positions_file" default="$(find ur5e_moveit_config)/config/2fg7/initial_positions.yaml"/>
+  <xacro:arg name="initial_positions_file" default="$(find cms_moveit_config)/config/epick/initial_positions.yaml"/>
   <xacro:property name="initial_positions_file" default="$(arg initial_positions_file)"/>
   <!-- create link fixed to the "map" -->
@@ -105,8 +106,21 @@
   <!-- Tool block attached to the Zivid arm mount (not the camera) -->
   <xacro:tool_block parent_link="zivid_arm_mount" xyz="0 0 0.049" rpy="-1.5708 0 3.14159"/>
-  <!-- OnRobot 2FG7 gripper — same mounting offset as ePick/Hand-E (same bolt pattern) -->
-  <xacro:onrobot_2fg7
-    parent="tool_block"
-    xyz="0 -0.03235 0"
-    rpy="-1.5708 0 3.1416"/>
+  <!-- Suction cup profile: dimensions loaded from suction_cups.yaml (single source of truth).
+       The cup_profile default MUST match the physically attached cup — the UR driver's
+       robot_state_publisher uses this default (it can't receive args from the orchestrator).
+       When changing cups, update this default AND the active beamline YAML's grippers.epick.cup_profile.
+       Available profiles: see epick_config/config/suction_cups.yaml -->
+  <xacro:property name="cups_yaml_path" value="$(find epick_config)/config/suction_cups.yaml"/>
+  <xacro:property name="cups_config" value="${xacro.load_yaml(cups_yaml_path)}"/>
+  <xacro:arg name="cup_profile" default="3mm_dia"/>
+  <xacro:property name="cup_profile_name" value="$(arg cup_profile)"/>
+  <xacro:property name="cup" value="${cups_config['cups'][cup_profile_name]}"/>
+  <!-- Epick Gripper -->
+  <xacro:epick_overlay use_mock_hardware="$(arg use_mock_hardware)" parent="tool_block"
+                  origin_xyz="0 -0.03235 0"
+                  origin_rpy="-1.5708 0 3.1416"
+                  extension_length="${cup['extension_length']}"
+                  extension_radius="${cup['extension_radius']}"
+                  suction_cup_height="${cup['suction_cup_height']}"
+                  suction_cup_radius="${cup['suction_cup_radius']}"/>
 </robot>

File: src/custom-ur-descriptions/cms_robot_description/urdf/ur_with_zivid_epick_isaac.urdf (robot description, URDF)
Before this commit: robot ur5e, 21 links, 20 joints
Links:
- removed link led_strip_link
- removed link pipette_base_link
- removed link pipette_body_link
- removed link pipette_tip_link
- added link epick_base_link
- added link epick_body; collision cylinder length=0.1023 radius=0.044; visual mesh filename=/home/aditya/work/erobs/src/end_effectors/ros2_epick_grippe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 scale=0.001 0.001 0.001
- added link epick_extension; collision cylinder length=0.018 radius=0.006; visual cylinder length=0.018 radius=0.006
- added link epick_suction_cup; collision cylinder length=0.006 radius=0.0035; visual cylinder length=0.006 radius=0.0035
- added link epick_tcp
- added link epick_tip
- added link epick_vacuum_state
- link tool_block: geometry collision mesh filename=/home/aditya/work/erobs/src/custom-ur-descriptions/cms_robo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 scale=0.001 0.001 0.001; visual mesh filename=/home/aditya/work/erobs/src/custom-ur-descriptions/cms_robo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 scale=0.001 0.001 0.001
- link zivid_arm_mount: geometry collision mesh filename=/home/aditya/work/erobs/src/custom-ur-descriptions/cms_robo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 scale=0.001 0.001 0.001; visual mesh filename=/home/aditya/work/erobs/src/custom-ur-descriptions/cms_robo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 scale=0.001 0.001 0.001
Joints:
- removed joint led_strip_joint
- removed joint pipette_attachment_joint
- removed joint pipette_orientation_joint
- removed joint pipette_tip_joint
- added joint epick_base_link_to_epick_body: type fixed, parent epick_base_link, child epick_body, origin xyz=0 0 0.05115 rpy=0 0 0
- added joint epick_body_to_epick_extension: type fixed, parent epick_body, child epick_extension, origin xyz=0 0 0.06015 rpy=0 0 0
- added joint epick_extension_to_epick_suction_cup: type fixed, parent epick_extension, child epick_suction_cup, origin xyz=0 0 0.012 rpy=0 0 0
- added joint epick_suction_cup_to_epick_tip: type fixed, parent epick_suction_cup, child epick_tip, origin xyz=0 0 0.003 rpy=0 0 0
- added joint epick_tip_to_epick_tcp: type fixed, parent epick_tip, child epick_tcp, origin xyz=0 0 -0.0 rpy=0 0 0
- added joint gripper: type revolute, parent epick_tcp, child epick_vacuum_state, origin xyz=0 0 0 rpy=0 0 0, limit lower=0.0 upper=1.0 effort=30 velocity=1.0
- added joint tool_block_to_epick_base_link: type fixed, parent tool_block, child epick_base_link, origin xyz=0 -0.02 0 rpy=-1.5708 0 3.1416
- joint tool_block_joint: origin xyz=0 0 0.049 rpy=-1.5708 0 3.14159 -> xyz=0 0 0.055 rpy=-1.5708 0 3.14159

File: src/custom-ur-descriptions/cms_robot_description/urdf/ur_with_zivid_hande.urdf (robot description, URDF)
Before this commit: robot ur5e, 22 links, 21 joints
Links:
- link base_link_inertia: geometry collision mesh filename=package://ur_description/meshes/ur5e/collision/base.stl; visual mesh filename=package://ur_description/meshes/ur5e/visual/base.dae
- link forearm_link: geometry collision mesh filename=package://ur_description/meshes/ur5e/collision/forearm.stl; visual mesh filename=package://ur_description/meshes/ur5e/visual/forearm.dae
- link robotiq_hande_coupler: geometry collision cylinder length=0.0169 radius=0.0385; visual mesh filename=package://robotiq_hande_description/meshes/io_coupler.dae
- link robotiq_hande_left_finger: geometry collision mesh filename=package://robotiq_hande_description/meshes/finger_collision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 scale=1.0 1.0 1.0; visual mesh filename=package://robotiq_hande_description/meshes/finger.dae scale=1.0 1.0 1.0
- link robotiq_hande_link: geometry collision cylinder length=0.10690000000000001 radius=0.0385; visual mesh filename=package://robotiq_hande_description/meshes/hande.dae scale=1.0 1.0 1.0
- link robotiq_hande_right_finger: geometry collision mesh filename=package://robotiq_hande_description/meshes/finger_collision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 scale=1.0 1.0 1.0; visual mesh filename=package://robotiq_hande_description/meshes/finger.dae scale=1.0 1.0 1.0
- link shoulder_link: geometry collision mesh filename=package://ur_description/meshes/ur5e/collision/shoulder.stl; visual mesh filename=package://ur_description/meshes/ur5e/visual/shoulder.dae
- link tool_block: geometry collision mesh filename=package://cms_robot_description/meshes/tool_exchanger/Tool_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 scale=0.001 0.001 0.001; visual mesh filename=package://cms_robot_description/meshes/tool_exchanger/Tool_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 scale=0.001 0.001 0.001
- link upper_arm_link: geometry collision mesh filename=package://ur_description/meshes/ur5e/collision/upperarm.stl; visual mesh filename=package://ur_description/meshes/ur5e/visual/upperarm.dae
- link wrist_1_link: geometry collision mesh filename=package://ur_description/meshes/ur5e/collision/wrist1.stl; visual mesh filename=package://ur_description/meshes/ur5e/visual/wrist1.dae
- link wrist_2_link: geometry collision mesh filename=package://ur_description/meshes/ur5e/collision/wrist2.stl; visual mesh filename=package://ur_description/meshes/ur5e/visual/wrist2.dae
- link wrist_3_link: geometry collision mesh filename=package://ur_description/meshes/ur5e/collision/wrist3.stl; visual mesh filename=package://ur_description/meshes/ur5e/visual/wrist3.dae
- link zivid_arm_mount: geometry collision mesh filename=package://cms_robot_description/meshes/zivid/zivid_onarm_mo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 scale=0.001 0.001 0.001; visual mesh filename=package://cms_robot_description/meshes/zivid/zivid_onarm_mo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 scale=0.001 0.001 0.001
- link zivid_base_link: geometry collision mesh filename=package://zivid_description/meshes/collision/zivid_2_plus_c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; visual mesh filename=package://zivid_description/meshes/visual/zivid_2_plus.stl

File: src/custom-ur-descriptions/cms_robot_description/urdf/ur_with_zivid_hande.xacro (robot description, xacro)
@@ -7,6 +7,6 @@
   <xacro:include filename="$(find ur_description)/urdf/ur_macro.xacro"/>
   <xacro:include filename="$(find ur_robot_driver)/urdf/ur.ros2_control.xacro"/>
-  <xacro:include filename="$(find ur5e_robot_description)/urdf/zivid_camera_mount.xacro"/>
-  <xacro:include filename="$(find ur5e_robot_description)/urdf/tool_block.xacro"/>
+  <xacro:include filename="$(find cms_robot_description)/urdf/zivid_camera_mount.xacro"/>
+  <xacro:include filename="$(find cms_robot_description)/urdf/tool_block.xacro"/>
   <xacro:include filename="$(find robotiq_hande_description)/urdf/robotiq_hande_gripper.xacro"/>
   <!-- possible 'ur_type' values: ur3, ur5e, ur5, ur10, ur10e, ur16e, ur20 -->
@@ -48,5 +48,5 @@
   <xacro:arg name="use_mock_hardware" default="false" />
   <!-- initial position for simulations (Fake Hardware, Gazebo, Ignition) -->
-  <xacro:arg name="initial_positions_file" default="$(find ur5e_moveit_config)/config/hande/initial_positions.yaml"/>
+  <xacro:arg name="initial_positions_file" default="$(find cms_moveit_config)/config/hande/initial_positions.yaml"/>
   <xacro:property name="initial_positions_file" default="$(arg initial_positions_file)"/>
   <!-- create link fixed to the "map" -->
