Commit message: refactor: rename ur5e_moveit_config → cms_moveit_config, ur5e_robot_description → cms_robot_description
These packages are CMS beamline-specific (gripper configs, URDF meshes,
controller params) but were named generically after the robot model. Since
multiple beamlines will each have their own UR5e, the generic name was
ambiguous. Beamline-prefixed names make ownership clear and let new beamlines
create their own packages (e.g. chx_moveit_config) without confusion.

Updated: package.xml, CMakeLists.txt, launch files, xacro includes, SRDF,
beamline YAML, visualization panel, docs, and all generated URDFs.

File: src/custom-ur-descriptions/cms_robot_description/urdf/ur_with_zivid_hande_isaac.urdf (robot description, URDF)
Before this commit: robot ur5e, 17 links, 16 joints
Links:
- removed link te_robotside
- added link robotiq_hande_coupler, mass 0.119; collision cylinder length=0.0169 radius=0.0385; visual mesh filename=/home/aditya/work/erobs/src/end_effectors/robotiq_hande_des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
- added link robotiq_hande_end
- added link robotiq_hande_left_finger, mass 0.03804; collision mesh filename=/home/aditya/work/erobs/src/end_effectors/robotiq_hande_des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 scale=1.0 1.0 1.0; visual mesh filename=/home/aditya/work/erobs/src/end_effectors/robotiq_hande_des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 scale=1.0 1.0 1.0
- added link robotiq_hande_link, mass 0.86387; collision cylinder length=0.10690000000000001 radius=0.0385; visual mesh filename=/home/aditya/work/erobs/src/end_effectors/robotiq_hande_des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 scale=1.0 1.0 1.0
- added link robotiq_hande_right_finger, mass 0.03804; collision mesh filename=/home/aditya/work/erobs/src/end_effectors/robotiq_hande_des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 scale=1.0 1.0 1.0; visual mesh filename=/home/aditya/work/erobs/src/end_effectors/robotiq_hande_des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 scale=1.0 1.0 1.0
- added link tool_block, mass 0.2; collision mesh filename=/home/aditya/work/erobs/src/custom-ur-descriptions/cms_robo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 scale=0.001 0.001 0.001; visual mesh filename=/home/aditya/work/erobs/src/custom-ur-descriptions/cms_robo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 scale=0.001 0.001 0.001
- link base_link_inertia: geometry collision mesh filename=/opt/ros/jazzy/share/ur_description/meshes/ur5e/collision/b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; visual mesh filename=/opt/ros/jazzy/share/ur_description/meshes/ur5e/visual/base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
- link forearm_link: geometry collision mesh filename=/opt/ros/jazzy/share/ur_description/meshes/ur5e/collision/f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; visual mesh filename=/opt/ros/jazzy/share/ur_description/meshes/ur5e/visual/fore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
- link shoulder_link: geometry collision mesh filename=/opt/ros/jazzy/share/ur_description/meshes/ur5e/collision/s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; visual mesh filename=/opt/ros/jazzy/share/ur_description/meshes/ur5e/visual/shou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
- link upper_arm_link: geometry collision mesh filename=/opt/ros/jazzy/share/ur_description/meshes/ur5e/collision/u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; visual mesh filename=/opt/ros/jazzy/share/ur_description/meshes/ur5e/visual/uppe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
- link wrist_1_link: geometry collision mesh filename=/opt/ros/jazzy/share/ur_description/meshes/ur5e/collision/w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; visual mesh filename=/opt/ros/jazzy/share/ur_description/meshes/ur5e/visual/wris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
- link wrist_2_link: geometry collision mesh filename=/opt/ros/jazzy/share/ur_description/meshes/ur5e/collision/w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; visual mesh filename=/opt/ros/jazzy/share/ur_description/meshes/ur5e/visual/wris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
- link wrist_3_link: geometry collision mesh filename=/opt/ros/jazzy/share/ur_description/meshes/ur5e/collision/w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; visual mesh filename=/opt/ros/jazzy/share/ur_description/meshes/ur5e/visual/wris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
- link zivid_arm_mount: geometry collision mesh filename=/home/aditya/work/erobs/src/custom-ur-descriptions/cms_robo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 scale=0.001 0.001 0.001; visual mesh filename=/home/aditya/work/erobs/src/custom-ur-descriptions/cms_robo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 scale=0.001 0.001 0.001
- link zivid_base_link: geometry collision mesh filename=/home/aditya/work/erobs/src/vision/zivid-ros/zivid_descript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; visual mesh filename=/home/aditya/work/erobs/src/vision/zivid-ros/zivid_descript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
Joints:
- removed joint te_robotside_joint
- added joint robotiq_hande_base_joint: type fixed, parent robotiq_hande_coupler, child robotiq_hande_link, origin xyz=0 0 0.011 rpy=0 0 0
- added joint robotiq_hande_coupler_joint: type fixed, parent tool_block, child robotiq_hande_coupler, origin xyz=0 -0.02 0 rpy=-1.5708 0 3.1416
- added joint robotiq_hande_end_joint: type fixed, parent robotiq_hande_link, child robotiq_hande_end, origin xyz=0 0 0.14550000000000002 rpy=0 0 0
- added joint robotiq_hande_left_finger_joint: type prismatic, parent robotiq_hande_link, child robotiq_hande_left_finger, origin xyz=0 0 0.099 rpy=0 0 0, axis 1 0 0, limit lower=0 upper=0.025 effort=130 velocity=0.15
- added joint robotiq_hande_right_finger_joint: type prismatic, parent robotiq_hande_link, child robotiq_hande_right_finger, origin xyz=0 0 0.099 rpy=0 0 0, axis -1 0 0, limit lower=0 upper=0.025 effort=130 velocity=0.15, mimic joint=robotiq_hande_left_finger_joint multiplier=1 offset=0
- added joint tool_block_joint: type fixed, parent zivid_arm_mount, child tool_block, origin xyz=0 0 0.055 rpy=-1.5708 0 3.14159

File: src/custom-ur-descriptions/cms_robot_description/urdf/ur_with_zivid_pipettor.urdf (robot description, URDF)
Before this commit: robot ur5e, 17 links, 16 joints
Links:
- removed link te_robotside
- added link led_strip_link; visual box size=0.002 0.001 0.02
- added link pipette_base_link
- added link pipette_body_link, mass 0.2; collision mesh filename=package://pipette_description/meshes/collision/pipettor_col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 scale=0.001 0.001 0.001; visual mesh filename=package://pipette_description/meshes/visual/pipettor_visual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 scale=0.001 0.001 0.001
- added link pipette_tip_link
- added link tool_block, mass 0.2; collision mesh filename=package://cms_robot_description/meshes/tool_exchanger/Tool_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 scale=0.001 0.001 0.001; visual mesh filename=package://cms_robot_description/meshes/tool_exchanger/Tool_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 scale=0.001 0.001 0.001
- link base_link_inertia: geometry collision mesh filename=package://ur_description/meshes/ur5e/collision/base.stl; visual mesh filename=package://ur_description/meshes/ur5e/visual/base.dae
- link forearm_link: geometry collision mesh filename=package://ur_description/meshes/ur5e/collision/forearm.stl; visual mesh filename=package://ur_description/meshes/ur5e/visual/forearm.dae
- link shoulder_link: geometry collision mesh filename=package://ur_description/meshes/ur5e/collision/shoulder.stl; visual mesh filename=package://ur_description/meshes/ur5e/visual/shoulder.dae
- link upper_arm_link: geometry collision mesh filename=package://ur_description/meshes/ur5e/collision/upperarm.stl; visual mesh filename=package://ur_description/meshes/ur5e/visual/upperarm.dae
- link wrist_1_link: geometry collision mesh filename=package://ur_description/meshes/ur5e/collision/wrist1.stl; visual mesh filename=package://ur_description/meshes/ur5e/visual/wrist1.dae
- link wrist_2_link: geometry collision mesh filename=package://ur_description/meshes/ur5e/collision/wrist2.stl; visual mesh filename=package://ur_description/meshes/ur5e/visual/wrist2.dae
- link wrist_3_link: geometry collision mesh filename=package://ur_description/meshes/ur5e/collision/wrist3.stl; visual mesh filename=package://ur_description/meshes/ur5e/visual/wrist3.dae
- link zivid_arm_mount: geometry collision mesh filename=package://cms_robot_description/meshes/zivid/zivid_onarm_mo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 scale=0.001 0.001 0.001; visual mesh filename=package://cms_robot_description/meshes/zivid/zivid_onarm_mo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 scale=0.001 0.001 0.001
- link zivid_base_link: geometry collision mesh filename=package://zivid_description/meshes/collision/zivid_2_plus_c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; visual mesh filename=package://zivid_description/meshes/visual/zivid_2_plus.stl
Joints:
- removed joint te_robotside_joint
- added joint led_strip_joint: type fixed, parent pipette_base_link, child led_strip_link, origin xyz=0 0.025 0.238 rpy=0 0 0
- added joint pipette_attachment_joint: type fixed, parent tool_block, child pipette_base_link, origin xyz=-0.005 -0.015 0 rpy=-1.5708 0 3.1416
- added joint pipette_orientation_joint: type fixed, parent pipette_base_link, child pipette_body_link, origin xyz=-0.09 -0.055 0.34 rpy=-1.5708 0 0
- added joint pipette_tip_joint: type fixed, parent pipette_base_link, child pipette_tip_link, origin xyz=0 0 0.34 rpy=0 0 0
- added joint tool_block_joint: type fixed, parent zivid_arm_mount, child tool_block, origin xyz=0 0 0.049 rpy=-1.5708 0 3.14159

File: src/custom-ur-descriptions/cms_robot_description/urdf/ur_with_zivid_pipettor.xacro (robot description, xacro)
@@ -1,5 +1,5 @@
 <?xml version="1.0"?>
 <robot xmlns:xacro="http://wiki.ros.org/xacro" name="$(arg name)">
-<!--   Chain: map -> UR -> flange -> zivid_camera_mount -> zivid_camera -> EPick gripper -->
+<!--Chain: map -> UR -> flange -> zivid_camera_mount -> zivid_camera -> tool_block -> pipettor -->
   <!-- robot name parameter -->
   <xacro:arg name="name" default="ur5e"/>
@@ -7,10 +7,9 @@
   <xacro:include filename="$(find ur_description)/urdf/ur_macro.xacro"/>
   <xacro:include filename="$(find ur_robot_driver)/urdf/ur.ros2_control.xacro"/>
-  <xacro:include filename="$(find ur5e_robot_description)/urdf/zivid_camera_mount.xacro"/>
-  <xacro:include filename="$(find ur5e_robot_description)/urdf/tool_block.xacro"/>
-  <xacro:include filename="$(find epick_config)/urdf/epick_overlay.xacro"/>
+  <xacro:include filename="$(find cms_robot_description)/urdf/zivid_camera_mount.xacro"/>
+  <xacro:include filename="$(find cms_robot_description)/urdf/tool_block.xacro"/>
+  <xacro:include filename="$(find pipette_description)/urdf/pipette_macro.urdf.xacro"/>
   <!-- possible 'ur_type' values: ur3, ur5e, ur5, ur10, ur10e, ur16e, ur20 -->
   <xacro:arg name="ur_type" default="ur5e"/>
-  <!--. -->
   <!-- Parameters from upstream UR description -->
   <xacro:arg name="tf_prefix" default="" />
@@ -36,6 +35,6 @@
   <xacro:arg name="robot_receive_timeout" default="0.2"/>
   <!-- tool communication related parameters -->
-  <xacro:arg name="use_tool_communication" default="false" />
-  <xacro:arg name="tool_voltage" default="0" />
+  <xacro:arg name="use_tool_communication" default="true" />
+  <xacro:arg name="tool_voltage" default="24" />
   <xacro:arg name="tool_parity" default="0" />
   <xacro:arg name="tool_baud_rate" default="115200" />
@@ -49,5 +48,5 @@
   <xacro:arg name="use_mock_hardware" default="false" />
   <!-- initial position for simulations (Fake Hardware, Gazebo, Ignition) -->
-  <xacro:arg name="initial_positions_file" default="$(find ur5e_moveit_config)/config/epick/initial_positions.yaml"/>
+  <xacro:arg name="initial_positions_file" default="$(find cms_moveit_config)/config/pipettor/initial_positions.yaml"/>
   <xacro:property name="initial_positions_file" default="$(arg initial_positions_file)"/>
   <!-- create link fixed to the "map" -->
@@ -106,21 +105,12 @@
   <!-- Tool block attached to the Zivid arm mount (not the camera) -->
   <xacro:tool_block parent_link="zivid_arm_mount" xyz="0 0 0.049" rpy="-1.5708 0 3.14159"/>
-  <!-- Suction cup profile: dimensions loaded from suction_cups.yaml (single source of truth).
-       The cup_profile default MUST match the physically attached cup — the UR driver's
-       robot_state_publisher uses this default (it can't receive args from the orchestrator).
-       When changing cups, update this default AND the active beamline YAML's grippers.epick.cup_profile.
-       Available profiles: see epick_config/config/suction_cups.yaml -->
-  <xacro:property name="cups_yaml_path" value="$(find epick_config)/config/suction_cups.yaml"/>
-  <xacro:property name="cups_config" value="${xacro.load_yaml(cups_yaml_path)}"/>
-  <xacro:arg name="cup_profile" default="3mm_dia"/>
-  <xacro:property name="cup_profile_name" value="$(arg cup_profile)"/>
-  <xacro:property name="cup" value="${cups_config['cups'][cup_profile_name]}"/>
-  <!-- Epick Gripper -->
-  <xacro:epick_overlay use_mock_hardware="$(arg use_mock_hardware)" parent="tool_block"
-                  origin_xyz="0 -0.03235 0"
-                  origin_rpy="-1.5708 0 3.1416"
-                  extension_length="${cup['extension_length']}"
-                  extension_radius="${cup['extension_radius']}"
-                  suction_cup_height="${cup['suction_cup_height']}"
-                  suction_cup_radius="${cup['suction_cup_radius']}"/>
+  <!-- Pipettor attached to tool block -->
+  <xacro:pipette
+    name="pipette"
+    prefix="$(arg tf_prefix)"
+    parent="tool_block"
+    pipette_mass="0.200"
+    xyz="-0.005 -0.015 0"
+    rpy="-1.5708 0 3.1416"
+  />
 </robot>

File: src/custom-ur-descriptions/cms_robot_description/urdf/ur_with_zivid_pipettor_isaac.urdf (robot description, URDF)
Before this commit: robot ur5e, 22 links, 21 joints
Links:
- removed link robotiq_hande_coupler
- removed link robotiq_hande_end
- removed link robotiq_hande_left_finger
- removed link robotiq_hande_link
- removed link robotiq_hande_right_finger
- added link led_strip_link; visual box size=0.002 0.001 0.02
- added link pipette_base_link
- added link pipette_body_link, mass 0.2; collision mesh filename=/home/aditya/work/erobs/src/end_effectors/pipettor/pipette_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 scale=0.001 0.001 0.001; visual mesh filename=/home/aditya/work/erobs/src/end_effectors/pipettor/pipette_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 scale=0.001 0.001 0.001
- added link pipette_tip_link
- link base_link_inertia: geometry collision mesh filename=/opt/ros/jazzy/share/ur_description/meshes/ur5e/collision/b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; visual mesh filename=/opt/ros/jazzy/share/ur_description/meshes/ur5e/visual/base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
- link forearm_link: geometry collision mesh filename=/opt/ros/jazzy/share/ur_description/meshes/ur5e/collision/f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; visual mesh filename=/opt/ros/jazzy/share/ur_description/meshes/ur5e/visual/fore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
- link shoulder_link: geometry collision mesh filename=/opt/ros/jazzy/share/ur_description/meshes/ur5e/collision/s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; visual mesh filename=/opt/ros/jazzy/share/ur_description/meshes/ur5e/visual/shou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
- link tool_block: geometry collision mesh filename=/home/aditya/work/erobs/src/custom-ur-descriptions/cms_robo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 scale=0.001 0.001 0.001; visual mesh filename=/home/aditya/work/erobs/src/custom-ur-descriptions/cms_robo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 scale=0.001 0.001 0.001
- link upper_arm_link: geometry collision mesh filename=/opt/ros/jazzy/share/ur_description/meshes/ur5e/collision/u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; visual mesh filename=/opt/ros/jazzy/share/ur_description/meshes/ur5e/visual/uppe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
- link wrist_1_link: geometry collision mesh filename=/opt/ros/jazzy/share/ur_description/meshes/ur5e/collision/w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; visual mesh filename=/opt/ros/jazzy/share/ur_description/meshes/ur5e/visual/wris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
- link wrist_2_link: geometry collision mesh filename=/opt/ros/jazzy/share/ur_description/meshes/ur5e/collision/w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; visual mesh filename=/opt/ros/jazzy/share/ur_description/meshes/ur5e/visual/wris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
- link wrist_3_link: geometry collision mesh filename=/opt/ros/jazzy/share/ur_description/meshes/ur5e/collision/w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; visual mesh filename=/opt/ros/jazzy/share/ur_description/meshes/ur5e/visual/wris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
- link zivid_arm_mount: geometry collision mesh filename=/home/aditya/work/erobs/src/custom-ur-descriptions/cms_robo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 scale=0.001 0.001 0.001; visual mesh filename=/home/aditya/work/erobs/src/custom-ur-descriptions/cms_robo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 scale=0.001 0.001 0.001
- link zivid_base_link: geometry collision mesh filename=/home/aditya/work/erobs/src/vision/zivid-ros/zivid_descript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; visual mesh filename=/home/aditya/work/erobs/src/vision/zivid-ros/zivid_descript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
Joints:
- removed joint robotiq_hande_base_joint
- removed joint robotiq_hande_coupler_joint
- removed joint robotiq_hande_end_joint
- removed joint robotiq_hande_left_finger_joint
- removed joint robotiq_hande_right_finger_joint
- added joint led_strip_joint: type fixed, parent pipette_base_link, child led_strip_link, origin xyz=0 0.025 0.238 rpy=0 0 0
- added joint pipette_attachment_joint: type fixed, parent tool_block, child pipette_base_link, origin xyz=-0.005 -0.015 0 rpy=-1.5708 0 3.1416
- added joint pipette_orientation_joint: type fixed, parent pipette_base_link, child pipette_body_link, origin xyz=-0.09 -0.055 0.34 rpy=-1.5708 0 0
- added joint pipette_tip_joint: type fixed, parent pipette_base_link, child pipette_tip_link, origin xyz=0 0 0.34 rpy=0 0 0
- joint tool_block_joint: origin xyz=0 0 0.055 rpy=-1.5708 0 3.14159 -> xyz=0 0 0.049 rpy=-1.5708 0 3.14159
