Commit message: add W-010-B tool-changer coupling to epick chain
The epick was mounted directly on the Wingman tool-side plate, missing the
W-010-B coupling adapter (16.9mm). This made the modeled epick_tip ~11mm short
of the real cup, causing vision approaches to drive into the surface.

Adds te_coupling.xacro + W-010-B mesh, inserting the coupling into the chain:
  te_toolside -> te_coupling -> epick
Total tool0->epick_tip now 214.2mm, matching a direct physical measurement.

Only epick is fixed here; hande/2fg7 likely need the same coupling treatment
(flagged, pending per-tool measurement).

File: src/custom-ur-descriptions/cms_robot_description/urdf/ur_with_zivid_epick.urdf (robot description, URDF)
Before this commit: robot ur5e, 26 links, 25 joints
Links:
- added link te_coupling, mass 0.2; collision mesh filename=package://cms_robot_description/meshes/tool_exchanger/W-010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 scale=0.001 0.001 0.001; visual mesh filename=package://cms_robot_description/meshes/tool_exchanger/W-010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 scale=0.001 0.001 0.001
Joints:
- removed joint te_toolside_to_epick_base_link
- added joint te_coupling_joint: type fixed, parent te_toolside, child te_coupling, origin xyz=0 -0.012 0 rpy=1.5708 0 0
- added joint te_coupling_to_epick_base_link: type fixed, parent te_coupling, child epick_base_link, origin xyz=0 0 0.0099 rpy=0 0 0

File: src/custom-ur-descriptions/cms_robot_description/urdf/ur_with_zivid_epick.xacro (robot description, xacro)
@@ -11,4 +11,5 @@
   <xacro:include filename="$(find cms_robot_description)/urdf/te_robotside.xacro"/>
   <xacro:include filename="$(find cms_robot_description)/urdf/te_toolside.xacro"/>
+  <xacro:include filename="$(find cms_robot_description)/urdf/te_coupling.xacro"/>
   <xacro:include filename="$(find epick_config)/urdf/epick_overlay.xacro"/>
   <!-- possible 'ur_type' values: ur3, ur5e, ur5, ur10, ur10e, ur16e, ur20 -->
@@ -131,8 +132,15 @@
   <xacro:property name="cup_profile_name" value="$(arg cup_profile)"/>
   <xacro:property name="cup" value="${cups_config['cups'][cup_profile_name]}"/>
-  <!-- Epick Gripper -->
-  <xacro:epick_overlay use_mock_hardware="$(arg use_mock_hardware)" parent="te_toolside"
-                  origin_xyz="0 -0.005 0"
-                  origin_rpy="-1.5708 0 3.1416"
+  <!-- Tool-changer coupling (W-010-B, 16.9mm axial) on the tool-side plate.
+       Mounts on te_toolside's outward (-Y) face; coupling axis (mesh Z) aligned
+       to te_toolside -Y via the rpy below. -->
+  <xacro:te_coupling
+    parent_link="te_toolside"
+    xyz="0 -0.012 0"
+    rpy="1.5708 0 0"/>
+  <!-- Epick Gripper — now mounted on the coupling far face -->
+  <xacro:epick_overlay use_mock_hardware="$(arg use_mock_hardware)" parent="te_coupling"
+                  origin_xyz="0 0 0.0099"
+                  origin_rpy="0 0 0"
                   extension_length="${cup['extension_length']}"
                   extension_radius="${cup['extension_radius']}"
