Commit message: updated zivid-calibration values

File: src/custom-ur-descriptions/cms_robot_description/urdf/ur_with_zivid_epick.urdf (robot description, URDF)
Before this commit: robot ur5e, 27 links, 26 joints
Joints:
- joint tool0_to_zivid_optical: origin xyz=0.05635 0.10228 0.06025 rpy=-0.03622 0.05218 3.13437 -> xyz=0.05594 0.10469 0.05890 rpy=-0.03511 0.05081 3.13360

File: src/custom-ur-descriptions/cms_robot_description/urdf/zivid_camera_mount.xacro (robot description, xacro)
@@ -21,7 +21,10 @@
       <!-- Hand-eye calibration: tool0 -> optical_frame -->
       <!-- Rotation: Euler XYZ extrinsic, radians | Translation: meters -->
-      <!-- Calibration (2026-03-27): 12 poses (pose 4 excluded as outlier). Residuals: rot < 0.33°, trans < 1.53mm -->
+      <!-- Calibration (2026-07-22): Zivid Studio GUI hand-eye recalibration (4x4 in hand_eye_calibration.yaml). Pending touch-test verification. -->
+      <origin xyz="0.05594 0.10469 0.05890"
+              rpy="-0.03511 0.05081 3.13360"/>
+      <!-- Calibration (2026-03-27): 12 poses (pose 4 excluded as outlier). Residuals: rot < 0.33°, trans < 1.53mm
       <origin xyz="0.05635 0.10228 0.06025"
-              rpy="-0.03622 0.05218 3.13437"/>
+              rpy="-0.03622 0.05218 3.13437"/> -->
       <!-- Calibration (2026-03-25): Residuals: rot < 0.15°, trans < 1.0mm
       <origin xyz="0.05475 0.10491 0.06013"
