Commit message: Derive workspace root in Isaac URDF conversion instead of hardcoding
The convert_urdf_for_isaac.sh script and the generated *_isaac.urdf files
hardcoded /home/aditya/work/erobs, which no longer exists after the checkout
moved to github_ws/jazzy — every mesh path in the committed Isaac URDFs was
dead. Derive the workspace root from the script location via
git rev-parse --show-toplevel (ROS_SHARE overridable), regenerate all four
*_isaac.urdf files, and fix a spurious bash warning in the leftover-URI check.

File: src/custom-ur-descriptions/cms_robot_description/urdf/ur_standalone_isaac.urdf (robot description, URDF)
Before this commit: robot ur5e, 17 links, 16 joints
Links:
- added link wrist_extension, mass 0.3; collision mesh filename=/home/aditya/work/github_ws/jazzy/src/custom-ur-description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 scale=0.001 0.001 0.001; visual mesh filename=/home/aditya/work/github_ws/jazzy/src/custom-ur-description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 scale=0.001 0.001 0.001
- link te_robotside: geometry collision mesh filename=/home/aditya/work/github_ws/jazzy/src/custom-ur-description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 scale=0.001 0.001 0.001; visual mesh filename=/home/aditya/work/github_ws/jazzy/src/custom-ur-description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 scale=0.001 0.001 0.001
- link zivid_arm_mount: geometry collision mesh filename=/home/aditya/work/github_ws/jazzy/src/custom-ur-description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 scale=0.001 0.001 0.001; visual mesh filename=/home/aditya/work/github_ws/jazzy/src/custom-ur-description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 scale=0.001 0.001 0.001
- link zivid_base_link: geometry collision mesh filename=/home/aditya/work/github_ws/jazzy/src/vision/zivid-ros/zivi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; visual mesh filename=/home/aditya/work/github_ws/jazzy/src/vision/zivid-ros/zivi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
Joints:
- added joint wrist_extension_joint: type fixed, parent tool0, child wrist_extension, origin xyz=0 0 0.016 rpy=1.5708 0 3.14159
- joint te_robotside_joint: origin xyz=0 0 0.055 rpy=-1.5708 0 3.14159 -> xyz=0 0.047 0 rpy=3.14159 0 0; parent zivid_arm_mount -> wrist_extension

File: src/custom-ur-descriptions/cms_robot_description/urdf/ur_with_zivid_epick_isaac.urdf (robot description, URDF)
Before this commit: robot ur5e, 24 links, 23 joints
Links:
- removed link tool_block
- added link te_coupling, mass 0.2; collision mesh filename=/home/aditya/work/github_ws/jazzy/src/custom-ur-description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 scale=0.001 0.001 0.001; visual mesh filename=/home/aditya/work/github_ws/jazzy/src/custom-ur-description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 scale=0.001 0.001 0.001
- added link te_robotside, mass 0.5; collision mesh filename=/home/aditya/work/github_ws/jazzy/src/custom-ur-description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 scale=0.001 0.001 0.001; visual mesh filename=/home/aditya/work/github_ws/jazzy/src/custom-ur-description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 scale=0.001 0.001 0.001
- added link te_toolside, mass 0.4; collision mesh filename=/home/aditya/work/github_ws/jazzy/src/custom-ur-description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 scale=0.001 0.001 0.001; visual mesh filename=/home/aditya/work/github_ws/jazzy/src/custom-ur-description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 scale=0.001 0.001 0.001
- added link wrist_extension, mass 0.3; collision mesh filename=/home/aditya/work/github_ws/jazzy/src/custom-ur-description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 scale=0.001 0.001 0.001; visual mesh filename=/home/aditya/work/github_ws/jazzy/src/custom-ur-description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 scale=0.001 0.001 0.001
- link epick_body: geometry collision cylinder length=0.1023 radius=0.044; visual mesh filename=/home/aditya/work/github_ws/jazzy/src/end_effectors/ros2_ep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 scale=0.001 0.001 0.001
- link epick_extension: geometry collision cylinder length=0.013 radius=0.004; visual cylinder length=0.013 radius=0.004
- link epick_suction_cup: geometry collision cylinder length=0.003 radius=0.0015; visual cylinder length=0.003 radius=0.0015
- link zivid_arm_mount: geometry collision mesh filename=/home/aditya/work/github_ws/jazzy/src/custom-ur-description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 scale=0.001 0.001 0.001; visual mesh filename=/home/aditya/work/github_ws/jazzy/src/custom-ur-description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 scale=0.001 0.001 0.001
- link zivid_base_link: geometry collision mesh filename=/home/aditya/work/github_ws/jazzy/src/vision/zivid-ros/zivi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; visual mesh filename=/home/aditya/work/github_ws/jazzy/src/vision/zivid-ros/zivi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
Joints:
- removed joint tool_block_joint
- removed joint tool_block_to_epick_base_link
- added joint te_coupling_joint: type fixed, parent te_toolside, child te_coupling, origin xyz=0 -0.012 0 rpy=1.5708 0 0
- added joint te_coupling_to_epick_base_link: type fixed, parent te_coupling, child epick_base_link, origin xyz=0 0 0.0099 rpy=0 0 3.14159
- added joint te_robotside_joint: type fixed, parent wrist_extension, child te_robotside, origin xyz=0 0.047 0 rpy=3.14159 0 0
- added joint te_toolside_joint: type fixed, parent te_robotside, child te_toolside, origin xyz=0 -0.011 0 rpy=0 0 0
- added joint wrist_extension_joint: type fixed, parent tool0, child wrist_extension, origin xyz=0 0 0.016 rpy=1.5708 0 3.14159
- joint epick_body_to_epick_extension: origin xyz=0 0 0.06015 rpy=0 0 0 -> xyz=0 0 0.05765 rpy=0 0 0
- joint epick_extension_to_epick_suction_cup: origin xyz=0 0 0.012 rpy=0 0 0 -> xyz=0 0 0.008 rpy=0 0 0
- joint epick_suction_cup_to_epick_tip: origin xyz=0 0 0.003 rpy=0 0 0 -> xyz=0 0 0.0015 rpy=0 0 0

File: src/custom-ur-descriptions/cms_robot_description/urdf/ur_with_zivid_hande_isaac.urdf (robot description, URDF)
Before this commit: robot ur5e, 22 links, 21 joints
Links:
- removed link tool_block
- added link te_robotside, mass 0.5; collision mesh filename=/home/aditya/work/github_ws/jazzy/src/custom-ur-description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 scale=0.001 0.001 0.001; visual mesh filename=/home/aditya/work/github_ws/jazzy/src/custom-ur-description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 scale=0.001 0.001 0.001
- added link te_toolside, mass 0.4; collision mesh filename=/home/aditya/work/github_ws/jazzy/src/custom-ur-description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 scale=0.001 0.001 0.001; visual mesh filename=/home/aditya/work/github_ws/jazzy/src/custom-ur-description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 scale=0.001 0.001 0.001
- added link wrist_extension, mass 0.3; collision mesh filename=/home/aditya/work/github_ws/jazzy/src/custom-ur-description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 scale=0.001 0.001 0.001; visual mesh filename=/home/aditya/work/github_ws/jazzy/src/custom-ur-description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 scale=0.001 0.001 0.001
- link robotiq_hande_coupler: geometry collision cylinder length=0.0169 radius=0.0385; visual mesh filename=/home/aditya/work/github_ws/jazzy/src/end_effectors/robotiq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
- link robotiq_hande_left_finger: geometry collision mesh filename=/home/aditya/work/github_ws/jazzy/src/end_effectors/robotiq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 scale=1.0 1.0 1.0; visual mesh filename=/home/aditya/work/github_ws/jazzy/src/end_effectors/robotiq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 scale=1.0 1.0 1.0
- link robotiq_hande_link: geometry collision cylinder length=0.10690000000000001 radius=0.0385; visual mesh filename=/home/aditya/work/github_ws/jazzy/src/end_effectors/robotiq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 scale=1.0 1.0 1.0
- link robotiq_hande_right_finger: geometry collision mesh filename=/home/aditya/work/github_ws/jazzy/src/end_effectors/robotiq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 scale=1.0 1.0 1.0; visual mesh filename=/home/aditya/work/github_ws/jazzy/src/end_effectors/robotiq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 scale=1.0 1.0 1.0
- link zivid_arm_mount: geometry collision mesh filename=/home/aditya/work/github_ws/jazzy/src/custom-ur-description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 scale=0.001 0.001 0.001; visual mesh filename=/home/aditya/work/github_ws/jazzy/src/custom-ur-description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 scale=0.001 0.001 0.001
- link zivid_base_link: geometry collision mesh filename=/home/aditya/work/github_ws/jazzy/src/vision/zivid-ros/zivi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; visual mesh filename=/home/aditya/work/github_ws/jazzy/src/vision/zivid-ros/zivi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
Joints:
- removed joint tool_block_joint
- added joint te_robotside_joint: type fixed, parent wrist_extension, child te_robotside, origin xyz=0 0.047 0 rpy=3.14159 0 0
- added joint te_toolside_joint: type fixed, parent te_robotside, child te_toolside, origin xyz=0 -0.011 0 rpy=0 0 0
- added joint wrist_extension_joint: type fixed, parent tool0, child wrist_extension, origin xyz=0 0 0.016 rpy=1.5708 0 3.14159
- joint robotiq_hande_coupler_joint: origin xyz=0 -0.02 0 rpy=-1.5708 0 3.1416 -> xyz=0 -0.005 0 rpy=-1.5708 0 3.1416; parent tool_block -> te_toolside

File: src/custom-ur-descriptions/cms_robot_description/urdf/ur_with_zivid_pipettor_isaac.urdf (robot description, URDF)
Before this commit: robot ur5e, 21 links, 20 joints
Links:
- removed link tool_block
- added link te_robotside, mass 0.5; collision mesh filename=/home/aditya/work/github_ws/jazzy/src/custom-ur-description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 scale=0.001 0.001 0.001; visual mesh filename=/home/aditya/work/github_ws/jazzy/src/custom-ur-description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 scale=0.001 0.001 0.001
- added link te_toolside, mass 0.4; collision mesh filename=/home/aditya/work/github_ws/jazzy/src/custom-ur-description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 scale=0.001 0.001 0.001; visual mesh filename=/home/aditya/work/github_ws/jazzy/src/custom-ur-description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 scale=0.001 0.001 0.001
- added link wrist_extension, mass 0.3; collision mesh filename=/home/aditya/work/github_ws/jazzy/src/custom-ur-description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 scale=0.001 0.001 0.001; visual mesh filename=/home/aditya/work/github_ws/jazzy/src/custom-ur-description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 scale=0.001 0.001 0.001
- link pipette_body_link: geometry collision mesh filename=/home/aditya/work/github_ws/jazzy/src/end_effectors/pipetto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 scale=0.001 0.001 0.001; visual mesh filename=/home/aditya/work/github_ws/jazzy/src/end_effectors/pipetto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 scale=0.001 0.001 0.001
- link zivid_arm_mount: geometry collision mesh filename=/home/aditya/work/github_ws/jazzy/src/custom-ur-description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 scale=0.001 0.001 0.001; visual mesh filename=/home/aditya/work/github_ws/jazzy/src/custom-ur-description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 scale=0.001 0.001 0.001
- link zivid_base_link: geometry collision mesh filename=/home/aditya/work/github_ws/jazzy/src/vision/zivid-ros/zivi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; visual mesh filename=/home/aditya/work/github_ws/jazzy/src/vision/zivid-ros/zivi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
Joints:
- removed joint tool_block_joint
- added joint te_robotside_joint: type fixed, parent wrist_extension, child te_robotside, origin xyz=0 0.047 0 rpy=3.14159 0 0
- added joint te_toolside_joint: type fixed, parent te_robotside, child te_toolside, origin xyz=0 -0.011 0 rpy=0 0 0
- added joint wrist_extension_joint: type fixed, parent tool0, child wrist_extension, origin xyz=0 0 0.016 rpy=1.5708 0 3.14159
- joint pipette_attachment_joint: origin xyz=-0.005 -0.015 0 rpy=-1.5708 0 3.1416 -> xyz=-0.005 -0.005 0 rpy=-1.5708 0 3.1416; parent tool_block -> te_toolside
